Commit message: added simplified mesh for contact and better tuned parameters

File: solo_description/urdfs/leg.xacro (robot description, xacro)
@@ -395,5 +395,5 @@
                 <origin xyz="0 0 0" rpy="0 0 0" />
                 <geometry>
-                    <mesh filename="package://solo_description/meshes/stl/with_foot/solo_foot.stl"/>
+                    <mesh filename="package://solo_description/meshes/stl/with_foot/solo_foot_simple.stl"/>
                 </geometry>
                 <material name="${color_name}">
