Commit message: Tuning and cleaning anymalc and minicheetah

File: minicheetah_description/robots/minicheetah.srdf.xacro (robot description, xacro)
@@ -60,3 +60,17 @@
     <joint name="rh_kfe_joint" value="-1.5"/>
   </group_state>
+  <group_state group="chains" name="standdown">
+    <joint name="lf_haa_joint" value="0.0"/>
+    <joint name="lf_hfe_joint" value="1.50"/>
+    <joint name="lf_kfe_joint" value="-2.60"/>
+    <joint name="rf_haa_joint" value="0.0"/>
+    <joint name="rf_hfe_joint" value="1.50"/>
+    <joint name="rf_kfe_joint" value="-2.60"/>
+    <joint name="lh_haa_joint" value="0.0"/>
+    <joint name="lh_hfe_joint" value="1.50"/>
+    <joint name="lh_kfe_joint" value="-2.60"/>
+    <joint name="rh_haa_joint" value="0.0"/>
+    <joint name="rh_hfe_joint" value="1.50"/>
+    <joint name="rh_kfe_joint" value="-2.60"/>
+  </group_state>
 </robot>
