Commit message: stand up procedure for solo

File: solo_description/robots/solo.srdf.xacro (robot description, xacro)
@@ -50,16 +50,30 @@
     </group>
     <group_state group="chains" name="standup">
-    <joint name="lf_haa_joint" value="0."       />
-    <joint name="lf_hfe_joint" value="0.78539816" />
-    <joint name="lf_kfe_joint" value="-1.57079633"/>
-    <joint name="rf_haa_joint" value="0."       />
-    <joint name="rf_hfe_joint" value="0.78539816" />
-    <joint name="rf_kfe_joint" value="-1.57079633"/>
-    <joint name="lh_haa_joint" value="0."       />
-    <joint name="lh_hfe_joint" value="-0.78539816"/>
-    <joint name="lh_kfe_joint" value="1.57079633" />
-    <joint name="rh_haa_joint" value="0."       />
-    <joint name="rh_hfe_joint" value="-0.78539816"/>
-    <joint name="rh_kfe_joint" value="1.57079633" />
+	    <joint name="lf_haa_joint" value="0."       />
+	    <joint name="lf_hfe_joint" value="0.78539816" />
+	    <joint name="lf_kfe_joint" value="-1.57079633"/>
+	    <joint name="rf_haa_joint" value="0."       />
+	    <joint name="rf_hfe_joint" value="0.78539816" />
+	    <joint name="rf_kfe_joint" value="-1.57079633"/>
+	    <joint name="lh_haa_joint" value="0."       />
+	    <joint name="lh_hfe_joint" value="-0.78539816"/>
+	    <joint name="lh_kfe_joint" value="1.57079633" />
+	    <joint name="rh_haa_joint" value="0."       />
+	    <joint name="rh_hfe_joint" value="-0.78539816"/>
+	    <joint name="rh_kfe_joint" value="1.57079633" />
+    </group_state>
+    <group_state group="chains" name="standdown">
+	    <joint name="lf_haa_joint" value="0."/>
+	    <joint name="lf_hfe_joint" value="1.5708" />
+	    <joint name="lf_kfe_joint" value="-3.1415"/>
+	    <joint name="rf_haa_joint" value="0."/>
+	    <joint name="rf_hfe_joint" value="1.5708" />
+	    <joint name="rf_kfe_joint" value="-3.1415"/>
+	    <joint name="lh_haa_joint" value="0."/>
+	    <joint name="lh_hfe_joint" value="-1.5708"/>
+	    <joint name="lh_kfe_joint" value="3.1415" />
+	    <joint name="rh_haa_joint" value="0."/>
+	    <joint name="rh_hfe_joint" value="-1.5708"/>
+	    <joint name="rh_kfe_joint" value="3.1415" />
     </group_state>
 </robot>

Commit message: Make solo stand up in < < configuration

File: solo_description/robots/solo.srdf.xacro (robot description, xacro)
@@ -65,14 +65,14 @@
     <group_state group="chains" name="standdown">
 	    <joint name="lf_haa_joint" value="0."/>
-	    <joint name="lf_hfe_joint" value="1.5708" />
-	    <joint name="lf_kfe_joint" value="-3.1415"/>
+            <joint name="lf_hfe_joint" value="1.5708" />
+            <joint name="lf_kfe_joint" value="3.1415"/>
 	    <joint name="rf_haa_joint" value="0."/>
-	    <joint name="rf_hfe_joint" value="1.5708" />
-	    <joint name="rf_kfe_joint" value="-3.1415"/>
+            <joint name="rf_hfe_joint" value="1.5708" />
+            <joint name="rf_kfe_joint" value="3.1415"/>
 	    <joint name="lh_haa_joint" value="0."/>
-	    <joint name="lh_hfe_joint" value="-1.5708"/>
+            <joint name="lh_hfe_joint" value="1.5708"/>
 	    <joint name="lh_kfe_joint" value="3.1415" />
 	    <joint name="rh_haa_joint" value="0."/>
-	    <joint name="rh_hfe_joint" value="-1.5708"/>
+            <joint name="rh_hfe_joint" value="1.5708"/>
 	    <joint name="rh_kfe_joint" value="3.1415" />
     </group_state>
