Commit message: Added simplified meshes (convex hulls). Moved simple foot mesh and using spehere for feet contacts

File: solo_description/robots/solo.urdf.xacro (robot description, xacro)
@@ -50,5 +50,5 @@
             <origin xyz="0 0 0" rpy="0 0 0" />
             <geometry>
-                <mesh filename="package://solo_description/meshes/stl/with_foot/solo_body.stl"/>
+                <mesh filename="package://solo_description/meshes/stl/with_foot/simple/solo_body.stl"/>
             </geometry>
             <material name="${color_name}">

File: solo_description/urdfs/leg.xacro (robot description, xacro)
@@ -95,5 +95,5 @@
                             <origin xyz="0.01950 0 0" rpy="0 0 0" />
                         	<geometry>
-                        	    <mesh filename="package://solo_description/meshes/stl/solo12/solo12_hip_fe_fl.stl"/>
+                        	    <mesh filename="package://solo_description/meshes/stl/solo12/simple/solo12_hip_fe_fl.stl"/>
                         	</geometry>
                         </xacro:unless>
@@ -102,5 +102,5 @@
                             <origin xyz="0.01950 0 0" rpy="0 0 0" />
                         	<geometry>
-                        	    <mesh filename="package://solo_description/meshes/stl/solo12/solo12_hip_fe_fr.stl"/>
+                        	    <mesh filename="package://solo_description/meshes/stl/solo12/simple/solo12_hip_fe_fr.stl"/>
                         	</geometry>
                         </xacro:if>
@@ -111,5 +111,5 @@
                             <origin xyz="-0.01950 0 0" rpy="0 0 0" />
                         	<geometry>
-                        	    <mesh filename="package://solo_description/meshes/stl/solo12/solo12_hip_fe_hl.stl"/>
+                        	    <mesh filename="package://solo_description/meshes/stl/solo12/simple/solo12_hip_fe_hl.stl"/>
                         	</geometry>
                         </xacro:unless>
@@ -118,5 +118,5 @@
                             <origin xyz="-0.01950 0 0" rpy="0 0 0" />
                         	<geometry>
-                        	    <mesh filename="package://solo_description/meshes/stl/solo12/solo12_hip_fe_hr.stl"/>
+                        	    <mesh filename="package://solo_description/meshes/stl/solo12/simple/solo12_hip_fe_hr.stl"/>
                         	</geometry>
                         </xacro:if>
@@ -254,8 +254,8 @@
                 <geometry>
                     <xacro:unless value="${is_right}">
-                        <mesh filename="package://solo_description/meshes/stl/with_foot/solo_upper_leg_left_side.stl"/>
-                    </xacro:unless>
-                    <xacro:if value="${is_right}">
-                        <mesh filename="package://solo_description/meshes/stl/with_foot/solo_upper_leg_right_side.stl"/>
+                        <mesh filename="package://solo_description/meshes/stl/with_foot/simple/solo_upper_leg_left_side.stl"/>
+                    </xacro:unless>
+                    <xacro:if value="${is_right}">
+                        <mesh filename="package://solo_description/meshes/stl/with_foot/simple/solo_upper_leg_right_side.stl"/>
                     </xacro:if>
                 </geometry>
@@ -340,8 +340,8 @@
                 <geometry>
                     <xacro:unless value="${is_right}">
-                        <mesh filename="package://solo_description/meshes/stl/with_foot/solo_lower_leg_left_side.stl"/>
-                    </xacro:unless>
-                    <xacro:if value="${is_right}">
-                        <mesh filename="package://solo_description/meshes/stl/with_foot/solo_lower_leg_right_side.stl"/>
+                        <mesh filename="package://solo_description/meshes/stl/with_foot/simple/solo_lower_leg_left_side.stl"/>
+                    </xacro:unless>
+                    <xacro:if value="${is_right}">
+                        <mesh filename="package://solo_description/meshes/stl/with_foot/simple/solo_lower_leg_right_side.stl"/>
                     </xacro:if>
                 </geometry>
@@ -395,5 +395,6 @@
                 <origin xyz="0 0 0" rpy="0 0 0" />
                 <geometry>
-                    <mesh filename="package://solo_description/meshes/stl/with_foot/solo_foot_simple.stl"/>
+                    <!-- mesh filename="package://solo_description/meshes/stl/with_foot/simple/solo_foot.stl"/ -->
+                    <sphere radius="0.015"/>
                 </geometry>
                 <material name="${color_name}">
