Commit message: Updated and tuned hyq

File: hyq_description/robots/hyq.srdf.xacro (robot description, xacro)
@@ -2,5 +2,5 @@
 <robot name="hyq" xmlns:xacro="http://ros.org/wiki/xacro">
   <group name="base">
-    <link name="base_link"/>
+    <link name="trunk"/>
   </group>
   <group name="lf_leg">
@@ -60,3 +60,17 @@
     <joint name="rh_kfe_joint" value="1.5"/>
   </group_state>
+  <group_state group="chains" name="standdown">
+      <joint name="lf_haa_joint" value="-0.1"/>
+      <joint name="lf_hfe_joint" value="0.8"/>
+      <joint name="lf_kfe_joint" value="-2.3"/>
+      <joint name="lh_haa_joint" value="-0.1"/>
+      <joint name="lh_hfe_joint" value="-0.8"/>
+      <joint name="lh_kfe_joint" value="2.3"/>
+      <joint name="rf_haa_joint" value="-0.1"/>
+      <joint name="rf_hfe_joint" value="0.8"/>
+      <joint name="rf_kfe_joint" value="-2.3"/>
+      <joint name="rh_haa_joint" value="-0.1"/>
+      <joint name="rh_hfe_joint" value="-0.8"/>
+      <joint name="rh_kfe_joint" value="2.3"/>
+  </group_state>
 </robot>

File: hyq_description/robots/hyq.urdf.xacro (robot description, xacro)
@@ -7,5 +7,5 @@
 	<xacro:arg name="floating_base_link" default="true"/>
         <xacro:arg name="robot_name"  default="hyq"/>
-        <xacro:arg name="base_name"   default="base_link"/>
+        <xacro:arg name="base_name"   default="trunk"/>
         <!-- load generic materials -->
         <xacro:include filename="$(find wolf_description_utils)/urdfs/materials.xacro"/>
