Commit message: Update hyq kinova and teleop

File: hyq_description/robots/hyq_kinova.srdf.xacro (robot description, xacro)
@@ -2,5 +2,5 @@
 <robot name="hyq" xmlns:xacro="http://ros.org/wiki/xacro">
  <group name="base">
-   <link name="base_link"/>
+   <link name="trunk"/>
  </group>
   <group name="kinova_arm">
@@ -72,3 +72,21 @@
     <joint name="kinova_joint_4" value="-1.5"/>
   </group_state>
+  <group_state group="chains" name="standdown">
+      <joint name="lf_haa_joint" value="-0.1"/>
+      <joint name="lf_hfe_joint" value="0.8"/>
+      <joint name="lf_kfe_joint" value="-2.3"/>
+      <joint name="lh_haa_joint" value="-0.1"/>
+      <joint name="lh_hfe_joint" value="-0.8"/>
+      <joint name="lh_kfe_joint" value="2.3"/>
+      <joint name="rf_haa_joint" value="-0.1"/>
+      <joint name="rf_hfe_joint" value="0.8"/>
+      <joint name="rf_kfe_joint" value="-2.3"/>
+      <joint name="rh_haa_joint" value="-0.1"/>
+      <joint name="rh_hfe_joint" value="-0.8"/>
+      <joint name="rh_kfe_joint" value="2.3"/>
+      <joint name="kinova_joint_1" value="0.0"/>
+      <joint name="kinova_joint_2" value="1.80"/>
+      <joint name="kinova_joint_3" value="4.0"/>
+      <joint name="kinova_joint_4" value="-1.5"/>
+  </group_state>
 </robot>

File: hyq_description/robots/hyq_teleop.srdf.xacro (robot description, xacro)
@@ -2,5 +2,5 @@
 <robot name="hyq" xmlns:xacro="http://ros.org/wiki/xacro">
   <group name="base">
-    <link name="base_link"/>
+    <link name="trunk"/>
   </group>
   <group name="teleop_arm">
@@ -74,3 +74,22 @@
     <joint name="joint5" value="0.0"/>
   </group_state>
+  <group_state group="chains" name="standdown">
+      <joint name="lf_haa_joint" value="-0.1"/>
+      <joint name="lf_hfe_joint" value="0.8"/>
+      <joint name="lf_kfe_joint" value="-2.3"/>
+      <joint name="lh_haa_joint" value="-0.1"/>
+      <joint name="lh_hfe_joint" value="-0.8"/>
+      <joint name="lh_kfe_joint" value="2.3"/>
+      <joint name="rf_haa_joint" value="-0.1"/>
+      <joint name="rf_hfe_joint" value="0.8"/>
+      <joint name="rf_kfe_joint" value="-2.3"/>
+      <joint name="rh_haa_joint" value="-0.1"/>
+      <joint name="rh_hfe_joint" value="-0.8"/>
+      <joint name="rh_kfe_joint" value="2.3"/>
+      <joint name="joint1" value="0.0"/>
+      <joint name="joint2" value="1.0"/>
+      <joint name="joint3" value="1.0"/>
+      <joint name="joint4" value="0.0"/>
+      <joint name="joint5" value="0.0"/>
+  </group_state>
 </robot>

File: hyq_description/urdfs/arm/kinova_adapter.urdf.xacro (robot description, xacro)
@@ -3,5 +3,5 @@
 <link name="kinova_adapter_link"/>
 <joint name="joint_base_robots" type="fixed">
-       <parent link="base_link"/>
+       <parent link="trunk"/>
        <child link="kinova_adapter_link"/>
        <origin xyz="0.5 0.0 0.0" rpy="0 1.57 0"/>

File: hyq_description/urdfs/arm/teleop_adapter.urdf.xacro (robot description, xacro)
@@ -2,10 +2,10 @@
 <robot xmlns:xacro="http://ros.org/wiki/xacro">
  <joint name="joint_base_robots" type="fixed">
-        <parent link="base_link"/>
+        <parent link="trunk"/>
         <child link="teleop_link0"/>
         <origin xyz="0.59 0 0" rpy="0 0 0"/>
  </joint>
 <xacro:include filename="$(find teleop_description)/urdf/teleop.urdf.xacro" />
-<xacro:include filename="$(find hyq_description)/urdfs/arm/arm.transmission.xacro"/>
+<xacro:include filename="$(find wolf_description_utils)/urdfs/arm.transmission.xacro"/>
 <xacro:arm_transmission name="joint1"/>
 <xacro:arm_transmission name="joint2"/>
