Commit message: Use VLP-16 with spot

File: sensors_description/urdfs/sensors/velodyne.gazebo.xacro (robot description, xacro)
@@ -1,9 +1,9 @@
 <?xml version="1.0"?>
 <root xmlns:xacro="http://ros.org/wiki/xacro">
-	<xacro:macro name="velodyne_sensor" params="link_name frame_name lidar_name">
+        <xacro:macro name="velodyne_sensor" params="link_name frame_name lidar_name update_rate">
 		<gazebo reference="${link_name}">
 			<sensor name="${link_name}_velodyne_sensor" type="ray">
 				<always_on>true</always_on>
-				<update_rate>1.0</update_rate>
+                                <update_rate>${update_rate}</update_rate>
 				<pose>0 0 0 0 0 0</pose>
 				<ray>
@@ -29,13 +29,18 @@
 				</ray>
                                 <!-- plugin -->
-                                <!-- <plugin name="${link_name}_controller" filename="libgazebo_ros_block_laser.so"> -->
-                                <plugin name="${link_name}_controller" filename="libgazebo_ros_velodyne_laser.so">
+                                <!--<plugin name="${link_name}_controller" filename="libgazebo_ros_block_laser.so">
 					<gaussianNoise>0.005</gaussianNoise>
 					<alwaysOn>true</alwaysOn>
-					<updateRate>10</updateRate>
+                                        <updateRate>10</updateRate>
 					<topicName>/${lidar_name}/velodyne_pointcloud</topicName>
 					<frameName>${frame_name}</frameName>
 					<hokuyoMinIntensity>101</hokuyoMinIntensity>
-				</plugin>
+                                </plugin>-->
+                                <plugin name="${link_name}_controller" filename="libgazebo_ros_velodyne_laser.so">
+                                    <gaussianNoise>0.005</gaussianNoise>
+                                    <updateRate>${update_rate}</updateRate>
+                                    <topicName>/${lidar_name}/velodyne_pointcloud</topicName>
+                                    <frameName>${frame_name}</frameName>
+                                </plugin>
 			</sensor>
 		</gazebo>

File: spot_description/urdfs/accessories.urdf.xacro (robot description, xacro)
@@ -2,5 +2,6 @@
 <robot xmlns:xacro="http://www.ros.org/wiki/xacro">
   <xacro:include filename="$(find sensors_description)/urdfs/common.xacro"/>
-  <xacro:include filename="$(find sensors_description)/urdfs/sensors/velodyne.gazebo.xacro"/>
+  <!--<xacro:include filename="$(find sensors_description)/urdfs/sensors/velodyne.gazebo.xacro"/>-->
+  <xacro:include filename="$(find velodyne_description)/urdf/VLP-16.urdf.xacro"/>
   <xacro:if value="$(optenv SPOT_PACK 1)">
     <joint name="pack_mount_joint" type="fixed">
@@ -63,5 +64,5 @@
         </collision>
       </link>
-      <joint name="velodyne_joint" type="fixed">
+      <!--<joint name="velodyne_joint" type="fixed">
         <parent link="velodyne_mount"/>
         <child link="velodyne"/>
@@ -69,5 +70,8 @@
       </joint>
       <link name="velodyne"/>
-      <xacro:velodyne_sensor link_name="velodyne" frame_name="velodyne" lidar_name="velodyne"/>
+      <xacro:velodyne_sensor link_name="velodyne" frame_name="velodyne" lidar_name="velodyne" update_rate="10.0"/>-->
+      <xacro:VLP-16 parent="velodyne_mount" name="velodyne" topic="/velodyne_pointcloud" organize_cloud="false" hz="10" samples="440" gpu="true">
+        <origin xyz="0 0 0.0377" rpy="0 0 0" />
+      </xacro:VLP-16>
     </xacro:if>
   </xacro:if>
