Commit message: Remove lumping and add a bit of inertia to the odom frame (is it really needed?)

File: sensors_description/urdfs/sensors/realsense_t265.xacro (robot description, xacro)
@@ -85,5 +85,16 @@
         <origin rpy="0 0 0" xyz="0 0 0"/> <!-- check on real hw -->
     </joint>
-    <link name="${sensor_name}_odom_frame"/>
+    <link name="${sensor_name}_odom_frame">
+    <inertial>
+        <mass value="0.0001"/>
+        <origin rpy="0 0 0" xyz="0 0 0"/>
+        <inertia ixx="0.0001"
+                 ixy="0"
+                 ixz="0"
+                 iyy="0.0001"
+                 iyz="0"
+                 izz="0.0001"/>
+    </inertial>
+    </link>
     <link name="${sensor_name}_pose_frame">
         <visual>
@@ -180,6 +191,9 @@
     </joint>
     <link name="${sensor_name}_accel_frame"/> <!-- dummy -->
+    <gazebo reference="${sensor_name}_odom_frame_joint">
+        <disableFixedJointLumping>true</disableFixedJointLumping>
+    </gazebo>
     <gazebo> <!-- odometry -->
-        <plugin name="p3d_base_controller" filename="libgazebo_ros_p3d.so">
+        <plugin name="t265_odom" filename="libgazebo_ros_p3d.so">
             <alwaysOn>true</alwaysOn>
             <updateRate>${rate}</updateRate>

Commit message: No need for the inertial values

File: sensors_description/urdfs/sensors/realsense_t265.xacro (robot description, xacro)
@@ -85,16 +85,5 @@
         <origin rpy="0 0 0" xyz="0 0 0"/> <!-- check on real hw -->
     </joint>
-    <link name="${sensor_name}_odom_frame">
-    <inertial>
-        <mass value="0.0001"/>
-        <origin rpy="0 0 0" xyz="0 0 0"/>
-        <inertia ixx="0.0001"
-                 ixy="0"
-                 ixz="0"
-                 iyy="0.0001"
-                 iyz="0"
-                 izz="0.0001"/>
-    </inertial>
-    </link>
+    <link name="${sensor_name}_odom_frame"/>
     <link name="${sensor_name}_pose_frame">
         <visual>

Commit message: Add disable_lumping param to t265 macro

File: sensors_description/urdfs/sensors/realsense_t265.xacro (robot description, xacro)
@@ -74,5 +74,5 @@
   </xacro:macro>
   <!-- INTEL REALSENSE T265 -->
-  <xacro:macro name="realsense_T265" params="sensor_name parent_link rate *origin">
+  <xacro:macro name="realsense_T265" params="sensor_name parent_link rate *origin disable_lumping:=true">
     <joint name="${sensor_name}_odom_frame_joint" type="fixed">
         <parent link="${parent_link}"/>
@@ -181,5 +181,5 @@
     <link name="${sensor_name}_accel_frame"/> <!-- dummy -->
     <gazebo reference="${sensor_name}_odom_frame_joint">
-        <disableFixedJointLumping>true</disableFixedJointLumping>
+        <disableFixedJointLumping>${disable_lumping}</disableFixedJointLumping>
     </gazebo>
     <gazebo> <!-- odometry -->
