Commit message: modified zed mini gazebo plugin

File: sensors_description/urdfs/sensors/zed_mini.xacro (robot description, xacro)
@@ -1,175 +1,95 @@
 <?xml version="1.0"?>
 <robot xmlns:xacro="http://www.ros.org/wiki/xacro">
-<!-- TODO make the zed camera eye for a single camera to be used after -->
-  <xacro:macro name="T265_fisheye" params="sensor_name reference_frame topic rate">
-    <gazebo reference="${reference_frame}">
-      <sensor name="camera" type="wideanglecamera">
-        <camera>
-          <horizontal_fov>6.283</horizontal_fov>
-          <image>
-            <width>800</width>
-            <height>848</height>
-          </image>
-          <clip>
-            <near>0.1</near>
-            <far>100</far>
-          </clip>
-          <lens>
-            <type>custom</type>
-            <custom_function>
-              <c1>1.05</c1>
-              <c2>4</c2>
-              <f>1.0</f>
-              <fun>tan</fun>
-            </custom_function>
-            <scale_to_hfov>true</scale_to_hfov>
-            <cutoff_angle>3.1415</cutoff_angle>
-            <env_texture_size>512</env_texture_size>
-          </lens>
-          <always_on>true</always_on>
-          <update_rate>30</update_rate>
-        </camera>
-        <plugin name="camera_controller" filename="libRealsenseGazeboPlugin.so">
-          <alwaysOn>true</alwaysOn>
-          <updateRate>${rate}</updateRate>
-          <cameraName>${sensor_name}/${topic}</cameraName>
-          <imageTopicName>image_raw</imageTopicName>
-          <cameraInfoTopicName>camera_info</cameraInfoTopicName>
-          <frameName>${reference_frame}</frameName>
-          <hackBaseline>0.07</hackBaseline>
-          <distortionK1>-0.007419134024530649</distortionK1>
-          <distortionK2>0.041209351271390915</distortionK2>
-          <distortionK3>-0.03811917081475258</distortionK3>
-          <distortionT1>0.006366158835589886</distortionT1>
-          <distortionT2>0.0</distortionT2>
-          <CxPrime>416.00531005859375</CxPrime>
-          <Cx>16.00531005859375</Cx>
-          <Cy>403.38909912109375</Cy>
-        </plugin>
-      </sensor>
-    </gazebo>
-  </xacro:macro>
-  <!-- INTEL REALSENSE T265 -->
-  <xacro:macro name="zed_mini" params="sensor_name parent_link rate *origin disable_lumping:=true">
+  <xacro:include filename="$(find sensors_description)/urdfs/sensors/zed_mini.gazebo.xacro"/>
+  <xacro:property name="M_PI"     value="3.1415926535897931" />
+  <xacro:property name="baseline" value="0.06" />
+  <xacro:property name="height" value="0.0265" />
+  <xacro:property name="bottom_slope" value="0.0" />
+  <xacro:property name="screw_offset_x" value="0.0" />
+  <xacro:property name="optical_offset_x" value="0.0" />
+  <xacro:property name="deg_to_rad" value="0.01745329251994329577" />
+  <!-- ZED MINI -->
+  <xacro:macro name="zed_mini" params="sensor_name parent_link rate *origin robot_name disable_lumping:=true">
+    <link name="${sensor_name}_odom_frame"/>
     <joint name="${sensor_name}_odom_frame_joint" type="fixed">
         <parent link="${parent_link}"/>
         <child link="${sensor_name}_odom_frame"/>
-        <xacro:insert_block name="origin"/>
+        <xacro:insert_block name="origin" />
     </joint>
-    <joint name="${sensor_name}_pose_frame_joint" type="fixed">
-        <parent link="${sensor_name}_odom_frame"/>
-        <child link="${sensor_name}_pose_frame"/>
-        <origin rpy="0 0 0" xyz="0 0 0"/> <!-- check on real hw -->
+    <!-- Camera mounting point (the threaded screw hole in the bottom) -->
+    <link name="${sensor_name}_base_link" />
+    <joint name="${sensor_name}_base_joint" type="fixed">
+      <parent link="${sensor_name}_odom_frame"/>
+      <child link="${sensor_name}_base_link"/>
+      <origin xyz="0 0 0" rpy="0 0 0"/>
     </joint>
-    <link name="${sensor_name}_odom_frame"/>
-    <link name="${sensor_name}_pose_frame">
-        <visual>
-            <origin rpy="0 0 0" xyz="0 0 0"/>
-            <geometry>
-                <mesh filename="package://sensors_description/meshes/sensors/zed_mini.stl" scale="1 1 1"/>
-            </geometry>
-        </visual>
-        <collision>
-            <geometry>
-                <box size="0.013 0.108 0.024"/>
-            </geometry>
-        </collision>
-        <inertial>
-            <mass value="0.055"/>
-            <origin rpy="0 0 0" xyz="0 0 0"/>
-            <inertia ixx="9.108e-05"
-                     ixy="0"
-                     ixz="0"
-                     iyy="2.51e-06"
-                     iyz="0"
-                     izz="8.931e-05"/>
-        </inertial>
+    <!-- Camera Center -->
+    <link name="${sensor_name}_camera_center">
+      <visual>
+        <origin xyz="${screw_offset_x} 0 0" rpy="0 0 0"/>
+        <geometry>
+          <mesh filename="package://sensors_description/meshes/sensors/zed_mini.stl" />
+        </geometry>
+        <!-- <material name="${model}_mat" /> -->
+      </visual>
+      <collision>
+        <geometry>
+          <mesh filename="package://sensors_description/meshes/sensors/zed_mini.stl" />
+        </geometry>
+      </collision>
     </link>
-    <joint name="${sensor_name}_joint" type="fixed">
-        <parent link="${sensor_name}_pose_frame"/>
-        <child link="${sensor_name}_link"/>
-        <origin rpy="0 0 0" xyz="0 0 0"/> <!-- check on real hw -->
+    <joint name="${sensor_name}_camera_center_joint" type="fixed">
+      <parent link="${sensor_name}_base_link"/>
+      <child link="${sensor_name}_camera_center"/>
+      <origin xyz="0 0 ${height/2}" rpy="0 ${bottom_slope} 0" />
     </joint>
-    <link name="${sensor_name}_link"/>
-    <joint name="${sensor_name}_fisheye1_joint" type="fixed">
-        <parent link="${sensor_name}_link"/>
-        <child link="${sensor_name}_fisheye1_frame"/>
-        <origin rpy="0 0 0" xyz="0 0.042 0"/>
+    <!-- Left Camera -->
+    <link name="${sensor_name}_l_camera_color_optical_frame" />
+    <joint name="${sensor_name}_left_camera_optical_joint" type="fixed">
+      <parent link="${sensor_name}_camera_center"/>
+      <child link="${sensor_name}_l_camera_color_optical_frame"/>
+      <origin xyz="0 ${baseline/2} 0" rpy="0 0 0" />
     </joint>
-    <link name="${sensor_name}_fisheye1_frame"/>
-    <joint name="${sensor_name}_fisheye1_optical_joint" type="fixed">
-        <parent link="${sensor_name}_fisheye1_frame"/>
-        <child link="${sensor_name}_fisheye1_optical_frame"/>
-        <origin rpy="0 0 0" xyz="0.01 0 0"/>
+    <link name="${sensor_name}_l_camera_depth_optical_frame"/>
+    <joint name="${sensor_name}_left_camera_depth_optical_joint" type="fixed">
+      <origin xyz="${optical_offset_x} 0 0" rpy="-${M_PI/2} 0.0 -${M_PI/2}"/>
+      <parent link="${sensor_name}_l_camera_color_optical_frame"/>
+      <child link="${sensor_name}_l_camera_depth_optical_frame"/>
     </joint>
-    <link name="${sensor_name}_fisheye1_optical_frame"/>
-    <xacro:T265_fisheye
-      sensor_name="${sensor_name}"
-      reference_frame="${sensor_name}_fisheye1_optical_frame"
-      topic="fisheye1"
-      rate="${rate}">
-    </xacro:T265_fisheye>
-    <joint name="${sensor_name}_fisheye2_joint" type="fixed">
-        <parent link="${sensor_name}_link"/>
-        <child link="${sensor_name}_fisheye2_frame"/>
-        <origin rpy="0 0 0" xyz="0 -0.022 0"/>
+    <!-- Right Camera -->
+    <link name="${sensor_name}_r_camera_color_optical_frame" />
+    <joint name="${sensor_name}_right_camera_optical_joint" type="fixed">
+      <parent link="${sensor_name}_camera_center"/>
+      <child link="${sensor_name}_r_camera_color_optical_frame"/>
+      <origin xyz="0 -${baseline/2} 0" rpy="0 0 0" />
     </joint>
-    <link name="${sensor_name}_fisheye2_frame"/>
-    <joint name="${sensor_name}_fisheye2_optical_joint" type="fixed">
-        <parent link="${sensor_name}_fisheye2_frame"/>
-        <child link="${sensor_name}_fisheye2_optical_frame"/>
-        <origin rpy="0 0 0" xyz="0.01 0 0"/>
-    </joint>
-    <link name="${sensor_name}_fisheye2_optical_frame"/>
-    <xacro:T265_fisheye
-      sensor_name="${sensor_name}"
-      reference_frame="${sensor_name}_fisheye2_optical_frame"
-      topic="fisheye2"
-      rate="${rate}">
-    </xacro:T265_fisheye>
-    <joint name="${sensor_name}_gyro_joint" type="fixed">
-        <parent link="${sensor_name}_link"/>
-        <child link="${sensor_name}_gyro_frame"/>
-        <origin rpy="0 0 0" xyz="0 0 0"/> <!-- check on real hw -->
+    <link name="${sensor_name}_r_camera_depth_optical_frame"/>
+    <joint name="${sensor_name}_right_camera_depth_optical_joint" type="fixed">
+      <origin xyz="${optical_offset_x} 0 0" rpy="-${M_PI/2} 0.0 -${M_PI/2}"/>
+      <parent link="${sensor_name}_r_camera_color_optical_frame"/>
+      <child link="${sensor_name}_r_camera_depth_optical_frame"/>
     </joint>
     <link name="${sensor_name}_gyro_frame"/>
-    <gazebo reference="${sensor_name}_gyro_frame">
-        <gravity>true</gravity>
-        <sensor name="${sensor_name}_imu" type="imu">
-            <always_on>true</always_on>
-            <update_rate>${rate}</update_rate>
-            <visualize>false</visualize>
-            <plugin filename="libgazebo_ros_imu_sensor.so" name="imu_plugin">
-                <topicName>${sensor_name}/gyro/sample</topicName>
-                <bodyName>${sensor_name}_pose_frame</bodyName>
-                <updateRateHZ>${rate}</updateRateHZ>
-                <gaussianNoise>0.000001</gaussianNoise>
-                <xyzOffset>0 0 0</xyzOffset>
-                <rpyOffset>0 0 0</rpyOffset>
-                <frameName>${sensor_name}_link</frameName>
-            </plugin>
-        </sensor>
-    </gazebo>
+    <joint name="${sensor_name}_gyro_joint" type="fixed">
+        <parent link="${sensor_name}_camera_center"/>
+        <child link="${sensor_name}_gyro_frame"/>
+        <origin rpy="0 0 0" xyz="0 0 0"/>
+    </joint>
+    <link name="${sensor_name}_accel_frame"/>
     <joint name="${sensor_name}_accel_joint" type="fixed">
-        <parent link="${sensor_name}_link"/>
+        <parent link="${sensor_name}_camera_center"/>
         <child link="${sensor_name}_accel_frame"/>
         <origin rpy="0 0 0" xyz="0 0 0"/>
     </joint>
-    <link name="${sensor_name}_accel_frame"/>
-    <gazebo reference="${sensor_name}_odom_frame_joint">
-        <disableFixedJointLumping>${disable_lumping}</disableFixedJointLumping>
-    </gazebo>
-    <gazebo> <!-- odometry -->
-        <plugin name="${sensor_name}_odom" filename="libgazebo_ros_p3d.so">
-            <alwaysOn>true</alwaysOn>
-            <updateRate>${rate}</updateRate>
-            <bodyName>${sensor_name}_odom_frame</bodyName>
-            <topicName>${sensor_name}/odom</topicName>
-            <gaussianNoise>0.001</gaussianNoise>
-            <frameName>world</frameName>
-            <xyzOffsets>0 0 0</xyzOffsets>
-            <rpyOffsets>0 0 0</rpyOffsets>
-        </plugin>
-    </gazebo>
+    <xacro:gazebo_zedm
+      camera_name="${sensor_name}" reference_frame="${sensor_name}_l_camera_color_optical_frame" baseline="${baseline}"
+      left_depth_optical_frame="${sensor_name}_l_camera_depth_optical_frame"
+      right_depth_optical_frame="${sensor_name}_r_camera_depth_optical_frame"
+      left_color_optical_frame="${sensor_name}_l_camera_color_optical_frame"
+      right_color_optical_frame="${sensor_name}_r_camera_color_optical_frame"
+      gyro_frame="${sensor_name}_gyro_frame" camera_center="${sensor_name}_camera_center"
+      odom_frame="${sensor_name}_odom_frame" odom_frame_joint="${sensor_name}_odom_frame_joint"
+      disable_lumping="false" robot_name="${robot_name}"
+    />
   </xacro:macro>
 </robot>
