Commit message: created intel d455 camera gazebo plugin

File: sensors_description/urdfs/sensors/realsense_d455.urdf.xacro (robot description, xacro)
@@ -8,24 +8,30 @@
 <robot name="sensor_d455" xmlns:xacro="http://ros.org/wiki/xacro">
   <!--File includes-->
-  <xacro:include filename="$(find sensors_description)/urdfs/sensors/realsense_d435.gazebo.xacro"/>
+  <xacro:include filename="$(find sensors_description)/urdfs/sensors/realsense_d455.gazebo.xacro"/>
   <xacro:macro name="sensor_d455" params="name:=camera topics_ns:=camera parent *origin">
     <xacro:property name="M_PI" value="3.1415926535897931" />
     <!-- The following values are approximate, and the camera node
      publishing TF values with actual calibrated camera extrinsic values -->
-    <xacro:property name="d435_cam_depth_to_left_ir_offset" value="0.0"/>
-    <xacro:property name="d435_cam_depth_to_right_ir_offset" value="-0.050"/>
-    <xacro:property name="d435_cam_depth_to_color_offset" value="0.015"/>
+    <xacro:property name="d455_cam_depth_to_infra1_offset" value="0.0"/>
+    <xacro:property name="d455_cam_depth_to_infra2_offset" value="-0.095"/>
+    <xacro:property name="d455_cam_depth_to_color_offset" value="-0.059"/>
     <!-- The following values model the aluminum peripherial case for the
-  	D435 camera, with the camera joint represented by the actual
+  	d455 camera, with the camera joint represented by the actual
   	peripherial camera tripod mount -->
-    <xacro:property name="d435_cam_width" value="0.090"/>
-    <xacro:property name="d435_cam_height" value="0.025"/>
-    <xacro:property name="d435_cam_depth" value="0.02505"/>
-    <xacro:property name="d435_cam_mount_from_center_offset" value="0.0149"/>
-    <!-- The following offset is relative the the physical D435 camera peripherial
+    <xacro:property name="d455_cam_width" value="0.124"/>
+    <xacro:property name="d455_cam_height" value="0.029"/>
+    <xacro:property name="d455_cam_depth" value="0.026"/>
+    <xacro:property name="d455_cam_mount_from_center_offset" value="0.0158"/>
+    <!-- glass cover is 0.1 mm inwards from front aluminium plate -->
+    <xacro:property name="d455_glass_to_front" value="0.1e-3"/>
+    <!-- see datasheet Revision 009, Fig. 4-4 page 68 -->
+    <xacro:property name="d455_zero_depth_to_glass" value="4.55e-3"/>
+    <!-- convenience precomputation to avoid clutter-->
+    <xacro:property name="d455_mesh_x_offset" value="${d455_cam_mount_from_center_offset-d455_glass_to_front-d455_zero_depth_to_glass}"/>
+    <!-- The following offset is relative to the physical d455 camera peripherial
   	camera tripod mount -->
-    <xacro:property name="d435_cam_depth_px" value="${d435_cam_mount_from_center_offset}"/>
-    <xacro:property name="d435_cam_depth_py" value="0.0175"/>
-    <xacro:property name="d435_cam_depth_pz" value="${d435_cam_height/2}"/>
+    <xacro:property name="d455_cam_depth_px" value="${d455_cam_mount_from_center_offset}"/>
+    <xacro:property name="d455_cam_depth_py" value="0.0475"/>
+    <xacro:property name="d455_cam_depth_pz" value="${d455_cam_height/2}"/>
     <material name="${name}_aluminum">
 	  <color rgba="0.5 0.5 0.5 1"/>
@@ -39,5 +45,5 @@
     <link name="${name}_bottom_screw_frame"/>
     <joint name="${name}_link_joint" type="fixed">
-      <origin xyz="0 ${d435_cam_depth_py} ${d435_cam_depth_pz}" rpy="0 0 0"/>
+      <origin xyz="${d455_mesh_x_offset} ${d455_cam_depth_py} ${d455_cam_depth_pz}" rpy="0 0 0"/>
       <parent link="${name}_bottom_screw_frame"/>
       <child link="${name}_link" />
@@ -45,5 +51,5 @@
     <link name="${name}_link">
       <visual>
-      <origin xyz="${d435_cam_mount_from_center_offset} ${-d435_cam_depth_py} 0" rpy="${M_PI/2} 0 ${M_PI/2}"/>
+      <origin xyz="${d455_zero_depth_to_glass + d455_glass_to_front} ${-d455_cam_depth_py} 0" rpy="${M_PI/2} 0 ${M_PI/2}"/>
         <geometry>
           <mesh filename="package://sensors_description/meshes/sensors/realsense_d455.stl" scale="0.001 0.001 0.001" />
@@ -52,12 +58,12 @@
       </visual>
       <collision>
-        <origin xyz="0 ${-d435_cam_depth_py} 0" rpy="0 0 0"/>
+        <origin xyz="${d455_zero_depth_to_glass-d455_cam_depth/2} ${-d455_cam_depth_py} 0" rpy="0 0 0"/>
         <geometry>
-        <box size="${d435_cam_depth} ${d435_cam_width} ${d435_cam_height}"/>
+          <box size="${d455_cam_depth} ${d455_cam_width} ${d455_cam_height}"/>
         </geometry>
       </collision>
       <inertial>
         <!-- The following are not reliable values, and should not be used for modeling -->
-        <mass value="0.564" />
+        <mass value="0.072" />
         <origin xyz="0 0 0" />
         <inertia ixx="0.003881243" ixy="0.0" ixz="0.0" iyy="0.000498940" iyz="0.0" izz="0.003879257" />
@@ -78,33 +84,33 @@
     <link name="${name}_depth_optical_frame"/>
     <!-- camera left IR joints and links -->
-    <joint name="${name}_left_ir_joint" type="fixed">
-      <origin xyz="0 ${d435_cam_depth_to_left_ir_offset} 0" rpy="0 0 0" />
-      <parent link="${name}_depth_frame" />
-      <child link="${name}_left_ir_frame" />
+    <joint name="${name}_infra1_joint" type="fixed">
+      <origin xyz="0 ${d455_cam_depth_to_infra1_offset} 0" rpy="0 0 0" />
+      <parent link="${name}_link" />
+      <child link="${name}_infra1_frame" />
     </joint>
-    <link name="${name}_left_ir_frame"/>
-    <joint name="${name}_left_ir_optical_joint" type="fixed">
+    <link name="${name}_infra1_frame"/>
+    <joint name="${name}_infra1_optical_joint" type="fixed">
       <origin xyz="0 0 0" rpy="${-M_PI/2} 0 ${-M_PI/2}" />
-      <parent link="${name}_left_ir_frame" />
-      <child link="${name}_left_ir_optical_frame" />
+      <parent link="${name}_infra1_frame" />
+      <child link="${name}_infra1_optical_frame" />
     </joint>
-    <link name="${name}_left_ir_optical_frame"/>
+    <link name="${name}_infra1_optical_frame"/>
     <!-- camera right IR joints and links -->
-    <joint name="${name}_right_ir_joint" type="fixed">
-      <origin xyz="0 ${d435_cam_depth_to_right_ir_offset} 0" rpy="0 0 0" />
-      <parent link="${name}_depth_frame" />
-      <child link="${name}_right_ir_frame" />
+    <joint name="${name}_infra2_joint" type="fixed">
+      <origin xyz="0 ${d455_cam_depth_to_infra2_offset} 0" rpy="0 0 0" />
+      <parent link="${name}_link" />
+      <child link="${name}_infra2_frame" />
     </joint>
-    <link name="${name}_right_ir_frame"/>
-    <joint name="${name}_right_ir_optical_joint" type="fixed">
+    <link name="${name}_infra2_frame"/>
+    <joint name="${name}_infra2_optical_joint" type="fixed">
       <origin xyz="0 0 0" rpy="${-M_PI/2} 0 ${-M_PI/2}" />
-      <parent link="${name}_right_ir_frame" />
-      <child link="${name}_right_ir_optical_frame" />
+      <parent link="${name}_infra2_frame" />
+      <child link="${name}_infra2_optical_frame" />
     </joint>
-    <link name="${name}_right_ir_optical_frame"/>
+    <link name="${name}_infra2_optical_frame"/>
     <!-- camera color joints and links -->
     <joint name="${name}_color_joint" type="fixed">
-      <origin xyz="0 ${d435_cam_depth_to_color_offset} 0" rpy="0 0 0" />
-      <parent link="${name}_depth_frame" />
+      <origin xyz="0 ${d455_cam_depth_to_color_offset} 0" rpy="0 0 0" />
+      <parent link="${name}_link" />
       <child link="${name}_color_frame" />
     </joint>
@@ -116,6 +122,45 @@
     </joint>
     <link name="${name}_color_optical_frame"/>
+    <!-- IMU -->
+    <!-- see datasheet Revision 009, page 114 -->
+    <xacro:property name="d455_imu_px" value="-0.01602"/>
+    <xacro:property name="d455_imu_py" value="-0.03022"/>
+    <xacro:property name="d455_imu_pz" value="+0.0074"/>
+    <link name="${name}_accel_frame" />
+    <link name="${name}_accel_optical_frame" />
+    <link name="${name}_gyro_frame" />
+    <link name="${name}_gyro_optical_frame" />
+    <link name="${name}_imu_optical_frame" />
+    <joint name="${name}_accel_joint" type="fixed">
+      <origin xyz = "${d455_imu_px} ${d455_imu_py} ${d455_imu_pz}" rpy = "0 0 0" />
+      <parent link="${name}_link" />
+      <child link="${name}_accel_frame" />
+    </joint>
+    <joint name="${name}_accel_optical_joint" type="fixed">
+      <origin xyz = "0 0 0" rpy = "${-M_PI/2} 0 ${-M_PI/2}" />
+      <parent link="${name}_accel_frame" />
+      <child link="${name}_accel_optical_frame" />
+    </joint>
+    <joint name="${name}_gyro_joint" type="fixed">
+      <origin xyz = "${d455_imu_px} ${d455_imu_py} ${d455_imu_pz}" rpy = "0 0 0" />
+      <parent link="${name}_link" />
+      <child link="${name}_gyro_frame" />
+    </joint>
+    <joint name="${name}_gyro_optical_joint" type="fixed">
+      <origin xyz = "0 0 0" rpy = "${-M_PI/2} 0 ${-M_PI/2}" />
+      <parent link="${name}_gyro_frame" />
+      <child link="${name}_gyro_optical_frame" />
+    </joint>
+    <joint name="${name}_imu_optical_joint" type="fixed">
+      <origin xyz = "0 0 0" rpy = "0 0 0" />
+      <parent link="${name}_gyro_optical_frame" />
+      <child link="${name}_imu_optical_frame" />
+    </joint>
     <!-- Realsense Gazebo Plugin -->
-    <xacro:gazebo_d435 camera_name="${name}" reference_link="${name}_link" topics_ns="${topics_ns}" depth_optical_frame="${name}_depth_optical_frame" color_optical_frame="${name}_color_optical_frame" infrared1_optical_frame="${name}_left_ir_optical_frame" infrared2_optical_frame="${name}_right_ir_optical_frame"/>
+    <xacro:gazebo_d455 camera_name="${name}" reference_link="${name}_link" topics_ns="${topics_ns}"
+      depth_optical_frame="${name}_depth_optical_frame" color_optical_frame="${name}_color_optical_frame"
+      infrared1_optical_frame="${name}_left_ir_optical_frame"
+      infrared2_optical_frame="${name}_right_ir_optical_frame"
+    />
   </xacro:macro>
 </robot>
