Commit message: detached camera_odom_frame from camera model (lumping block camera publishing)

File: sensors_description/urdfs/sensors/zed_mini.urdf.xacro (robot description, xacro)
@@ -11,15 +11,16 @@
   <!-- ZED MINI -->
   <xacro:macro name="zed_mini" params="sensor_name parent_link rate *origin robot_name disable_lumping:=true">
-    <link name="${sensor_name}_odom_frame"/>
-    <joint name="${sensor_name}_odom_frame_joint" type="fixed">
-        <parent link="${parent_link}"/>
-        <child link="${sensor_name}_odom_frame"/>
-        <xacro:insert_block name="origin" />
-    </joint>
     <!-- Camera mounting point (the threaded screw hole in the bottom) -->
     <link name="${sensor_name}_base_link" />
     <joint name="${sensor_name}_base_joint" type="fixed">
-      <parent link="${sensor_name}_odom_frame"/>
+      <parent link="${parent_link}"/>
       <child link="${sensor_name}_base_link"/>
+      <xacro:insert_block name="origin" />
+    </joint>
+    <!-- odom frame for odometry -->
+    <link name="${sensor_name}_odom_frame"/>
+    <joint name="${sensor_name}_odom_frame_joint" type="fixed">
+      <parent link="${sensor_name}_base_link"/>
+      <child link="${sensor_name}_odom_frame"/>
       <origin xyz="0 0 0" rpy="0 0 0"/>
     </joint>

Commit message: added inertia to zed mini otherwise gazebo disable_lumping does not work

File: sensors_description/urdfs/sensors/zed_mini.urdf.xacro (robot description, xacro)
@@ -25,4 +25,22 @@
       <origin xyz="0 0 0" rpy="0 0 0"/>
     </joint>
+    <!-- fake odom frame to disable odom lumping -->
+    <link name="${sensor_name}_fake_odom">
+      <inertial>
+        <mass value="0.001"/>
+        <origin rpy="0 0 0" xyz="0 0 0"/>
+        <inertia ixx="9.108e-08"
+                  ixy="0"
+                  ixz="0"
+                  iyy="2.51e-08"
+                  iyz="0"
+                  izz="8.931e-08"/>
+      </inertial>
+    </link>
+    <joint name="${sensor_name}_odom_fake_joint" type="fixed">
+      <parent link="${sensor_name}_odom_frame"/>
+      <child link="${sensor_name}_fake_odom"/>
+      <origin xyz="0 0 0" rpy="0 0 0" />
+    </joint>
     <!-- Camera Center -->
     <link name="${sensor_name}_camera_center">
@@ -39,4 +57,14 @@
         </geometry>
       </collision>
+      <inertial>
+        <mass value="0.055"/>
+        <origin rpy="0 0 0" xyz="0 0 0"/>
+        <inertia ixx="9.108e-05"
+                  ixy="0"
+                  ixz="0"
+                  iyy="2.51e-06"
+                  iyz="0"
+                  izz="8.931e-05"/>
+      </inertial>
     </link>
     <joint name="${sensor_name}_camera_center_joint" type="fixed">
