Commit message: renamed realsense d435 xacros files

File: sensors_description/urdfs/sensors/realsense_d435.urdf.xacro (robot description, xacro)
@@ -8,5 +8,5 @@
 <robot name="sensor_d435" xmlns:xacro="http://ros.org/wiki/xacro">
   <!--File includes-->
-  <xacro:include filename="$(find sensors_description)/urdfs/sensors/_d435.gazebo.xacro"/>
+  <xacro:include filename="$(find sensors_description)/urdfs/sensors/realsense_d435.gazebo.xacro"/>
   <xacro:macro name="sensor_d435" params="name:=camera topics_ns:=camera parent *origin">
     <xacro:property name="M_PI" value="3.1415926535897931" />
@@ -48,5 +48,6 @@
         <geometry>
           <!-- <box size="${d435_cam_width} ${d435_cam_height} ${d435_cam_depth}"/> -->
-          <mesh filename="package://realsense2_description/meshes/d435.dae" />
+<!--          <mesh filename="package://realsense2_description/meshes/d435.dae" />-->
+          <mesh filename="package://sensors_description/meshes/sensors/realsense_d435.stl" />
           <!--<mesh filename="package://realsense2_description/meshes/d435/d435.dae" />-->
         </geometry>

Commit message: Making the sensor macros look alike

File: sensors_description/urdfs/sensors/realsense_d435.urdf.xacro (robot description, xacro)
@@ -6,8 +6,8 @@
 aluminum peripherial evaluation case.
 -->
-<robot name="sensor_d435" xmlns:xacro="http://ros.org/wiki/xacro">
+<robot name="realsense_d435" xmlns:xacro="http://ros.org/wiki/xacro">
   <!--File includes-->
   <xacro:include filename="$(find sensors_description)/urdfs/sensors/realsense_d435.gazebo.xacro"/>
-  <xacro:macro name="sensor_d435" params="name:=camera topics_ns:=camera parent *origin">
+  <xacro:macro name="realsense_d435" params="name:=camera topics_ns:=camera parent *origin">
     <xacro:property name="M_PI" value="3.1415926535897931" />
     <!-- The following values are approximate, and the camera node

File: sensors_description/urdfs/sensors/realsense_t265.urdf.xacro (robot description, xacro)
@@ -25,5 +25,5 @@
   <Cy>403.38909912109375</Cy>
   -->
-  <xacro:macro name="T265_fisheye" params="sensor_name reference_frame topic rate">
+  <xacro:macro name="T265_fisheye" params="name reference_frame topic rate">
     <gazebo reference="${reference_frame}">
       <sensor name="camera" type="wideanglecamera">
@@ -56,5 +56,5 @@
           <alwaysOn>true</alwaysOn>
           <updateRate>${rate}</updateRate>
-          <cameraName>${sensor_name}/${topic}</cameraName>
+          <cameraName>${name}/${topic}</cameraName>
           <imageTopicName>image_raw</imageTopicName>
           <cameraInfoTopicName>camera_info</cameraInfoTopicName>
@@ -74,17 +74,17 @@
   </xacro:macro>
   <!-- INTEL REALSENSE T265 -->
-  <xacro:macro name="realsense_T265" params="sensor_name parent_link rate *origin disable_lumping:=true">
-    <joint name="${sensor_name}_odom_frame_joint" type="fixed">
-        <parent link="${parent_link}"/>
-        <child link="${sensor_name}_odom_frame"/>
+  <xacro:macro name="realsense_T265" params="name topics_ns parent rate *origin disable_lumping:=true">
+    <joint name="${name}_odom_frame_joint" type="fixed">
+        <parent link="${parent}"/>
+        <child link="${name}_odom_frame"/>
         <xacro:insert_block name="origin"/>
     </joint>
-    <joint name="${sensor_name}_pose_frame_joint" type="fixed">
-        <parent link="${sensor_name}_odom_frame"/>
-        <child link="${sensor_name}_pose_frame"/>
+    <joint name="${name}_pose_frame_joint" type="fixed">
+        <parent link="${name}_odom_frame"/>
+        <child link="${name}_pose_frame"/>
         <origin rpy="0 0 0" xyz="0 0 0"/> <!-- check on real hw -->
     </joint>
-    <link name="${sensor_name}_odom_frame"/>
-    <link name="${sensor_name}_pose_frame">
+    <link name="${name}_odom_frame"/>
+    <link name="${name}_pose_frame">
         <visual>
             <origin rpy="1.57 0 1.57" xyz="0 0 0"/>
@@ -109,76 +109,76 @@
         </inertial>
     </link>
-    <joint name="${sensor_name}_joint" type="fixed">
-        <parent link="${sensor_name}_pose_frame"/>
-        <child link="${sensor_name}_link"/>
+    <joint name="${name}_joint" type="fixed">
+        <parent link="${name}_pose_frame"/>
+        <child link="${name}_link"/>
         <origin rpy="0 0 0" xyz="0 0 0"/> <!-- check on real hw -->
     </joint>
-    <link name="${sensor_name}_link"/>
-    <joint name="${sensor_name}_fisheye1_joint" type="fixed">
-        <parent link="${sensor_name}_link"/>
-        <child link="${sensor_name}_fisheye1_frame"/>
+    <link name="${name}_link"/>
+    <joint name="${name}_fisheye1_joint" type="fixed">
+        <parent link="${name}_link"/>
+        <child link="${name}_fisheye1_frame"/>
         <origin rpy="0 0 0" xyz="0 0.042 0"/>
     </joint>
-    <link name="${sensor_name}_fisheye1_frame"/>
-    <joint name="${sensor_name}_fisheye1_optical_joint" type="fixed">
-        <parent link="${sensor_name}_fisheye1_frame"/>
-        <child link="${sensor_name}_fisheye1_optical_frame"/>
+    <link name="${name}_fisheye1_frame"/>
+    <joint name="${name}_fisheye1_optical_joint" type="fixed">
+        <parent link="${name}_fisheye1_frame"/>
+        <child link="${name}_fisheye1_optical_frame"/>
         <origin rpy="0 0 0" xyz="0.01 0 0"/>
     </joint>
-    <link name="${sensor_name}_fisheye1_optical_frame"/>
+    <link name="${name}_fisheye1_optical_frame"/>
     <xacro:T265_fisheye
-      sensor_name="${sensor_name}"
-      reference_frame="${sensor_name}_fisheye1_optical_frame"
+      name="${name}"
+      reference_frame="${name}_fisheye1_optical_frame"
       topic="fisheye1"
       rate="${rate}">
     </xacro:T265_fisheye>
-    <joint name="${sensor_name}_fisheye2_joint" type="fixed">
-        <parent link="${sensor_name}_link"/>
-        <child link="${sensor_name}_fisheye2_frame"/>
+    <joint name="${name}_fisheye2_joint" type="fixed">
+        <parent link="${name}_link"/>
+        <child link="${name}_fisheye2_frame"/>
         <origin rpy="0 0 0" xyz="0 -0.022 0"/>
     </joint>
-    <link name="${sensor_name}_fisheye2_frame"/>
-    <joint name="${sensor_name}_fisheye2_optical_joint" type="fixed">
-        <parent link="${sensor_name}_fisheye2_frame"/>
-        <child link="${sensor_name}_fisheye2_optical_frame"/>
+    <link name="${name}_fisheye2_frame"/>
+    <joint name="${name}_fisheye2_optical_joint" type="fixed">
+        <parent link="${name}_fisheye2_frame"/>
+        <child link="${name}_fisheye2_optical_frame"/>
         <origin rpy="0 0 0" xyz="0.01 0 0"/>
     </joint>
-    <link name="${sensor_name}_fisheye2_optical_frame"/>
+    <link name="${name}_fisheye2_optical_frame"/>
     <xacro:T265_fisheye
-      sensor_name="${sensor_name}"
-      reference_frame="${sensor_name}_fisheye2_optical_frame"
+      name="${name}"
+      reference_frame="${name}_fisheye2_optical_frame"
       topic="fisheye2"
       rate="${rate}">
     </xacro:T265_fisheye>
-    <joint name="${sensor_name}_gyro_joint" type="fixed">
-        <parent link="${sensor_name}_link"/>
-        <child link="${sensor_name}_gyro_frame"/>
+    <joint name="${name}_gyro_joint" type="fixed">
+        <parent link="${name}_link"/>
+        <child link="${name}_gyro_frame"/>
         <origin rpy="0 0 0" xyz="0 0 0"/> <!-- check on real hw -->
     </joint>
-    <link name="${sensor_name}_gyro_frame"/>
-    <gazebo reference="${sensor_name}_gyro_frame">
+    <link name="${name}_gyro_frame"/>
+    <gazebo reference="${name}_gyro_frame">
         <gravity>true</gravity>
-        <sensor name="${sensor_name}_imu" type="imu">
+        <sensor name="${name}_imu" type="imu">
             <always_on>true</always_on>
             <update_rate>${rate}</update_rate>
             <visualize>false</visualize>
             <plugin filename="libgazebo_ros_imu_sensor.so" name="imu_plugin">
-                <topicName>${sensor_name}/gyro/sample</topicName>
-                <bodyName>${sensor_name}_pose_frame</bodyName>
+                <topicName>${topics_ns}/gyro/sample</topicName>
+                <bodyName>${name}_pose_frame</bodyName>
                 <updateRateHZ>${rate}</updateRateHZ>
                 <gaussianNoise>0.000001</gaussianNoise>
                 <xyzOffset>0 0 0</xyzOffset>
                 <rpyOffset>0 0 0</rpyOffset>
-                <frameName>${sensor_name}_link</frameName>
+                <frameName>${name}_link</frameName>
             </plugin>
         </sensor>
     </gazebo>
-    <joint name="${sensor_name}_accel_joint" type="fixed">
-        <parent link="${sensor_name}_link"/>
-        <child link="${sensor_name}_accel_frame"/>
+    <joint name="${name}_accel_joint" type="fixed">
+        <parent link="${name}_link"/>
+        <child link="${name}_accel_frame"/>
         <origin rpy="0 0 0" xyz="0 0 0"/> <!-- check on real hw -->
     </joint>
-    <link name="${sensor_name}_accel_frame"/> <!-- dummy -->
-    <gazebo reference="${sensor_name}_odom_frame_joint">
+    <link name="${name}_accel_frame"/> <!-- dummy -->
+    <gazebo reference="${name}_odom_frame_joint">
         <disableFixedJointLumping>${disable_lumping}</disableFixedJointLumping>
     </gazebo>
@@ -187,6 +187,6 @@
             <alwaysOn>true</alwaysOn>
             <updateRate>${rate}</updateRate>
-            <bodyName>${sensor_name}_odom_frame</bodyName>
-            <topicName>${sensor_name}/odom</topicName>
+            <bodyName>${name}_odom_frame</bodyName>
+            <topicName>${topics_ns}/odom</topicName>
             <gaussianNoise>0.001</gaussianNoise>
             <frameName>world</frameName>

File: spot_description/urdfs/accessories.urdf.xacro (robot description, xacro)
@@ -72,8 +72,8 @@
         <origin xyz="0 0 0" rpy="0 0 0" />
       </xacro:VLP-16>
-      <xacro:sensor_d435 name="d435" topics_ns="/$(arg robot_name)/d435" parent="front_rail">
+      <xacro:realsense_d435 name="d435" topics_ns="/$(arg robot_name)/d435" parent="front_rail">
         <origin xyz="0.13 0 0" rpy="0 0 0" />
-      </xacro:sensor_d435>
-      <xacro:realsense_T265 sensor_name="/$(arg robot_name)/t265" parent_link="front_rail" rate="30.0">
+      </xacro:realsense_d435>
+      <xacro:realsense_T265 name="t265" topics_ns="/$(arg robot_name)/t265" parent="front_rail" rate="30.0">
         <origin xyz="0.13 0 0.04" rpy="0 0 0" />
       </xacro:realsense_T265>
