Commit message: Update sensors
add ad namespace filter for the frames in imu and gps

File: sensors_description/urdfs/sensors/gps.gazebo.xacro (robot description, xacro)
@@ -1,13 +1,19 @@
 <?xml version="1.0"?>
 <robot xmlns:xacro="http://ros.org/wiki/xacro">
-        <xacro:macro name="gps_sensor" params="gps_name gps_topic vel_topic robot_name frame_name update_rate">
+        <xacro:macro name="gps_sensor" params="gps_topic vel_topic namespace frame_name update_rate">
+            <xacro:if value="${namespace == ''}">
+                <xacro:property name="frame_name_ns" value="${frame_name}"/>
+            </xacro:if>
+            <xacro:if value="${namespace != ''}">
+                <xacro:property name="frame_name_ns" value="${namespace+'/'+frame_name}"/>
+            </xacro:if>
             <gazebo>
                 <!-- plugins are in hector_gazebo_plugins ros package -->
-                <plugin name="${gps_name}" filename="libhector_gazebo_ros_gps.so">
-                    <robotNamespace>${robot_name}/gps/</robotNamespace>
+                <plugin name="gps_sensor_plugin" filename="libhector_gazebo_ros_gps.so">
+                    <robotNamespace>${namespace}/gps/</robotNamespace>
                     <alwaysOn>1</alwaysOn>
                     <updateRate>10.0</updateRate>
                     <bodyName>${frame_name}</bodyName>
-                    <frameId>${frame_name}</frameId>
+                    <frameId>${frame_name_ns}</frameId>
                     <topicName>${gps_topic}</topicName>
                     <velocityTopicName>${vel_topic}</velocityTopicName>

File: sensors_description/urdfs/sensors/imu.gazebo.xacro (robot description, xacro)
@@ -1,5 +1,5 @@
 <?xml version="1.0"?>
 <robot xmlns:xacro="http://ros.org/wiki/xacro">
-	<xacro:macro name="imu_sensor" params="imu_name imu_topic update_rate rate_mean rate_stddev
+        <xacro:macro name="imu_sensor" params="imu_name imu_topic namespace update_rate rate_mean rate_stddev
 		rate_bias_mean rate_bias_stddev accel_mean accel_stddev accel_bias_mean accel_bias_stddev">
                 <!-- old plugin -->
@@ -41,4 +41,10 @@
                 </gazebo>-->
                 <!-- recent plugin with gravity acceleration -->
+                <xacro:if value="${namespace == ''}">
+                    <xacro:property name="frame_name" value="${imu_name}"/>
+                </xacro:if>
+                <xacro:if value="${namespace != ''}">
+                    <xacro:property name="frame_name" value="${namespace+'/'+imu_name}"/>
+                </xacro:if>
                 <gazebo reference="${imu_name}">
                    <gravity>true</gravity>
@@ -48,5 +54,6 @@
                      <visualize>true</visualize>
                      <topic>__default_topic__</topic>
-                     <plugin filename="libgazebo_ros_imu_sensor.so" name="imu_plugin">
+                     <plugin name="imu_sensor_plugin" filename="libgazebo_ros_imu_sensor.so">
+                       <robotNamespace>${namespace}</robotNamespace>
                        <topicName>${imu_topic}</topicName>
                        <bodyName>${imu_name}</bodyName>
@@ -55,5 +62,5 @@
                        <xyzOffset>0 0 0</xyzOffset>
                        <rpyOffset>0 0 0</rpyOffset>
-                       <frameName>${imu_name}</frameName>
+                       <frameName>${frame_name}</frameName>
                        <initialOrientationAsReference>false</initialOrientationAsReference>
                      </plugin>

File: sensors_description/urdfs/sensors/realsense_t265.urdf.xacro (robot description, xacro)
@@ -25,5 +25,5 @@
   <Cy>403.38909912109375</Cy>
   -->
-  <xacro:macro name="T265_fisheye" params="name reference_frame topic rate">
+  <xacro:macro name="fisheye_t265" params="name topics_ns reference_frame rate">
     <gazebo reference="${reference_frame}">
       <sensor name="camera" type="wideanglecamera">
@@ -56,7 +56,7 @@
           <alwaysOn>true</alwaysOn>
           <updateRate>${rate}</updateRate>
-          <cameraName>${name}/${topic}</cameraName>
-          <imageTopicName>image_raw</imageTopicName>
-          <cameraInfoTopicName>camera_info</cameraInfoTopicName>
+          <cameraName>${name}</cameraName>
+          <imageTopicName>${topics_ns}/${name}_image_raw</imageTopicName>
+          <cameraInfoTopicName>${topics_ns}/${name}_camera_info</cameraInfoTopicName>
           <frameName>${reference_frame}</frameName>
           <hackBaseline>0.07</hackBaseline>
@@ -127,10 +127,10 @@
     </joint>
     <link name="${name}_fisheye1_optical_frame"/>
-    <xacro:T265_fisheye
-      name="${name}"
+    <xacro:fisheye_t265
+      name="${name}_fisheye1"
       reference_frame="${name}_fisheye1_optical_frame"
-      topic="fisheye1"
+      topics_ns="${topics_ns}"
       rate="${rate}">
-    </xacro:T265_fisheye>
+    </xacro:fisheye_t265>
     <joint name="${name}_fisheye2_joint" type="fixed">
         <parent link="${name}_link"/>
@@ -145,10 +145,10 @@
     </joint>
     <link name="${name}_fisheye2_optical_frame"/>
-    <xacro:T265_fisheye
-      name="${name}"
+    <xacro:fisheye_t265
+      name="${name}_fisheye2"
       reference_frame="${name}_fisheye2_optical_frame"
-      topic="fisheye2"
+      topics_ns="${topics_ns}"
       rate="${rate}">
-    </xacro:T265_fisheye>
+    </xacro:fisheye_t265>
     <joint name="${name}_gyro_joint" type="fixed">
         <parent link="${name}_link"/>
@@ -164,4 +164,5 @@
             <visualize>false</visualize>
             <plugin filename="libgazebo_ros_imu_sensor.so" name="imu_plugin">
+                <robotNamespace>${topics_ns}</robotNamespace>
                 <topicName>${topics_ns}/gyro/sample</topicName>
                 <bodyName>${name}_pose_frame</bodyName>
@@ -183,10 +184,12 @@
         <disableFixedJointLumping>${disable_lumping}</disableFixedJointLumping>
     </gazebo>
-    <gazebo> <!-- odometry -->
+    <gazebo>
+    <!-- odometry -->
         <plugin name="t265_odom" filename="libgazebo_ros_p3d.so">
             <alwaysOn>true</alwaysOn>
             <updateRate>${rate}</updateRate>
+            <robotNamespace>${topics_ns}</robotNamespace>
             <bodyName>${name}_odom_frame</bodyName>
-            <topicName>${topics_ns}/odom</topicName>
+            <topicName>${name}/odom</topicName>
             <gaussianNoise>0.001</gaussianNoise>
             <frameName>world</frameName>

Commit message: Add frame_name_ns in sensors

File: sensors_description/urdfs/sensors/gps.gazebo.xacro (robot description, xacro)
@@ -13,4 +13,10 @@
   -->
   <xacro:macro name="gazebo_gps_sensor" params="sensor_name namespace gps_topic velocity_topic update_rate frame_id">
+      <xacro:if value="${namespace == ''}">
+                    <xacro:property name="frame_name_ns" value="${frame_id}"/>
+      </xacro:if>
+      <xacro:if value="${namespace != ''}">
+                    <xacro:property name="frame_name_ns" value="${namespace+'/'+frame_id}"/>
+      </xacro:if>
     <gazebo reference="${frame_id}">
       <sensor type="gps" name="${sensor_name}">
@@ -27,5 +33,5 @@
             <remapping>gps_plugin/vel:=${velocity_topic}</remapping>
           </ros>
-          <frameId>${frame_id}</frameId>
+          <frame_name>${frame_name_ns}</frame_name>
         </plugin>
       </sensor>

File: sensors_description/urdfs/sensors/imu.gazebo.xacro (robot description, xacro)
@@ -3,4 +3,10 @@
     <xacro:macro name="imu_sensor" params="frame_name imu_topic namespace update_rate rate_mean rate_stddev
         rate_bias_mean rate_bias_stddev accel_mean accel_stddev accel_bias_mean accel_bias_stddev">
+      <xacro:if value="${namespace == ''}">
+                    <xacro:property name="frame_name_ns" value="${frame_name}"/>
+      </xacro:if>
+      <xacro:if value="${namespace != ''}">
+                    <xacro:property name="frame_name_ns" value="${namespace+'/'+frame_name}"/>
+      </xacro:if>
         <gazebo reference="trunk_imu">
             <gravity>true</gravity>
@@ -19,5 +25,5 @@
                     <xyz_offset>0 0 0</xyz_offset>
                     <rpy_offset>0 0 0</rpy_offset>
-                    <frame_name>${frame_name}</frame_name>
+                    <frame_name>${frame_name_ns}</frame_name>
                     <initial_orientation_as_reference>false</initial_orientation_as_reference>
                 </plugin>

File: sensors_description/urdfs/sensors/lidar.gazebo.xacro (robot description, xacro)
@@ -2,4 +2,10 @@
 <robot xmlns:xacro="http://ros.org/wiki/xacro">
 <xacro:macro name="velodyne_laser_gazebo_sensor" params="sensor_name topic_name update_rate frame_id namespace min_range max_range number_of_beams horizontal_samples horizontal_fov vertical_fov noise_stddev">
+      <xacro:if value="${namespace == ''}">
+                    <xacro:property name="frame_name_ns" value="${frame_id}"/>
+      </xacro:if>
+      <xacro:if value="${namespace != ''}">
+                    <xacro:property name="frame_name_ns" value="${namespace+'/'+frame_id}"/>
+      </xacro:if>
   <gazebo reference="${frame_id}">
         <sensor type="ray" name="${sensor_name}">
@@ -38,5 +44,5 @@
               <remapping>gazebo_ros_laser_controller/out:=${topic_name}</remapping>
             </ros>
-            <frame_name>${frame_id}</frame_name>
+            <frame_name>${frame_name_ns}</frame_name>
             <organize_cloud>true</organize_cloud>
             <min_range>${min_range}</min_range>
