Commit message: Change param names in imu macro

File: sensors_description/urdfs/sensors/imu.gazebo.xacro (robot description, xacro)
@@ -1,5 +1,5 @@
 <?xml version="1.0"?>
 <robot xmlns:xacro="http://ros.org/wiki/xacro">
-        <xacro:macro name="imu_sensor" params="imu_name imu_topic namespace update_rate rate_mean rate_stddev
+        <xacro:macro name="imu_sensor" params="frame_name imu_topic namespace update_rate rate_mean rate_stddev
 		rate_bias_mean rate_bias_stddev accel_mean accel_stddev accel_bias_mean accel_bias_stddev">
                 <!-- old plugin -->
@@ -42,12 +42,12 @@
                 <!-- recent plugin with gravity acceleration -->
                 <xacro:if value="${namespace == ''}">
-                    <xacro:property name="frame_name" value="${imu_name}"/>
+                    <xacro:property name="frame_name_ns" value="${frame_name}"/>
                 </xacro:if>
                 <xacro:if value="${namespace != ''}">
-                    <xacro:property name="frame_name" value="${namespace+'/'+imu_name}"/>
+                    <xacro:property name="frame_name_ns" value="${namespace+'/'+frame_name}"/>
                 </xacro:if>
-                <gazebo reference="${imu_name}">
+                <gazebo reference="${frame_name}">
                    <gravity>true</gravity>
-                   <sensor name="${imu_name}" type="imu">
+                   <sensor name="${frame_name}_sensor" type="imu">
                      <always_on>true</always_on>
                      <update_rate>${update_rate}</update_rate>
@@ -57,10 +57,10 @@
                        <robotNamespace>${namespace}</robotNamespace>
                        <topicName>${imu_topic}</topicName>
-                       <bodyName>${imu_name}</bodyName>
+                       <bodyName>${frame_name_ns}</bodyName>
                        <updateRateHZ>${update_rate}</updateRateHZ>
                        <gaussianNoise>${rate_stddev*rate_stddev}</gaussianNoise>
                        <xyzOffset>0 0 0</xyzOffset>
                        <rpyOffset>0 0 0</rpyOffset>
-                       <frameName>${frame_name}</frameName>
+                       <frameName>${frame_name_ns}</frameName>
                        <initialOrientationAsReference>false</initialOrientationAsReference>
                      </plugin>

File: spot_description/urdfs/accessories.urdf.xacro (robot description, xacro)
@@ -80,5 +80,5 @@
       <!-- IMU sensor -->
       <xacro:imu_sensor
-          imu_name="trunk_imu"
+          frame_name="trunk_imu"
           imu_topic="trunk_imu/data"
           namespace="$(arg robot_name)"

Commit message: Attempt to use ignition

File: sensors_description/urdfs/sensors/imu.gazebo.xacro (robot description, xacro)
@@ -15,6 +15,6 @@
                      <update_rate>${update_rate}</update_rate>
                      <visualize>true</visualize>
-                     <topic>__default_topic__</topic>
-                     <plugin name="imu_sensor_plugin" filename="libgazebo_ros_imu_sensor.so">
+                     <topic>${imu_topic}</topic>
+                    <plugin name="ignition::gazebo::systems::Imu" filename="libignition-gazebo-imu-system.so">
                        <robotNamespace>${namespace}</robotNamespace>
                        <topicName>${imu_topic}</topicName>

File: spot_description/robots/spot.urdf.xacro (robot description, xacro)
@@ -17,5 +17,5 @@
     <xacro:include filename="$(find wolf_description_utils)/urdfs/leg.hardware.xacro"/>
     <xacro:include filename="$(find wolf_description_utils)/urdfs/leg.gazebo.xacro"/>
-    <xacro:include filename="$(find wolf_description_utils)/urdfs/imu.hardware.xacro"/>
+    <!--<xacro:include filename="$(find wolf_description_utils)/urdfs/imu.hardware.xacro"/> -->
     <xacro:include filename="$(find sensors_description)/urdfs/sensors/imu.gazebo.xacro"/>
     <!-- dynamics inertial value -->
@@ -651,5 +651,5 @@
     <xacro:leg_hardware prefix="lh"/>
     <xacro:leg_gazebo prefix="lh" robot_name="$(arg robot_name)" load_force_sensors="$(arg load_force_sensors)"/>
-    <xacro:imu_hardware imu_name="trunk_imu" imu_frame="trunk_imu"/>
+    <!--<xacro:imu_hardware imu_name="trunk_imu" imu_frame="trunk_imu"/>-->
     <xacro:if value="$(eval arm_name != '')">
            <xacro:include filename="$(find spot_description)/urdfs/arm/$(arg arm_name)_adapter.urdf.xacro" />

File: wolf_description_utils/urdfs/gazebo.urdf.xacro (robot description, xacro)
@@ -5,26 +5,39 @@
 <xacro:arg name="robot_model" default=""/>
 <xacro:arg name="base_name"   default="base_link"/>
+<xacro:arg name="sim_engine"  default="ignition"/>
 <xacro:property name="model_name" value="$(arg robot_model)"/>
 	<gazebo>
-        <plugin name="gazebo_ros_controller_manager" filename="libgazebo_ros_control.so">
-                <robotNamespace>$(arg robot_name)</robotNamespace>
-                <robotSimType>wolf_gazebo_interface/WolfRobotHwSim</robotSimType>
-                <controlPeriod>$(arg period)</controlPeriod>
-        </plugin>
-        <plugin name="gazebo_ros2_controller_manager" filename="libgazebo_ros2_control.so">
-                <parameters>$(find wolf_controller)/params/config.ros2.yaml</parameters>
-                <parameters>$(find ${model_name}_description)/params/${model_name}_params.ros2.yaml</parameters>
-        </plugin>
-    	<plugin filename="libgazebo_ros_p3d.so" name="ground_truth">
-                <robotNamespace>$(arg robot_name)</robotNamespace>
-                <bodyName>$(arg base_name)</bodyName>
-                <topicName>ground_truth</topicName>
-                <frameName>world</frameName>
-                <xyzOffsets>0 0 0</xyzOffsets>
-                <rpyOffsets>0 0 0</rpyOffsets>
-                <gaussianNoise>0</gaussianNoise>
-                <alwaysOn>true</alwaysOn>
-                <updateRate>${1/ $(arg period)}</updateRate>
-        </plugin>
+        <xacro:if value="$(eval sim_engine == 'classic')">
+                <!-- ROS1 -->
+                <plugin name="gazebo_ros_controller_manager" filename="libgazebo_ros_control.so">
+                        <robotNamespace>$(arg robot_name)</robotNamespace>
+                        <robotSimType>wolf_gazebo_interface/WolfRobotHwSim</robotSimType>
+                        <controlPeriod>$(arg period)</controlPeriod>
+                </plugin>
+                <plugin filename="libgazebo_ros_p3d.so" name="ground_truth">
+                        <robotNamespace>$(arg robot_name)</robotNamespace>
+                        <bodyName>$(arg base_name)</bodyName>
+                        <topicName>ground_truth</topicName>
+                        <frameName>world</frameName>
+                        <xyzOffsets>0 0 0</xyzOffsets>
+                        <rpyOffsets>0 0 0</rpyOffsets>
+                        <gaussianNoise>0</gaussianNoise>
+                        <alwaysOn>true</alwaysOn>
+                        <updateRate>${1/ $(arg period)}</updateRate>
+                </plugin>
+                <!-- ROS2 -->
+                <plugin name="gazebo_ros2_controller_manager" filename="libgazebo_ros2_control.so">
+                        <parameters>$(find wolf_controller)/params/config.ros2.yaml</parameters>
+                        <parameters>$(find ${model_name}_description)/params/${model_name}_params.ros2.yaml</parameters>
+                </plugin>
+        </xacro:if>
+        <xacro:if value="$(eval sim_engine == 'ignition')">
+                <!-- ROS1 -->
+                <plugin filename="ign_ros_control_plugin" name="ign_ros_control::IgnitionROSControlPlugin">
+                        <updateRate>${1/ $(arg period)}</updateRate>
+                        <robotSimType>wolf_ign_interface/WolfRobotHwIgn</robotSimType>
+                        <robotNamespace>$(arg robot_name)</robotNamespace>
+                </plugin>
+        </xacro:if>
 	</gazebo>
 </robot>

File: wolf_description_utils/urdfs/leg.gazebo.xacro (robot description, xacro)
@@ -1,97 +1,76 @@
 <?xml version="1.0"?>
 <robot xmlns:xacro="http://ros.org/wiki/xacro">
-	<xacro:macro name="leg_gazebo" params="prefix robot_name load_force_sensors">
-		<gazebo reference="${prefix}_haa_joint">
-			<provideFeedback>true</provideFeedback>
-		</gazebo>
-		<xacro:if value="${load_force_sensors}">
-			<gazebo>
-				<plugin name="${prefix}_haa_sensor" filename="libgazebo_ros_ft_sensor.so">
-					<robotNamespace>/${robot_name}/internal_wrench/</robotNamespace>
-					<updateRate>100.0</updateRate>
-					<topicName>${prefix}_haa_joint</topicName>
-					<jointName>${prefix}_haa_joint</jointName>
-				</plugin>
-			</gazebo>
-		</xacro:if>
-		<gazebo reference="${prefix}_hfe_joint">
-			<provideFeedback>true</provideFeedback>
-		</gazebo>
-		<xacro:if value="${load_force_sensors}">
-			<gazebo>
-				<plugin name="${prefix}_hfe_sensor" filename="libgazebo_ros_ft_sensor.so">
-					<robotNamespace>/${robot_name}/internal_wrench/</robotNamespace>
-					<updateRate>100.0</updateRate>
-					<topicName>${prefix}_hfe_joint</topicName>
-					<jointName>${prefix}_hfe_joint</jointName>
-				</plugin>
-			</gazebo>
-		</xacro:if>
-                <gazebo reference="${prefix}_kfe_joint">
-                        <provideFeedback>true</provideFeedback>
-                </gazebo>
-                <xacro:if value="${load_force_sensors}">
-                        <gazebo>
-                                <plugin name="${prefix}_kfe_sensor" filename="libgazebo_ros_ft_sensor.so">
-                                        <robotNamespace>/${robot_name}/internal_wrench/</robotNamespace>
-                                        <updateRate>100.0</updateRate>
-                                        <topicName>${prefix}_kfe_joint</topicName>
-                                        <jointName>${prefix}_kfe_joint</jointName>
-                                </plugin>
-                        </gazebo>
-                </xacro:if>
-               <gazebo reference="${prefix}_foot_joint">
-                       <disableFixedJointLumping>true</disableFixedJointLumping>
-               </gazebo>
-                <gazebo reference="${prefix}_upperleg">
-			<kp>1000000.0</kp>
-			<kd>100.0</kd>
-			<mu1>1.5</mu1>
-			<mu2>1.5</mu2>
-			<fdir1>1 0 0</fdir1>
-			<maxVel>1.0</maxVel>
-                        <maxContacts>1</maxContacts>
-			<minDepth>0.00</minDepth>
-		</gazebo>
-		<gazebo reference="${prefix}_lowerleg">
-			<kp>1000000.0</kp>
-			<kd>100.0</kd>
-			<mu1>1.0</mu1>
-			<mu2>1.0</mu2>
-			<maxVel>1.0</maxVel>
-			<maxContacts>1</maxContacts>
-			<sensor name="${prefix}_shin_contact_sensor" type="contact">
-					<always_on>true</always_on>
-					<update_rate>250.0</update_rate>
-					<contact>
-						<collision>${prefix}_lowerleg_collision</collision>
-					</contact>
-					<plugin name="${prefix}_shin_bumper" filename="libgazebo_ros_bumper.so">
-						<bumperTopicName>/${robot_name}/${prefix}_shin_bumper</bumperTopicName>
-						<robotNamespace>${robot_name}</robotNamespace>
-						<frameName>${prefix}_lowerleg</frameName>
-					</plugin>
-			</sensor>
-		</gazebo>
-                <gazebo reference="${prefix}_foot">
-                        <kp>1000000.0</kp>
-                        <kd>100.0</kd>
-                        <mu1>1.0</mu1>
-                        <mu2>1.0</mu2>
-                        <maxVel>1.0</maxVel>
-                        <maxContacts>1</maxContacts>
-                        <sensor name="${prefix}_foot_contact_sensor" type="contact">
-				<always_on>true</always_on>
-				<update_rate>250.0</update_rate>
-				<contact>
-						<collision>${prefix}_foot_collision</collision>
-				</contact>
-				<plugin name="${prefix}_foot_bumper" filename="libgazebo_ros_bumper.so">
-						<bumperTopicName>/${robot_name}/${prefix}_foot_bumper</bumperTopicName>
-						<robotNamespace>${robot_name}</robotNamespace>
-						<frameName>${prefix}_foot</frameName>
-				</plugin>
-			</sensor>
-		</gazebo>
-	</xacro:macro>
+  <xacro:macro name="leg_gazebo" params="prefix robot_name load_force_sensors">
+    <!-- Joint feedback -->
+    <gazebo reference="${prefix}_haa_joint">
+      <provideFeedback>true</provideFeedback>
+    </gazebo>
+    <gazebo reference="${prefix}_hfe_joint">
+      <provideFeedback>true</provideFeedback>
+    </gazebo>
+    <gazebo reference="${prefix}_kfe_joint">
+      <provideFeedback>true</provideFeedback>
+    </gazebo>
+    <!-- Joint controller plugins for Ignition -->
+    <gazebo>
+      <plugin name="ignition::gazebo::systems::JointPositionController" filename="libignition-gazebo-joint-position-controller-system.so">
+        <joint_name>${prefix}_haa_joint</joint_name>
+        <joint_name>${prefix}_hfe_joint</joint_name>
+        <joint_name>${prefix}_kfe_joint</joint_name>
+      </plugin>
+    </gazebo>
+    <!-- Fixed joint handling -->
+    <gazebo reference="${prefix}_foot_joint">
+      <disableFixedJointLumping>true</disableFixedJointLumping>
+    </gazebo>
+    <!-- Visual/collision and contact sensors -->
+    <gazebo reference="${prefix}_upperleg">
+      <kp>1000000.0</kp>
+      <kd>100.0</kd>
+      <mu1>1.5</mu1>
+      <mu2>1.5</mu2>
+      <fdir1>1 0 0</fdir1>
+      <maxVel>1.0</maxVel>
+      <maxContacts>1</maxContacts>
+      <minDepth>0.00</minDepth>
+    </gazebo>
+    <gazebo reference="${prefix}_lowerleg">
+      <kp>1000000.0</kp>
+      <kd>100.0</kd>
+      <mu1>1.0</mu1>
+      <mu2>1.0</mu2>
+      <maxVel>1.0</maxVel>
+      <maxContacts>1</maxContacts>
+      <sensor name="${prefix}_shin_contact_sensor" type="contact">
+        <always_on>true</always_on>
+        <update_rate>250.0</update_rate>
+        <contact>
+          <collision>${prefix}_lowerleg_collision</collision>
+        </contact>
+        <plugin name="ignition::gazebo::systems::Contact" filename="libignition-gazebo-contact-system.so">
+          <topic>/${robot_name}/${prefix}_shin_bumper</topic>
+          <frame_name>${prefix}_lowerleg</frame_name>
+        </plugin>
+      </sensor>
+    </gazebo>
+    <gazebo reference="${prefix}_foot">
+      <kp>1000000.0</kp>
+      <kd>100.0</kd>
+      <mu1>1.0</mu1>
+      <mu2>1.0</mu2>
+      <maxVel>1.0</maxVel>
+      <maxContacts>1</maxContacts>
+      <sensor name="${prefix}_foot_contact_sensor" type="contact">
+        <always_on>true</always_on>
+        <update_rate>250.0</update_rate>
+        <contact>
+          <collision>${prefix}_foot_collision</collision>
+        </contact>
+        <plugin name="ignition::gazebo::systems::Contact" filename="libignition-gazebo-contact-system.so">
+          <topic>/${robot_name}/${prefix}_foot_bumper</topic>
+          <frame_name>${prefix}_foot</frame_name>
+        </plugin>
+      </sensor>
+    </gazebo>
+  </xacro:macro>
 </robot>

File: wolf_description_utils/urdfs/leg.hardware.xacro (robot description, xacro)
@@ -37,9 +37,8 @@
 		</transmission>
                 <!-- ROS2 -->
-                <ros2_control name="quadruped_system" type="system">
+                <!--<ros2_control name="quadruped_system" type="system">
                     <hardware>
                       <plugin>gazebo_ros2_control/GazeboSystem</plugin>
                     </hardware>
-                    <!-- Hip assembly -->
                     <joint name="${prefix}_haa_joint">
                       <command_interface name="effort">
@@ -51,5 +50,4 @@
                       <state_interface name="effort"/>
                     </joint>
-                    <!-- Upper leg -->
                     <joint name="${prefix}_hfe_joint">
                       <command_interface name="effort">
@@ -61,5 +59,4 @@
                       <state_interface name="effort"/>
                     </joint>
-                    <!-- Lower leg -->
                     <joint name="${prefix}_kfe_joint">
                       <command_interface name="effort">
@@ -71,5 +68,5 @@
                       <state_interface name="effort"/>
                     </joint>
-            </ros2_control>
+            </ros2_control>-->
 	</xacro:macro>
 </robot>
