Commit message: Working with namespaces
only spot at the moment

File: sensors_description/urdfs/sensors/depth_camera.gazebo.xacro (robot description, xacro)
@@ -2,5 +2,5 @@
 <robot xmlns:xacro="http://ros.org/wiki/xacro">
   <xacro:macro name="depth_camera" params="
-    name update_rate image_width image_height fov near far parent_link
+    name namespace update_rate image_width image_height fov near far parent_link
     image_topic camera_info_topic depth_topic pointcloud_topic origin_xyz origin_rpy
   ">
@@ -54,9 +54,9 @@
         <plugin name="gazebo_ros_camera_plugin" filename="libgazebo_ros_camera.so">
           <ros>
-            <namespace>/${name}</namespace>
+            <namespace>${namespace}</namespace>
             <remapping>~/image_raw:=${image_topic}</remapping>
             <remapping>~/camera_info:=${camera_info_topic}</remapping>
           </ros>
-          <camera_name>${name}_camera</camera_name>
+          <camera_name>${name}</camera_name>
           <frame_name>${name}_link</frame_name>
           <update_rate>${update_rate}</update_rate>

File: sensors_description/urdfs/sensors/imu.gazebo.xacro (robot description, xacro)
@@ -1,33 +1,28 @@
 <?xml version="1.0"?>
 <robot xmlns:xacro="http://ros.org/wiki/xacro">
-        <xacro:macro name="imu_sensor" params="frame_name imu_topic namespace update_rate rate_mean rate_stddev
-		rate_bias_mean rate_bias_stddev accel_mean accel_stddev accel_bias_mean accel_bias_stddev">
-                <xacro:if value="${namespace == ''}">
-                    <xacro:property name="frame_name_ns" value="${frame_name}"/>
-                </xacro:if>
-                <xacro:if value="${namespace != ''}">
-                    <xacro:property name="frame_name_ns" value="${namespace+'/'+frame_name}"/>
-                </xacro:if>
-                <gazebo reference="trunk_imu">
-                   <gravity>true</gravity>
-                   <sensor name="trunk_imu" type="imu">
-                     <always_on>true</always_on>
-                     <update_rate>${update_rate}</update_rate>
-                     <visualize>true</visualize>
-                     <topic>__default_topic__</topic>
-                     <plugin name="imu_sensor_plugin" filename="libgazebo_ros_imu_sensor.so">
-                       <robotNamespace>${namespace}</robotNamespace>
-                       <topicName>${imu_topic}</topicName>
-                       <bodyName>${frame_name_ns}</bodyName>
-                       <updateRateHZ>${update_rate}</updateRateHZ>
-                       <gaussianNoise>${rate_stddev*rate_stddev}</gaussianNoise>
-                       <xyzOffset>0 0 0</xyzOffset>
-                       <rpyOffset>0 0 0</rpyOffset>
-                       <frameName>${frame_name_ns}</frameName>
-                       <initialOrientationAsReference>false</initialOrientationAsReference>
-                     </plugin>
-                     <pose>0 0 0 0 0 0</pose>
-                   </sensor>
-                 </gazebo>
-	</xacro:macro>
+    <xacro:macro name="imu_sensor" params="frame_name imu_topic namespace update_rate rate_mean rate_stddev
+        rate_bias_mean rate_bias_stddev accel_mean accel_stddev accel_bias_mean accel_bias_stddev">
+        <gazebo reference="trunk_imu">
+            <gravity>true</gravity>
+            <sensor name="trunk_imu" type="imu">
+                <always_on>true</always_on>
+                <update_rate>${update_rate}</update_rate>
+                <visualize>true</visualize>
+                <topic>${imu_topic}</topic>
+                <plugin name="imu_sensor_plugin" filename="libgazebo_ros_imu_sensor.so">
+                    <ros>
+                        <namespace>${namespace}</namespace>
+                        <remapping>imu_sensor_plugin/out:=${imu_topic}</remapping>
+                    </ros>
+                    <update_rate>${update_rate}</update_rate>
+                    <gaussian_noise>${rate_stddev*rate_stddev}</gaussian_noise>
+                    <xyz_offset>0 0 0</xyz_offset>
+                    <rpy_offset>0 0 0</rpy_offset>
+                    <frame_name>${frame_name}</frame_name>
+                    <initial_orientation_as_reference>false</initial_orientation_as_reference>
+                </plugin>
+                <pose>0 0 0 0 0 0</pose>
+            </sensor>
+        </gazebo>
+    </xacro:macro>
 </robot>

File: spot_description/urdfs/accessories.urdf.xacro (robot description, xacro)
@@ -63,4 +63,5 @@
    <xacro:depth_camera
      name="camera"
+     namespace="$(arg robot_name)"
      update_rate="30"
      image_width="640"
@@ -70,8 +71,8 @@
      far="10.0"
      parent_link="front_rail"
-     image_topic="/camera/rgb/image_raw"
-     depth_topic="/camera/depth/image_raw"
-     pointcloud_topic="/camera/points"
-     camera_info_topic="/camera/camera_info"
+     image_topic="camera/rgb/image_raw"
+     depth_topic="camera/depth/image_raw"
+     pointcloud_topic="camera/points"
+     camera_info_topic="camera/camera_info"
      origin_xyz="0.13 0 0"
      origin_rpy="0 0 0"/>
@@ -94,5 +95,5 @@
     gps_topic="fix"
     velocity_topic="velocity_fix"
-    update_rate="40.0"
+    update_rate="10.0"
     frame_id="base_link" />
 </robot>

File: wolf_description_utils/urdfs/gazebo.urdf.xacro (robot description, xacro)
@@ -7,18 +7,20 @@
 <xacro:property name="model_name" value="$(arg robot_model)"/>
 	<gazebo>
-        <plugin name="gazebo_ros2_controller_manager" filename="libgazebo_ros2_control.so">
+        <plugin name="controller_manager" filename="libgazebo_ros2_control.so">
+                <ros>
+                        <namespace>/$(arg robot_name)</namespace>
+                        <!--<remapping>tf:=$(arg robot_name)/tf</remapping>-->
+                </ros>
                 <parameters>$(find wolf_controller)/params/config.ros2.yaml</parameters>
                 <parameters>$(find ${model_name}_description)/params/${model_name}_params.ros2.yaml</parameters>
         </plugin>
-    	<plugin filename="libgazebo_ros_p3d.so" name="ground_truth">
-                <robotNamespace>$(arg robot_name)</robotNamespace>
-                <bodyName>$(arg base_name)</bodyName>
-                <topicName>ground_truth</topicName>
-                <frameName>world</frameName>
-                <xyzOffsets>0 0 0</xyzOffsets>
-                <rpyOffsets>0 0 0</rpyOffsets>
-                <gaussianNoise>0</gaussianNoise>
-                <alwaysOn>true</alwaysOn>
-                <updateRate>${1/ $(arg period)}</updateRate>
+    	<plugin name="ground_truth" filename="libgazebo_ros_p3d.so">
+                <ros>
+                    <namespace>/$(arg robot_name)</namespace>
+                    <remapping>odom:=ground_truth</remapping>
+                </ros>
+                <frame_name>world</frame_name>
+                <body_name>$(arg base_name)</body_name>
+                <update_rate>${1/ $(arg period)}</update_rate>
         </plugin>
         <plugin name="set_joint_positions_plugin" filename="libgazebo_set_joint_positions_plugin.so">

File: wolf_description_utils/urdfs/leg.gazebo.xacro (robot description, xacro)
@@ -8,8 +8,9 @@
 			<gazebo>
 				<plugin name="${prefix}_haa_sensor" filename="libgazebo_ros_ft_sensor.so">
-					<robotNamespace>/${robot_name}/internal_wrench/</robotNamespace>
-					<updateRate>100.0</updateRate>
-					<topicName>${prefix}_haa_joint</topicName>
-					<jointName>${prefix}_haa_joint</jointName>
+					<ros>
+                        <namespace>${robot_name}</namespace>
+                    </ros>
+					<update_rate>100.0</update_rate>
+					<joint_name>${prefix}_haa_joint</joint_name>
 				</plugin>
 			</gazebo>
@@ -21,28 +22,30 @@
 			<gazebo>
 				<plugin name="${prefix}_hfe_sensor" filename="libgazebo_ros_ft_sensor.so">
-					<robotNamespace>/${robot_name}/internal_wrench/</robotNamespace>
-					<updateRate>100.0</updateRate>
-					<topicName>${prefix}_hfe_joint</topicName>
-					<jointName>${prefix}_hfe_joint</jointName>
+					<ros>
+                        <namespace>${robot_name}</namespace>
+                    </ros>
+					<update_rate>100.0</update_rate>
+					<joint_name>${prefix}_hfe_joint</joint_name>
 				</plugin>
 			</gazebo>
 		</xacro:if>
-                <gazebo reference="${prefix}_kfe_joint">
-                        <provideFeedback>true</provideFeedback>
-                </gazebo>
-                <xacro:if value="${load_force_sensors}">
-                        <gazebo>
-                                <plugin name="${prefix}_kfe_sensor" filename="libgazebo_ros_ft_sensor.so">
-                                        <robotNamespace>/${robot_name}/internal_wrench/</robotNamespace>
-                                        <updateRate>100.0</updateRate>
-                                        <topicName>${prefix}_kfe_joint</topicName>
-                                        <jointName>${prefix}_kfe_joint</jointName>
-                                </plugin>
-                        </gazebo>
-                </xacro:if>
-               <gazebo reference="${prefix}_foot_joint">
-                       <disableFixedJointLumping>true</disableFixedJointLumping>
-               </gazebo>
-                <gazebo reference="${prefix}_upperleg">
+		<gazebo reference="${prefix}_kfe_joint">
+				<provideFeedback>true</provideFeedback>
+		</gazebo>
+		<xacro:if value="${load_force_sensors}">
+				<gazebo>
+						<plugin name="${prefix}_kfe_sensor" filename="libgazebo_ros_ft_sensor.so">
+								<ros>
+									<namespace>${robot_name}</namespace>
+								</ros>
+								<update_rate>100.0</update_rate>
+								<joint_name>${prefix}_kfe_joint</joint_name>
+						</plugin>
+				</gazebo>
+		</xacro:if>
+		<gazebo reference="${prefix}_foot_joint">
+			<disableFixedJointLumping>true</disableFixedJointLumping>
+		</gazebo>
+		<gazebo reference="${prefix}_upperleg">
 			<kp>1000000.0</kp>
 			<kd>100.0</kd>
@@ -51,5 +54,5 @@
 			<fdir1>1 0 0</fdir1>
 			<maxVel>1.0</maxVel>
-                        <maxContacts>1</maxContacts>
+			<maxContacts>1</maxContacts>
 			<minDepth>0.00</minDepth>
 		</gazebo>
@@ -68,7 +71,9 @@
 					</contact>
 					<plugin name="${prefix}_shin_bumper" filename="libgazebo_ros_bumper.so">
-						<bumperTopicName>/${robot_name}/${prefix}_shin_bumper</bumperTopicName>
-						<robotNamespace>${robot_name}</robotNamespace>
-						<frameName>${prefix}_lowerleg</frameName>
+						<frame_name>${prefix}_lowerleg</frame_name>
+						   <ros>
+							<namespace>${robot_name}</namespace>
+							<remapping>bumper_states:=${prefix}_shin_bumper</remapping>
+						  </ros>
 					</plugin>
 			</sensor>
@@ -88,7 +93,9 @@
 				</contact>
 				<plugin name="${prefix}_foot_bumper" filename="libgazebo_ros_bumper.so">
-						<bumperTopicName>/${robot_name}/${prefix}_foot_bumper</bumperTopicName>
-						<robotNamespace>${robot_name}</robotNamespace>
-						<frameName>${prefix}_foot</frameName>
+						<frame_name>${prefix}_foot</frame_name>
+						  <ros>
+							<namespace>${robot_name}</namespace>
+							<remapping>bumper_states:=${prefix}_foot_bumper</remapping>
+						  </ros>
 				</plugin>
 			</sensor>

Commit message: Fix frame names in sensors (ign)

File: sensors_description/urdfs/sensors/depth_camera.gazebo.xacro (robot description, xacro)
@@ -34,7 +34,9 @@
     <xacro:if value="${namespace == ''}">
       <xacro:property name="camera_topic_ns" value="${name}"/>
+      <xacro:property name="camera_frame_id" value="${name + '_link'}"/>
     </xacro:if>
     <xacro:if value="${namespace != ''}">
       <xacro:property name="camera_topic_ns" value="${namespace + '/' + name}"/>
+      <xacro:property name="camera_frame_id" value="${namespace + '/' + name + '_link'}"/>
     </xacro:if>
     <!-- Gazebo Sim depth camera sensor -->
@@ -45,4 +47,5 @@
         <pose>${origin_xyz} ${origin_rpy}</pose>
         <topic>${camera_topic_ns}</topic>
+        <gz_frame_id>${camera_frame_id}</gz_frame_id>
         <camera name="${name}">
           <horizontal_fov>${fov}</horizontal_fov>

File: sensors_description/urdfs/sensors/gps.gazebo.xacro (robot description, xacro)
@@ -15,7 +15,9 @@
       <xacro:if value="${namespace == ''}">
                     <xacro:property name="gps_topic_ns" value="${gps_topic}"/>
+                    <xacro:property name="gps_frame_id_ns" value="${frame_id}"/>
       </xacro:if>
       <xacro:if value="${namespace != ''}">
                     <xacro:property name="gps_topic_ns" value="${namespace+'/'+gps_topic}"/>
+                    <xacro:property name="gps_frame_id_ns" value="${namespace+'/'+frame_id}"/>
       </xacro:if>
     <gazebo reference="${frame_id}">
@@ -24,4 +26,5 @@
         <update_rate>${update_rate}</update_rate>
         <topic>${gps_topic_ns}</topic>
+        <gz_frame_id>${gps_frame_id_ns}</gz_frame_id>
         <gps>
           <!-- Optionally, include additional sensor-specific parameters here -->

File: sensors_description/urdfs/sensors/imu.gazebo.xacro (robot description, xacro)
@@ -3,10 +3,12 @@
     <xacro:macro name="imu_sensor" params="sensor_name frame_name imu_topic namespace update_rate rate_mean rate_stddev
         rate_bias_mean rate_bias_stddev accel_mean accel_stddev accel_bias_mean accel_bias_stddev">
-      <xacro:if value="${namespace == ''}">
+    <xacro:if value="${namespace == ''}">
                 <xacro:property name="imu_topic_ns" value="${'/' + imu_topic}"/>
-      </xacro:if>
-      <xacro:if value="${namespace != ''}">
+                <xacro:property name="imu_frame_id" value="${frame_name}"/>
+    </xacro:if>
+    <xacro:if value="${namespace != ''}">
                 <xacro:property name="imu_topic_ns" value="${'/' + namespace + '/' + imu_topic}"/>
-      </xacro:if>
+                <xacro:property name="imu_frame_id" value="${namespace + '/' + frame_name}"/>
+    </xacro:if>
         <gazebo reference="${frame_name}">
             <gravity>true</gravity>
@@ -16,4 +18,5 @@
                 <visualize>true</visualize>
                 <topic>${imu_topic_ns}</topic>
+                <gz_frame_id>${imu_frame_id}</gz_frame_id>
                 <pose>0 0 0 0 0 0</pose>
             </sensor>

File: sensors_description/urdfs/sensors/lidar.gazebo.xacro (robot description, xacro)
@@ -4,7 +4,9 @@
     <xacro:if value="${namespace == ''}">
       <xacro:property name="lidar_topic_ns" value="${topic_name}"/>
+      <xacro:property name="lidar_frame_id_ns" value="${frame_id}"/>
     </xacro:if>
     <xacro:if value="${namespace != ''}">
       <xacro:property name="lidar_topic_ns" value="${namespace + '/' + topic_name}"/>
+      <xacro:property name="lidar_frame_id_ns" value="${namespace + '/' + frame_id}"/>
     </xacro:if>
     <!-- Sensor definition -->
@@ -16,5 +18,5 @@
         <update_rate>${update_rate}</update_rate>
         <topic>${lidar_topic_ns}</topic>
-        <gz_frame_id>${frame_id}</gz_frame_id>
+        <gz_frame_id>${lidar_frame_id_ns}</gz_frame_id>
         <lidar>
           <scan>
