Commit message: Update params to the new impedance interface, remove unused tasks waistZ and postural

File: aliengo_description/robots/aliengo.urdf.xacro (robot description, xacro)
@@ -3,8 +3,8 @@
      <!-- This argument allows us to load joint sensors that measure the internal wrenches -->
     <xacro:arg name="load_force_sensors" default="false"/>
+    <xacro:arg name="sensors" default="false"/>
     <xacro:arg name="task_period" default="0.004"/>
     <xacro:arg name="arm_enabled" default="false"/>
     <xacro:arg name="arm_name" default="kinova"/>
-    <xacro:arg name="sensors" default="false"/>
     <xacro:arg name="floating_base_link" default="true"/>
     <xacro:arg name="robot_name"  default="aliengo"/>
@@ -25,13 +25,4 @@
     <!-- Rollover Protection mode will add an additional stick on the top, use "true" or "false" to switch it. -->
     <xacro:property name="rolloverProtection" value="false"/>
-    <!-- Debug mode will hung up the robot, use "true" or "false" to switch it. -->
-    <!-- <xacro:if value="$(arg DEBUG)">
-        <link name="world"/>
-        <joint name="base_static_joint" type="fixed">
-            <origin rpy="0 0 0" xyz="0 0 0"/>
-            <parent link="world"/>
-            <child link="base"/>
-        </joint>
-    </xacro:if>  -->
     <!-- Floating-base Joint -->
     <xacro:if value="$(arg floating_base_link)">

File: anymal_description/robots/anymal.srdf.xacro (robot description, xacro)
@@ -60,3 +60,17 @@
       <joint name="rh_kfe_joint" value="1.0"/>
   </group_state>
+  <group_state group="chains" name="standdown">
+    <joint name="lf_haa_joint" value="0.0"/>
+    <joint name="lf_hfe_joint" value="1.60"/>
+    <joint name="lf_kfe_joint" value="2.60"/>
+    <joint name="rf_haa_joint" value="0.0"/>
+    <joint name="rf_hfe_joint" value="1.60"/>
+    <joint name="rf_kfe_joint" value="2.60"/>
+    <joint name="lh_haa_joint" value="0.0"/>
+    <joint name="lh_hfe_joint" value="-1.60"/>
+    <joint name="lh_kfe_joint" value="2.60"/>
+    <joint name="rh_haa_joint" value="0.0"/>
+    <joint name="rh_hfe_joint" value="-1.60"/>
+    <joint name="rh_kfe_joint" value="2.60"/>
+  </group_state>
 </robot>
