Commit message: added camera to accessories

File: spot_description/urdfs/accessories.urdf.xacro (robot description, xacro)
@@ -4,4 +4,5 @@
   <!--<xacro:include filename="$(find sensors_description)/urdfs/sensors/velodyne.gazebo.xacro"/>-->
   <xacro:include filename="$(find velodyne_description)/urdf/VLP-16.urdf.xacro"/>
+  <xacro:include filename="$(find sensors_description)/urdfs/sensors/_d435.urdf.xacro" />
   <xacro:if value="$(optenv SPOT_PACK 1)">
     <joint name="pack_mount_joint" type="fixed">
@@ -64,14 +65,10 @@
         </collision>
       </link>
-      <!--<joint name="velodyne_joint" type="fixed">
-        <parent link="velodyne_mount"/>
-        <child link="velodyne"/>
-        <origin xyz="0 0 0.0377" rpy="0 0 0"/>
-      </joint>
-      <link name="velodyne"/>
-      <xacro:velodyne_sensor link_name="velodyne" frame_name="velodyne" lidar_name="velodyne" update_rate="10.0"/>-->
       <xacro:VLP-16 parent="velodyne_mount" name="velodyne" topic="/velodyne_pointcloud" organize_cloud="false" hz="10" samples="440" gpu="true">
         <origin xyz="0 0 0.0377" rpy="0 0 0" />
       </xacro:VLP-16>
+      <xacro:sensor_d435 parent="front_rail">
+        <origin xyz="0.13 0 0" rpy="0 0 0" />
+      </xacro:sensor_d435>
     </xacro:if>
   </xacro:if>

Commit message: added t265 to spot accessories

File: spot_description/urdfs/accessories.urdf.xacro (robot description, xacro)
@@ -5,4 +5,5 @@
   <xacro:include filename="$(find velodyne_description)/urdf/VLP-16.urdf.xacro"/>
   <xacro:include filename="$(find sensors_description)/urdfs/sensors/_d435.urdf.xacro" />
+  <xacro:include filename="$(find sensors_description)/urdfs/sensors/realsense_t265.xacro" />
   <xacro:if value="$(optenv SPOT_PACK 1)">
     <joint name="pack_mount_joint" type="fixed">
@@ -71,4 +72,7 @@
         <origin xyz="0.13 0 0" rpy="0 0 0" />
       </xacro:sensor_d435>
+      <xacro:realsense_T265 sensor_name="t265" parent_link="d435_bottom_screw_frame" rate="30.0">
+        <origin xyz="0 0 0.04" rpy="0 0 0" />
+      </xacro:realsense_T265>
     </xacro:if>
   </xacro:if>

Commit message: improved velodyne mesh sensor position on spot

File: spot_description/urdfs/accessories.urdf.xacro (robot description, xacro)
@@ -67,5 +67,5 @@
       </link>
       <xacro:VLP-16 parent="velodyne_mount" name="velodyne" topic="/velodyne_pointcloud" organize_cloud="false" hz="10" samples="440" gpu="true">
-        <origin xyz="0 0 0.0377" rpy="0 0 0" />
+        <origin xyz="0 0 0" rpy="0 0 0" />
       </xacro:VLP-16>
       <xacro:sensor_d435 parent="front_rail">

Commit message: reorganized velodyne importing and attached t265 to another frame

File: spot_description/urdfs/accessories.urdf.xacro (robot description, xacro)
@@ -66,5 +66,6 @@
         </collision>
       </link>
-      <xacro:VLP-16 parent="velodyne_mount" name="velodyne" topic="/velodyne_pointcloud" organize_cloud="false" hz="10" samples="440" gpu="true">
+      <xacro:VLP-16 parent="velodyne_mount" name="velodyne" topic="/velodyne_pointcloud"
+                    organize_cloud="false" hz="10" samples="440" gpu="true">
         <origin xyz="0 0 0" rpy="0 0 0" />
       </xacro:VLP-16>
@@ -72,6 +73,6 @@
         <origin xyz="0.13 0 0" rpy="0 0 0" />
       </xacro:sensor_d435>
-      <xacro:realsense_T265 sensor_name="t265" parent_link="d435_bottom_screw_frame" rate="30.0">
-        <origin xyz="0 0 0.04" rpy="0 0 0" />
+      <xacro:realsense_T265 sensor_name="t265" parent_link="front_rail" rate="30.0">
+        <origin xyz="0.13 0 0.04" rpy="0 0 0" />
       </xacro:realsense_T265>
     </xacro:if>
