Commit message: updates on xacro/objects

File: ylo2_description/robots/ylo2.srdf.xacro (robot description, xacro)
@@ -61,14 +61,14 @@
     </group_state>
     <group_state group="chains" name="standdown">
-        <joint name="lf_haa_joint" value="0.8"/>
+        <joint name="lf_haa_joint" value="0.60"/>
         <joint name="lf_hfe_joint" value="1.70"/>
         <joint name="lf_kfe_joint" value="-2.77"/>
-        <joint name="rf_haa_joint" value="-0.8"/>
+        <joint name="rf_haa_joint" value="-0.60"/>
         <joint name="rf_hfe_joint" value="1.70"/>
         <joint name="rf_kfe_joint" value="-2.77"/>
-        <joint name="lh_haa_joint" value="0.8"/>
+        <joint name="lh_haa_joint" value="0.60"/>
         <joint name="lh_hfe_joint" value="1.52"/>
         <joint name="lh_kfe_joint" value="-2.77"/>
-        <joint name="rh_haa_joint" value="-0.8"/>
+        <joint name="rh_haa_joint" value="-0.60"/>
         <joint name="rh_hfe_joint" value="1.52"/>
         <joint name="rh_kfe_joint" value="-2.77"/>

File: ylo2_description/robots/ylo2.urdf.xacro (robot description, xacro)
@@ -19,8 +19,17 @@
         <xacro:include filename="$(find sensors_description)/urdfs/sensors/imu.gazebo.xacro"/>
     </xacro:if>
-    <xacro:include filename="$(find ylo2_description)/urdfs/const.xacro"/>
-    <xacro:include filename="$(find ylo2_description)/urdfs/leg.xacro"/>
+    <xacro:include filename="$(find ylo2_urdf_2022_description)/urdfs/const.xacro"/>
+    <xacro:include filename="$(find ylo2_urdf_2022_description)/urdfs/leg.xacro"/>
     <!-- Rollover Protection mode will add an additional stick on the top, use "true" or "false" to switch it. -->
     <xacro:property name="rolloverProtection" value="false"/>
+    <!-- Debug mode will hung up the robot, use "true" or "false" to switch it. -->
+    <!-- <xacro:if value="$(arg DEBUG)">
+        <link name="world"/>
+        <joint name="base_static_joint" type="fixed">
+            <origin rpy="0 0 0" xyz="0 0 0"/>
+            <parent link="world"/>
+            <child link="base"/>
+        </joint>
+    </xacro:if>  -->
     <!-- Floating-base Joint -->
     <xacro:if value="$(arg floating_base_link)">
@@ -34,22 +43,16 @@
     <link name="trunk">
         <visual>
-            <origin rpy="0 0 0" xyz="${trunk_offset_x} ${trunk_offset_y} ${trunk_offset_z}"/>
-            <geometry>
-                <mesh filename="package://ylo2_description/meshes/base_link_resized.stl" scale="-1 1 1"/>
-            </geometry>
-            <material name="orange"/>
+            <origin rpy="0 0 0" xyz="${trunk_offset_x} 0 ${abab_motors_offset_z}"/>
+            <geometry>
+                <mesh filename="package://ylo2_urdf_2022_description/meshes/body/body_parts.stl" scale="1 1 1"/>
+            </geometry>
+            <material name="grey"/>
         </visual>
         <collision>
-            <origin rpy="0 0 0" xyz="0 0 0"/>
-            <geometry>
-                <box size="${trunk_length} ${trunk_width} ${trunk_height}"/>
+            <origin rpy="0 0 0" xyz="${trunk_offset_x} 0 ${abab_motors_offset_z}"/>
+            <geometry>
+                <mesh filename="package://ylo2_urdf_2022_description/meshes/body/covers_collision.stl" scale="1 1 1"/>
             </geometry>
         </collision>
-        <!-- <collision>
-            <origin rpy="0 0 0" xyz="0 0 0"/>
-            <geometry>
-                <mesh filename="package://ylo2_description/meshes/base_link_resized.stl" scale="1 1 1"/>
-            </geometry>
-        </collision> -->
         <inertial>
             <origin rpy="0 0 0" xyz="${trunk_com_x} ${trunk_com_y} ${trunk_com_z}"/>
@@ -61,4 +64,75 @@
         </inertial>
     </link>
+    <link name="abad_motors">
+        <visual>
+            <origin rpy="0 0 0" xyz="${trunk_offset_x} ${trunk_offset_y} ${abab_motors_offset_z}"/>
+            <geometry>
+                <mesh filename="package://ylo2_urdf_2022_description/meshes/body/abad_motors.stl" scale="1 1 1"/>
+            </geometry>
+            <material name="white"/>
+        </visual>
+    </link>
+    <joint name="abad_motors_joint" type="fixed">
+        <parent link="trunk"/>
+        <child link="abad_motors"/>
+        <origin rpy="0 0 0" xyz="0 0 0"/>
+    </joint>
+    <link name="battery">
+        <visual>
+            <origin rpy="0 0 0" xyz="${trunk_offset_x} ${trunk_offset_y} ${abab_motors_offset_z}"/>
+            <geometry>
+                <mesh filename="package://ylo2_urdf_2022_description/meshes/body/battery.stl" scale="1 1 1"/>
+            </geometry>
+            <material name="blue"/>
+        </visual>
+    </link>
+    <joint name="battery_joint" type="fixed">
+        <parent link="trunk"/>
+        <child link="battery"/>
+        <origin rpy="0 0 0" xyz="0 0 0"/>
+    </joint>
+    <link name="covers">
+        <visual>
+            <origin rpy="0 0 0" xyz="${trunk_offset_x} ${trunk_offset_y} ${abab_motors_offset_z}"/>
+            <geometry>
+                <mesh filename="package://ylo2_urdf_2022_description/meshes/body/covers.stl" scale="1 1 1"/>
+            </geometry>
+            <material name="orange"/>
+        </visual>
+    </link>
+    <joint name="covers_joint" type="fixed">
+        <parent link="trunk"/>
+        <child link="covers"/>
+        <origin rpy="0 0 0" xyz="0 0 0"/>
+    </joint>
+    <link name="D435">
+        <visual>
+            <origin rpy="0 0 0" xyz="${trunk_offset_x} ${trunk_offset_y} ${abab_motors_offset_z}"/>
+            <geometry>
+                <mesh filename="package://ylo2_urdf_2022_description/meshes/body/D435_fake_camera.stl" scale="1 1 1"/>
+            </geometry>
+            <material name="black"/>
+        </visual>
+    </link>
+    <joint name="D435_joint" type="fixed">
+        <parent link="trunk"/>
+        <child link="D435"/>
+        <origin rpy="0 0 0" xyz="0 0 0"/>
+    </joint>
+    <link name="T265">
+        <visual>
+            <origin rpy="0 0 0" xyz="${trunk_offset_x} ${trunk_offset_y} ${abab_motors_offset_z}"/>
+            <geometry>
+                <mesh filename="package://ylo2_urdf_2022_description/meshes/body/T265_fake_camera.stl" scale="1 1 1"/>
+            </geometry>
+            <material name="black"/>
+        </visual>
+    </link>
+    <joint name="T265_joint" type="fixed">
+        <parent link="trunk"/>
+        <child link="T265"/>
+        <origin rpy="0 0 0" xyz="0 0 0"/>
+    </joint>
+    <!-- adding a lateral cylinder as collision object, to avoid robot to fall on it side-->
     <xacro:if value="${(rolloverProtection == 'true')}">
         <joint name="stick_joint" type="fixed">
@@ -117,14 +191,14 @@
     <!-- ABAD POSITION OK pas touche-->
     <xacro:leg name="rf" mirror="-1" mirror_dae= "False" front_hind="1" front_hind_dae="True">
-        <origin rpy="0 0 0" xyz="${leg_offset_x} ${trunk_offset_y-leg_offset_y} 0.014"/>
+        <origin rpy="0 0 0" xyz="${leg_offset_x-0.019} ${0-leg_offset_y+0.006} ${0-leg_offset_z}"/>
     </xacro:leg>
     <xacro:leg name="lf" mirror="1" mirror_dae="True" front_hind="1" front_hind_dae="True">
-        <origin rpy="0 0 0" xyz="${leg_offset_x} ${trunk_offset_y+leg_offset_y} 0.014"/>
+        <origin rpy="0 0 0" xyz="${leg_offset_x-0.019} ${0+leg_offset_y+0.006} ${0-leg_offset_z}"/>
     </xacro:leg>
     <xacro:leg name="rh" mirror="-1" mirror_dae="False" front_hind="-1" front_hind_dae="False">
-        <origin rpy="0 0 0" xyz="${-leg_offset_x} ${trunk_offset_y-leg_offset_y} 0.014"/>
+        <origin rpy="0 0 0" xyz="${-leg_offset_x-0.019} ${0-leg_offset_y+0.006} ${0-leg_offset_z}"/>
     </xacro:leg>
     <xacro:leg name="lh" mirror="1" mirror_dae="True" front_hind="-1" front_hind_dae="False">
-        <origin rpy="0 0 0" xyz="${-leg_offset_x} ${trunk_offset_y+leg_offset_y} 0.014"/>
+        <origin rpy="0 0 0" xyz="${-leg_offset_x-0.019} ${0+leg_offset_y+0.006} ${0-leg_offset_z}"/>
     </xacro:leg>
     <!-- <xacro:stairs stairs="15" xpos="0" ypos="2.0" zpos="0" /> -->

File: ylo2_description/urdfs/const.xacro (robot description, xacro)
@@ -7,11 +7,11 @@
     <!-- corps -->
     <xacro:property name="trunk_width" value="0.350"/>
-    <xacro:property name="trunk_length" value="0.500"/>
+    <xacro:property name="trunk_length" value="0.568"/>
     <xacro:property name="trunk_height" value="0.130"/>
     <!-- adjust center of robot -->
-    <xacro:property name="trunk_offset_x" value="0.011"/>
-    <xacro:property name="trunk_offset_y" value="0.005"/>
-    <xacro:property name="trunk_offset_z" value="0.000"/>
-    <xacro:property name="hip_radius" value="0.046"/>
+    <xacro:property name="trunk_offset_x" value="0.0"/>
+    <xacro:property name="trunk_offset_y" value="0.0"/>
+    <xacro:property name="abab_motors_offset_z" value="0.0"/>
+    <xacro:property name="hip_radius" value="0.050"/>
     <xacro:property name="hip_length" value="0.418"/>
     <xacro:property name="upperleg_shoulder_radius" value="0.044"/>
@@ -25,10 +25,11 @@
     <xacro:property name="stick_length" value="0.2"/>
     <!-- kinematic value -->
-    <xacro:property name="upperleg_offset" value="0.092"/> <!-- ecart centre abad et axe de la upper/lower leg -->
-    <xacro:property name="upperleg_length" value="0.215427"/>
-    <xacro:property name="lowerleg_length" value="0.229819"/> <!-- TODO a regler apres avoir positionne le bas de patte silicone -->
+    <xacro:property name="upperleg_offset" value="0.092"/> <!-- decalage lateral HIP -> upper_leg - lateral difference between HIP and upper_leg -->
+    <xacro:property name="upperleg_length" value="0.215427"/> <!-- upper leg size, from HIP axis, to lower leg axis-->
+    <xacro:property name="lowerleg_length" value="0.229819"/> <!-- lower leg size, from lower leg axis to end foot -->
     <!-- leg offset from trunk center value -->
-    <xacro:property name="leg_offset_x" value="${0.387/2}"/> <!-- ecart longueur axes pattes -->
-    <xacro:property name="leg_offset_y" value="${0.115/2}"/> <!-- ecart largeur axes pattes  demande reglage mais semble ok-->
+    <xacro:property name="leg_offset_x" value="${0.387/2}"/> <!-- ecart centres HIP avant/arriere - HIP distance front/back -->
+    <xacro:property name="leg_offset_y" value="${0.1144/2}"/> <!-- ecart centres HIP gauche/droite - HIP distance left/right-->
+    <xacro:property name="leg_offset_z" value="-0.023"/> <!-- decalage hauteur axes pattes/abad - vertical difference HIP -> ABAD -->
     <xacro:property name="trunk_offset_z" value="0.01675"/>
     <xacro:property name="hip_offset" value="0.083"/>
@@ -39,56 +40,56 @@
     <xacro:property name="hip_position_min" value="${-70*PI/180.0}"/>
     <xacro:property name="hip_velocity_max" value="20"/>
-    <xacro:property name="hip_torque_max" value="44"/>
+    <xacro:property name="hip_torque_max" value="16"/>
     <xacro:property name="upperleg_velocity_max" value="20"/>
-    <xacro:property name="upperleg_torque_max" value="44"/>
+    <xacro:property name="upperleg_torque_max" value="16"/>
     <xacro:property name="lowerleg_position_max" value="${-37*PI/180.0}"/>
     <xacro:property name="lowerleg_position_min" value="${-159*PI/180.0}"/>
     <xacro:property name="lowerleg_velocity_max" value="16"/>
-    <xacro:property name="lowerleg_torque_max" value="55"/>
+    <xacro:property name="lowerleg_torque_max" value="16"/>
     <!-- dynamics inertial value -->
     <!-- trunk -->
-    <xacro:property name="trunk_mass" value="11.041"/>
+    <xacro:property name="trunk_mass" value="3.6601201387244187"/>
     <xacro:property name="trunk_com_x" value="0.008465"/>
     <xacro:property name="trunk_com_y" value="0.004045"/>
     <xacro:property name="trunk_com_z" value="-0.000763"/>
-    <xacro:property name="trunk_ixx" value="0.050874"/>
-    <xacro:property name="trunk_ixy" value="-0.000451628"/>
-    <xacro:property name="trunk_ixz" value="0.000487603"/>
-    <xacro:property name="trunk_iyy" value="0.64036"/>
-    <xacro:property name="trunk_iyz" value="0.000048356"/>
-    <xacro:property name="trunk_izz" value="0.65655"/>
+    <xacro:property name="trunk_ixx" value="0.01991"/>
+    <xacro:property name="trunk_ixy" value="-0.000303"/>
+    <xacro:property name="trunk_ixz" value="-0.000443"/>
+    <xacro:property name="trunk_iyy" value="0.068086"/>
+    <xacro:property name="trunk_iyz" value="2.7e-05"/>
+    <xacro:property name="trunk_izz" value="0.074459"/>
     <!-- hip (left front) -->
-    <xacro:property name="hip_mass" value="1.993"/>
+    <xacro:property name="hip_mass" value="0.45927445698625047"/>
     <xacro:property name="hip_com_x" value="-0.022191"/>
     <xacro:property name="hip_com_y" value="0.015144"/>
     <xacro:property name="hip_com_z" value="-0.000015"/>
-    <xacro:property name="hip_ixx" value="0.002903894"/>
-    <xacro:property name="hip_ixy" value="-0.000071850"/>
-    <xacro:property name="hip_ixz" value="-0.000001262"/>
-    <xacro:property name="hip_iyy" value="0.004907517"/>
-    <xacro:property name="hip_iyz" value="-0.00000175"/>
-    <xacro:property name="hip_izz" value="0.005586944"/>
+    <xacro:property name="hip_ixx" value="0.000412"/>
+    <xacro:property name="hip_ixy" value="8e-06"/>
+    <xacro:property name="hip_ixz" value="-0.0"/>
+    <xacro:property name="hip_iyy" value="0.000689"/>
+    <xacro:property name="hip_iyz" value="-0.0"/>
+    <xacro:property name="hip_izz" value="0.000457"/>
     <!-- upperleg -->
-    <xacro:property name="upperleg_mass" value="0.639"/>
+    <xacro:property name="upperleg_mass" value="0.6130196221001395"/>
     <xacro:property name="upperleg_com_x" value="-0.005607"/>
     <xacro:property name="upperleg_com_y" value="-0.003877"/>
     <xacro:property name="upperleg_com_z" value="-0.048199"/>
-    <xacro:property name="upperleg_ixx" value="0.005666803"/>
-    <xacro:property name="upperleg_ixy" value="0.000003597"/>
-    <xacro:property name="upperleg_ixz" value="0.000491446"/>
-    <xacro:property name="upperleg_iyy" value="0.005847229"/>
-    <xacro:property name="upperleg_iyz" value="0.000010086"/>
-    <xacro:property name="upperleg_izz" value="0.000369811"/>
+    <xacro:property name="upperleg_ixx" value="0.004041"/>
+    <xacro:property name="upperleg_ixy" value="2e-06"/>
+    <xacro:property name="upperleg_ixz" value="0.0001"/>
+    <xacro:property name="upperleg_iyy" value="0.004028"/>
+    <xacro:property name="upperleg_iyz" value="-0.000397"/>
+    <xacro:property name="upperleg_izz" value="0.000788"/>
     <!-- lowerleg -->
-    <xacro:property name="lowerleg_mass" value="0.207"/>
+    <xacro:property name="lowerleg_mass" value="0.17546927346672364"/>
     <xacro:property name="lowerleg_com_x" value="0.002781"/>
     <xacro:property name="lowerleg_com_y" value="0.000063"/>
     <xacro:property name="lowerleg_com_z" value="-0.142518"/>
-    <xacro:property name="lowerleg_ixx" value="0.006341369"/>
-    <xacro:property name="lowerleg_ixy" value="-0.000000003"/>
-    <xacro:property name="lowerleg_ixz" value="-0.000087951"/>
-    <xacro:property name="lowerleg_iyy" value="0.006355157"/>
-    <xacro:property name="lowerleg_iyz" value="-0.000001336"/>
-    <xacro:property name="lowerleg_izz" value="0.000039188"/>
+    <xacro:property name="lowerleg_ixx" value="0.000462"/>
+    <xacro:property name="lowerleg_ixy" value="-0.0"/>
+    <xacro:property name="lowerleg_ixz" value="-3.2e-05"/>
+    <xacro:property name="lowerleg_iyy" value="0.000473"/>
+    <xacro:property name="lowerleg_iyz" value="-0.0"/>
+    <xacro:property name="lowerleg_izz" value="3e-05"/>
     <!-- foot -->
     <xacro:property name="foot_mass" value="0.03157"/>

File: ylo2_description/urdfs/leg.xacro (robot description, xacro)
@@ -18,17 +18,17 @@
             <visual>
                 <xacro:if value="${(mirror_dae == True) and (front_hind_dae == True)}">
-                    <origin rpy="0 0 0" xyz="-0.059 -0.046 0"/>
+                    <origin rpy="0 0 0" xyz="-0.06 0 0"/>
                 </xacro:if>
                 <xacro:if value="${(mirror_dae == False) and (front_hind_dae == True)}">
-                    <origin rpy="${PI} 0 0" xyz="-0.059 0.046 0"/>
+                    <origin rpy="${PI} 0 0" xyz="-0.06 0 0"/>
                 </xacro:if>
                 <xacro:if value="${(mirror_dae == True) and (front_hind_dae == False)}">
-                    <origin rpy="0 ${PI} 0" xyz="0.059 -0.046 0"/>
+                    <origin rpy="0 ${PI} 0" xyz="0.06 0 0"/>
                 </xacro:if>
                 <xacro:if value="${(mirror_dae == False) and (front_hind_dae == False)}">
-                    <origin rpy="${PI} ${PI} 0" xyz="0.059 0.046 0"/>
+                    <origin rpy="${PI} ${PI} 0" xyz="0.06 0 0"/>
                 </xacro:if>
                 <geometry>
-                    <mesh filename="package://ylo2_description/meshes/abduct_fl_resized.stl" scale="-1 -1 1"/>
+                    <mesh filename="package://ylo2_urdf_2022_description/meshes/leg/fl_hip.stl" scale="1 1 1"/>
                 </geometry>
                 <material name="grey"/>
@@ -49,18 +49,4 @@
             </inertial>
         </link>
-        <!-- <joint name="${name}_hip_fixed" type="fixed">
-            <origin rpy="0 0 0" xyz="0 ${(upperleg_shoulder_length/2.0+hip_offset)*mirror} 0"/>
-            <parent link="${name}_hip"/>
-            <child link="${name}_upperleg_shoulder"/>
-        </joint> -->
-        <!-- this link is only for collision -->
-        <!-- <link name="${name}_upperleg_shoulder">
-            <collision>
-                <origin rpy="${PI/2.0} 0 0" xyz="0 0 0"/>
-                <geometry>
-                    <cylinder length="${upperleg_shoulder_length}" radius="${upperleg_shoulder_radius}"/>
-                </geometry>
-            </collision>
-        </link> -->
         <joint name="${name}_hfe_joint" type="continuous">
             <origin rpy="0 0 0" xyz="0.0 ${upperleg_offset*mirror} 0"/>
@@ -76,8 +62,8 @@
                 <geometry>
                     <xacro:if value="${mirror_dae == True}">
-                        <mesh filename="package://ylo2_description/meshes/thigh_fl_resized.stl" scale="-1 -1 1"/>
+                        <mesh filename="package://ylo2_urdf_2022_description/meshes/leg/fl_upper_leg.stl" scale="1 1 1"/>
                     </xacro:if>
                     <xacro:if value="${mirror_dae == False}">
-                        <mesh filename="package://ylo2_description/meshes/thigh_fl_resized.stl" scale="-1 1 1"/>
+                        <mesh filename="package://ylo2_urdf_2022_description/meshes/leg/fl_upper_leg.stl" scale="1 -1 1"/>
                     </xacro:if>
                 </geometry>
@@ -85,8 +71,14 @@
             </visual>
             <collision>
-                <origin rpy="0 ${PI/2.0} 0" xyz="0 0 ${-upperleg_length/2.0}"/>
+                <origin rpy="0 0 0" xyz="0 ${-0.0732*mirror} 0"/> <!-- positionnement des 4 axes en meme temps -->
                 <geometry>
-                    <box size="${upperleg_length} ${upperleg_width} ${upperleg_height}"/>
+                    <xacro:if value="${mirror_dae == True}">
+                        <mesh filename="package://ylo2_urdf_2022_description/meshes/leg/fl_upper_leg_collision.stl" scale="1 1 1"/>
+                    </xacro:if>
+                    <xacro:if value="${mirror_dae == False}">
+                        <mesh filename="package://ylo2_urdf_2022_description/meshes/leg/fl_upper_leg_collision.stl" scale="1 -1 1"/>
+                    </xacro:if>
                 </geometry>
+                <material name="red"/>
             </collision>
             <inertial>
@@ -111,13 +103,14 @@
                 <origin rpy="0 0 0" xyz="0 ${0.001*mirror} 0"/>
                 <geometry>
-                    <mesh filename="package://ylo2_description/meshes/shank_fl_resized.stl" scale="-1 1 1"/>
+                    <mesh filename="package://ylo2_urdf_2022_description/meshes/leg/fl_lower_leg.stl" scale="1 1 1"/>
                 </geometry>
                 <material name="grey"/>
             </visual>
             <collision>
-                <origin rpy="0 ${PI/2.0} 0" xyz="0 0 ${-lowerleg_length/2.0}"/>
+                <origin rpy="0 0 0" xyz="0 ${0.001*mirror} 0"/>
                 <geometry>
-                    <box size="${lowerleg_length} ${lowerleg_width} ${lowerleg_height}"/>
+                    <mesh filename="package://ylo2_urdf_2022_description/meshes/leg/fl_lower_leg_collision.stl" scale="1 -1 1"/>
                 </geometry>
+                <material name="red"/>
             </collision>
             <inertial>
@@ -135,28 +128,4 @@
             <child link="${name}_foot"/>
         </joint>
-        <!--
-        <link name="${name}_foot">
-            <visual>
-                <origin rpy="0 0 0" xyz="0 0 0"/>
-                <geometry>
-                    <sphere radius="${foot_radius-0.01}"/>
-                </geometry>
-                <material name="green"/>
-            </visual>
-            <collision>
-                <origin rpy="0 0 0" xyz="0 0 0"/>
-                <geometry>
-                    <sphere radius="${foot_radius}"/>
-                </geometry>
-            </collision>
-            <inertial>
-                <mass value="${foot_mass}"/>
-                <inertia
-                    ixx="${(2*foot_mass)/5.0*(foot_radius*foot_radius)}" ixy="0.0" ixz="0.0"
-                    iyy="${(2*foot_mass)/5.0*(foot_radius*foot_radius)}" iyz="0.0"
-                    izz="${(2*foot_mass)/5.0*(foot_radius*foot_radius)}"/>
-            </inertial>
-        </link>
-        -->
         <link name="${name}_foot">
             <inertial>
@@ -171,13 +140,14 @@
                 <origin rpy="0 0 0" xyz="0.009 ${(0.001*mirror)+0.001} 0.069"/>
                 <geometry>
-                    <mesh filename="package://ylo2_description/meshes/toe_fl_resized.stl" scale="-1.0 1.0 1.0"/>
+                    <mesh filename="package://ylo2_urdf_2022_description/meshes/leg/fl_foot.stl" scale="1.0 1.0 1.0"/>
                 </geometry>
                 <material name="white"/>
             </visual>
             <collision>
-                <origin rpy="0 0 0" xyz="0 0 0"/>
+                <origin rpy="0 0 0" xyz="0.009 ${(0.001*mirror)+0.001} 0.069"/>
                 <geometry>
-                    <mesh filename="package://ylo2_description/meshes/toe_fl_resized.stl" scale="-1.0 1.0 1.0"/>
+                    <mesh filename="package://ylo2_urdf_2022_description/meshes/leg/fl_foot_collision.stl" scale="1.0 1.0 1.0"/>
                 </geometry>
+                <material name="red"/>
             </collision>
         </link>
