Commit message: Make the standup position for ylo2 more stable by increasing slighlty the haa angles

File: ylo2_description/robots/ylo2.srdf.xacro (robot description, xacro)
@@ -47,28 +47,28 @@
     </group>
     <group_state group="chains" name="standup">
-        <joint name="lf_haa_joint" value="0.1"/>
-        <joint name="lf_hfe_joint" value="0.67"/>
-        <joint name="lf_kfe_joint" value="-1.3"/>
-        <joint name="rf_haa_joint" value="-0.1"/>
-        <joint name="rf_hfe_joint" value="0.67"/>
-        <joint name="rf_kfe_joint" value="-1.3"/>
-        <joint name="lh_haa_joint" value="0.1"/>
-        <joint name="lh_hfe_joint" value="0.67"/>
-        <joint name="lh_kfe_joint" value="-1.3"/>
-        <joint name="rh_haa_joint" value="-0.1"/>
-        <joint name="rh_hfe_joint" value="0.67"/>
-        <joint name="rh_kfe_joint" value="-1.3"/>
+        <joint name="lf_haa_joint" value="0.051"/>
+        <joint name="lf_hfe_joint" value="1.0"/>
+        <joint name="lf_kfe_joint" value="-1.7"/>
+        <joint name="rf_haa_joint" value="-0.051"/>
+        <joint name="rf_hfe_joint" value="1.0"/>
+        <joint name="rf_kfe_joint" value="-1.7"/>
+        <joint name="lh_haa_joint" value="0.051"/>
+        <joint name="lh_hfe_joint" value="1.0"/>
+        <joint name="lh_kfe_joint" value="-1.7"/>
+        <joint name="rh_haa_joint" value="-0.051"/>
+        <joint name="rh_hfe_joint" value="1.0"/>
+        <joint name="rh_kfe_joint" value="-1.7"/>
     </group_state>
     <group_state group="chains" name="standdown">
-        <joint name="lf_haa_joint" value="0.8"/>
+        <joint name="lf_haa_joint" value="0.60"/>
         <joint name="lf_hfe_joint" value="1.70"/>
         <joint name="lf_kfe_joint" value="-2.77"/>
-        <joint name="rf_haa_joint" value="-0.8"/>
+        <joint name="rf_haa_joint" value="-0.60"/>
         <joint name="rf_hfe_joint" value="1.70"/>
         <joint name="rf_kfe_joint" value="-2.77"/>
-        <joint name="lh_haa_joint" value="0.8"/>
+        <joint name="lh_haa_joint" value="0.60"/>
         <joint name="lh_hfe_joint" value="1.52"/>
         <joint name="lh_kfe_joint" value="-2.77"/>
-        <joint name="rh_haa_joint" value="-0.8"/>
+        <joint name="rh_haa_joint" value="-0.60"/>
         <joint name="rh_hfe_joint" value="1.52"/>
         <joint name="rh_kfe_joint" value="-2.77"/>

Commit message: Update ylo2, remove hip collisions

File: ylo2_description/robots/ylo2.srdf.xacro (robot description, xacro)
@@ -47,14 +47,14 @@
     </group>
     <group_state group="chains" name="standup">
-        <joint name="lf_haa_joint" value="0.051"/>
+        <joint name="lf_haa_joint" value="-0.051"/>
         <joint name="lf_hfe_joint" value="1.0"/>
         <joint name="lf_kfe_joint" value="-1.7"/>
-        <joint name="rf_haa_joint" value="-0.051"/>
+        <joint name="rf_haa_joint" value="0.051"/>
         <joint name="rf_hfe_joint" value="1.0"/>
         <joint name="rf_kfe_joint" value="-1.7"/>
-        <joint name="lh_haa_joint" value="0.051"/>
+        <joint name="lh_haa_joint" value="-0.051"/>
         <joint name="lh_hfe_joint" value="1.0"/>
         <joint name="lh_kfe_joint" value="-1.7"/>
-        <joint name="rh_haa_joint" value="-0.051"/>
+        <joint name="rh_haa_joint" value="0.051"/>
         <joint name="rh_hfe_joint" value="1.0"/>
         <joint name="rh_kfe_joint" value="-1.7"/>

File: ylo2_description/urdfs/const.xacro (robot description, xacro)
@@ -5,5 +5,5 @@
     <xacro:property name="stick_mass" value="0.00001"/>
     <!-- simplified collision value for ylo2 -->
-    <!-- corps -->
+    <!-- body -->
     <xacro:property name="trunk_width" value="0.350"/>
     <xacro:property name="trunk_length" value="0.569125"/>
@@ -65,5 +65,5 @@
     <!-- hip (left front) -->
     <xacro:property name="hip_mass" value="0.599"/>
-    <xacro:property name="hip_com_x" value="-0.011957"/> <!-- com bon-->
+    <xacro:property name="hip_com_x" value="-0.011957"/>
     <xacro:property name="hip_com_y" value="0.000306"/>
     <xacro:property name="hip_com_z" value="0.000366"/>
@@ -76,5 +76,5 @@
     <!-- upperleg -->
     <xacro:property name="upperleg_mass" value="1.080"/>
-    <xacro:property name="upperleg_com_x" value="-0.000684"/> <!-- com bon-->
+    <xacro:property name="upperleg_com_x" value="-0.000684"/>
     <xacro:property name="upperleg_com_y" value="-0.010999"/>
     <xacro:property name="upperleg_com_z" value="-0.035487"/>
@@ -87,5 +87,5 @@
     <!-- lowerleg -->
     <xacro:property name="lowerleg_mass" value="0.175"/>
-    <xacro:property name="lowerleg_com_x" value="0.000252"/> <!-- com bon-->
+    <xacro:property name="lowerleg_com_x" value="0.000252"/>
     <xacro:property name="lowerleg_com_y" value="0.000194"/>
     <xacro:property name="lowerleg_com_z" value="-0.05192"/>

File: ylo2_description/urdfs/leg.xacro (robot description, xacro)
@@ -34,10 +34,4 @@
                 <material name="white"/>
             </visual>
-            <collision>
-                <origin rpy="${PI/2.0} 0 0" xyz="0 ${hip_offset*mirror} 0"/>
-                <geometry>
-                    <cylinder length="${hip_length}" radius="${hip_radius}"/>
-                </geometry>
-            </collision>
             <inertial>
                 <origin rpy="0 0 0" xyz="${hip_com_x*front_hind} ${hip_com_y*mirror} ${hip_com_z}"/>
