Commit message: ylo2 improving gaits

File: ylo2_description/urdfs/leg.xacro (robot description, xacro)
@@ -18,26 +18,20 @@
             <visual>
                 <xacro:if value="${(mirror_dae == True) and (front_hind_dae == True)}">
-                    <origin rpy="0 0 0" xyz="-0.059 -0.046 0"/>
+                    <origin rpy="0 0 0" xyz="-0.06 0 0"/>
                 </xacro:if>
                 <xacro:if value="${(mirror_dae == False) and (front_hind_dae == True)}">
-                    <origin rpy="${PI} 0 0" xyz="-0.059 0.046 0"/>
+                    <origin rpy="${PI} 0 0" xyz="-0.06 0 0"/>
                 </xacro:if>
                 <xacro:if value="${(mirror_dae == True) and (front_hind_dae == False)}">
-                    <origin rpy="0 ${PI} 0" xyz="0.059 -0.046 0"/>
+                    <origin rpy="0 ${PI} 0" xyz="0.06 0 0"/>
                 </xacro:if>
                 <xacro:if value="${(mirror_dae == False) and (front_hind_dae == False)}">
-                    <origin rpy="${PI} ${PI} 0" xyz="0.059 0.046 0"/>
+                    <origin rpy="${PI} ${PI} 0" xyz="0.06 0 0"/>
                 </xacro:if>
                 <geometry>
-                    <mesh filename="package://ylo2_description/meshes/abduct_fl_resized.stl" scale="-1 -1 1"/>
+                    <mesh filename="package://ylo2_description/meshes/leg/textured/ylo2texturedhip.dae" scale="1 1 1"/>
                 </geometry>
-                <material name="grey"/>
+                <material name="white"/>
             </visual>
-            <collision>
-                <origin rpy="${PI/2.0} 0 0" xyz="0 ${hip_offset*mirror} 0"/>
-                <geometry>
-                    <cylinder length="${hip_length}" radius="${hip_radius}"/>
-                </geometry>
-            </collision>
             <inertial>
                 <origin rpy="0 0 0" xyz="${hip_com_x*front_hind} ${hip_com_y*mirror} ${hip_com_z}"/>
@@ -49,18 +43,4 @@
             </inertial>
         </link>
-        <!-- <joint name="${name}_hip_fixed" type="fixed">
-            <origin rpy="0 0 0" xyz="0 ${(upperleg_shoulder_length/2.0+hip_offset)*mirror} 0"/>
-            <parent link="${name}_hip"/>
-            <child link="${name}_upperleg_shoulder"/>
-        </joint> -->
-        <!-- this link is only for collision -->
-        <!-- <link name="${name}_upperleg_shoulder">
-            <collision>
-                <origin rpy="${PI/2.0} 0 0" xyz="0 0 0"/>
-                <geometry>
-                    <cylinder length="${upperleg_shoulder_length}" radius="${upperleg_shoulder_radius}"/>
-                </geometry>
-            </collision>
-        </link> -->
         <joint name="${name}_hfe_joint" type="continuous">
             <origin rpy="0 0 0" xyz="0.0 ${upperleg_offset*mirror} 0"/>
@@ -76,8 +56,8 @@
                 <geometry>
                     <xacro:if value="${mirror_dae == True}">
-                        <mesh filename="package://ylo2_description/meshes/thigh_fl_resized.stl" scale="-1 -1 1"/>
+                        <mesh filename="package://ylo2_description/meshes/leg/textured/ylo2_textured_upper_leg.dae" scale="1 1 1"/>
                     </xacro:if>
                     <xacro:if value="${mirror_dae == False}">
-                        <mesh filename="package://ylo2_description/meshes/thigh_fl_resized.stl" scale="-1 1 1"/>
+                        <mesh filename="package://ylo2_description/meshes/leg/textured/ylo2_textured_upper_leg.dae" scale="1 -1 1"/>
                     </xacro:if>
                 </geometry>
@@ -85,8 +65,14 @@
             </visual>
             <collision>
-                <origin rpy="0 ${PI/2.0} 0" xyz="0 0 ${-upperleg_length/2.0}"/>
+                <origin rpy="0 0 0" xyz="0 ${-0.0732*mirror} 0"/> <!-- positionnement des 4 axes en meme temps -->
                 <geometry>
-                    <box size="${upperleg_length} ${upperleg_width} ${upperleg_height}"/>
+                    <xacro:if value="${mirror_dae == True}">
+                        <mesh filename="package://ylo2_description/meshes/leg/fl_upper_leg_collision.stl" scale="1 1 1"/>
+                    </xacro:if>
+                    <xacro:if value="${mirror_dae == False}">
+                        <mesh filename="package://ylo2_description/meshes/leg/fl_upper_leg_collision.stl" scale="1 -1 1"/>
+                    </xacro:if>
                 </geometry>
+                <material name="red"/>
             </collision>
             <inertial>
@@ -111,13 +97,14 @@
                 <origin rpy="0 0 0" xyz="0 ${0.001*mirror} 0"/>
                 <geometry>
-                    <mesh filename="package://ylo2_description/meshes/shank_fl_resized.stl" scale="-1 1 1"/>
+                    <mesh filename="package://ylo2_description/meshes/leg/textured/lower_leg.dae" scale="1 1 1"/>
                 </geometry>
-                <material name="grey"/>
+                <material name="white"/>
             </visual>
             <collision>
-                <origin rpy="0 ${PI/2.0} 0" xyz="0 0 ${-lowerleg_length/2.0}"/>
+                <origin rpy="0 0 0" xyz="0 ${0.001*mirror} 0"/>
                 <geometry>
-                    <box size="${lowerleg_length} ${lowerleg_width} ${lowerleg_height}"/>
+                    <mesh filename="package://ylo2_description/meshes/leg/fl_lower_leg_collision.stl" scale="1 -1 1"/>
                 </geometry>
+                <material name="red"/>
             </collision>
             <inertial>
@@ -135,28 +122,4 @@
             <child link="${name}_foot"/>
         </joint>
-        <!--
-        <link name="${name}_foot">
-            <visual>
-                <origin rpy="0 0 0" xyz="0 0 0"/>
-                <geometry>
-                    <sphere radius="${foot_radius-0.01}"/>
-                </geometry>
-                <material name="green"/>
-            </visual>
-            <collision>
-                <origin rpy="0 0 0" xyz="0 0 0"/>
-                <geometry>
-                    <sphere radius="${foot_radius}"/>
-                </geometry>
-            </collision>
-            <inertial>
-                <mass value="${foot_mass}"/>
-                <inertia
-                    ixx="${(2*foot_mass)/5.0*(foot_radius*foot_radius)}" ixy="0.0" ixz="0.0"
-                    iyy="${(2*foot_mass)/5.0*(foot_radius*foot_radius)}" iyz="0.0"
-                    izz="${(2*foot_mass)/5.0*(foot_radius*foot_radius)}"/>
-            </inertial>
-        </link>
-        -->
         <link name="${name}_foot">
             <inertial>
@@ -171,13 +134,14 @@
                 <origin rpy="0 0 0" xyz="0.009 ${(0.001*mirror)+0.001} 0.069"/>
                 <geometry>
-                    <mesh filename="package://ylo2_description/meshes/toe_fl_resized.stl" scale="-1.0 1.0 1.0"/>
+                    <mesh filename="package://ylo2_description/meshes/leg/fl_foot.dae" scale="1.0 1.0 1.0"/>
                 </geometry>
-                <material name="white"/>
+                <material name="orange"/>
             </visual>
             <collision>
-                <origin rpy="0 0 0" xyz="0 0 0"/>
+                <origin rpy="0 0 0" xyz="0.009 ${(0.001*mirror)+0.001} 0.069"/>
                 <geometry>
-                    <mesh filename="package://ylo2_description/meshes/toe_fl_resized.stl" scale="-1.0 1.0 1.0"/>
+                    <mesh filename="package://ylo2_description/meshes/leg/fl_foot_collision.stl" scale="1.0 1.0 1.0"/>
                 </geometry>
+                <material name="red"/>
             </collision>
         </link>
