Commit message: Add postural

File: anymal_description/robots/anymal.srdf.xacro (robot description, xacro)
@@ -47,29 +47,29 @@
   </group>
   <group_state group="chains" name="standup">
-      <joint name="lf_haa_joint" value="0.0"/>
-      <joint name="lf_hfe_joint" value="0.75"/>
-      <joint name="lf_kfe_joint" value="-1.0"/>
-      <joint name="rf_haa_joint" value="0.0"/>
-      <joint name="rf_hfe_joint" value="0.75"/>
-      <joint name="rf_kfe_joint" value="-1.0"/>
-      <joint name="lh_haa_joint" value="0.0"/>
-      <joint name="lh_hfe_joint" value="-0.75"/>
-      <joint name="lh_kfe_joint" value="1.0"/>
-      <joint name="rh_haa_joint" value="0.0"/>
-      <joint name="rh_hfe_joint" value="-0.75"/>
-      <joint name="rh_kfe_joint" value="1.0"/>
+    <joint name="lf_haa_joint" value="-0.15"/>
+    <joint name="lf_hfe_joint" value="0.75"/>
+    <joint name="lf_kfe_joint" value="5.08"/>
+    <joint name="rf_haa_joint" value="0.15"/>
+    <joint name="rf_hfe_joint" value="0.75"/>
+    <joint name="rf_kfe_joint" value="5.08"/>
+    <joint name="lh_haa_joint" value="-0.15"/>
+    <joint name="lh_hfe_joint" value="-0.75"/>
+    <joint name="lh_kfe_joint" value="1.20"/>
+    <joint name="rh_haa_joint" value="0.15"/>
+    <joint name="rh_hfe_joint" value="-0.75"/>
+    <joint name="rh_kfe_joint" value="1.20"/>
   </group_state>
   <group_state group="chains" name="standdown">
     <joint name="lf_haa_joint" value="0.0"/>
-    <joint name="lf_hfe_joint" value="1.60"/>
-    <joint name="lf_kfe_joint" value="2.60"/>
+    <joint name="lf_hfe_joint" value="1.7"/>
+    <joint name="lf_kfe_joint" value="3.66"/>
     <joint name="rf_haa_joint" value="0.0"/>
-    <joint name="rf_hfe_joint" value="1.60"/>
-    <joint name="rf_kfe_joint" value="2.60"/>
+    <joint name="rf_hfe_joint" value="1.7"/>
+    <joint name="rf_kfe_joint" value="3.66"/>
     <joint name="lh_haa_joint" value="0.0"/>
-    <joint name="lh_hfe_joint" value="-1.60"/>
+    <joint name="lh_hfe_joint" value="-1.7"/>
     <joint name="lh_kfe_joint" value="2.60"/>
     <joint name="rh_haa_joint" value="0.0"/>
-    <joint name="rh_hfe_joint" value="-1.60"/>
+    <joint name="rh_hfe_joint" value="-1.7"/>
     <joint name="rh_kfe_joint" value="2.60"/>
   </group_state>
