Commit message: Some anymalc updates

File: anymalc_description/robots/anymalc.srdf.xacro (robot description, xacro)
@@ -63,8 +63,8 @@
     <joint name="lf_haa_joint" value="0.0"/>
     <joint name="lf_hfe_joint" value="1.60"/>
-    <joint name="lf_kfe_joint" value="-2.60"/>
+    <joint name="lf_kfe_joint" value="2.60"/>
     <joint name="rf_haa_joint" value="0.0"/>
     <joint name="rf_hfe_joint" value="1.60"/>
-    <joint name="rf_kfe_joint" value="-2.60"/>
+    <joint name="rf_kfe_joint" value="2.60"/>
     <joint name="lh_haa_joint" value="0.0"/>
     <joint name="lh_hfe_joint" value="-1.60"/>

Commit message: Working anymalc

File: anymalc_description/robots/anymalc.srdf.xacro (robot description, xacro)
@@ -47,29 +47,29 @@
   </group>
   <group_state group="chains" name="standup">
-    <joint name="lf_haa_joint" value="0.0"/>
+    <joint name="lf_haa_joint" value="-0.15"/>
     <joint name="lf_hfe_joint" value="0.75"/>
-    <joint name="lf_kfe_joint" value="-1.0"/>
-    <joint name="rf_haa_joint" value="0.0"/>
+    <joint name="lf_kfe_joint" value="-1.20"/>
+    <joint name="rf_haa_joint" value="0.15"/>
     <joint name="rf_hfe_joint" value="0.75"/>
-    <joint name="rf_kfe_joint" value="-1.0"/>
-    <joint name="lh_haa_joint" value="0.0"/>
+    <joint name="rf_kfe_joint" value="-1.20"/>
+    <joint name="lh_haa_joint" value="-0.15"/>
     <joint name="lh_hfe_joint" value="-0.75"/>
-    <joint name="lh_kfe_joint" value="1.0"/>
-    <joint name="rh_haa_joint" value="0.0"/>
+    <joint name="lh_kfe_joint" value="1.20"/>
+    <joint name="rh_haa_joint" value="0.15"/>
     <joint name="rh_hfe_joint" value="-0.75"/>
-    <joint name="rh_kfe_joint" value="1.0"/>
+    <joint name="rh_kfe_joint" value="1.20"/>
   </group_state>
   <group_state group="chains" name="standdown">
     <joint name="lf_haa_joint" value="0.0"/>
-    <joint name="lf_hfe_joint" value="1.60"/>
+    <joint name="lf_hfe_joint" value="1.7"/>
     <joint name="lf_kfe_joint" value="2.60"/>
     <joint name="rf_haa_joint" value="0.0"/>
-    <joint name="rf_hfe_joint" value="1.60"/>
+    <joint name="rf_hfe_joint" value="1.67"/>
     <joint name="rf_kfe_joint" value="2.60"/>
     <joint name="lh_haa_joint" value="0.0"/>
-    <joint name="lh_hfe_joint" value="-1.60"/>
+    <joint name="lh_hfe_joint" value="-1.7"/>
     <joint name="lh_kfe_joint" value="2.60"/>
     <joint name="rh_haa_joint" value="0.0"/>
-    <joint name="rh_hfe_joint" value="-1.60"/>
+    <joint name="rh_hfe_joint" value="-1.7"/>
     <joint name="rh_kfe_joint" value="2.60"/>
   </group_state>

Commit message: Fix anymalc postures

File: anymalc_description/robots/anymalc.srdf.xacro (robot description, xacro)
@@ -49,8 +49,8 @@
     <joint name="lf_haa_joint" value="-0.15"/>
     <joint name="lf_hfe_joint" value="0.75"/>
-    <joint name="lf_kfe_joint" value="-1.20"/>
+    <joint name="lf_kfe_joint" value="5.08"/>
     <joint name="rf_haa_joint" value="0.15"/>
     <joint name="rf_hfe_joint" value="0.75"/>
-    <joint name="rf_kfe_joint" value="-1.20"/>
+    <joint name="rf_kfe_joint" value="5.08"/>
     <joint name="lh_haa_joint" value="-0.15"/>
     <joint name="lh_hfe_joint" value="-0.75"/>
@@ -63,8 +63,8 @@
     <joint name="lf_haa_joint" value="0.0"/>
     <joint name="lf_hfe_joint" value="1.7"/>
-    <joint name="lf_kfe_joint" value="2.60"/>
+    <joint name="lf_kfe_joint" value="3.66"/>
     <joint name="rf_haa_joint" value="0.0"/>
-    <joint name="rf_hfe_joint" value="1.67"/>
-    <joint name="rf_kfe_joint" value="2.60"/>
+    <joint name="rf_hfe_joint" value="1.7"/>
+    <joint name="rf_kfe_joint" value="3.66"/>
     <joint name="lh_haa_joint" value="0.0"/>
     <joint name="lh_hfe_joint" value="-1.7"/>

Commit message: Add anymalc sensors

File: anymalc_description/robots/anymalc.srdf.xacro (robot description, xacro)
@@ -3,4 +3,7 @@
   <group name="base">
     <link name="base"/>
+  </group>
+  <group name="imu">
+    <link name="imu_link"/>
   </group>
   <group name="lf_leg">

File: anymalc_description/robots/anymalc.urdf.xacro (robot description, xacro)
@@ -7,4 +7,5 @@
    <!-- This argument allows us to load joint sensors that measure the internal wrenches -->
    <xacro:arg name="load_force_sensors" default="false"/>
+   <xacro:arg name="sensors" default="false"/>
    <xacro:arg name="task_period" default="0.004"/>
    <xacro:arg name="floating_base_link" default="true"/>
@@ -18,4 +19,5 @@
    <xacro:include filename="$(find wolf_description_utils)/urdfs/leg.transmission.xacro"/>
    <xacro:include filename="$(find wolf_description_utils)/urdfs/leg.gazebo.xacro"/>
+   <xacro:property name="foot_radius" value="0.03"/>
     <!-- Base link -->
     <link name="base">
@@ -467,5 +469,5 @@
         <parent link="base"/>
         <child link="imu_link"/>
-        <origin rpy="0.0 0.0 1.57079632679" xyz="0.2488 0.00835 0.04628"/>
+        <origin rpy="0.0 0.0 0.0" xyz="0.2488 0.00835 0.04628"/>
     </joint>
     <!-- Camera joint -->
@@ -858,5 +860,5 @@
             <origin xyz="0 0 0.0225"/>
             <geometry>
-                <sphere radius="0.03"/>
+                <sphere radius="${foot_radius}"/>
             </geometry>
         </collision>
@@ -1102,5 +1104,5 @@
             <origin xyz="0 0 0.0225"/>
             <geometry>
-                <sphere radius="0.03"/>
+                <sphere radius="${foot_radius}"/>
             </geometry>
         </collision>
@@ -1346,5 +1348,5 @@
             <origin xyz="0 0 0.0225"/>
             <geometry>
-                <sphere radius="0.03"/>
+                <sphere radius="${foot_radius}"/>
             </geometry>
         </collision>
@@ -1590,5 +1592,5 @@
             <origin xyz="0 0 0.0225"/>
             <geometry>
-                <sphere radius="0.03"/>
+                <sphere radius="${foot_radius}"/>
             </geometry>
         </collision>
@@ -1628,3 +1630,42 @@
     <xacro:leg_transmission prefix="lh"/>
     <xacro:leg_gazebo prefix="lh" robot_name="$(arg robot_name)" load_force_sensors="$(arg load_force_sensors)"/>
+    <!-- Standard accessories. -->
+    <xacro:if value="$(arg sensors)">
+        <xacro:include filename="$(find sensors_description)/urdfs/common.xacro"/>
+        <xacro:include filename="$(find velodyne_description)/urdf/VLP-16.urdf.xacro"/>
+        <xacro:include filename="$(find sensors_description)/urdfs/sensors/realsense_d435.urdf.xacro" />
+        <xacro:include filename="$(find sensors_description)/urdfs/sensors/realsense_t265.xacro" />
+        <xacro:include filename="$(find sensors_description)/urdfs/sensors/imu.gazebo.xacro"/>
+        <xacro:include filename="$(find sensors_description)/urdfs/sensors/wideangle_camera.urdf.xacro"/>
+        <xacro:imu_sensor
+            imu_name="imu_link"
+            imu_topic="imu_link/data"
+            update_rate="${1.0 / $(arg task_period)}"
+            rate_mean="0"
+            rate_stddev="0"
+            rate_bias_mean="0"
+            rate_bias_stddev="0"
+            accel_mean="0"
+            accel_stddev="0"
+            accel_bias_mean="0"
+            accel_bias_stddev="0">
+        </xacro:imu_sensor>
+        <xacro:VLP-16 parent="lidar" name="velodyne" topic="/velodyne_pointcloud"
+                      organize_cloud="true" hz="10" gpu="true">
+          <origin xyz="0 0 0" rpy="0 0 0" />
+        </xacro:VLP-16>
+        <xacro:sensor_d435 name="d435_front" topics_ns="d435_front" parent="depth_camera_front_camera">
+          <origin xyz="0 0 0" rpy="0 0 0" />
+        </xacro:sensor_d435>
+        <xacro:sensor_d435 name="d435_rear" topics_ns="d435_rear" parent="depth_camera_rear_camera">
+          <origin xyz="0 0 0" rpy="0 0 0" />
+        </xacro:sensor_d435>
+        <xacro:realsense_T265 sensor_name="t265_right" parent_link="depth_camera_right_camera" rate="30.0">
+          <origin xyz="0 0 0" rpy="0 0 0" />
+        </xacro:realsense_T265>
+        <xacro:realsense_T265 sensor_name="t265_left" parent_link="depth_camera_left_camera" rate="30.0">
+          <origin xyz="0 0 0" rpy="0 0 0" />
+        </xacro:realsense_T265>
+       <xacro:wideangle_camera reference="wide_angle_camera_front_camera" ns="wide_angle_camera_front_camera" frame_id="wide_angle_camera_front_camera" update_rate="30.0"/>
+    </xacro:if>
 </robot>

Commit message: Working on waistZ branch

File: anymalc_description/robots/anymalc.srdf.xacro (robot description, xacro)
@@ -6,4 +6,10 @@
   <group name="imu">
     <link name="imu_link"/>
+  </group>
+  <group name="contacts">
+    <link name="lf_foot"/>
+    <link name="rf_foot"/>
+    <link name="lh_foot"/>
+    <link name="rh_foot"/>
   </group>
   <group name="lf_leg">
@@ -50,16 +56,16 @@
   </group>
   <group_state group="chains" name="standup">
-    <joint name="lf_haa_joint" value="-0.15"/>
-    <joint name="lf_hfe_joint" value="0.75"/>
-    <joint name="lf_kfe_joint" value="5.08"/>
-    <joint name="rf_haa_joint" value="0.15"/>
-    <joint name="rf_hfe_joint" value="0.75"/>
-    <joint name="rf_kfe_joint" value="5.08"/>
-    <joint name="lh_haa_joint" value="-0.15"/>
-    <joint name="lh_hfe_joint" value="-0.75"/>
-    <joint name="lh_kfe_joint" value="1.20"/>
-    <joint name="rh_haa_joint" value="0.15"/>
-    <joint name="rh_hfe_joint" value="-0.75"/>
-    <joint name="rh_kfe_joint" value="1.20"/>
+    <joint name="lf_haa_joint" value="-0.12"/>
+    <joint name="lf_hfe_joint" value="0.83"/>
+    <joint name="lf_kfe_joint" value="5.0"/>
+    <joint name="rf_haa_joint" value="0.12"/>
+    <joint name="rf_hfe_joint" value="0.83"/>
+    <joint name="rf_kfe_joint" value="5.0"/>
+    <joint name="lh_haa_joint" value="-0.12"/>
+    <joint name="lh_hfe_joint" value="-0.83"/>
+    <joint name="lh_kfe_joint" value="-5.0"/>
+    <joint name="rh_haa_joint" value="0.12"/>
+    <joint name="rh_hfe_joint" value="-0.83"/>
+    <joint name="rh_kfe_joint" value="-5.0"/>
   </group_state>
   <group_state group="chains" name="standdown">

Commit message: Make anymal and anymalc walk again

File: anymalc_description/robots/anymalc.srdf.xacro (robot description, xacro)
@@ -3,4 +3,13 @@
   <group name="base">
     <link name="base"/>
+  </group>
+  <group name="imu">
+    <link name="imu_link"/>
+  </group>
+  <group name="contacts">
+    <link name="lf_foot"/>
+    <link name="rf_foot"/>
+    <link name="lh_foot"/>
+    <link name="rh_foot"/>
   </group>
   <group name="lf_leg">
@@ -47,24 +56,24 @@
   </group>
   <group_state group="chains" name="standup">
-    <joint name="lf_haa_joint" value="-0.15"/>
-    <joint name="lf_hfe_joint" value="0.75"/>
-    <joint name="lf_kfe_joint" value="-1.20"/>
-    <joint name="rf_haa_joint" value="0.15"/>
-    <joint name="rf_hfe_joint" value="0.75"/>
-    <joint name="rf_kfe_joint" value="-1.20"/>
-    <joint name="lh_haa_joint" value="-0.15"/>
-    <joint name="lh_hfe_joint" value="-0.75"/>
-    <joint name="lh_kfe_joint" value="1.20"/>
-    <joint name="rh_haa_joint" value="0.15"/>
-    <joint name="rh_hfe_joint" value="-0.75"/>
-    <joint name="rh_kfe_joint" value="1.20"/>
+    <joint name="lf_haa_joint" value="-0.12"/>
+    <joint name="lf_hfe_joint" value="0.83"/>
+    <joint name="lf_kfe_joint" value="5.0"/>
+    <joint name="rf_haa_joint" value="0.12"/>
+    <joint name="rf_hfe_joint" value="0.83"/>
+    <joint name="rf_kfe_joint" value="5.0"/>
+    <joint name="lh_haa_joint" value="-0.12"/>
+    <joint name="lh_hfe_joint" value="-0.83"/>
+    <joint name="lh_kfe_joint" value="-5.0"/>
+    <joint name="rh_haa_joint" value="0.12"/>
+    <joint name="rh_hfe_joint" value="-0.83"/>
+    <joint name="rh_kfe_joint" value="-5.0"/>
   </group_state>
   <group_state group="chains" name="standdown">
     <joint name="lf_haa_joint" value="0.0"/>
     <joint name="lf_hfe_joint" value="1.7"/>
-    <joint name="lf_kfe_joint" value="2.60"/>
+    <joint name="lf_kfe_joint" value="3.66"/>
     <joint name="rf_haa_joint" value="0.0"/>
-    <joint name="rf_hfe_joint" value="1.67"/>
-    <joint name="rf_kfe_joint" value="2.60"/>
+    <joint name="rf_hfe_joint" value="1.7"/>
+    <joint name="rf_kfe_joint" value="3.66"/>
     <joint name="lh_haa_joint" value="0.0"/>
     <joint name="lh_hfe_joint" value="-1.7"/>
