Commit message: Flip velodyne for aliengo and anymalc

File: aliengo_description/urdfs/accessories.urdf.xacro (robot description, xacro)
@@ -54,5 +54,5 @@
   <xacro:VLP-16 parent="lidar" name="velodyne" topic="/velodyne_points"
                 organize_cloud="true" hz="10" gpu="true">
-    <origin xyz="0 0 0" rpy="0 0 0" />
+    <origin xyz="0 0 0" rpy="0 0 1.57" />
   </xacro:VLP-16>
   <xacro:sensor_d435 name="d435" topics_ns="d435" parent="trunk">

File: anymalc_description/robots/anymalc.urdf.xacro (robot description, xacro)
@@ -1653,5 +1653,5 @@
         <xacro:VLP-16 parent="lidar" name="velodyne" topic="/velodyne_points"
                       organize_cloud="true" hz="10" gpu="true">
-          <origin xyz="0 0 0" rpy="0 0 0" />
+          <origin xyz="0 0 0" rpy="0 0 1.57"/>
         </xacro:VLP-16>
         <xacro:sensor_d435 name="d435_front" topics_ns="d435_front" parent="depth_camera_front_camera">
