Commit message: Testing

File: spot_description/robots/spot.srdf.xacro (robot description, xacro)
@@ -3,4 +3,13 @@
     <group name="base">
       <link name="base_link"/>
+    </group>
+    <group name="imu">
+      <link name="imu_link"/>
+    </group>
+    <group name="contacts">
+      <link name="lf_foot"/>
+      <link name="rf_foot"/>
+      <link name="lh_foot"/>
+      <link name="rh_foot"/>
     </group>
     <group name="lf_leg">

Commit message: Add imu to spot

File: spot_description/robots/spot.srdf.xacro (robot description, xacro)
@@ -5,5 +5,5 @@
     </group>
     <group name="imu">
-      <link name="imu_link"/>
+      <link name="trunk_imu"/>
     </group>
     <group name="contacts">

File: spot_description/robots/spot.urdf.xacro (robot description, xacro)
@@ -17,4 +17,8 @@
     <xacro:include filename="$(find wolf_description_utils)/urdfs/leg.transmission.xacro"/>
     <xacro:include filename="$(find wolf_description_utils)/urdfs/leg.gazebo.xacro"/>
+    <!-- sensors -->
+    <xacro:if value="$(arg sensors)">
+        <xacro:include filename="$(find sensors_description)/urdfs/sensors/imu.gazebo.xacro"/>
+    </xacro:if>
     <!-- dynamics inertial value -->
     <!-- body -->
@@ -69,11 +73,17 @@
     <!-- Floating-base Joint -->
     <xacro:if value="$(arg floating_base_link)">
-	    <link name="world"/>
-	    <joint name="floating_base_joint" type="floating">
-	      <origin rpy="0 0 0" xyz="0 0 0"/>
-	      <parent link="world"/>
-	      <child link="base_link"/>
-	    </joint>
+        <link name="world"/>
+        <joint name="floating_base_joint" type="floating">
+          <origin rpy="0 0 0" xyz="0 0 0"/>
+          <parent link="world"/>
+          <child link="base_link"/>
+        </joint>
     </xacro:if>
+    <joint name="imu_joint" type="fixed">
+        <parent link="base_link"/>
+        <child link="trunk_imu"/>
+        <origin rpy="0 0 0" xyz="0 0 0"/>
+    </joint>
+    <link name="trunk_imu"/>
     <link name="base_link">
         <visual>
@@ -527,4 +537,17 @@
     <xacro:if value="$(arg sensors)">
         <xacro:include filename="$(find spot_description)/urdfs/accessories.urdf.xacro" />
+        <xacro:imu_sensor
+            imu_name="trunk_imu"
+            imu_topic="trunk_imu/data"
+            update_rate="${1.0 / $(arg task_period)}"
+            rate_mean="0"
+            rate_stddev="0"
+            rate_bias_mean="0"
+            rate_bias_stddev="0"
+            accel_mean="0"
+            accel_stddev="0"
+            accel_bias_mean="0"
+            accel_bias_stddev="0">
+        </xacro:imu_sensor>
     </xacro:if>
     <!-- Extensions -->

Commit message: Use disable lumping to get the forces at the feet

File: spot_description/robots/spot.srdf.xacro (robot description, xacro)
@@ -4,8 +4,8 @@
       <link name="base_link"/>
     </group>
-    <group name="imu">
+    <group name="imu"> <!-- where the imu sensor is mounted -->
       <link name="trunk_imu"/>
     </group>
-    <group name="contacts">
+    <group name="contacts"> <!-- where the contact sensors are mounted -->
       <link name="lf_foot"/>
       <link name="rf_foot"/>

File: wolf_description_utils/urdfs/leg.gazebo.xacro (robot description, xacro)
@@ -15,17 +15,4 @@
 			</gazebo>
 		</xacro:if>
-		<gazebo reference="${prefix}_kfe_joint">
-			<provideFeedback>true</provideFeedback>
-		</gazebo>
-		<xacro:if value="${load_force_sensors}">
-			<gazebo>
-				<plugin name="${prefix}_kfe_sensor" filename="libgazebo_ros_ft_sensor.so">
-                                        <robotNamespace>/${robot_name}/internal_wrench/</robotNamespace>
-					<updateRate>100.0</updateRate>
-					<topicName>${prefix}_kfe_joint</topicName>
-					<jointName>${prefix}_kfe_joint</jointName>
-				</plugin>
-			</gazebo>
-		</xacro:if>
 		<gazebo reference="${prefix}_hfe_joint">
 			<provideFeedback>true</provideFeedback>
@@ -41,4 +28,20 @@
 			</gazebo>
 		</xacro:if>
+                <gazebo reference="${prefix}_kfe_joint">
+                        <provideFeedback>true</provideFeedback>
+                </gazebo>
+                <xacro:if value="${load_force_sensors}">
+                        <gazebo>
+                                <plugin name="${prefix}_kfe_sensor" filename="libgazebo_ros_ft_sensor.so">
+                                        <robotNamespace>/${robot_name}/internal_wrench/</robotNamespace>
+                                        <updateRate>100.0</updateRate>
+                                        <topicName>${prefix}_kfe_joint</topicName>
+                                        <jointName>${prefix}_kfe_joint</jointName>
+                                </plugin>
+                        </gazebo>
+                </xacro:if>
+               <gazebo reference="${prefix}_foot_joint">
+                       <disableFixedJointLumping>true</disableFixedJointLumping>
+               </gazebo>
 		<gazebo reference="${prefix}_upperleg">
 			<kp>1000000.0</kp>
@@ -50,5 +53,5 @@
 			<minDepth>0.00</minDepth>
 		</gazebo>
-		<gazebo reference="${prefix}_lowerleg">
+                <gazebo reference="${prefix}_lowerleg">
 			<kp>1000000.0</kp>
 			<kd>100.0</kd>
@@ -58,16 +61,15 @@
 			<maxContacts>1</maxContacts>
 			<sensor name="${prefix}_shin_contact_sensor" type="contact">
-                <always_on>true</always_on>
-                <update_rate>250.0</update_rate>
-                <contact>
-                  <collision>${prefix}_lowerleg_collision</collision>
-                </contact>
-                <!-- the sensor readings in terms of force torques are expressed in the lowerleg frame
-                because gazebo lumps the fake footframe with the real parent link, the normals are in the world frame-->
-                 <plugin name="${prefix}_shin_bumper" filename="libgazebo_ros_bumper.so">
-                  <bumperTopicName>/${robot_name}/${prefix}_shin_bumper</bumperTopicName>
-                </plugin>
-            </sensor>
-		</gazebo>
+                                <always_on>true</always_on>
+                                <update_rate>250.0</update_rate>
+                                <contact>
+                                    <collision>${prefix}_lowerleg_collision</collision>
+                                </contact>
+                                <plugin name="${prefix}_shin_bumper" filename="libgazebo_ros_bumper.so">
+                                    <bumperTopicName>/${robot_name}/${prefix}_shin_bumper</bumperTopicName>
+                                    <robotNamespace>${robot_name}</robotNamespace>
+                                </plugin>
+                        </sensor>
+                </gazebo>
 		<gazebo reference="${prefix}_foot">
                         <kp>1000000.0</kp>
@@ -77,12 +79,10 @@
                         <maxVel>1.0</maxVel>
 			<maxContacts>1</maxContacts>
-			<sensor name="${prefix}_foot_contact_sensor" type="contact">
+                        <sensor name="${prefix}_foot_contact_sensor" type="contact">
 				<always_on>true</always_on>
 				<update_rate>250.0</update_rate>
 				<contact>
-					<collision>${prefix}_lowerleg_fixed_joint_lump__${prefix}_foot_collision_1</collision>
+                                    <collision>${prefix}_foot_collision</collision>
 				</contact>
-                                <!-- the sensor readings in terms of force torques are expressed in the lowerleg frame
-                                because gazebo lumps the fake footframe with the real parent link, the normals are in the world frame-->
 				<plugin name="${prefix}_foot_bumper" filename="libgazebo_ros_bumper.so">
                                         <bumperTopicName>/${robot_name}/${prefix}_foot_bumper</bumperTopicName>
@@ -90,5 +90,4 @@
 				</plugin>
 			</sensor>
-			<material>Gazebo/Black</material>
 		</gazebo>
 	</xacro:macro>
