Commit message: Working on the arm

File: spot_description/robots/spot_kinova.srdf.xacro (robot description, xacro)
@@ -86,7 +86,7 @@
       <joint name="rh_kfe_joint" value="-2.7"/>
       <joint name="kinova_joint_1" value="0.0"/>
-      <joint name="kinova_joint_2" value="4.9"/>
+      <joint name="kinova_joint_2" value="4.0"/>
       <joint name="kinova_joint_3" value="5.6"/>
-      <joint name="kinova_joint_4" value="0.0"/>
+      <joint name="kinova_joint_4" value="3.14"/>
     </group_state>
 </robot>

Commit message: Update spot arm params

File: spot_description/robots/spot_kinova.srdf.xacro (robot description, xacro)
@@ -1,7 +1,16 @@
 <?xml version="1.0" ?>
 <robot name="spot" xmlns:xacro="http://ros.org/wiki/xacro">
-    <group name="base">
-      <link name="base_link"/>
-    </group>
+   <group name="base">
+     <link name="base_link"/>
+   </group>
+   <group name="imu"> <!-- where the imu sensor is mounted -->
+     <link name="trunk_imu"/>
+   </group>
+   <group name="contacts"> <!-- where the contact sensors are mounted -->
+     <link name="lf_foot"/>
+     <link name="rf_foot"/>
+     <link name="lh_foot"/>
+     <link name="rh_foot"/>
+   </group>
     <group name="kinova_arm">
       <chain base_link="kinova_link_base" tip_link="kinova_end_effector"/>
