Commit message: Remove pisellino

File: spot_description/robots/spot.urdf.xacro (robot description, xacro)
@@ -203,10 +203,4 @@
         </material>
     </visual>
-    <collision>
-        <origin rpy="0 0 0" xyz="0 0 0"/>
-        <geometry>
-            <sphere radius="${foot_radius}"/>
-        </geometry>
-    </collision>
     <inertial>
         <mass value="${foot_mass}"/>
@@ -313,10 +307,4 @@
         </material>
     </visual>
-    <collision>
-        <origin rpy="0 0 0" xyz="0 0 0"/>
-        <geometry>
-            <sphere radius="${foot_radius}"/>
-        </geometry>
-    </collision>
     <inertial>
         <mass value="${foot_mass}"/>
@@ -423,10 +411,4 @@
         </material>
     </visual>
-    <collision>
-        <origin rpy="0 0 0" xyz="0 0 0"/>
-        <geometry>
-            <sphere radius="${foot_radius}"/>
-        </geometry>
-    </collision>
     <inertial>
         <mass value="${foot_mass}"/>
@@ -533,10 +515,4 @@
         </material>
     </visual>
-    <collision>
-        <origin rpy="0 0 0" xyz="0 0 0"/>
-        <geometry>
-            <sphere radius="${foot_radius}"/>
-        </geometry>
-    </collision>
     <inertial>
         <mass value="${foot_mass}"/>

Commit message: Add velocity limits to spot

File: spot_description/robots/spot.urdf.xacro (robot description, xacro)
@@ -132,5 +132,5 @@
         <parent link="base_link" />
         <child link="lf_hip" />
-        <limit effort="50" velocity="1000.00" lower="-0.78539816339744827899" upper="0.78539816339744827899" />
+        <limit effort="50" velocity="10" lower="-0.78539816339744827899" upper="0.78539816339744827899" />
     </joint>
     <link name="lf_upperleg">
@@ -159,5 +159,5 @@
         <parent link="lf_hip" />
         <child link="lf_upperleg" />
-        <limit effort="50" velocity="1000.00" lower="-0.89884456477707963539" upper="2.2951079663725435509" />
+        <limit effort="50" velocity="10" lower="-0.89884456477707963539" upper="2.2951079663725435509" />
     </joint>
     <link name="lf_lowerleg">
@@ -186,5 +186,5 @@
         <parent link="lf_upperleg" />
         <child link="lf_lowerleg" />
-        <limit effort="50" velocity="1000.00" lower="-2.7929" upper="-0.254801" />
+        <limit effort="50" velocity="10" lower="-2.7929" upper="-0.254801" />
     </joint>
     <joint name="lf_foot_joint" type="fixed">
@@ -236,5 +236,5 @@
         <parent link="base_link" />
         <child link="rf_hip" />
-        <limit effort="50" velocity="1000.00" lower="-0.78539816339744827899" upper="0.78539816339744827899" />
+        <limit effort="50" velocity="10" lower="-0.78539816339744827899" upper="0.78539816339744827899" />
     </joint>
     <link name="rf_upperleg">
@@ -263,5 +263,5 @@
         <parent link="rf_hip" />
         <child link="rf_upperleg" />
-        <limit effort="50" velocity="1000.00" lower="-0.89884456477707963539" upper="2.2951079663725435509" />
+        <limit effort="50" velocity="10" lower="-0.89884456477707963539" upper="2.2951079663725435509" />
     </joint>
     <link name="rf_lowerleg">
@@ -290,5 +290,5 @@
         <parent link="rf_upperleg" />
         <child link="rf_lowerleg" />
-        <limit effort="50" velocity="1000.00" lower="-2.7929" upper="-0.247563" />
+        <limit effort="50" velocity="10" lower="-2.7929" upper="-0.247563" />
     </joint>
     <joint name="rf_foot_joint" type="fixed">
@@ -340,5 +340,5 @@
         <parent link="base_link" />
         <child link="lh_hip" />
-        <limit effort="50" velocity="1000.00" lower="-0.78539816339744827899" upper="0.78539816339744827899" />
+        <limit effort="50" velocity="10" lower="-0.78539816339744827899" upper="0.78539816339744827899" />
     </joint>
     <link name="lh_upperleg">
@@ -367,5 +367,5 @@
         <parent link="lh_hip" />
         <child link="lh_upperleg" />
-        <limit effort="50" velocity="1000.00" lower="-0.89884456477707963539" upper="2.2951079663725435509" />
+        <limit effort="50" velocity="10" lower="-0.89884456477707963539" upper="2.2951079663725435509" />
     </joint>
     <link name="lh_lowerleg">
@@ -394,5 +394,5 @@
         <parent link="lh_upperleg" />
         <child link="lh_lowerleg" />
-        <limit effort="50" velocity="1000.00" lower="-2.7929" upper="-0.267153" />
+        <limit effort="50" velocity="10" lower="-2.7929" upper="-0.267153" />
     </joint>
     <joint name="lh_foot_joint" type="fixed">
@@ -444,5 +444,5 @@
         <parent link="base_link" />
         <child link="rh_hip" />
-        <limit effort="50" velocity="1000.00" lower="-0.78539816339744827899" upper="0.78539816339744827899" />
+        <limit effort="50" velocity="10" lower="-0.78539816339744827899" upper="0.78539816339744827899" />
     </joint>
     <link name="rh_upperleg">
@@ -471,5 +471,5 @@
         <parent link="rh_hip" />
         <child link="rh_upperleg" />
-        <limit effort="50" velocity="1000.00" lower="-0.89884456477707963539" upper="2.2951079663725435509" />
+        <limit effort="50" velocity="10" lower="-0.89884456477707963539" upper="2.2951079663725435509" />
     </joint>
     <link name="rh_lowerleg">
@@ -498,5 +498,5 @@
         <parent link="rh_upperleg" />
         <child link="rh_lowerleg" />
-        <limit effort="50" velocity="1000.00" lower="-2.7929" upper="-0.257725" />
+        <limit effort="50" velocity="10" lower="-2.7929" upper="-0.257725" />
     </joint>
     <joint name="rh_foot_joint" type="fixed">

Commit message: Add reduced meshes for spot

File: spot_description/robots/spot.urdf.xacro (robot description, xacro)
@@ -94,5 +94,5 @@
         <collision>
             <geometry>
-                <mesh filename="package://spot_description/meshes/body_collision.stl" />
+                <mesh filename="package://spot_description/meshes/body_collision_low.stl" />
             </geometry>
         </collision>
@@ -126,5 +126,5 @@
         <collision>
             <geometry>
-                <mesh filename="package://spot_description/meshes/front_left_hip_collision.stl" />
+                <mesh filename="package://spot_description/meshes/front_left_hip_collision_low.stl" />
             </geometry>
         </collision>
@@ -153,5 +153,5 @@
         <collision>
             <geometry>
-                <mesh filename="package://spot_description/meshes/front_left_upper_leg_collision.stl" />
+                <mesh filename="package://spot_description/meshes/front_left_upper_leg_collision_low.stl" />
             </geometry>
         </collision>
@@ -180,5 +180,5 @@
         <collision>
             <geometry>
-                <mesh filename="package://spot_description/meshes/front_left_lower_leg_collision.stl" />
+                <mesh filename="package://spot_description/meshes/front_left_lower_leg_collision_low.stl" />
             </geometry>
         </collision>
@@ -230,5 +230,5 @@
         <collision>
             <geometry>
-                <mesh filename="package://spot_description/meshes/front_right_hip_collision.stl" />
+                <mesh filename="package://spot_description/meshes/front_right_hip_collision_low.stl" />
             </geometry>
         </collision>
@@ -257,5 +257,5 @@
         <collision>
             <geometry>
-                <mesh filename="package://spot_description/meshes/front_right_upper_leg_collision.stl" />
+                <mesh filename="package://spot_description/meshes/front_right_upper_leg_collision_low.stl" />
             </geometry>
         </collision>
@@ -284,5 +284,5 @@
         <collision>
             <geometry>
-                <mesh filename="package://spot_description/meshes/front_right_lower_leg_collision.stl" />
+                <mesh filename="package://spot_description/meshes/front_right_lower_leg_collision_low.stl" />
             </geometry>
         </collision>
@@ -334,5 +334,5 @@
         <collision>
             <geometry>
-                <mesh filename="package://spot_description/meshes/rear_left_hip_collision.stl" />
+                <mesh filename="package://spot_description/meshes/rear_left_hip_collision_low.stl" />
             </geometry>
         </collision>
@@ -361,5 +361,5 @@
         <collision>
             <geometry>
-                <mesh filename="package://spot_description/meshes/rear_left_upper_leg_collision.stl" />
+                <mesh filename="package://spot_description/meshes/rear_left_upper_leg_collision_low.stl" />
             </geometry>
         </collision>
@@ -388,5 +388,5 @@
         <collision>
             <geometry>
-                <mesh filename="package://spot_description/meshes/rear_left_lower_leg_collision.stl" />
+                <mesh filename="package://spot_description/meshes/rear_left_lower_leg_collision_low.stl" />
             </geometry>
         </collision>
@@ -438,5 +438,5 @@
         <collision>
             <geometry>
-                <mesh filename="package://spot_description/meshes/rear_right_hip_collision.stl" />
+                <mesh filename="package://spot_description/meshes/rear_right_hip_collision_low.stl" />
             </geometry>
         </collision>
@@ -465,5 +465,5 @@
         <collision>
             <geometry>
-                <mesh filename="package://spot_description/meshes/rear_right_upper_leg_collision.stl" />
+                <mesh filename="package://spot_description/meshes/rear_right_upper_leg_collision_low.stl" />
             </geometry>
         </collision>
@@ -492,5 +492,5 @@
         <collision>
             <geometry>
-                <mesh filename="package://spot_description/meshes/rear_right_lower_leg_collision.stl" />
+                <mesh filename="package://spot_description/meshes/rear_right_lower_leg_collision_low.stl" />
             </geometry>
         </collision>

Commit message: Use box shape for lower leg collision and sphere for the feet, remove hip and upperleg collision

File: spot_description/robots/spot.urdf.xacro (robot description, xacro)
@@ -22,4 +22,6 @@
     </xacro:if>
     <!-- dynamics inertial value -->
+    <!-- Constants for robot dimensions -->
+    <xacro:property name="PI" value="3.1415926535897931"/>
     <!-- body -->
     <xacro:property name="body_mass" value="11.041"/>
@@ -71,4 +73,20 @@
     <xacro:property name="foot_x" value="-0.005"/>
     <xacro:property name="foot_z" value="-0.348"/>
+    <!-- simplified collision value -->
+    <xacro:property name="trunk_width" value="0.150"/>
+    <xacro:property name="trunk_length" value="0.647"/>
+    <xacro:property name="trunk_height" value="0.112"/>
+    <xacro:property name="hip_radius" value="0.046"/>
+    <xacro:property name="hip_length" value="0.0418"/>
+    <xacro:property name="upperleg_shoulder_radius" value="0.044"/>
+    <xacro:property name="upperleg_shoulder_length" value="0.08"/>
+    <xacro:property name="upperleg_width" value="0.0374"/>
+    <xacro:property name="upperleg_height" value="0.05"/>
+    <xacro:property name="lowerleg_length" value="0.34"/>
+    <xacro:property name="lowerleg_width" value="0.04"/>
+    <xacro:property name="lowerleg_height" value="0.06"/>
+    <xacro:property name="foot_radius" value="0.0265"/>
+    <xacro:property name="stick_radius" value="0.01"/>
+    <xacro:property name="stick_length" value="0.2"/>
     <!-- Floating-base Joint -->
     <xacro:if value="$(arg floating_base_link)">
@@ -94,5 +112,5 @@
         <collision>
             <geometry>
-                <mesh filename="package://spot_description/meshes/body_collision_low.stl" />
+                <mesh filename="package://spot_description/meshes/body_collision.stl" />
             </geometry>
         </collision>
@@ -124,9 +142,4 @@
             </geometry>
         </visual>
-        <collision>
-            <geometry>
-                <mesh filename="package://spot_description/meshes/front_left_hip_collision_low.stl" />
-            </geometry>
-        </collision>
         <inertial>
             <origin rpy="0 0 0" xyz="${hip_com_x*1} ${hip_com_y*1} ${hip_com_z}"/>
@@ -151,9 +164,4 @@
             </geometry>
         </visual>
-        <collision>
-            <geometry>
-                <mesh filename="package://spot_description/meshes/front_left_upper_leg_collision_low.stl" />
-            </geometry>
-        </collision>
         <inertial>
             <origin rpy="0 0 0" xyz="${upperleg_com_x} ${upperleg_com_y*1} ${upperleg_com_z}"/>
@@ -179,6 +187,7 @@
         </visual>
         <collision>
-            <geometry>
-                <mesh filename="package://spot_description/meshes/front_left_lower_leg_collision_low.stl" />
+            <origin rpy="0 ${PI/2.0} 0" xyz="0 0 ${-lowerleg_length/2.0}"/>
+            <geometry>
+                <box size="${lowerleg_length} ${lowerleg_width} ${lowerleg_height}"/>
             </geometry>
         </collision>
@@ -214,4 +223,10 @@
         </material>
     </visual>
+    <collision>
+        <origin rpy="0 0 0" xyz="0 0 0"/>
+        <geometry>
+            <sphere radius="${foot_radius}"/>
+        </geometry>
+    </collision>
     <inertial>
         <mass value="${foot_mass}"/>
@@ -228,9 +243,4 @@
             </geometry>
         </visual>
-        <collision>
-            <geometry>
-                <mesh filename="package://spot_description/meshes/front_right_hip_collision_low.stl" />
-            </geometry>
-        </collision>
         <inertial>
             <origin rpy="0 0 0" xyz="${hip_com_x*1} ${hip_com_y*-1} ${hip_com_z}"/>
@@ -255,9 +265,4 @@
             </geometry>
         </visual>
-        <collision>
-            <geometry>
-                <mesh filename="package://spot_description/meshes/front_right_upper_leg_collision_low.stl" />
-            </geometry>
-        </collision>
         <inertial>
             <origin rpy="0 0 0" xyz="${upperleg_com_x} ${upperleg_com_y*-1} ${upperleg_com_z}"/>
@@ -283,6 +288,7 @@
         </visual>
         <collision>
-            <geometry>
-                <mesh filename="package://spot_description/meshes/front_right_lower_leg_collision_low.stl" />
+            <origin rpy="0 ${PI/2.0} 0" xyz="0 0 ${-lowerleg_length/2.0}"/>
+            <geometry>
+                <box size="${lowerleg_length} ${lowerleg_width} ${lowerleg_height}"/>
             </geometry>
         </collision>
@@ -318,4 +324,10 @@
         </material>
     </visual>
+    <collision>
+        <origin rpy="0 0 0" xyz="0 0 0"/>
+        <geometry>
+            <sphere radius="${foot_radius}"/>
+        </geometry>
+    </collision>
     <inertial>
         <mass value="${foot_mass}"/>
@@ -332,9 +344,4 @@
             </geometry>
         </visual>
-        <collision>
-            <geometry>
-                <mesh filename="package://spot_description/meshes/rear_left_hip_collision_low.stl" />
-            </geometry>
-        </collision>
         <inertial>
             <origin rpy="0 0 0" xyz="${hip_com_x*-1} ${hip_com_y*1} ${hip_com_z}"/>
@@ -359,9 +366,4 @@
             </geometry>
         </visual>
-        <collision>
-            <geometry>
-                <mesh filename="package://spot_description/meshes/rear_left_upper_leg_collision_low.stl" />
-            </geometry>
-        </collision>
         <inertial>
             <origin rpy="0 0 0" xyz="${upperleg_com_x} ${upperleg_com_y*1} ${upperleg_com_z}"/>
@@ -387,6 +389,7 @@
         </visual>
         <collision>
-            <geometry>
-                <mesh filename="package://spot_description/meshes/rear_left_lower_leg_collision_low.stl" />
+            <origin rpy="0 ${PI/2.0} 0" xyz="0 0 ${-lowerleg_length/2.0}"/>
+            <geometry>
+                <box size="${lowerleg_length} ${lowerleg_width} ${lowerleg_height}"/>
             </geometry>
         </collision>
@@ -422,4 +425,10 @@
         </material>
     </visual>
+    <collision>
+        <origin rpy="0 0 0" xyz="0 0 0"/>
+        <geometry>
+            <sphere radius="${foot_radius}"/>
+        </geometry>
+    </collision>
     <inertial>
         <mass value="${foot_mass}"/>
@@ -436,9 +445,4 @@
             </geometry>
         </visual>
-        <collision>
-            <geometry>
-                <mesh filename="package://spot_description/meshes/rear_right_hip_collision_low.stl" />
-            </geometry>
-        </collision>
         <inertial>
             <origin rpy="0 0 0" xyz="${hip_com_x*-1} ${hip_com_y*-1} ${hip_com_z}"/>
@@ -463,9 +467,4 @@
             </geometry>
         </visual>
-        <collision>
-            <geometry>
-                <mesh filename="package://spot_description/meshes/rear_right_upper_leg_collision_low.stl" />
-            </geometry>
-        </collision>
         <inertial>
             <origin rpy="0 0 0" xyz="${upperleg_com_x} ${upperleg_com_y*-1} ${upperleg_com_z}"/>
@@ -491,6 +490,7 @@
         </visual>
         <collision>
-            <geometry>
-                <mesh filename="package://spot_description/meshes/rear_right_lower_leg_collision_low.stl" />
+            <origin rpy="0 ${PI/2.0} 0" xyz="0 0 ${-lowerleg_length/2.0}"/>
+            <geometry>
+                <box size="${lowerleg_length} ${lowerleg_width} ${lowerleg_height}"/>
             </geometry>
         </collision>
@@ -526,4 +526,10 @@
         </material>
     </visual>
+    <collision>
+        <origin rpy="0 0 0" xyz="0 0 0"/>
+        <geometry>
+            <sphere radius="${foot_radius}"/>
+        </geometry>
+    </collision>
     <inertial>
         <mass value="${foot_mass}"/>
