Commit message: Simplified base collision mesh

File: spot_description/robots/spot.urdf.xacro (robot description, xacro)
@@ -74,19 +74,17 @@
     <xacro:property name="foot_z" value="-0.348"/>
     <!-- simplified collision value -->
-    <xacro:property name="trunk_width" value="0.150"/>
-    <xacro:property name="trunk_length" value="0.647"/>
-    <xacro:property name="trunk_height" value="0.112"/>
-    <xacro:property name="hip_radius" value="0.046"/>
-    <xacro:property name="hip_length" value="0.0418"/>
-    <xacro:property name="upperleg_shoulder_radius" value="0.044"/>
-    <xacro:property name="upperleg_shoulder_length" value="0.08"/>
-    <xacro:property name="upperleg_width" value="0.0374"/>
-    <xacro:property name="upperleg_height" value="0.05"/>
+    <xacro:property name="base_width" value="0.23"/>
+    <xacro:property name="base_length" value="0.9"/>
+    <xacro:property name="base_height" value="0.17"/>
+    <xacro:property name="hip_radius" value="0.0"/>
+    <xacro:property name="hip_length" value="0.0"/>
+    <xacro:property name="upperleg_shoulder_radius" value="0.0"/>
+    <xacro:property name="upperleg_shoulder_length" value="0.0"/>
+    <xacro:property name="upperleg_width" value="0.0"/>
+    <xacro:property name="upperleg_height" value="0.0"/>
     <xacro:property name="lowerleg_length" value="0.34"/>
     <xacro:property name="lowerleg_width" value="0.04"/>
     <xacro:property name="lowerleg_height" value="0.06"/>
-    <xacro:property name="foot_radius" value="0.0265"/>
-    <xacro:property name="stick_radius" value="0.01"/>
-    <xacro:property name="stick_length" value="0.2"/>
+    <xacro:property name="foot_radius" value="0.02"/>
     <!-- Floating-base Joint -->
     <xacro:if value="$(arg floating_base_link)">
@@ -110,7 +108,13 @@
             </geometry>
         </visual>
+        <!--<collision>
+            <geometry>
+                <mesh filename="package://spot_description/meshes/body_collision.stl" />
+            </geometry>
+        </collision>-->
         <collision>
-            <geometry>
-                <mesh filename="package://spot_description/meshes/body_collision.stl" />
+            <origin rpy="0 0 0" xyz="0 0 0"/>
+            <geometry>
+                <box size="${base_length} ${base_width} ${base_height}"/>
             </geometry>
         </collision>
@@ -142,4 +146,9 @@
             </geometry>
         </visual>
+        <!--<collision>
+            <geometry>
+                <mesh filename="package://spot_description/meshes/front_left_hip_collision.stl" />
+            </geometry>
+        </collision>-->
         <inertial>
             <origin rpy="0 0 0" xyz="${hip_com_x*1} ${hip_com_y*1} ${hip_com_z}"/>
@@ -164,4 +173,9 @@
             </geometry>
         </visual>
+        <!--<collision>
+            <geometry>
+                <mesh filename="package://spot_description/meshes/front_left_upper_leg_collision.stl" />
+            </geometry>
+        </collision>-->
         <inertial>
             <origin rpy="0 0 0" xyz="${upperleg_com_x} ${upperleg_com_y*1} ${upperleg_com_z}"/>
@@ -186,4 +200,9 @@
             </geometry>
         </visual>
+        <!--<collision>
+            <geometry>
+                <mesh filename="package://spot_description/meshes/front_left_lower_leg_collision.stl" />
+            </geometry>
+        </collision>-->
         <collision>
             <origin rpy="0 ${PI/2.0} 0" xyz="0 0 ${-lowerleg_length/2.0}"/>
@@ -243,4 +262,9 @@
             </geometry>
         </visual>
+        <!--<collision>
+            <geometry>
+                <mesh filename="package://spot_description/meshes/front_right_hip_collision.stl" />
+            </geometry>
+        </collision>-->
         <inertial>
             <origin rpy="0 0 0" xyz="${hip_com_x*1} ${hip_com_y*-1} ${hip_com_z}"/>
@@ -265,4 +289,9 @@
             </geometry>
         </visual>
+        <!--<collision>
+            <geometry>
+                <mesh filename="package://spot_description/meshes/front_right_upper_leg_collision.stl" />
+            </geometry>
+        </collision>-->
         <inertial>
             <origin rpy="0 0 0" xyz="${upperleg_com_x} ${upperleg_com_y*-1} ${upperleg_com_z}"/>
@@ -287,4 +316,9 @@
             </geometry>
         </visual>
+        <!--<collision>
+            <geometry>
+                <mesh filename="package://spot_description/meshes/front_right_lower_leg_collision.stl" />
+            </geometry>
+        </collision>-->
         <collision>
             <origin rpy="0 ${PI/2.0} 0" xyz="0 0 ${-lowerleg_length/2.0}"/>
@@ -344,4 +378,9 @@
             </geometry>
         </visual>
+        <!--<collision>
+            <geometry>
+                <mesh filename="package://spot_description/meshes/rear_left_hip_collision.stl" />
+            </geometry>
+        </collision>-->
         <inertial>
             <origin rpy="0 0 0" xyz="${hip_com_x*-1} ${hip_com_y*1} ${hip_com_z}"/>
@@ -366,4 +405,9 @@
             </geometry>
         </visual>
+        <!--<collision>
+            <geometry>
+                <mesh filename="package://spot_description/meshes/rear_left_upper_leg_collision.stl" />
+            </geometry>
+        </collision>-->
         <inertial>
             <origin rpy="0 0 0" xyz="${upperleg_com_x} ${upperleg_com_y*1} ${upperleg_com_z}"/>
@@ -388,4 +432,9 @@
             </geometry>
         </visual>
+        <!--<collision>
+            <geometry>
+                <mesh filename="package://spot_description/meshes/rear_left_lower_leg_collision.stl" />
+            </geometry>
+        </collision>-->
         <collision>
             <origin rpy="0 ${PI/2.0} 0" xyz="0 0 ${-lowerleg_length/2.0}"/>
@@ -445,4 +494,9 @@
             </geometry>
         </visual>
+        <!--<collision>
+            <geometry>
+                <mesh filename="package://spot_description/meshes/rear_right_hip_collision.stl" />
+            </geometry>
+        </collision>-->
         <inertial>
             <origin rpy="0 0 0" xyz="${hip_com_x*-1} ${hip_com_y*-1} ${hip_com_z}"/>
@@ -467,4 +521,9 @@
             </geometry>
         </visual>
+        <!--<collision>
+            <geometry>
+                <mesh filename="package://spot_description/meshes/rear_right_upper_leg_collision.stl" />
+            </geometry>
+        </collision>-->
         <inertial>
             <origin rpy="0 0 0" xyz="${upperleg_com_x} ${upperleg_com_y*-1} ${upperleg_com_z}"/>
@@ -489,4 +548,9 @@
             </geometry>
         </visual>
+        <!--<collision>
+            <geometry>
+                <mesh filename="package://spot_description/meshes/rear_right_lower_leg_collision.stl" />
+            </geometry>
+        </collision>-->
         <collision>
             <origin rpy="0 ${PI/2.0} 0" xyz="0 0 ${-lowerleg_length/2.0}"/>

Commit message: Add upper leg collision

File: spot_description/robots/spot.urdf.xacro (robot description, xacro)
@@ -77,10 +77,7 @@
     <xacro:property name="base_length" value="0.9"/>
     <xacro:property name="base_height" value="0.17"/>
-    <xacro:property name="hip_radius" value="0.0"/>
-    <xacro:property name="hip_length" value="0.0"/>
-    <xacro:property name="upperleg_shoulder_radius" value="0.0"/>
-    <xacro:property name="upperleg_shoulder_length" value="0.0"/>
-    <xacro:property name="upperleg_width" value="0.0"/>
-    <xacro:property name="upperleg_height" value="0.0"/>
+    <xacro:property name="upperleg_length" value="0.42"/>
+    <xacro:property name="upperleg_width" value="0.12"/>
+    <xacro:property name="upperleg_height" value="0.1"/>
     <xacro:property name="lowerleg_length" value="0.34"/>
     <xacro:property name="lowerleg_width" value="0.04"/>
@@ -178,4 +175,10 @@
             </geometry>
         </collision>-->
+        <collision>
+            <origin rpy="0 ${PI/2.0} 0" xyz="0 0 ${-upperleg_length/3.0}"/>
+            <geometry>
+                <box size="${upperleg_length} ${upperleg_width} ${upperleg_height}"/>
+            </geometry>
+        </collision>
         <inertial>
             <origin rpy="0 0 0" xyz="${upperleg_com_x} ${upperleg_com_y*1} ${upperleg_com_z}"/>
@@ -294,4 +297,10 @@
             </geometry>
         </collision>-->
+        <collision>
+            <origin rpy="0 ${PI/2.0} 0" xyz="0 0 ${-upperleg_length/3.0}"/>
+            <geometry>
+                <box size="${upperleg_length} ${upperleg_width} ${upperleg_height}"/>
+            </geometry>
+        </collision>
         <inertial>
             <origin rpy="0 0 0" xyz="${upperleg_com_x} ${upperleg_com_y*-1} ${upperleg_com_z}"/>
@@ -410,4 +419,10 @@
             </geometry>
         </collision>-->
+        <collision>
+            <origin rpy="0 ${PI/2.0} 0" xyz="0 0 ${-upperleg_length/3.0}"/>
+            <geometry>
+                <box size="${upperleg_length} ${upperleg_width} ${upperleg_height}"/>
+            </geometry>
+        </collision>
         <inertial>
             <origin rpy="0 0 0" xyz="${upperleg_com_x} ${upperleg_com_y*1} ${upperleg_com_z}"/>
@@ -526,4 +541,10 @@
             </geometry>
         </collision>-->
+        <collision>
+            <origin rpy="0 ${PI/2.0} 0" xyz="0 0 ${-upperleg_length/3.0}"/>
+            <geometry>
+                <box size="${upperleg_length} ${upperleg_width} ${upperleg_height}"/>
+            </geometry>
+        </collision>
         <inertial>
             <origin rpy="0 0 0" xyz="${upperleg_com_x} ${upperleg_com_y*-1} ${upperleg_com_z}"/>

Commit message: Use find instead of package://

File: spot_description/robots/spot.urdf.xacro (robot description, xacro)
@@ -102,10 +102,10 @@
         <visual>
             <geometry>
-                <mesh filename="package://spot_description/meshes/body.dae" />
-            </geometry>
-        </visual>
-        <!--<collision>
-            <geometry>
-                <mesh filename="package://spot_description/meshes/body_collision.stl" />
+                <mesh filename="$(find spot_description)/meshes/body.dae" />
+            </geometry>
+        </visual>
+        <!--<collision>
+            <geometry>
+                <mesh filename="$(find spot_description)/meshes/body_collision.stl" />
             </geometry>
         </collision>-->
@@ -140,10 +140,10 @@
         <visual>
             <geometry>
-                <mesh filename="package://spot_description/meshes/front_left_hip.dae" />
-            </geometry>
-        </visual>
-        <!--<collision>
-            <geometry>
-                <mesh filename="package://spot_description/meshes/front_left_hip_collision.stl" />
+                <mesh filename="$(find spot_description)/meshes/front_left_hip.dae" />
+            </geometry>
+        </visual>
+        <!--<collision>
+            <geometry>
+                <mesh filename="$(find spot_description)/meshes/front_left_hip_collision.stl" />
             </geometry>
         </collision>-->
@@ -167,10 +167,10 @@
         <visual>
             <geometry>
-                <mesh filename="package://spot_description/meshes/front_left_upper_leg.dae" />
-            </geometry>
-        </visual>
-        <!--<collision>
-            <geometry>
-                <mesh filename="package://spot_description/meshes/front_left_upper_leg_collision.stl" />
+                <mesh filename="$(find spot_description)/meshes/front_left_upper_leg.dae" />
+            </geometry>
+        </visual>
+        <!--<collision>
+            <geometry>
+                <mesh filename="$(find spot_description)/meshes/front_left_upper_leg_collision.stl" />
             </geometry>
         </collision>-->
@@ -200,10 +200,10 @@
         <visual>
             <geometry>
-                <mesh filename="package://spot_description/meshes/front_left_lower_leg.dae" />
-            </geometry>
-        </visual>
-        <!--<collision>
-            <geometry>
-                <mesh filename="package://spot_description/meshes/front_left_lower_leg_collision.stl" />
+                <mesh filename="$(find spot_description)/meshes/front_left_lower_leg.dae" />
+            </geometry>
+        </visual>
+        <!--<collision>
+            <geometry>
+                <mesh filename="$(find spot_description)/meshes/front_left_lower_leg_collision.stl" />
             </geometry>
         </collision>-->
@@ -262,10 +262,10 @@
         <visual>
             <geometry>
-                <mesh filename="package://spot_description/meshes/front_right_hip.dae" />
-            </geometry>
-        </visual>
-        <!--<collision>
-            <geometry>
-                <mesh filename="package://spot_description/meshes/front_right_hip_collision.stl" />
+                <mesh filename="$(find spot_description)/meshes/front_right_hip.dae" />
+            </geometry>
+        </visual>
+        <!--<collision>
+            <geometry>
+                <mesh filename="$(find spot_description)/meshes/front_right_hip_collision.stl" />
             </geometry>
         </collision>-->
@@ -289,10 +289,10 @@
         <visual>
             <geometry>
-                <mesh filename="package://spot_description/meshes/front_right_upper_leg.dae" />
-            </geometry>
-        </visual>
-        <!--<collision>
-            <geometry>
-                <mesh filename="package://spot_description/meshes/front_right_upper_leg_collision.stl" />
+                <mesh filename="$(find spot_description)/meshes/front_right_upper_leg.dae" />
+            </geometry>
+        </visual>
+        <!--<collision>
+            <geometry>
+                <mesh filename="$(find spot_description)/meshes/front_right_upper_leg_collision.stl" />
             </geometry>
         </collision>-->
@@ -322,10 +322,10 @@
         <visual>
             <geometry>
-                <mesh filename="package://spot_description/meshes/front_right_lower_leg.dae" />
-            </geometry>
-        </visual>
-        <!--<collision>
-            <geometry>
-                <mesh filename="package://spot_description/meshes/front_right_lower_leg_collision.stl" />
+                <mesh filename="$(find spot_description)/meshes/front_right_lower_leg.dae" />
+            </geometry>
+        </visual>
+        <!--<collision>
+            <geometry>
+                <mesh filename="$(find spot_description)/meshes/front_right_lower_leg_collision.stl" />
             </geometry>
         </collision>-->
@@ -384,10 +384,10 @@
         <visual>
             <geometry>
-                <mesh filename="package://spot_description/meshes/rear_left_hip.dae" />
-            </geometry>
-        </visual>
-        <!--<collision>
-            <geometry>
-                <mesh filename="package://spot_description/meshes/rear_left_hip_collision.stl" />
+                <mesh filename="$(find spot_description)/meshes/rear_left_hip.dae" />
+            </geometry>
+        </visual>
+        <!--<collision>
+            <geometry>
+                <mesh filename="$(find spot_description)/meshes/rear_left_hip_collision.stl" />
             </geometry>
         </collision>-->
@@ -411,10 +411,10 @@
         <visual>
             <geometry>
-                <mesh filename="package://spot_description/meshes/rear_left_upper_leg.dae" />
-            </geometry>
-        </visual>
-        <!--<collision>
-            <geometry>
-                <mesh filename="package://spot_description/meshes/rear_left_upper_leg_collision.stl" />
+                <mesh filename="$(find spot_description)/meshes/rear_left_upper_leg.dae" />
+            </geometry>
+        </visual>
+        <!--<collision>
+            <geometry>
+                <mesh filename="$(find spot_description)/meshes/rear_left_upper_leg_collision.stl" />
             </geometry>
         </collision>-->
@@ -444,10 +444,10 @@
         <visual>
             <geometry>
-                <mesh filename="package://spot_description/meshes/rear_left_lower_leg.dae" />
-            </geometry>
-        </visual>
-        <!--<collision>
-            <geometry>
-                <mesh filename="package://spot_description/meshes/rear_left_lower_leg_collision.stl" />
+                <mesh filename="$(find spot_description)/meshes/rear_left_lower_leg.dae" />
+            </geometry>
+        </visual>
+        <!--<collision>
+            <geometry>
+                <mesh filename="$(find spot_description)/meshes/rear_left_lower_leg_collision.stl" />
             </geometry>
         </collision>-->
@@ -506,10 +506,10 @@
         <visual>
             <geometry>
-                <mesh filename="package://spot_description/meshes/rear_right_hip.dae" />
-            </geometry>
-        </visual>
-        <!--<collision>
-            <geometry>
-                <mesh filename="package://spot_description/meshes/rear_right_hip_collision.stl" />
+                <mesh filename="$(find spot_description)/meshes/rear_right_hip.dae" />
+            </geometry>
+        </visual>
+        <!--<collision>
+            <geometry>
+                <mesh filename="$(find spot_description)/meshes/rear_right_hip_collision.stl" />
             </geometry>
         </collision>-->
@@ -533,10 +533,10 @@
         <visual>
             <geometry>
-                <mesh filename="package://spot_description/meshes/rear_right_upper_leg.dae" />
-            </geometry>
-        </visual>
-        <!--<collision>
-            <geometry>
-                <mesh filename="package://spot_description/meshes/rear_right_upper_leg_collision.stl" />
+                <mesh filename="$(find spot_description)/meshes/rear_right_upper_leg.dae" />
+            </geometry>
+        </visual>
+        <!--<collision>
+            <geometry>
+                <mesh filename="$(find spot_description)/meshes/rear_right_upper_leg_collision.stl" />
             </geometry>
         </collision>-->
@@ -566,10 +566,10 @@
         <visual>
             <geometry>
-                <mesh filename="package://spot_description/meshes/rear_right_lower_leg.dae" />
-            </geometry>
-        </visual>
-        <!--<collision>
-            <geometry>
-                <mesh filename="package://spot_description/meshes/rear_right_lower_leg_collision.stl" />
+                <mesh filename="$(find spot_description)/meshes/rear_right_lower_leg.dae" />
+            </geometry>
+        </visual>
+        <!--<collision>
+            <geometry>
+                <mesh filename="$(find spot_description)/meshes/rear_right_lower_leg_collision.stl" />
             </geometry>
         </collision>-->
