Commit message: Fix rviz meshes problem

File: spot_description/robots/spot.urdf.xacro (robot description, xacro)
@@ -102,10 +102,10 @@
         <visual>
             <geometry>
-                <mesh filename="$(find spot_description)/meshes/body.dae" />
-            </geometry>
-        </visual>
-        <!--<collision>
-            <geometry>
-                <mesh filename="$(find spot_description)/meshes/body_collision.stl" />
+                <mesh filename="file://$(find spot_description)/meshes/body.dae" />
+            </geometry>
+        </visual>
+        <!--<collision>
+            <geometry>
+                <mesh filename="file://$(find spot_description)/meshes/body_collision.stl" />
             </geometry>
         </collision>-->
@@ -140,10 +140,10 @@
         <visual>
             <geometry>
-                <mesh filename="$(find spot_description)/meshes/front_left_hip.dae" />
-            </geometry>
-        </visual>
-        <!--<collision>
-            <geometry>
-                <mesh filename="$(find spot_description)/meshes/front_left_hip_collision.stl" />
+                <mesh filename="file://$(find spot_description)/meshes/front_left_hip.dae" />
+            </geometry>
+        </visual>
+        <!--<collision>
+            <geometry>
+                <mesh filename="file://$(find spot_description)/meshes/front_left_hip_collision.stl" />
             </geometry>
         </collision>-->
@@ -167,10 +167,10 @@
         <visual>
             <geometry>
-                <mesh filename="$(find spot_description)/meshes/front_left_upper_leg.dae" />
-            </geometry>
-        </visual>
-        <!--<collision>
-            <geometry>
-                <mesh filename="$(find spot_description)/meshes/front_left_upper_leg_collision.stl" />
+                <mesh filename="file://$(find spot_description)/meshes/front_left_upper_leg.dae" />
+            </geometry>
+        </visual>
+        <!--<collision>
+            <geometry>
+                <mesh filename="file://$(find spot_description)/meshes/front_left_upper_leg_collision.stl" />
             </geometry>
         </collision>-->
@@ -200,10 +200,10 @@
         <visual>
             <geometry>
-                <mesh filename="$(find spot_description)/meshes/front_left_lower_leg.dae" />
-            </geometry>
-        </visual>
-        <!--<collision>
-            <geometry>
-                <mesh filename="$(find spot_description)/meshes/front_left_lower_leg_collision.stl" />
+                <mesh filename="file://$(find spot_description)/meshes/front_left_lower_leg.dae" />
+            </geometry>
+        </visual>
+        <!--<collision>
+            <geometry>
+                <mesh filename="file://$(find spot_description)/meshes/front_left_lower_leg_collision.stl" />
             </geometry>
         </collision>-->
@@ -262,10 +262,10 @@
         <visual>
             <geometry>
-                <mesh filename="$(find spot_description)/meshes/front_right_hip.dae" />
-            </geometry>
-        </visual>
-        <!--<collision>
-            <geometry>
-                <mesh filename="$(find spot_description)/meshes/front_right_hip_collision.stl" />
+                <mesh filename="file://$(find spot_description)/meshes/front_right_hip.dae" />
+            </geometry>
+        </visual>
+        <!--<collision>
+            <geometry>
+                <mesh filename="file://$(find spot_description)/meshes/front_right_hip_collision.stl" />
             </geometry>
         </collision>-->
@@ -289,10 +289,10 @@
         <visual>
             <geometry>
-                <mesh filename="$(find spot_description)/meshes/front_right_upper_leg.dae" />
-            </geometry>
-        </visual>
-        <!--<collision>
-            <geometry>
-                <mesh filename="$(find spot_description)/meshes/front_right_upper_leg_collision.stl" />
+                <mesh filename="file://$(find spot_description)/meshes/front_right_upper_leg.dae" />
+            </geometry>
+        </visual>
+        <!--<collision>
+            <geometry>
+                <mesh filename="file://$(find spot_description)/meshes/front_right_upper_leg_collision.stl" />
             </geometry>
         </collision>-->
@@ -322,10 +322,10 @@
         <visual>
             <geometry>
-                <mesh filename="$(find spot_description)/meshes/front_right_lower_leg.dae" />
-            </geometry>
-        </visual>
-        <!--<collision>
-            <geometry>
-                <mesh filename="$(find spot_description)/meshes/front_right_lower_leg_collision.stl" />
+                <mesh filename="file://$(find spot_description)/meshes/front_right_lower_leg.dae" />
+            </geometry>
+        </visual>
+        <!--<collision>
+            <geometry>
+                <mesh filename="file://$(find spot_description)/meshes/front_right_lower_leg_collision.stl" />
             </geometry>
         </collision>-->
@@ -384,10 +384,10 @@
         <visual>
             <geometry>
-                <mesh filename="$(find spot_description)/meshes/rear_left_hip.dae" />
-            </geometry>
-        </visual>
-        <!--<collision>
-            <geometry>
-                <mesh filename="$(find spot_description)/meshes/rear_left_hip_collision.stl" />
+                <mesh filename="file://$(find spot_description)/meshes/rear_left_hip.dae" />
+            </geometry>
+        </visual>
+        <!--<collision>
+            <geometry>
+                <mesh filename="file://$(find spot_description)/meshes/rear_left_hip_collision.stl" />
             </geometry>
         </collision>-->
@@ -411,10 +411,10 @@
         <visual>
             <geometry>
-                <mesh filename="$(find spot_description)/meshes/rear_left_upper_leg.dae" />
-            </geometry>
-        </visual>
-        <!--<collision>
-            <geometry>
-                <mesh filename="$(find spot_description)/meshes/rear_left_upper_leg_collision.stl" />
+                <mesh filename="file://$(find spot_description)/meshes/rear_left_upper_leg.dae" />
+            </geometry>
+        </visual>
+        <!--<collision>
+            <geometry>
+                <mesh filename="file://$(find spot_description)/meshes/rear_left_upper_leg_collision.stl" />
             </geometry>
         </collision>-->
@@ -444,10 +444,10 @@
         <visual>
             <geometry>
-                <mesh filename="$(find spot_description)/meshes/rear_left_lower_leg.dae" />
-            </geometry>
-        </visual>
-        <!--<collision>
-            <geometry>
-                <mesh filename="$(find spot_description)/meshes/rear_left_lower_leg_collision.stl" />
+                <mesh filename="file://$(find spot_description)/meshes/rear_left_lower_leg.dae" />
+            </geometry>
+        </visual>
+        <!--<collision>
+            <geometry>
+                <mesh filename="file://$(find spot_description)/meshes/rear_left_lower_leg_collision.stl" />
             </geometry>
         </collision>-->
@@ -506,10 +506,10 @@
         <visual>
             <geometry>
-                <mesh filename="$(find spot_description)/meshes/rear_right_hip.dae" />
-            </geometry>
-        </visual>
-        <!--<collision>
-            <geometry>
-                <mesh filename="$(find spot_description)/meshes/rear_right_hip_collision.stl" />
+                <mesh filename="file://$(find spot_description)/meshes/rear_right_hip.dae" />
+            </geometry>
+        </visual>
+        <!--<collision>
+            <geometry>
+                <mesh filename="file://$(find spot_description)/meshes/rear_right_hip_collision.stl" />
             </geometry>
         </collision>-->
@@ -533,10 +533,10 @@
         <visual>
             <geometry>
-                <mesh filename="$(find spot_description)/meshes/rear_right_upper_leg.dae" />
-            </geometry>
-        </visual>
-        <!--<collision>
-            <geometry>
-                <mesh filename="$(find spot_description)/meshes/rear_right_upper_leg_collision.stl" />
+                <mesh filename="file://$(find spot_description)/meshes/rear_right_upper_leg.dae" />
+            </geometry>
+        </visual>
+        <!--<collision>
+            <geometry>
+                <mesh filename="file://$(find spot_description)/meshes/rear_right_upper_leg_collision.stl" />
             </geometry>
         </collision>-->
@@ -566,10 +566,10 @@
         <visual>
             <geometry>
-                <mesh filename="$(find spot_description)/meshes/rear_right_lower_leg.dae" />
-            </geometry>
-        </visual>
-        <!--<collision>
-            <geometry>
-                <mesh filename="$(find spot_description)/meshes/rear_right_lower_leg_collision.stl" />
+                <mesh filename="file://$(find spot_description)/meshes/rear_right_lower_leg.dae" />
+            </geometry>
+        </visual>
+        <!--<collision>
+            <geometry>
+                <mesh filename="file://$(find spot_description)/meshes/rear_right_lower_leg_collision.stl" />
             </geometry>
         </collision>-->

Commit message: Fix meshes path when using multiple pcs

File: spot_description/robots/spot.urdf.xacro (robot description, xacro)
@@ -102,10 +102,10 @@
         <visual>
             <geometry>
-                <mesh filename="file://$(find spot_description)/meshes/body.dae" />
-            </geometry>
-        </visual>
-        <!--<collision>
-            <geometry>
-                <mesh filename="file://$(find spot_description)/meshes/body_collision.stl" />
+                <mesh filename="package://spot_description/meshes/body.dae" />
+            </geometry>
+        </visual>
+        <!--<collision>
+            <geometry>
+                <mesh filename="package://spot_description/meshes/body_collision.stl" />
             </geometry>
         </collision>-->
@@ -140,10 +140,10 @@
         <visual>
             <geometry>
-                <mesh filename="file://$(find spot_description)/meshes/front_left_hip.dae" />
-            </geometry>
-        </visual>
-        <!--<collision>
-            <geometry>
-                <mesh filename="file://$(find spot_description)/meshes/front_left_hip_collision.stl" />
+                <mesh filename="package://spot_description/meshes/front_left_hip.dae" />
+            </geometry>
+        </visual>
+        <!--<collision>
+            <geometry>
+                <mesh filename="package://spot_description/meshes/front_left_hip_collision.stl" />
             </geometry>
         </collision>-->
@@ -167,10 +167,10 @@
         <visual>
             <geometry>
-                <mesh filename="file://$(find spot_description)/meshes/front_left_upper_leg.dae" />
-            </geometry>
-        </visual>
-        <!--<collision>
-            <geometry>
-                <mesh filename="file://$(find spot_description)/meshes/front_left_upper_leg_collision.stl" />
+                <mesh filename="package://spot_description/meshes/front_left_upper_leg.dae" />
+            </geometry>
+        </visual>
+        <!--<collision>
+            <geometry>
+                <mesh filename="package://spot_description/meshes/front_left_upper_leg_collision.stl" />
             </geometry>
         </collision>-->
@@ -200,10 +200,10 @@
         <visual>
             <geometry>
-                <mesh filename="file://$(find spot_description)/meshes/front_left_lower_leg.dae" />
-            </geometry>
-        </visual>
-        <!--<collision>
-            <geometry>
-                <mesh filename="file://$(find spot_description)/meshes/front_left_lower_leg_collision.stl" />
+                <mesh filename="package://spot_description/meshes/front_left_lower_leg.dae" />
+            </geometry>
+        </visual>
+        <!--<collision>
+            <geometry>
+                <mesh filename="package://spot_description/meshes/front_left_lower_leg_collision.stl" />
             </geometry>
         </collision>-->
@@ -262,10 +262,10 @@
         <visual>
             <geometry>
-                <mesh filename="file://$(find spot_description)/meshes/front_right_hip.dae" />
-            </geometry>
-        </visual>
-        <!--<collision>
-            <geometry>
-                <mesh filename="file://$(find spot_description)/meshes/front_right_hip_collision.stl" />
+                <mesh filename="package://spot_description/meshes/front_right_hip.dae" />
+            </geometry>
+        </visual>
+        <!--<collision>
+            <geometry>
+                <mesh filename="package://spot_description/meshes/front_right_hip_collision.stl" />
             </geometry>
         </collision>-->
@@ -289,10 +289,10 @@
         <visual>
             <geometry>
-                <mesh filename="file://$(find spot_description)/meshes/front_right_upper_leg.dae" />
-            </geometry>
-        </visual>
-        <!--<collision>
-            <geometry>
-                <mesh filename="file://$(find spot_description)/meshes/front_right_upper_leg_collision.stl" />
+                <mesh filename="package://spot_description/meshes/front_right_upper_leg.dae" />
+            </geometry>
+        </visual>
+        <!--<collision>
+            <geometry>
+                <mesh filename="package://spot_description/meshes/front_right_upper_leg_collision.stl" />
             </geometry>
         </collision>-->
@@ -322,10 +322,10 @@
         <visual>
             <geometry>
-                <mesh filename="file://$(find spot_description)/meshes/front_right_lower_leg.dae" />
-            </geometry>
-        </visual>
-        <!--<collision>
-            <geometry>
-                <mesh filename="file://$(find spot_description)/meshes/front_right_lower_leg_collision.stl" />
+                <mesh filename="package://spot_description/meshes/front_right_lower_leg.dae" />
+            </geometry>
+        </visual>
+        <!--<collision>
+            <geometry>
+                <mesh filename="package://spot_description/meshes/front_right_lower_leg_collision.stl" />
             </geometry>
         </collision>-->
@@ -384,10 +384,10 @@
         <visual>
             <geometry>
-                <mesh filename="file://$(find spot_description)/meshes/rear_left_hip.dae" />
-            </geometry>
-        </visual>
-        <!--<collision>
-            <geometry>
-                <mesh filename="file://$(find spot_description)/meshes/rear_left_hip_collision.stl" />
+                <mesh filename="package://spot_description/meshes/rear_left_hip.dae" />
+            </geometry>
+        </visual>
+        <!--<collision>
+            <geometry>
+                <mesh filename="package://spot_description/meshes/rear_left_hip_collision.stl" />
             </geometry>
         </collision>-->
@@ -411,10 +411,10 @@
         <visual>
             <geometry>
-                <mesh filename="file://$(find spot_description)/meshes/rear_left_upper_leg.dae" />
-            </geometry>
-        </visual>
-        <!--<collision>
-            <geometry>
-                <mesh filename="file://$(find spot_description)/meshes/rear_left_upper_leg_collision.stl" />
+                <mesh filename="package://spot_description/meshes/rear_left_upper_leg.dae" />
+            </geometry>
+        </visual>
+        <!--<collision>
+            <geometry>
+                <mesh filename="package://spot_description/meshes/rear_left_upper_leg_collision.stl" />
             </geometry>
         </collision>-->
@@ -444,10 +444,10 @@
         <visual>
             <geometry>
-                <mesh filename="file://$(find spot_description)/meshes/rear_left_lower_leg.dae" />
-            </geometry>
-        </visual>
-        <!--<collision>
-            <geometry>
-                <mesh filename="file://$(find spot_description)/meshes/rear_left_lower_leg_collision.stl" />
+                <mesh filename="package://spot_description/meshes/rear_left_lower_leg.dae" />
+            </geometry>
+        </visual>
+        <!--<collision>
+            <geometry>
+                <mesh filename="package://spot_description/meshes/rear_left_lower_leg_collision.stl" />
             </geometry>
         </collision>-->
@@ -506,10 +506,10 @@
         <visual>
             <geometry>
-                <mesh filename="file://$(find spot_description)/meshes/rear_right_hip.dae" />
-            </geometry>
-        </visual>
-        <!--<collision>
-            <geometry>
-                <mesh filename="file://$(find spot_description)/meshes/rear_right_hip_collision.stl" />
+                <mesh filename="package://spot_description/meshes/rear_right_hip.dae" />
+            </geometry>
+        </visual>
+        <!--<collision>
+            <geometry>
+                <mesh filename="package://spot_description/meshes/rear_right_hip_collision.stl" />
             </geometry>
         </collision>-->
@@ -533,10 +533,10 @@
         <visual>
             <geometry>
-                <mesh filename="file://$(find spot_description)/meshes/rear_right_upper_leg.dae" />
-            </geometry>
-        </visual>
-        <!--<collision>
-            <geometry>
-                <mesh filename="file://$(find spot_description)/meshes/rear_right_upper_leg_collision.stl" />
+                <mesh filename="package://spot_description/meshes/rear_right_upper_leg.dae" />
+            </geometry>
+        </visual>
+        <!--<collision>
+            <geometry>
+                <mesh filename="package://spot_description/meshes/rear_right_upper_leg_collision.stl" />
             </geometry>
         </collision>-->
@@ -566,10 +566,10 @@
         <visual>
             <geometry>
-                <mesh filename="file://$(find spot_description)/meshes/rear_right_lower_leg.dae" />
-            </geometry>
-        </visual>
-        <!--<collision>
-            <geometry>
-                <mesh filename="file://$(find spot_description)/meshes/rear_right_lower_leg_collision.stl" />
+                <mesh filename="package://spot_description/meshes/rear_right_lower_leg.dae" />
+            </geometry>
+        </visual>
+        <!--<collision>
+            <geometry>
+                <mesh filename="package://spot_description/meshes/rear_right_lower_leg_collision.stl" />
             </geometry>
         </collision>-->
