Commit message: Remove comments
they are causing issues when parsed because of tabs...

File: kinova_description/urdf/kinova_common.xacro (robot description, xacro)
@@ -98,14 +98,4 @@
             <limit lower="0" upper="1.51" effort="2" velocity="1"/>
         </joint>
-        <!--	    <transmission name="${prefix}joint_finger_${finger_number}_trans">
-					<type>transmission_interface/SimpleTransmission</type>
-					<joint name="${prefix}joint_finger_${finger_number}">
-					  <hardwareInterface>hardware_interface/EffortJointInterface</hardwareInterface>
-					</joint>
-					<actuator name="${prefix}joint_finger_${finger_number}_actuator">
-					<hardwareInterface>hardware_interface/EffortJointInterface</hardwareInterface>
-					<mechanicalReduction>1</mechanicalReduction>
-					</actuator>
-                    </transmission> -->
         <xacro:kinova_armlink link_name="${prefix}link_finger_tip_${finger_number}" link_mesh="finger_distal" mesh_no="58"/>
         <joint name="${prefix}joint_finger_tip_${finger_number}" type="fixed">
@@ -116,14 +106,4 @@
             <limit lower="0" upper="2" effort="2" velocity="1"/>
         </joint>
-        <!-- <transmission name="${prefix}joint_finger_tip_${finger_number}_trans">
-					<type>transmission_interface/SimpleTransmission</type>
-					<joint name="${prefix}joint_finger_tip_${finger_number}">
-					  <hardwareInterface>hardware_interface/EffortJointInterface</hardwareInterface>
-					</joint>
-					<actuator name="${prefix}joint_finger_tip_${finger_number}_actuator">
-					<hardwareInterface>hardware_interface/EffortJointInterface</hardwareInterface>
-					<mechanicalReduction>1</mechanicalReduction>
-					</actuator>
-        </transmission> -->
     </xacro:macro>
 </root>

File: kinova_description/urdf/kinova_inertial.xacro (robot description, xacro)
@@ -13,19 +13,19 @@
     xmlns:physics="http://playerstage.sourceforge.net/gazebo/xmlschema/#physics"
 	xmlns:xacro="http://www.ros.org/wiki/xacro">
-<!-- links      		mesh_no
-   base           		0
-   shoulder       		1
-   arm            		2
-   forearm        		3
-   wrist          		4
-   arm_mico       		5
-   arm_half1 (7dof)		6
-   arm_half2 (7dof)		7
-   wrist_spherical_1  8
-   wrist_spherical_2  9
-   hand 3 finger  		55
-   hand_2finger   		56
-   finger_proximal		57
-   finger_distal      58
+<!-- links mesh_no
+   base 0
+   shoulder 1
+   arm 2
+   forearm 3
+   wrist 4
+   arm_mico 5
+   arm_half1 (7dof) 6
+   arm_half2 (7dof) 7
+   wrist_spherical_1 8
+   wrist_spherical_2 9
+   hand 3 finger 55
+   hand_2finger 56
+   finger_proximal 57
+   finger_distal 58
 -->
 <xacro:macro name="inertia_cylinder" params="mass height radius axis:=0">
