Commit message: Format

File: wolf_description_utils/urdfs/gazebo.urdf.xacro (robot description, xacro)
@@ -6,11 +6,11 @@
 	<gazebo>
 		<plugin name="gazebo_ros_controller_manager" filename="libgazebo_ros_control.so">
-                        <robotNamespace>$(arg robot_name)</robotNamespace>
-                        <robotSimType>wolf_gazebo_interface/WolfRobotHwSim</robotSimType>
-                        <controlPeriod>$(arg period)</controlPeriod>
+            <robotNamespace>$(arg robot_name)</robotNamespace>
+            <robotSimType>wolf_gazebo_interface/WolfRobotHwSim</robotSimType>
+            <controlPeriod>$(arg period)</controlPeriod>
 		</plugin>
-              <plugin filename="libgazebo_ros_p3d.so" name="ground_truth">
-                        <robotNamespace>$(arg robot_name)</robotNamespace>
-                        <bodyName>$(arg base_name)</bodyName>
+    	<plugin filename="libgazebo_ros_p3d.so" name="ground_truth">
+            <robotNamespace>$(arg robot_name)</robotNamespace>
+            <bodyName>$(arg base_name)</bodyName>
 			<topicName>ground_truth</topicName>
 			<frameName>world</frameName>
@@ -19,6 +19,6 @@
 			<gaussianNoise>0</gaussianNoise>
 			<alwaysOn>true</alwaysOn>
-                        <updateRate>${1/ $(arg period)}</updateRate>
-                </plugin>
+            <updateRate>${1/ $(arg period)}</updateRate>
+        </plugin>
 	</gazebo>
 </robot>

File: wolf_description_utils/urdfs/leg.gazebo.xacro (robot description, xacro)
@@ -8,5 +8,5 @@
 			<gazebo>
 				<plugin name="${prefix}_haa_sensor" filename="libgazebo_ros_ft_sensor.so">
-                                        <robotNamespace>/${robot_name}/internal_wrench/</robotNamespace>
+					<robotNamespace>/${robot_name}/internal_wrench/</robotNamespace>
 					<updateRate>100.0</updateRate>
 					<topicName>${prefix}_haa_joint</topicName>
@@ -21,5 +21,5 @@
 			<gazebo>
 				<plugin name="${prefix}_hfe_sensor" filename="libgazebo_ros_ft_sensor.so">
-                                        <robotNamespace>/${robot_name}/internal_wrench/</robotNamespace>
+					<robotNamespace>/${robot_name}/internal_wrench/</robotNamespace>
 					<updateRate>100.0</updateRate>
 					<topicName>${prefix}_hfe_joint</topicName>
@@ -54,5 +54,5 @@
 			<minDepth>0.00</minDepth>
 		</gazebo>
-                <gazebo reference="${prefix}_lowerleg">
+		<gazebo reference="${prefix}_lowerleg">
 			<kp>1000000.0</kp>
 			<kd>100.0</kd>
@@ -62,16 +62,16 @@
 			<maxContacts>1</maxContacts>
 			<sensor name="${prefix}_shin_contact_sensor" type="contact">
-                                <always_on>true</always_on>
-                                <update_rate>250.0</update_rate>
-                                <contact>
-                                    <collision>${prefix}_lowerleg_collision</collision>
-                                </contact>
-                                <plugin name="${prefix}_shin_bumper" filename="libgazebo_ros_bumper.so">
-                                    <bumperTopicName>/${robot_name}/${prefix}_shin_bumper</bumperTopicName>
-                                    <robotNamespace>${robot_name}</robotNamespace>
-                                    <frameName>${prefix}_lowerleg</frameName>
-                                </plugin>
-                        </sensor>
-                </gazebo>
+					<always_on>true</always_on>
+					<update_rate>250.0</update_rate>
+					<contact>
+						<collision>${prefix}_lowerleg_collision</collision>
+					</contact>
+					<plugin name="${prefix}_shin_bumper" filename="libgazebo_ros_bumper.so">
+						<bumperTopicName>/${robot_name}/${prefix}_shin_bumper</bumperTopicName>
+						<robotNamespace>${robot_name}</robotNamespace>
+						<frameName>${prefix}_lowerleg</frameName>
+					</plugin>
+			</sensor>
+		</gazebo>
                 <gazebo reference="${prefix}_foot">
                         <kp>1000000.0</kp>
@@ -84,11 +84,11 @@
 				<always_on>true</always_on>
 				<update_rate>250.0</update_rate>
-                                <contact>
-                                    <collision>${prefix}_foot_collision</collision>
+				<contact>
+						<collision>${prefix}_foot_collision</collision>
 				</contact>
 				<plugin name="${prefix}_foot_bumper" filename="libgazebo_ros_bumper.so">
-                                        <bumperTopicName>/${robot_name}/${prefix}_foot_bumper</bumperTopicName>
-                                        <robotNamespace>${robot_name}</robotNamespace>
-                                        <frameName>${prefix}_foot</frameName>
+						<bumperTopicName>/${robot_name}/${prefix}_foot_bumper</bumperTopicName>
+						<robotNamespace>${robot_name}</robotNamespace>
+						<frameName>${prefix}_foot</frameName>
 				</plugin>
 			</sensor>

Commit message: Add ros2 control plugin

File: wolf_description_utils/urdfs/gazebo.urdf.xacro (robot description, xacro)
@@ -1,23 +1,30 @@
 <?xml version="1.0"?>
 <robot xmlns:xacro="http://ros.org/wiki/xacro">
-<xacro:arg name="period"     default="0.001"/>
-<xacro:arg name="robot_name" default=""/>
-<xacro:arg name="base_name"  default="base"/>
+<xacro:arg name="period"      default="0.001"/>
+<xacro:arg name="robot_name"  default=""/>
+<xacro:arg name="robot_model" default=""/>
+<xacro:arg name="base_name"   default="base_link"/>
+<xacro:property name="model_name" value="$(arg robot_model)"/>
 	<gazebo>
-		<plugin name="gazebo_ros_controller_manager" filename="libgazebo_ros_control.so">
-            <robotNamespace>$(arg robot_name)</robotNamespace>
-            <robotSimType>wolf_gazebo_interface/WolfRobotHwSim</robotSimType>
-            <controlPeriod>$(arg period)</controlPeriod>
-		</plugin>
+        <plugin name="gazebo_ros_controller_manager" filename="libgazebo_ros_control.so">
+                <robotNamespace>$(arg robot_name)</robotNamespace>
+                <robotSimType>wolf_gazebo_interface/WolfRobotHwSim</robotSimType>
+                <controlPeriod>$(arg period)</controlPeriod>
+        </plugin>
+        <plugin name="gazebo_ros2_controller_manager" filename="libgazebo_ros2_control.so">
+                <robotNamespace>$(arg robot_name)</robotNamespace>
+                <robotSimType>wolf_gazebo_interface/WolfRobotHwSim</robotSimType>
+                <parameters>$(find ${model_name}_description)/params/${model_name}_params.yaml</parameters>
+        </plugin>
     	<plugin filename="libgazebo_ros_p3d.so" name="ground_truth">
             <robotNamespace>$(arg robot_name)</robotNamespace>
-            <bodyName>$(arg base_name)</bodyName>
-			<topicName>ground_truth</topicName>
-			<frameName>world</frameName>
-			<xyzOffsets>0 0 0</xyzOffsets>
-			<rpyOffsets>0 0 0</rpyOffsets>
-			<gaussianNoise>0</gaussianNoise>
-			<alwaysOn>true</alwaysOn>
-            <updateRate>${1/ $(arg period)}</updateRate>
+                <body_name>$(arg base_name)</body_name>
+                <topicName>ground_truth</topicName>
+                <frameName>world</frameName>
+                <xyzOffsets>0 0 0</xyzOffsets>
+                <rpyOffsets>0 0 0</rpyOffsets>
+                <gaussianNoise>0</gaussianNoise>
+                <alwaysOn>true</alwaysOn>
+                <updateRate>${1/ $(arg period)}</updateRate>
         </plugin>
 	</gazebo>
