Commit message: Add floating base

File: husky_description/urdfs/husky_macro.urdf.xacro (robot description, xacro)
@@ -20,5 +20,5 @@
   <xacro:include filename="$(find husky_description)/urdfs/accessories/sensor_arch.urdf.xacro"/>
   <xacro:property name="M_PI" value="3.14159"/>
-  <xacro:macro name="husky" params="prefix">
+  <xacro:macro name="husky" params="prefix floating_base_link">
     <!-- Base Size -->
     <xacro:property name="base_x_size" value="0.98740000" />
@@ -32,4 +32,13 @@
     <xacro:property name="wheel_length" value="0.1143" />
     <xacro:property name="wheel_radius" value="0.1651" />
+    <!-- Floating-base Joint -->
+    <xacro:if value="$(arg floating_base_link)">
+        <link name="world"/>
+        <joint name="${prefix}floating_base_joint" type="floating">
+          <origin rpy="0 0 0" xyz="0 0 0"/>
+          <parent link="world"/>
+          <child link="${prefix}base_link"/>
+        </joint>
+    </xacro:if>
     <!-- Base link is the center of the robot's bottom plate -->
     <link name="${prefix}base_link">

Commit message: Fix base footprint

File: husky_description/urdfs/husky_macro.urdf.xacro (robot description, xacro)
@@ -25,7 +25,13 @@
         <origin rpy="0 0 0" xyz="0 0 0"/>
         <parent link="world"/>
-        <child link="base_link"/>
+        <child link="base_footprint"/>
       </joint>
     </xacro:if>
+    <link name="base_footprint" />
+    <joint name="base_footprint_joint" type="fixed">
+      <origin xyz="0 0 ${wheel_radius - wheel_vertical_offset}" rpy="0 0 0" />
+      <parent link="base_footprint" />
+      <child link="base_link" />
+    </joint>
     <!-- Base Link -->
     <link name="base_link">
@@ -49,10 +55,4 @@
       </collision>
     </link>
-    <link name="base_footprint" />
-    <joint name="base_footprint_joint" type="fixed">
-      <origin xyz="0 0 ${wheel_vertical_offset - wheel_radius}" rpy="0 0 0" />
-      <parent link="base_link" />
-      <child link="base_footprint" />
-    </joint>
     <!-- Inertial -->
     <link name="inertial_link">
