Commit message: Tune go1 for simulation

File: go1_description/robots/go1.srdf.xacro (robot description, xacro)
@@ -51,15 +51,15 @@
     <group_state group="chains" name="standup">
         <joint name="lf_haa_joint" value="0.1"/>
-        <joint name="lf_hfe_joint" value="0.67"/>
-        <joint name="lf_kfe_joint" value="-1.3"/>
+        <joint name="lf_hfe_joint" value="0.8"/>
+        <joint name="lf_kfe_joint" value="-1.45"/>
         <joint name="rf_haa_joint" value="-0.1"/>
-        <joint name="rf_hfe_joint" value="0.67"/>
-        <joint name="rf_kfe_joint" value="-1.3"/>
+        <joint name="rf_hfe_joint" value="0.8"/>
+        <joint name="rf_kfe_joint" value="-1.45"/>
         <joint name="lh_haa_joint" value="0.1"/>
-        <joint name="lh_hfe_joint" value="0.67"/>
-        <joint name="lh_kfe_joint" value="-1.3"/>
+        <joint name="lh_hfe_joint" value="0.8"/>
+        <joint name="lh_kfe_joint" value="-1.45"/>
         <joint name="rh_haa_joint" value="-0.1"/>
-        <joint name="rh_hfe_joint" value="0.67"/>
-        <joint name="rh_kfe_joint" value="-1.3"/>
+        <joint name="rh_hfe_joint" value="0.8"/>
+        <joint name="rh_kfe_joint" value="-1.45"/>
     </group_state>
     <group_state group="chains" name="standdown">

Commit message: trunk -> base_link

File: go1_description/robots/go1.srdf.xacro (robot description, xacro)
@@ -2,5 +2,5 @@
 <robot name="go1" xmlns:xacro="http://ros.org/wiki/xacro">
     <group name="base">
-      <link name="trunk"/>
+      <link name="base_link"/>
     </group>
     <group name="imu">
@@ -8,5 +8,5 @@
     </group>
     <group name="lf_leg">
-      <chain base_link="trunk" tip_link="lf_foot"/>
+      <chain base_link="base_link" tip_link="lf_foot"/>
       <joint name="lf_haa_joint"/>
       <joint name="lf_hfe_joint"/>
@@ -14,5 +14,5 @@
     </group>
     <group name="rf_leg">
-      <chain base_link="trunk" tip_link="rf_foot"/>
+      <chain base_link="base_link" tip_link="rf_foot"/>
       <joint name="rf_haa_joint"/>
       <joint name="rf_hfe_joint"/>
@@ -20,5 +20,5 @@
     </group>
     <group name="lh_leg">
-      <chain base_link="trunk" tip_link="lh_foot"/>
+      <chain base_link="base_link" tip_link="lh_foot"/>
       <joint name="lh_haa_joint"/>
       <joint name="lh_hfe_joint"/>
@@ -26,5 +26,5 @@
     </group>
     <group name="rh_leg">
-      <chain base_link="trunk" tip_link="rh_foot"/>
+      <chain base_link="base_link" tip_link="rh_foot"/>
       <joint name="rh_haa_joint"/>
       <joint name="rh_hfe_joint"/>
@@ -32,14 +32,14 @@
     </group>
     <group name="lf_hip">
-      <chain base_link="trunk" tip_link="lf_hip"/>
+      <chain base_link="base_link" tip_link="lf_hip"/>
     </group>
     <group name="rf_hip">
-      <chain base_link="trunk" tip_link="rf_hip"/>
+      <chain base_link="base_link" tip_link="rf_hip"/>
     </group>
     <group name="lh_hip">
-      <chain base_link="trunk" tip_link="lh_hip"/>
+      <chain base_link="base_link" tip_link="lh_hip"/>
     </group>
     <group name="rh_hip">
-      <chain base_link="trunk" tip_link="rh_hip"/>
+      <chain base_link="base_link" tip_link="rh_hip"/>
     </group>
     <group name="chains">

File: go1_description/robots/go1.urdf.xacro (robot description, xacro)
@@ -10,5 +10,5 @@
     <xacro:arg name="robot_model"        default="go1"/>
     <xacro:arg name="robot_name"         default=""/>
-    <xacro:arg name="base_name"          default="trunk"/>
+    <xacro:arg name="base_name"          default="base_link"/>
     <!-- load generic materials -->
     <xacro:include filename="$(find wolf_description_utils)/urdfs/materials.xacro"/>
@@ -28,8 +28,8 @@
               <origin rpy="0 0 0" xyz="0 0 0"/>
               <parent link="world"/>
-              <child link="trunk"/>
+              <child link="base_link"/>
             </joint>
     </xacro:if>
-    <link name="trunk">
+    <link name="base_link">
         <visual>
             <origin rpy="0 0 0" xyz="0 0 0"/>
@@ -62,5 +62,5 @@
     <xacro:if value="${(rolloverProtection == 'true')}">
         <joint name="stick_joint" type="fixed">
-            <parent link="trunk"/>
+            <parent link="base_link"/>
             <child link="stick_link"/>
             <origin rpy="0 0 0" xyz="${0.18} 0 ${stick_length/2.0+0.08}"/>
@@ -90,5 +90,5 @@
     </xacro:if>
     <joint name="imu_joint" type="fixed">
-        <parent link="trunk"/>
+        <parent link="base_link"/>
         <child link="trunk_imu"/>
         <origin rpy="0 0 0" xyz="-0.01592 -0.06659 -0.00617"/>
@@ -115,9 +115,9 @@
     </link>
     <joint name="lidar_cage_to_lidar" type="fixed">
-        <parent link="trunk"/>
-        <child link="rslidar"/>
+        <parent link="base_link"/>
+        <child link="lidar_mount"/>
         <origin rpy="0.0 0.0 0.0" xyz="0.0 0.0 0.05"/>
     </joint>
-    <link name="rslidar">
+    <link name="lidar_mount">
         <inertial>
             <origin rpy="0.0 0.0 0.0" xyz="-0.012 0.001 -0.008"/>

File: go1_description/urdfs/accessories.urdf.xacro (robot description, xacro)
@@ -9,5 +9,5 @@
   <xacro:include filename="$(find sensors_description)/urdfs/sensors/gps.gazebo.xacro"/>
   <xacro:include filename="$(find sensors_description)/urdfs/sensors/realsense_d435.urdf.xacro" />
-  <xacro:realsense_d435 name="d435" topics_ns="/$(arg robot_name)/d435" parent="trunk">
+  <xacro:realsense_d435 name="d435" topics_ns="/$(arg robot_name)/d435" parent="base_link">
       <origin xyz="0.14 0 0.15" rpy="0 0.3 0" />
   </xacro:realsense_d435>
@@ -53,8 +53,8 @@
   </xacro:ultraSound>
    -->
-  <xacro:realsense_T265 name="t265" topics_ns="/$(arg robot_name)" parent="trunk" rate="30.0">
+  <xacro:realsense_T265 name="t265" topics_ns="/$(arg robot_name)" parent="base_link" rate="30.0">
     <origin xyz="0.3 0 0.05" rpy="0 0.24 0" />
   </xacro:realsense_T265>
-  <xacro:VLP-16 parent="rslidar" name="rslidar-16" topic="/$(arg robot_name)/lidar_points"
+  <xacro:VLP-16 parent="lidar_mount" name="rslidar" topic="/$(arg robot_name)/lidar_points"
                 organize_cloud="true" hz="10" gpu="true">
     <origin xyz="0.1 0 0" rpy="0 0 0" />
@@ -80,5 +80,5 @@
       vel_topic="velocity_fix"
       namespace="$(arg robot_name)"
-      frame_name="trunk"
+      frame_name="base_link"
       update_rate="10.0">
   </xacro:gps_sensor>

File: go1_description/urdfs/depthCamera.xacro (robot description, xacro)
@@ -4,5 +4,5 @@
         <joint name="camera_joint_${name}" type="fixed">
             <xacro:insert_block name="origin"/>
-            <parent link="trunk"/>
+            <parent link="base_link"/>
             <child link="camera_${name}"/>
         </joint>

File: go1_description/urdfs/leg.xacro (robot description, xacro)
@@ -4,5 +4,5 @@
         <joint name="${name}_haa_joint" type="revolute">
             <xacro:insert_block name="origin"/>
-            <parent link="trunk"/>
+            <parent link="base_link"/>
             <child link="${name}_hip"/>
             <axis xyz="1 0 0"/>

File: go1_description/urdfs/ultraSound.xacro (robot description, xacro)
@@ -4,5 +4,5 @@
         <joint name="ultraSound_joint_${name}" type="fixed">
             <xacro:insert_block name="origin"/>
-            <parent link="trunk"/>
+            <parent link="base_link"/>
             <child link="ultraSound_${name}"/>
         </joint>

Commit message: Update go1 to work with the new humble branch

File: go1_description/robots/go1.srdf.xacro (robot description, xacro)
@@ -6,4 +6,10 @@
     <group name="imu">
       <link name="trunk_imu"/>
+    </group>
+    <group name="contacts"> <!-- where the contact sensors are mounted -->
+      <link name="lf_foot"/>
+      <link name="rf_foot"/>
+      <link name="lh_foot"/>
+      <link name="rh_foot"/>
     </group>
     <group name="lf_leg">

File: go1_description/robots/go1.urdf.xacro (robot description, xacro)
@@ -5,5 +5,4 @@
     <xacro:arg name="sensors"            default="false"/>
     <xacro:arg name="period"             default="0.004"/>
-    <xacro:arg name="arm_enabled"        default="false"/>
     <xacro:arg name="arm_name"           default=""/>
     <xacro:arg name="floating_base_link" default="true"/>
@@ -94,38 +93,7 @@
         <parent link="base_link"/>
         <child link="trunk_imu"/>
-        <origin rpy="0 0 0" xyz="-0.01592 -0.06659 -0.00617"/>
+        <origin rpy="0 0 0" xyz="0 0 0"/>
     </joint>
-    <link name="trunk_imu">
-        <inertial>
-            <mass value="0.001"/>
-            <origin rpy="0 0 0" xyz="0 0 0"/>
-            <inertia ixx="0.0001" ixy="0" ixz="0" iyy="0.0001" iyz="0" izz="0.0001"/>
-        </inertial>
-        <visual>
-            <origin rpy="0 0 0" xyz="0 0 0"/>
-            <geometry>
-                <box size="0.001 0.001 0.001"/>
-            </geometry>
-            <!-- <material name="red"/> -->
-        </visual>
-        <collision>
-            <origin rpy="0 0 0" xyz="0 0 0"/>
-            <geometry>
-                <box size=".001 .001 .001"/>
-            </geometry>
-        </collision>
-    </link>
-    <joint name="lidar_cage_to_lidar" type="fixed">
-        <parent link="base_link"/>
-        <child link="lidar_mount"/>
-        <origin rpy="0.0 0.0 0.0" xyz="0.0 0.0 0.05"/>
-    </joint>
-    <link name="lidar_mount">
-        <inertial>
-            <origin rpy="0.0 0.0 0.0" xyz="-0.012 0.001 -0.008"/>
-            <mass value="0.695"/>
-            <inertia ixx="0.000846765" ixy="6.9565e-05" ixz="0.00027111" iyy="0.001367583" iyz="5.8984e-05" izz="0.001363673"/>
-        </inertial>
-    </link>
+    <link name="trunk_imu"/>
     <xacro:leg name="rf" mirror="-1" mirror_dae= "False" front_hind="1" front_hind_dae="True">
         <origin rpy="0 0 0" xyz="${leg_offset_x} ${-leg_offset_y} 0"/>

File: go1_description/urdfs/accessories.urdf.xacro (robot description, xacro)
@@ -5,4 +5,38 @@
   <xacro:include filename="$(find sensors_description)/urdfs/sensors/gps.gazebo.xacro"/>
   <xacro:include filename="$(find sensors_description)/urdfs/sensors/lidar.gazebo.xacro"/>
+    <joint name="lidar_cage_to_lidar" type="fixed">
+        <parent link="base_link"/>
+        <child link="lidar_mount"/>
+        <origin rpy="0.0 0.0 0.0" xyz="0.0 0.0 0.05"/>
+    </joint>
+    <link name="lidar_mount">
+        <inertial>
+            <origin rpy="0.0 0.0 0.0" xyz="-0.012 0.001 -0.008"/>
+            <mass value="0.695"/>
+            <inertia ixx="0.000846765" ixy="6.9565e-05" ixz="0.00027111" iyy="0.001367583" iyz="5.8984e-05" izz="0.001363673"/>
+        </inertial>
+        <visual>
+          <geometry>
+            <mesh filename="file://$(find go1_description)/meshes/lidar.dae"/>
+          </geometry>
+        </visual>
+    </link>
+    <joint name="base_link_to_camera" type="fixed">
+        <parent link="base_link"/>
+        <child link="camera_mount"/>
+        <origin rpy="0 0.3 0" xyz="0.3 0 0.05"/>
+    </joint>
+    <link name="camera_mount">
+        <inertial>
+            <origin rpy="0 0.0 0" xyz="0.0 0 0.0"/>
+            <mass value="0.001"/>
+            <inertia ixx="0.000846765" ixy="6.9565e-05" ixz="0.00027111" iyy="0.001367583" iyz="5.8984e-05" izz="0.001363673"/>
+        </inertial>
+        <visual>
+          <geometry>
+            <mesh filename="file://$(find go1_description)/meshes/depth_camera.dae"/>
+          </geometry>
+        </visual>
+    </link>
    <xacro:depth_camera
      name="camera"
@@ -14,7 +48,7 @@
      near="0.1"
      far="10.0"
-     parent_link="base_link"
-     origin_xyz="0.14 0 0.15"
-     origin_rpy="0 0.3 0"/>
+     parent_link="camera_mount"
+     origin_xyz="0.0 0 0.0"
+     origin_rpy="0 0.0 0"/>
   <xacro:velodyne_laser_gazebo_sensor
     sensor_name="$(arg robot_name)_lidar"
