Commit message: Move the rslidar link into the go1.urdf.xacro
Because there is a weird bug... to investigate

File: go1_description/robots/go1.urdf.xacro (robot description, xacro)
@@ -114,4 +114,16 @@
         </collision>
     </link>
+    <joint name="lidar_cage_to_lidar" type="fixed">
+        <parent link="trunk"/>
+        <child link="rslidar"/>
+        <origin rpy="0.0 0.0 0.0" xyz="0.0 0.0 0.05"/>
+    </joint>
+    <link name="rslidar">
+        <inertial>
+            <origin rpy="0.0 0.0 0.0" xyz="-0.012 0.001 -0.008"/>
+            <mass value="0.695"/>
+            <inertia ixx="0.000846765" ixy="6.9565e-05" ixz="0.00027111" iyy="0.001367583" iyz="5.8984e-05" izz="0.001363673"/>
+        </inertial>
+    </link>
     <xacro:leg name="rf" mirror="-1" mirror_dae= "False" front_hind="1" front_hind_dae="True">
         <origin rpy="0 0 0" xyz="${leg_offset_x} ${-leg_offset_y} 0"/>

File: go1_description/urdfs/accessories.urdf.xacro (robot description, xacro)
@@ -51,16 +51,4 @@
     <origin xyz="0.3 0 0.05" rpy="0 0.24 0" />
   </xacro:realsense_T265>
-  <joint name="lidar_cage_to_lidar" type="fixed">
-      <parent link="trunk"/>
-      <child link="rslidar"/>
-      <origin rpy="0.0 0.0 0.0" xyz="0.0 0.0 0.05"/>
-  </joint>
-  <link name="rslidar">
-      <inertial>
-          <origin rpy="0.0 0.0 0.0" xyz="-0.012 0.001 -0.008"/>
-          <mass value="0.695"/>
-          <inertia ixx="0.000846765" ixy="6.9565e-05" ixz="0.00027111" iyy="0.001367583" iyz="5.8984e-05" izz="0.001363673"/>
-      </inertial>
-  </link>
   <xacro:VLP-16 parent="rslidar" name="rslidar-16" topic="/$(arg robot_name)/rslidar_points"
                 organize_cloud="true" hz="10" gpu="true">

Commit message: Fix package -> file

File: go1_description/robots/go1.urdf.xacro (robot description, xacro)
@@ -35,5 +35,5 @@
             <origin rpy="0 0 0" xyz="0 0 0"/>
             <geometry>
-                <mesh filename="package://go1_description/meshes/trunk.dae" scale="1 1 1"/>
+                <mesh filename="file://$(find go1_description)/meshes/trunk.dae" scale="1 1 1"/>
             </geometry>
             <material name="orange"/>
@@ -48,5 +48,5 @@
             <origin rpy="0 0 0" xyz="0 0 0"/>
             <geometry>
-                <mesh filename="file://$"$(find go1_description)/meshes/trunk.dae" scale="1 1 1"/>
+                <mesh filename="file://$(find go1_description)/meshes/trunk.dae" scale="1 1 1"/>
             </geometry>
         </collision> -->

File: go1_description/urdfs/depthCamera.xacro (robot description, xacro)
@@ -17,5 +17,5 @@
             <origin xyz="0 0 0" rpy="0 0 0"/>
             <geometry>
-                <mesh filename="package://go1_description/meshes/depthCamera.dae" scale="1 1 1"/>
+                <mesh filename="file://$(find go1_description)/meshes/depthCamera.dae" scale="1 1 1"/>
             </geometry>
             </visual>

File: go1_description/urdfs/leg.xacro (robot description, xacro)
@@ -30,5 +30,5 @@
                 </xacro:if>
                 <geometry>
-                    <mesh filename="package://go1_description/meshes/hip.dae" scale="1 1 1"/>
+                    <mesh filename="file://$(find go1_description)/meshes/hip.dae" scale="1 1 1"/>
                 </geometry>
                 <!-- <material name="orange"/> -->
@@ -76,8 +76,8 @@
                 <geometry>
                     <xacro:if value="${mirror_dae == True}">
-                        <mesh filename="package://go1_description/meshes/thigh.dae" scale="1 1 1"/>
+                        <mesh filename="file://$(find go1_description)/meshes/thigh.dae" scale="1 1 1"/>
                     </xacro:if>
                     <xacro:if value="${mirror_dae == False}">
-                        <mesh filename="package://go1_description/meshes/thigh_mirror.dae" scale="1 1 1"/>
+                        <mesh filename="file://$(find go1_description)/meshes/thigh_mirror.dae" scale="1 1 1"/>
                     </xacro:if>
                 </geometry>
@@ -111,5 +111,5 @@
                 <origin rpy="0 0 0" xyz="0 0 0"/>
                 <geometry>
-                    <mesh filename="package://go1_description/meshes/calf.dae" scale="1 1 1"/>
+                    <mesh filename="file://$(find go1_description)/meshes/calf.dae" scale="1 1 1"/>
                 </geometry>
                 <!-- <material name="orange"/> -->

File: go1_description/urdfs/ultraSound.xacro (robot description, xacro)
@@ -17,5 +17,5 @@
             <origin xyz="0 0 0" rpy="0 0 0"/>
             <geometry>
-                <mesh filename="package://go1_description/meshes/ultraSound.dae" scale="1 1 1"/>
+                <mesh filename="file://$(find go1_description)/meshes/ultraSound.dae" scale="1 1 1"/>
             </geometry>
             <material name="black"/>

File: sensors_description/urdfs/sensors/bumblebee.urdf.xacro (robot description, xacro)
@@ -19,5 +19,5 @@
 				<origin xyz="0 0 0.018" rpy="${PI/2} 0 ${PI/2}"/>
 				<geometry>
-					<mesh filename="package://sensors_description/meshes/sensors/bumblebee.dae"/>
+					<mesh filename="file://$(find sensors_description)/meshes/sensors/bumblebee.dae"/>
 				</geometry>
 			</visual>
@@ -25,5 +25,5 @@
 				<origin xyz="0 0 0.018" rpy="${PI/2} 0 ${PI/2}"/>
 				<geometry>
-					<mesh filename="package://sensors_description/meshes/sensors/bumblebee.dae"/>
+					<mesh filename="file://$(find sensors_description)/meshes/sensors/bumblebee.dae"/>
 				</geometry>
 			</collision>

File: sensors_description/urdfs/sensors/hokuyo_laser.urdf.xacro (robot description, xacro)
@@ -25,5 +25,5 @@
 				<origin xyz="0 0 0" rpy="0 0 0" />
 				<geometry>
-					<mesh filename="package://sensors_description/meshes/sensors/hokuyo.dae" scale="0.0254 0.0254 0.0254" />
+					<mesh filename="file://$(find sensors_description)/meshes/sensors/hokuyo.dae" scale="0.0254 0.0254 0.0254" />
 				</geometry>
 			</visual>

File: sensors_description/urdfs/sensors/kinect.urdf.xacro (robot description, xacro)
@@ -46,5 +46,5 @@
 				<origin xyz="0.0 0.0 0.0" rpy="0.0 0.0 0"/>
 				<geometry>
-					<mesh filename="package://sensors_description/meshes/sensors/kinect.dae" scale="1 1 1" />
+					<mesh filename="file://$(find sensors_description)/meshes/sensors/kinect.dae" scale="1 1 1" />
 				</geometry>
 				<material name="gray">
@@ -55,5 +55,5 @@
 				<origin xyz="0.0 0.0 0.0" rpy="0.0 0.0 0.0"/>
 				<geometry>
-					<mesh filename="package://sensors_description/meshes/sensors/kinect.dae" scale="1 1 1" />
+					<mesh filename="file://$(find sensors_description)/meshes/sensors/kinect.dae" scale="1 1 1" />
 				</geometry>
 			</collision>

File: sensors_description/urdfs/sensors/kvh_1775_imu.urdf.xacro (robot description, xacro)
@@ -115,5 +115,5 @@
 				<origin xyz="0.0 0.0 0.0" rpy="0 0 0"/>
 				<geometry>
-					<mesh filename="package://sensors_description/meshes/sensors/kvh_1775.dae" scale="1 1 1" />
+					<mesh filename="file://$(find sensors_description)/meshes/sensors/kvh_1775.dae" scale="1 1 1" />
 				</geometry>
 				<material name="aluminium">

File: sensors_description/urdfs/sensors/realsense_d435.urdf.xacro (robot description, xacro)
@@ -49,5 +49,5 @@
           <!-- <box size="${d435_cam_width} ${d435_cam_height} ${d435_cam_depth}"/> -->
 <!--          <mesh filename="package://realsense2_description/meshes/d435.dae" />-->
-          <mesh filename="package://sensors_description/meshes/sensors/realsense_d435.stl" />
+          <mesh filename="file://$(find sensors_description)/meshes/sensors/realsense_d435.stl" />
           <!--<mesh filename="package://realsense2_description/meshes/d435/d435.dae" />-->
         </geometry>

File: sensors_description/urdfs/sensors/realsense_d455.urdf.xacro (robot description, xacro)
@@ -53,5 +53,5 @@
       <origin xyz="${d455_zero_depth_to_glass + d455_glass_to_front} ${-d455_cam_depth_py} 0" rpy="${M_PI/2} 0 ${M_PI/2}"/>
         <geometry>
-          <mesh filename="package://sensors_description/meshes/sensors/realsense_d455.stl" scale="0.001 0.001 0.001" />
+          <mesh filename="file://$(find sensors_description)/meshes/sensors/realsense_d455.stl" scale="0.001 0.001 0.001" />
         </geometry>
         <material name="${name}_aluminum"/>

File: sensors_description/urdfs/sensors/realsense_t265.urdf.xacro (robot description, xacro)
@@ -90,5 +90,5 @@
             <origin rpy="1.57 0 1.57" xyz="0 0 0"/>
             <geometry>
-                <mesh filename="package://sensors_description/meshes/sensors/realsense_t265.stl" scale="0.001 0.001 0.001"/>
+                <mesh filename="file://$(find sensors_description)/meshes/sensors/realsense_t265.stl" scale="0.001 0.001 0.001"/>
             </geometry>
         </visual>
@@ -190,5 +190,5 @@
             <updateRate>${rate}</updateRate>
             <robotNamespace>${topics_ns}</robotNamespace>
-            <bodyName>${name}_odom_frame</bodyName>
+            <body_name>${name}_odom_frame</body_name>
             <topicName>${name}/odom</topicName>
             <gaussianNoise>0.001</gaussianNoise>

File: sensors_description/urdfs/sensors/velodyne.urdf.xacro (robot description, xacro)
@@ -27,5 +27,5 @@
 				<origin xyz="0 0 0" rpy="0 0 0"/>
 				<geometry>
-					<mesh filename="package://sensors_description/meshes/sensors/velodyne_hdl32e.dae" scale="1 1 1" />
+					<mesh filename="file://$(find sensors_description)/meshes/sensors/velodyne_hdl32e.dae" scale="1 1 1" />
 				</geometry>
 				<material name="gray">
@@ -36,5 +36,5 @@
 				<origin xyz="0 0 0" rpy="0 0 0"/>
 				<geometry>
-					<mesh filename="package://sensors_description/meshes/sensors/velodyne_hdl32e.dae" scale="1 1 1" />
+					<mesh filename="file://$(find sensors_description)/meshes/sensors/velodyne_hdl32e.dae" scale="1 1 1" />
 				</geometry>
 			</collision>

File: sensors_description/urdfs/sensors/vislab_3dve.urdf.xacro (robot description, xacro)
@@ -18,5 +18,5 @@
 				<origin xyz="0.018 0 0" rpy="${PI/2} 0 ${-PI/2}"/>
 				<geometry>
-					<mesh filename="package://sensors_description/meshes/sensors/vislab_3dve.stl"/>
+					<mesh filename="file://$(find sensors_description)/meshes/sensors/vislab_3dve.stl"/>
 				</geometry>
 			</visual>
@@ -24,5 +24,5 @@
 				<origin xyz="0.018 0 0" rpy="${PI/2} 0 ${-PI/2}"/>
 				<geometry>
-					<mesh filename="package://sensors_description/meshes/sensors/vislab_3dve.stl"/>
+					<mesh filename="file://$(find sensors_description)/meshes/sensors/vislab_3dve.stl"/>
 				</geometry>
 			</collision>

File: sensors_description/urdfs/sensors/zed_mini.urdf.xacro (robot description, xacro)
@@ -68,5 +68,5 @@
         <origin xyz="${screw_offset_x} 0 0" rpy="0 0 0"/>
         <geometry>
-          <mesh filename="package://sensors_description/meshes/sensors/zed_mini.stl" />
+          <mesh filename="file://$(find sensors_description)/meshes/sensors/zed_mini.stl" />
         </geometry>
         <!-- <material name="${model}_mat" /> -->
@@ -74,5 +74,5 @@
       <collision>
         <geometry>
-          <mesh filename="package://sensors_description/meshes/sensors/zed_mini.stl" />
+          <mesh filename="file://$(find sensors_description)/meshes/sensors/zed_mini.stl" />
         </geometry>
       </collision>

File: spot_description/robots/spot.urdf.xacro (robot description, xacro)
@@ -98,10 +98,10 @@
         <visual>
             <geometry>
-                <mesh filename="package://spot_description/meshes/body.dae" />
-            </geometry>
-        </visual>
-        <!--<collision>
-            <geometry>
-                <mesh filename="package://spot_description/meshes/body_collision.stl" />
+                <mesh filename="file://$(find spot_description)/meshes/body.dae" />
+            </geometry>
+        </visual>
+        <!--<collision>
+            <geometry>
+                <mesh filename="file://$(find spot_description)/meshes/body_collision.stl" />
             </geometry>
         </collision>-->
@@ -136,10 +136,10 @@
         <visual>
             <geometry>
-                <mesh filename="package://spot_description/meshes/front_left_hip.dae" />
-            </geometry>
-        </visual>
-        <!--<collision>
-            <geometry>
-                <mesh filename="package://spot_description/meshes/front_left_hip_collision.stl" />
+                <mesh filename="file://$(find spot_description)/meshes/front_left_hip.dae" />
+            </geometry>
+        </visual>
+        <!--<collision>
+            <geometry>
+                <mesh filename="file://$(find spot_description)/meshes/front_left_hip_collision.stl" />
             </geometry>
         </collision>-->
@@ -163,10 +163,10 @@
         <visual>
             <geometry>
-                <mesh filename="package://spot_description/meshes/front_left_upper_leg.dae" />
-            </geometry>
-        </visual>
-        <!--<collision>
-            <geometry>
-                <mesh filename="package://spot_description/meshes/front_left_upper_leg_collision.stl" />
+                <mesh filename="file://$(find spot_description)/meshes/front_left_upper_leg.dae" />
+            </geometry>
+        </visual>
+        <!--<collision>
+            <geometry>
+                <mesh filename="file://$(find spot_description)/meshes/front_left_upper_leg_collision.stl" />
             </geometry>
         </collision>-->
@@ -196,10 +196,10 @@
         <visual>
             <geometry>
-                <mesh filename="package://spot_description/meshes/front_left_lower_leg.dae" />
-            </geometry>
-        </visual>
-        <!--<collision>
-            <geometry>
-                <mesh filename="package://spot_description/meshes/front_left_lower_leg_collision.stl" />
+                <mesh filename="file://$(find spot_description)/meshes/front_left_lower_leg.dae" />
+            </geometry>
+        </visual>
+        <!--<collision>
+            <geometry>
+                <mesh filename="file://$(find spot_description)/meshes/front_left_lower_leg_collision.stl" />
             </geometry>
         </collision>-->
@@ -258,10 +258,10 @@
         <visual>
             <geometry>
-                <mesh filename="package://spot_description/meshes/front_right_hip.dae" />
-            </geometry>
-        </visual>
-        <!--<collision>
-            <geometry>
-                <mesh filename="package://spot_description/meshes/front_right_hip_collision.stl" />
+                <mesh filename="file://$(find spot_description)/meshes/front_right_hip.dae" />
+            </geometry>
+        </visual>
+        <!--<collision>
+            <geometry>
+                <mesh filename="file://$(find spot_description)/meshes/front_right_hip_collision.stl" />
             </geometry>
         </collision>-->
@@ -285,10 +285,10 @@
         <visual>
             <geometry>
-                <mesh filename="package://spot_description/meshes/front_right_upper_leg.dae" />
-            </geometry>
-        </visual>
-        <!--<collision>
-            <geometry>
-                <mesh filename="package://spot_description/meshes/front_right_upper_leg_collision.stl" />
+                <mesh filename="file://$(find spot_description)/meshes/front_right_upper_leg.dae" />
+            </geometry>
+        </visual>
+        <!--<collision>
+            <geometry>
+                <mesh filename="file://$(find spot_description)/meshes/front_right_upper_leg_collision.stl" />
             </geometry>
         </collision>-->
@@ -318,10 +318,10 @@
         <visual>
             <geometry>
-                <mesh filename="package://spot_description/meshes/front_right_lower_leg.dae" />
-            </geometry>
-        </visual>
-        <!--<collision>
-            <geometry>
-                <mesh filename="package://spot_description/meshes/front_right_lower_leg_collision.stl" />
+                <mesh filename="file://$(find spot_description)/meshes/front_right_lower_leg.dae" />
+            </geometry>
+        </visual>
+        <!--<collision>
+            <geometry>
+                <mesh filename="file://$(find spot_description)/meshes/front_right_lower_leg_collision.stl" />
             </geometry>
         </collision>-->
@@ -380,10 +380,10 @@
         <visual>
             <geometry>
-                <mesh filename="package://spot_description/meshes/rear_left_hip.dae" />
-            </geometry>
-        </visual>
-        <!--<collision>
-            <geometry>
-                <mesh filename="package://spot_description/meshes/rear_left_hip_collision.stl" />
+                <mesh filename="file://$(find spot_description)/meshes/rear_left_hip.dae" />
+            </geometry>
+        </visual>
+        <!--<collision>
+            <geometry>
+                <mesh filename="file://$(find spot_description)/meshes/rear_left_hip_collision.stl" />
             </geometry>
         </collision>-->
@@ -407,10 +407,10 @@
         <visual>
             <geometry>
-                <mesh filename="package://spot_description/meshes/rear_left_upper_leg.dae" />
-            </geometry>
-        </visual>
-        <!--<collision>
-            <geometry>
-                <mesh filename="package://spot_description/meshes/rear_left_upper_leg_collision.stl" />
+                <mesh filename="file://$(find spot_description)/meshes/rear_left_upper_leg.dae" />
+            </geometry>
+        </visual>
+        <!--<collision>
+            <geometry>
+                <mesh filename="file://$(find spot_description)/meshes/rear_left_upper_leg_collision.stl" />
             </geometry>
         </collision>-->
@@ -440,10 +440,10 @@
         <visual>
             <geometry>
-                <mesh filename="package://spot_description/meshes/rear_left_lower_leg.dae" />
-            </geometry>
-        </visual>
-        <!--<collision>
-            <geometry>
-                <mesh filename="package://spot_description/meshes/rear_left_lower_leg_collision.stl" />
+                <mesh filename="file://$(find spot_description)/meshes/rear_left_lower_leg.dae" />
+            </geometry>
+        </visual>
+        <!--<collision>
+            <geometry>
+                <mesh filename="file://$(find spot_description)/meshes/rear_left_lower_leg_collision.stl" />
             </geometry>
         </collision>-->
@@ -502,10 +502,10 @@
         <visual>
             <geometry>
-                <mesh filename="package://spot_description/meshes/rear_right_hip.dae" />
-            </geometry>
-        </visual>
-        <!--<collision>
-            <geometry>
-                <mesh filename="package://spot_description/meshes/rear_right_hip_collision.stl" />
+                <mesh filename="file://$(find spot_description)/meshes/rear_right_hip.dae" />
+            </geometry>
+        </visual>
+        <!--<collision>
+            <geometry>
+                <mesh filename="file://$(find spot_description)/meshes/rear_right_hip_collision.stl" />
             </geometry>
         </collision>-->
@@ -529,10 +529,10 @@
         <visual>
             <geometry>
-                <mesh filename="package://spot_description/meshes/rear_right_upper_leg.dae" />
-            </geometry>
-        </visual>
-        <!--<collision>
-            <geometry>
-                <mesh filename="package://spot_description/meshes/rear_right_upper_leg_collision.stl" />
+                <mesh filename="file://$(find spot_description)/meshes/rear_right_upper_leg.dae" />
+            </geometry>
+        </visual>
+        <!--<collision>
+            <geometry>
+                <mesh filename="file://$(find spot_description)/meshes/rear_right_upper_leg_collision.stl" />
             </geometry>
         </collision>-->
@@ -562,10 +562,10 @@
         <visual>
             <geometry>
-                <mesh filename="package://spot_description/meshes/rear_right_lower_leg.dae" />
-            </geometry>
-        </visual>
-        <!--<collision>
-            <geometry>
-                <mesh filename="package://spot_description/meshes/rear_right_lower_leg_collision.stl" />
+                <mesh filename="file://$(find spot_description)/meshes/rear_right_lower_leg.dae" />
+            </geometry>
+        </visual>
+        <!--<collision>
+            <geometry>
+                <mesh filename="file://$(find spot_description)/meshes/rear_right_lower_leg_collision.stl" />
             </geometry>
         </collision>-->

File: spot_description/urdfs/accessories.urdf.xacro (robot description, xacro)
@@ -17,15 +17,15 @@
       <visual>
         <geometry>
-          <mesh filename="package://spot_description/meshes/pack_top.dae"/>
+          <mesh filename="file://$(find spot_description)/meshes/pack_top.dae"/>
         </geometry>
       </visual>
       <visual>
         <geometry>
-          <mesh filename="package://spot_description/meshes/pack_body.dae"/>
+          <mesh filename="file://$(find spot_description)/meshes/pack_body.dae"/>
         </geometry>
       </visual>
       <collision>
         <geometry>
-          <mesh filename="package://spot_description/meshes/pack_body.dae"/>
+          <mesh filename="file://$(find spot_description)/meshes/pack_body.dae"/>
         </geometry>
       </collision>
@@ -41,10 +41,10 @@
       <visual>
         <geometry>
-          <mesh filename="package://spot_description/meshes/lidar_mount.dae"/>
+          <mesh filename="file://$(find spot_description)/meshes/lidar_mount.dae"/>
         </geometry>
       </visual>
       <collision>
         <geometry>
-          <mesh filename="package://spot_description/meshes/lidar_mount_collision.stl"/>
+          <mesh filename="file://$(find spot_description)/meshes/lidar_mount_collision.stl"/>
         </geometry>
       </collision>
@@ -59,10 +59,10 @@
         <visual>
           <geometry>
-            <mesh filename="package://spot_description/meshes/velo.dae"/>
+            <mesh filename="file://$(find spot_description)/meshes/velo.dae"/>
           </geometry>
         </visual>
         <collision>
           <geometry>
-            <mesh filename="package://spot_description/meshes/velo_collision.stl"/>
+            <mesh filename="file://$(find spot_description)/meshes/velo_collision.stl"/>
           </geometry>
         </collision>
