Commit message: Running both with ros1 and ros2
work in progress

File: go1_description/robots/go1.urdf.xacro (robot description, xacro)
@@ -16,6 +16,8 @@
     <xacro:include filename="$(find wolf_description_utils)/urdfs/gazebo.urdf.xacro"/>
     <!-- legs transmission and gazebo plugins -->
-    <xacro:include filename="$(find wolf_description_utils)/urdfs/leg.transmission.xacro"/>
+    <xacro:include filename="$(find wolf_description_utils)/urdfs/leg.hardware.xacro"/>
     <xacro:include filename="$(find wolf_description_utils)/urdfs/leg.gazebo.xacro"/>
+    <xacro:include filename="$(find wolf_description_utils)/urdfs/imu.hardware.xacro"/>
+    <xacro:include filename="$(find sensors_description)/urdfs/sensors/imu.gazebo.xacro"/>
     <xacro:include filename="$(find go1_description)/urdfs/const.xacro"/>
     <xacro:include filename="$(find go1_description)/urdfs/leg.xacro"/>
@@ -142,12 +144,28 @@
         <xacro:include filename="$(find go1_description)/urdfs/accessories.urdf.xacro" />
     </xacro:if>
+    <!-- IMU sensor -->
+    <xacro:imu_sensor
+        frame_name="trunk_imu"
+        imu_topic="trunk_imu/data"
+        namespace="$(arg robot_name)"
+        update_rate="${1.0 / $(arg period)}"
+        rate_mean="0"
+        rate_stddev="0.01"
+        rate_bias_mean="0"
+        rate_bias_stddev="0"
+        accel_mean="0"
+        accel_stddev="0.001"
+        accel_bias_mean="0"
+        accel_bias_stddev="0">
+    </xacro:imu_sensor>
     <!-- Extensions -->
-    <xacro:leg_transmission prefix="rf"/>
+    <xacro:leg_hardware prefix="rf"/>
     <xacro:leg_gazebo prefix="rf" robot_name="$(arg robot_name)" load_force_sensors="$(arg load_force_sensors)"/>
-    <xacro:leg_transmission prefix="lf"/>
+    <xacro:leg_hardware prefix="lf"/>
     <xacro:leg_gazebo prefix="lf" robot_name="$(arg robot_name)" load_force_sensors="$(arg load_force_sensors)"/>
-    <xacro:leg_transmission prefix="rh"/>
+    <xacro:leg_hardware prefix="rh"/>
     <xacro:leg_gazebo prefix="rh" robot_name="$(arg robot_name)" load_force_sensors="$(arg load_force_sensors)"/>
-    <xacro:leg_transmission prefix="lh"/>
+    <xacro:leg_hardware prefix="lh"/>
     <xacro:leg_gazebo prefix="lh" robot_name="$(arg robot_name)" load_force_sensors="$(arg load_force_sensors)"/>
+    <xacro:imu_hardware imu_name="trunk_imu" imu_frame="trunk_imu"/>
 </robot>

File: go1_description/urdfs/accessories.urdf.xacro (robot description, xacro)
@@ -6,5 +6,4 @@
   <xacro:include filename="$(find velodyne_description)/urdf/VLP-16.urdf.xacro"/>
   <xacro:include filename="$(find sensors_description)/urdfs/sensors/realsense_t265.urdf.xacro"/>
-  <xacro:include filename="$(find sensors_description)/urdfs/sensors/imu.gazebo.xacro"/>
   <xacro:include filename="$(find sensors_description)/urdfs/sensors/gps.gazebo.xacro"/>
   <xacro:include filename="$(find sensors_description)/urdfs/sensors/realsense_d435.urdf.xacro" />
@@ -60,19 +59,4 @@
     <origin xyz="0.1 0 0" rpy="0 0 0" />
   </xacro:VLP-16>
-  <!-- IMU sensor -->
-  <xacro:imu_sensor
-      frame_name="trunk_imu"
-      imu_topic="trunk_imu/data"
-      namespace="$(arg robot_name)"
-      update_rate="${1.0 / $(arg period)}"
-      rate_mean="0"
-      rate_stddev="0.01"
-      rate_bias_mean="0"
-      rate_bias_stddev="0"
-      accel_mean="0"
-      accel_stddev="0.001"
-      accel_bias_mean="0"
-      accel_bias_stddev="0">
-  </xacro:imu_sensor>
   <!-- GPS sensor -->
   <xacro:gps_sensor

File: sensors_description/urdfs/sensors/imu.gazebo.xacro (robot description, xacro)
@@ -3,42 +3,4 @@
         <xacro:macro name="imu_sensor" params="frame_name imu_topic namespace update_rate rate_mean rate_stddev
 		rate_bias_mean rate_bias_stddev accel_mean accel_stddev accel_bias_mean accel_bias_stddev">
-                <!-- old plugin -->
-                <!--<gazebo>
-                        <plugin name="${imu_name}_controller" filename="libgazebo_ros_imu.so">
-                                <alwaysOn>true</alwaysOn>
-                                <updateRate>${update_rate}</updateRate>
-                                <bodyName>${imu_name}</bodyName>
-                                <topicName>${imu_topic}</topicName>
-                                <gaussianNoise>${rate_stddev*rate_stddev}</gaussianNoise>
-                                <xyzOffset>0 0 0</xyzOffset>
-                                <rpyOffset>0 0 0</rpyOffset>
-                                <serviceName>${imu_name}</serviceName>
-			</plugin>
-                </gazebo>-->
-                <!-- Imu definition required for the hardware interface of ros control -->
-                <!--<gazebo reference="${imu_name}">
-                        <sensor name="${imu_name}" type="imu">
-                                <always_on>1</always_on>
-                                <update_rate>${update_rate}</update_rate>
-                                <imu>
-                                        <noise>
-                                                <type>gaussian</type>
-                                                <rate>
-                                                        <mean>${rate_mean}</mean>
-                                                        <stddev>${rate_stddev}</stddev>
-                                                        <bias_mean>${rate_bias_mean}</bias_mean>
-                                                        <bias_stddev>${rate_bias_stddev}</bias_stddev>
-                                                </rate>
-                                                <accel>
-                                                        <mean>${accel_mean}</mean>
-                                                        <stddev>${accel_stddev}</stddev>
-                                                        <bias_mean>${accel_bias_mean}</bias_mean>
-                                                        <bias_stddev>${accel_bias_stddev}</bias_stddev>
-                                                </accel>
-                                        </noise>
-                                </imu>
-                        </sensor>
-                </gazebo>-->
-                <!-- recent plugin with gravity acceleration -->
                 <xacro:if value="${namespace == ''}">
                     <xacro:property name="frame_name_ns" value="${frame_name}"/>
@@ -47,7 +9,7 @@
                     <xacro:property name="frame_name_ns" value="${namespace+'/'+frame_name}"/>
                 </xacro:if>
-                <gazebo reference="${frame_name}">
+                <gazebo reference="trunk_imu">
                    <gravity>true</gravity>
-                   <sensor name="${frame_name}_sensor" type="imu">
+                   <sensor name="trunk_imu" type="imu">
                      <always_on>true</always_on>
                      <update_rate>${update_rate}</update_rate>

File: sensors_description/urdfs/sensors/realsense_t265.urdf.xacro (robot description, xacro)
@@ -1,5 +1,5 @@
 <?xml version="1.0"?>
 <robot xmlns:xacro="http://www.ros.org/wiki/xacro">
-  <!-- T265 Fisheye:
+<!-- T265 Fisheye:
   gazebo_ros_camera supports only plumb_bob
   D: [-0.007419134024530649, 0.041209351271390915, -0.03811917081475258, 0.006366158835589886, 0.0]
@@ -190,5 +190,5 @@
             <updateRate>${rate}</updateRate>
             <robotNamespace>${topics_ns}</robotNamespace>
-            <body_name>${name}_odom_frame</body_name>
+            <bodyName>${name}_odom_frame</bodyName>
             <topicName>${name}/odom</topicName>
             <gaussianNoise>0.001</gaussianNoise>

File: spot_description/robots/spot.urdf.xacro (robot description, xacro)
@@ -15,6 +15,8 @@
     <xacro:include filename="$(find wolf_description_utils)/urdfs/gazebo.urdf.xacro"/>
     <!-- legs transmission and gazebo plugins -->
-    <xacro:include filename="$(find wolf_description_utils)/urdfs/leg.transmission.xacro"/>
+    <xacro:include filename="$(find wolf_description_utils)/urdfs/leg.hardware.xacro"/>
     <xacro:include filename="$(find wolf_description_utils)/urdfs/leg.gazebo.xacro"/>
+    <xacro:include filename="$(find wolf_description_utils)/urdfs/imu.hardware.xacro"/>
+    <xacro:include filename="$(find sensors_description)/urdfs/sensors/imu.gazebo.xacro"/>
     <!-- dynamics inertial value -->
     <!-- Constants for robot dimensions -->
@@ -625,13 +627,29 @@
         <xacro:include filename="$(find spot_description)/urdfs/accessories.urdf.xacro" />
     </xacro:if>
+    <!-- IMU sensor -->
+    <xacro:imu_sensor
+        frame_name="trunk_imu"
+        imu_topic="trunk_imu/data"
+        namespace="$(arg robot_name)"
+        update_rate="${1.0 / $(arg period)}"
+        rate_mean="0"
+        rate_stddev="0.01"
+        rate_bias_mean="0"
+        rate_bias_stddev="0"
+        accel_mean="0"
+        accel_stddev="0.001"
+        accel_bias_mean="0"
+        accel_bias_stddev="0">
+    </xacro:imu_sensor>
     <!-- Extensions -->
-    <xacro:leg_transmission prefix="rf"/>
+    <xacro:leg_hardware prefix="rf"/>
     <xacro:leg_gazebo prefix="rf" robot_name="$(arg robot_name)" load_force_sensors="$(arg load_force_sensors)"/>
-    <xacro:leg_transmission prefix="lf"/>
+    <xacro:leg_hardware prefix="lf"/>
     <xacro:leg_gazebo prefix="lf" robot_name="$(arg robot_name)" load_force_sensors="$(arg load_force_sensors)"/>
-    <xacro:leg_transmission prefix="rh"/>
+    <xacro:leg_hardware prefix="rh"/>
     <xacro:leg_gazebo prefix="rh" robot_name="$(arg robot_name)" load_force_sensors="$(arg load_force_sensors)"/>
-    <xacro:leg_transmission prefix="lh"/>
+    <xacro:leg_hardware prefix="lh"/>
     <xacro:leg_gazebo prefix="lh" robot_name="$(arg robot_name)" load_force_sensors="$(arg load_force_sensors)"/>
+    <xacro:imu_hardware imu_name="trunk_imu" imu_frame="trunk_imu"/>
     <xacro:if value="$(eval arm_name != '')">
            <xacro:include filename="$(find spot_description)/urdfs/arm/$(arg arm_name)_adapter.urdf.xacro" />

File: spot_description/urdfs/accessories.urdf.xacro (robot description, xacro)
@@ -2,9 +2,7 @@
 <robot xmlns:xacro="http://www.ros.org/wiki/xacro">
   <xacro:include filename="$(find sensors_description)/urdfs/common.xacro"/>
-  <!--<xacro:include filename="$(find sensors_description)/urdfs/sensors/velodyne.gazebo.xacro"/>-->
   <xacro:include filename="$(find velodyne_description)/urdf/VLP-16.urdf.xacro"/>
   <xacro:include filename="$(find sensors_description)/urdfs/sensors/realsense_d435.urdf.xacro" />
   <xacro:include filename="$(find sensors_description)/urdfs/sensors/realsense_t265.urdf.xacro" />
-  <xacro:include filename="$(find sensors_description)/urdfs/sensors/imu.gazebo.xacro"/>
   <xacro:include filename="$(find sensors_description)/urdfs/sensors/gps.gazebo.xacro"/>
   <xacro:if value="$(optenv SPOT_PACK 1)">
@@ -78,19 +76,4 @@
         <origin xyz="0.13 0 0.04" rpy="0 0 0" />
       </xacro:realsense_T265>
-      <!-- IMU sensor -->
-      <xacro:imu_sensor
-          frame_name="trunk_imu"
-          imu_topic="trunk_imu/data"
-          namespace="$(arg robot_name)"
-          update_rate="${1.0 / $(arg period)}"
-          rate_mean="0"
-          rate_stddev="0.01"
-          rate_bias_mean="0"
-          rate_bias_stddev="0"
-          accel_mean="0"
-          accel_stddev="0.001"
-          accel_bias_mean="0"
-          accel_bias_stddev="0">
-      </xacro:imu_sensor>
       <!-- GPS sensor -->
       <xacro:gps_sensor

File: wolf_description_utils/urdfs/arm.hardware.xacro (robot description, xacro)
@@ -1,5 +1,5 @@
 <?xml version="1.0"?>
 <robot xmlns:xacro="http://ros.org/wiki/xacro">
-        <xacro:macro name="arm_transmission" params="name">
+        <xacro:macro name="arm_hardware" params="name">
                 <transmission name="${name}_trans">
                         <type>transmission_interface/SimpleTransmission</type>

File: wolf_description_utils/urdfs/gazebo.urdf.xacro (robot description, xacro)
@@ -13,11 +13,10 @@
         </plugin>
         <plugin name="gazebo_ros2_controller_manager" filename="libgazebo_ros2_control.so">
-                <robotNamespace>$(arg robot_name)</robotNamespace>
-                <robotSimType>wolf_gazebo_interface/WolfRobotHwSim</robotSimType>
-                <parameters>$(find ${model_name}_description)/params/${model_name}_params.yaml</parameters>
+                <parameters>$(find wolf_controller)/params/config.ros2.yaml</parameters>
+                <parameters>$(find ${model_name}_description)/params/${model_name}_params.ros2.yaml</parameters>
         </plugin>
     	<plugin filename="libgazebo_ros_p3d.so" name="ground_truth">
-            <robotNamespace>$(arg robot_name)</robotNamespace>
-                <body_name>$(arg base_name)</body_name>
+                <robotNamespace>$(arg robot_name)</robotNamespace>
+                <bodyName>$(arg base_name)</bodyName>
                 <topicName>ground_truth</topicName>
                 <frameName>world</frameName>

File: wolf_description_utils/urdfs/leg.hardware.xacro (robot description, xacro)
@@ -1,5 +1,5 @@
 <?xml version="1.0"?>
 <robot xmlns:xacro="http://ros.org/wiki/xacro">
-        <xacro:macro name="leg_transmission" params="prefix">
+        <xacro:macro name="leg_hardware" params="prefix">
         <!-- ROS1 -->
     	<!-- Hip assembly -->
@@ -44,6 +44,6 @@
                     <joint name="${prefix}_haa_joint">
                       <command_interface name="effort">
-                        <param name="min">-6.28</param>
-                        <param name="max">6.28</param>
+                        <param name="min">-500.0</param>
+                        <param name="max">500.0</param>
                       </command_interface>
                       <state_interface name="position"/>
@@ -54,6 +54,6 @@
                     <joint name="${prefix}_hfe_joint">
                       <command_interface name="effort">
-                        <param name="min">-6.28</param>
-                        <param name="max">6.28</param>
+                        <param name="min">-500.0</param>
+                        <param name="max">500.0</param>
                       </command_interface>
                       <state_interface name="position"/>
@@ -64,6 +64,6 @@
                     <joint name="${prefix}_kfe_joint">
                       <command_interface name="effort">
-                        <param name="min">-6.28</param>
-                        <param name="max">6.28</param>
+                        <param name="min">-500.0</param>
+                        <param name="max">500.0</param>
                       </command_interface>
                       <state_interface name="position"/>
