Commit message: Use Ignition

File: go1_description/robots/go1.urdf.xacro (robot description, xacro)
@@ -10,4 +10,5 @@
     <xacro:arg name="robot_name"         default=""/>
     <xacro:arg name="base_name"          default="base_link"/>
+    <xacro:arg name="simulator"          default="ignition"/>
     <!-- load generic materials -->
     <xacro:include filename="$(find wolf_description_utils)/urdfs/materials.xacro"/>
@@ -129,12 +130,11 @@
     </xacro:imu_sensor>
     <!-- Extensions -->
-    <xacro:leg_hardware prefix="rf"/>
+    <xacro:leg_hardware prefix="rf" imu_name="$(arg robot_name)_imu" imu_frame="trunk_imu"/>
     <xacro:leg_gazebo prefix="rf" robot_name="$(arg robot_name)" load_force_sensors="$(arg load_force_sensors)"/>
-    <xacro:leg_hardware prefix="lf"/>
+    <xacro:leg_hardware prefix="lf" imu_name="" imu_frame=""/>
     <xacro:leg_gazebo prefix="lf" robot_name="$(arg robot_name)" load_force_sensors="$(arg load_force_sensors)"/>
-    <xacro:leg_hardware prefix="rh"/>
+    <xacro:leg_hardware prefix="rh" imu_name="" imu_frame=""/>
     <xacro:leg_gazebo prefix="rh" robot_name="$(arg robot_name)" load_force_sensors="$(arg load_force_sensors)"/>
-    <xacro:leg_hardware prefix="lh"/>
+    <xacro:leg_hardware prefix="lh" imu_name="" imu_frame=""/>
     <xacro:leg_gazebo prefix="lh" robot_name="$(arg robot_name)" load_force_sensors="$(arg load_force_sensors)"/>
-    <xacro:imu_hardware imu_name="$(arg robot_name)_imu" imu_frame="trunk_imu"/>
 </robot>

File: go1_description/urdfs/accessories.urdf.xacro (robot description, xacro)
@@ -1,4 +1,5 @@
 <?xml version="1.0"?>
 <robot xmlns:xacro="http://www.ros.org/wiki/xacro">
+  <xacro:arg name="simulator" default="ignition"/>
   <xacro:include filename="$(find sensors_description)/urdfs/common.xacro"/>
   <xacro:include filename="$(find sensors_description)/urdfs/sensors/depth_camera.gazebo.xacro"/>
@@ -39,16 +40,16 @@
         </visual>
     </link>
-   <xacro:depth_camera
-     name="camera"
-     namespace="$(arg robot_name)"
-     update_rate="30"
-     image_width="640"
-     image_height="480"
-     fov="1.047"
-     near="0.1"
-     far="10.0"
-     parent_link="camera_mount"
-     origin_xyz="0.0 0 0.0"
-     origin_rpy="0 0.0 0"/>
+  <xacro:depth_camera
+    name="camera"
+    namespace="$(arg robot_name)"
+    update_rate="30"
+    image_width="640"
+    image_height="480"
+    fov="1.047"
+    near="0.1"
+    far="10.0"
+    parent_link="camera_mount"
+    origin_xyz="0.0 0 0.0"
+    origin_rpy="0 0.0 0"/>
   <xacro:velodyne_laser_gazebo_sensor
     sensor_name="$(arg robot_name)_lidar"

File: husky_description/robots/husky.urdf.xacro (robot description, xacro)
@@ -9,4 +9,5 @@
   <xacro:arg name="robot_name"         default=""/>
   <xacro:arg name="base_name"          default="base_link"/>
+  <xacro:arg name="simulator"          default="ignition"/>
   <!-- generic simulator_gazebo plugins for starting mechanism control, ros time -->
   <xacro:include filename="$(find wolf_description_utils)/urdfs/gazebo.urdf.xacro"/>
@@ -35,5 +36,4 @@
         accel_bias_stddev="0">
     </xacro:imu_sensor>
-    <xacro:imu_hardware imu_name="$(arg robot_name)_imu" imu_frame="trunk_imu"/>
     <!-- Standard accessories. -->
     <xacro:if value="$(arg sensors)">

File: sensors_description/urdfs/sensors/depth_camera.gazebo.xacro (robot description, xacro)
@@ -32,10 +32,17 @@
       <origin xyz="${origin_xyz}" rpy="${origin_rpy}"/>
     </joint>
-    <!-- Depth Camera Sensor -->
+    <xacro:if value="${namespace == ''}">
+      <xacro:property name="camera_topic_ns" value="${name}"/>
+    </xacro:if>
+    <xacro:if value="${namespace != ''}">
+      <xacro:property name="camera_topic_ns" value="${namespace + '/' + name}"/>
+    </xacro:if>
+    <!-- Gazebo Sim depth camera sensor -->
     <gazebo reference="${name}_link">
-      <sensor type="depth" name="${name}">
+      <sensor type="depth_camera" name="${name}">
         <update_rate>${update_rate}</update_rate>
         <always_on>true</always_on>
         <pose>${origin_xyz} ${origin_rpy}</pose>
+        <topic>${camera_topic_ns}</topic>
         <camera name="${name}">
           <horizontal_fov>${fov}</horizontal_fov>
@@ -50,26 +57,4 @@
           </clip>
         </camera>
-        <!-- Plugin for Depth Camera -->
-        <plugin name="${namespace}_${name}_plugin" filename="libgazebo_ros_camera.so">
-          <robotNamespace>/${namespace}</robotNamespace>
-          <ros>
-            <namespace>/${namespace}</namespace>
-            <remapping>${name}/image_raw:=/${namespace}/${name}/image_raw</remapping>
-            <remapping>${name}/image_raw/compressed:=/${namespace}/${name}/image_raw/compressed</remapping>
-            <remapping>${name}/image_raw/compressedDepth:=/${namespace}/${name}/image_raw/compressedDepth</remapping>
-            <remapping>${name}/image_raw/theora:=/${namespace}/${name}/image_raw/theora</remapping>
-            <remapping>${name}/depth/image_raw:=/${namespace}/${name}/depth/image_raw</remapping>
-            <remapping>${name}/depth/camera_info:=/${namespace}/${name}/depth/camera_info</remapping>
-            <remapping>${name}/depth/image_raw/compressed:=/${namespace}/${name}/depth/image_raw/compressed</remapping>
-            <remapping>${name}/depth/image_raw/compressedDepth:=/${namespace}/${name}/depth/image_raw/compressedDepth</remapping>
-            <remapping>${name}/depth/image_raw/theora:=/${namespace}/${name}/depth/image_raw/theora</remapping>
-            <remapping>${name}/camera_info:=/${namespace}/${name}/camera_info</remapping>
-            <remapping>${name}/points:=/${namespace}/${name}/points</remapping>
-          </ros>
-          <camera_name>${name}</camera_name>
-          <frame_name>${name}_link</frame_name>
-          <update_rate>${update_rate}</update_rate>
-          <point_cloud>true</point_cloud> <!-- Optional -->
-        </plugin>
       </sensor>
     </gazebo>

File: sensors_description/urdfs/sensors/gps.gazebo.xacro (robot description, xacro)
@@ -3,5 +3,5 @@
   <!--
     Macro: gazebo_gps_sensor
-    Description: Inserts a GPS sensor with the gazebo_ros_gps_sensor plugin.
+    Description: Inserts a Gazebo Sim GPS sensor (bridge to ROS with ros_gz_bridge).
     Parameters:
       sensor_name    - Name for the sensor element.
@@ -14,8 +14,8 @@
   <xacro:macro name="gazebo_gps_sensor" params="sensor_name namespace gps_topic velocity_topic update_rate frame_id">
       <xacro:if value="${namespace == ''}">
-                    <xacro:property name="frame_name_ns" value="${frame_id}"/>
+                    <xacro:property name="gps_topic_ns" value="${gps_topic}"/>
       </xacro:if>
       <xacro:if value="${namespace != ''}">
-                    <xacro:property name="frame_name_ns" value="${namespace+'/'+frame_id}"/>
+                    <xacro:property name="gps_topic_ns" value="${namespace+'/'+gps_topic}"/>
       </xacro:if>
     <gazebo reference="${frame_id}">
@@ -23,17 +23,8 @@
         <always_on>1</always_on>
         <update_rate>${update_rate}</update_rate>
+        <topic>${gps_topic_ns}</topic>
         <gps>
           <!-- Optionally, include additional sensor-specific parameters here -->
         </gps>
-        <plugin name="${sensor_name}_plugin" filename="libgazebo_ros_gps_sensor.so">
-          <robotNamespace>/${namespace}</robotNamespace>
-          <ros>
-            <namespace>/${namespace}</namespace>
-            <!-- Additional ROS plugin configuration can be added here -->
-            <remapping>${sensor_name}_plugin/out:=/${namespace}/${gps_topic}</remapping>
-            <remapping>${sensor_name}_plugin/vel:=/${namespace}/${velocity_topic}</remapping>
-          </ros>
-          <frame_name>${frame_name_ns}</frame_name>
-        </plugin>
       </sensor>
     </gazebo>

File: sensors_description/urdfs/sensors/imu.gazebo.xacro (robot description, xacro)
@@ -4,8 +4,8 @@
         rate_bias_mean rate_bias_stddev accel_mean accel_stddev accel_bias_mean accel_bias_stddev">
       <xacro:if value="${namespace == ''}">
-                <xacro:property name="frame_name_ns" value="${frame_name}"/>
+                <xacro:property name="imu_topic_ns" value="${imu_topic}"/>
       </xacro:if>
       <xacro:if value="${namespace != ''}">
-                <xacro:property name="frame_name_ns" value="${namespace+'/'+frame_name}"/>
+                <xacro:property name="imu_topic_ns" value="${namespace+'/'+imu_topic}"/>
       </xacro:if>
         <gazebo reference="${frame_name}">
@@ -15,18 +15,5 @@
                 <update_rate>${update_rate}</update_rate>
                 <visualize>true</visualize>
-                <topic>${imu_topic}</topic>
-                <plugin name="${sensor_name}_plugin" filename="libgazebo_ros_imu_sensor.so">
-                    <robotNamespace>/${namespace}</robotNamespace>
-                    <ros>
-                        <namespace>/${namespace}</namespace>
-                        <remapping>${sensor_name}_plugin/out:=/${namespace}/${imu_topic}</remapping>
-                    </ros>
-                    <update_rate>${update_rate}</update_rate>
-                    <gaussian_noise>${rate_stddev*rate_stddev}</gaussian_noise>
-                    <xyz_offset>0 0 0</xyz_offset>
-                    <rpy_offset>0 0 0</rpy_offset>
-                    <frame_name>${frame_name_ns}</frame_name>
-                    <initial_orientation_as_reference>false</initial_orientation_as_reference>
-                </plugin>
+                <topic>${imu_topic_ns}</topic>
                 <pose>0 0 0 0 0 0</pose>
             </sensor>

File: sensors_description/urdfs/sensors/lidar.gazebo.xacro (robot description, xacro)
@@ -2,10 +2,9 @@
 <robot xmlns:xacro="http://ros.org/wiki/xacro">
   <xacro:macro name="velodyne_laser_gazebo_sensor" params="sensor_name topic_name update_rate frame_id namespace min_range max_range number_of_beams horizontal_samples horizontal_fov vertical_fov noise_stddev">
-    <!-- Construct full frame name -->
     <xacro:if value="${namespace == ''}">
-      <xacro:property name="frame_name_ns" value="${frame_id}"/>
+      <xacro:property name="lidar_topic_ns" value="${topic_name}"/>
     </xacro:if>
     <xacro:if value="${namespace != ''}">
-      <xacro:property name="frame_name_ns" value="${namespace + '/' + frame_id}"/>
+      <xacro:property name="lidar_topic_ns" value="${namespace + '/' + topic_name}"/>
     </xacro:if>
     <!-- Sensor definition -->
@@ -15,4 +14,5 @@
         <visualize>false</visualize>
         <update_rate>${update_rate}</update_rate>
+        <topic>${lidar_topic_ns}</topic>
         <ray>
           <scan>
@@ -41,16 +41,4 @@
           </noise>
         </ray>
-        <plugin name="${sensor_name}_plugin" filename="libgazebo_ros_velodyne_laser.so">
-          <robotNamespace>/${namespace}</robotNamespace>
-          <ros>
-            <namespace>/${namespace}</namespace>
-            <remapping>${sensor_name}_plugin/out:=/${namespace}/${topic_name}</remapping>
-          </ros>
-          <frame_name>${frame_name_ns}</frame_name>
-          <organize_cloud>true</organize_cloud>
-          <min_range>${min_range}</min_range>
-          <max_range>${max_range}</max_range>
-          <gaussian_noise>${noise_stddev}</gaussian_noise>
-        </plugin>
       </sensor>
     </gazebo>

File: spot_description/robots/spot.urdf.xacro (robot description, xacro)
@@ -10,4 +10,5 @@
     <xacro:arg name="robot_name"         default=""/>
     <xacro:arg name="base_name"          default="base_link"/>
+    <xacro:arg name="simulator"          default="ignition"/>
     <!-- load generic materials -->
     <xacro:include filename="$(find wolf_description_utils)/urdfs/materials.xacro"/>
@@ -644,13 +645,12 @@
     </xacro:imu_sensor>
     <!-- Extensions -->
-    <xacro:leg_hardware prefix="rf"/>
+    <xacro:leg_hardware prefix="rf" imu_name="$(arg robot_name)_imu" imu_frame="trunk_imu"/>
     <xacro:leg_gazebo prefix="rf" robot_name="$(arg robot_name)" load_force_sensors="$(arg load_force_sensors)"/>
-    <xacro:leg_hardware prefix="lf"/>
+    <xacro:leg_hardware prefix="lf" imu_name="" imu_frame=""/>
     <xacro:leg_gazebo prefix="lf" robot_name="$(arg robot_name)" load_force_sensors="$(arg load_force_sensors)"/>
-    <xacro:leg_hardware prefix="rh"/>
+    <xacro:leg_hardware prefix="rh" imu_name="" imu_frame=""/>
     <xacro:leg_gazebo prefix="rh" robot_name="$(arg robot_name)" load_force_sensors="$(arg load_force_sensors)"/>
-    <xacro:leg_hardware prefix="lh"/>
+    <xacro:leg_hardware prefix="lh" imu_name="" imu_frame=""/>
     <xacro:leg_gazebo prefix="lh" robot_name="$(arg robot_name)" load_force_sensors="$(arg load_force_sensors)"/>
-    <xacro:imu_hardware imu_name="$(arg robot_name)_imu" imu_frame="trunk_imu"/>
     <xacro:if value="$(eval arm_name != '')">
         <xacro:include filename="$(find spot_description)/urdfs/arm/$(arg arm_name)_adapter.urdf.xacro" />

File: spot_description/urdfs/accessories.urdf.xacro (robot description, xacro)
@@ -1,4 +1,5 @@
 <?xml version="1.0"?>
 <robot xmlns:xacro="http://www.ros.org/wiki/xacro">
+  <xacro:arg name="simulator" default="ignition"/>
   <xacro:include filename="$(find sensors_description)/urdfs/common.xacro"/>
   <xacro:include filename="$(find sensors_description)/urdfs/sensors/depth_camera.gazebo.xacro"/>
@@ -61,16 +62,16 @@
     </collision>
   </link>
-   <xacro:depth_camera
-     name="camera"
-     namespace="$(arg robot_name)"
-     update_rate="30"
-     image_width="640"
-     image_height="480"
-     fov="1.047"
-     near="0.1"
-     far="10.0"
-     parent_link="front_rail"
-     origin_xyz="0.13 0 0"
-     origin_rpy="0 0 0"/>
+  <xacro:depth_camera
+    name="camera"
+    namespace="$(arg robot_name)"
+    update_rate="30"
+    image_width="640"
+    image_height="480"
+    fov="1.047"
+    near="0.1"
+    far="10.0"
+    parent_link="front_rail"
+    origin_xyz="0.13 0 0"
+    origin_rpy="0 0 0"/>
   <xacro:velodyne_laser_gazebo_sensor
     sensor_name="$(arg robot_name)_lidar"
@@ -86,5 +87,5 @@
     vertical_fov="0.2618"
     noise_stddev="0.01" />
-<xacro:gazebo_gps_sensor
+  <xacro:gazebo_gps_sensor
     sensor_name="$(arg robot_name)_gps"
     namespace="$(arg robot_name)"

File: wolf_description_utils/urdfs/gazebo.urdf.xacro (robot description, xacro)
@@ -7,6 +7,6 @@
 <xacro:property name="model_name" value="$(arg robot_model)"/>
 	<gazebo>
-        <plugin name="$(arg robot_name)_controller_manager" filename="libgazebo_ros2_control.so">
-                <robot_param_node>/$(arg robot_name)/robot_state_publisher</robot_param_node>
+        <plugin name="ign_ros2_control::IgnitionROS2ControlPlugin" filename="libign_ros2_control-system.so">
+                <robot_param_node>robot_state_publisher</robot_param_node>
                 <ros>
                         <namespace>/$(arg robot_name)</namespace>
@@ -17,17 +17,4 @@
                 <parameters>$(find ${model_name}_description)/params/${model_name}_params_$(arg robot_name).ros2.yaml</parameters>
         </plugin>
-    	<plugin name="$(arg robot_name)_ground_truth" filename="libgazebo_ros_p3d.so">
-                <ros>
-                    <namespace>/$(arg robot_name)</namespace>
-                    <remapping>odom:=ground_truth</remapping>
-                </ros>
-                <frame_name>world</frame_name>
-                <body_name>$(arg base_name)</body_name>
-                <update_rate>${1/ $(arg period)}</update_rate>
-        </plugin>
-        <plugin name="$(arg robot_name)_set_joint_positions_plugin" filename="libgazebo_set_joint_positions_plugin.so">
-            <robot_namespace>$(arg robot_name)</robot_namespace>
-            <topic_name>set_joint_states</topic_name>
-        </plugin>
 	</gazebo>
 </robot>

File: wolf_description_utils/urdfs/imu.hardware.xacro (robot description, xacro)
@@ -5,5 +5,5 @@
                 <ros2_control name="sim_hardware_system" type="system">
                     <hardware>
-                      <plugin>gazebo_ros2_control/GazeboSystem</plugin>
+                      <plugin>ign_ros2_control/IgnitionSystem</plugin>
                     </hardware>
                     <sensor name="${imu_name}">

File: wolf_description_utils/urdfs/leg.gazebo.xacro (robot description, xacro)
@@ -1,104 +1,59 @@
 <?xml version="1.0"?>
 <robot xmlns:xacro="http://ros.org/wiki/xacro">
-	<xacro:macro name="leg_gazebo" params="prefix robot_name load_force_sensors">
-		<gazebo reference="${prefix}_haa_joint">
-			<provideFeedback>true</provideFeedback>
-		</gazebo>
-		<xacro:if value="${load_force_sensors}">
-			<gazebo>
-				<plugin name="${prefix}_haa_sensor" filename="libgazebo_ros_ft_sensor.so">
-					<ros>
-                        <namespace>${robot_name}</namespace>
-                    </ros>
-					<update_rate>100.0</update_rate>
-					<joint_name>${prefix}_haa_joint</joint_name>
-				</plugin>
-			</gazebo>
-		</xacro:if>
-		<gazebo reference="${prefix}_hfe_joint">
-			<provideFeedback>true</provideFeedback>
-		</gazebo>
-		<xacro:if value="${load_force_sensors}">
-			<gazebo>
-				<plugin name="${prefix}_hfe_sensor" filename="libgazebo_ros_ft_sensor.so">
-					<ros>
-                        <namespace>${robot_name}</namespace>
-                    </ros>
-					<update_rate>100.0</update_rate>
-					<joint_name>${prefix}_hfe_joint</joint_name>
-				</plugin>
-			</gazebo>
-		</xacro:if>
-		<gazebo reference="${prefix}_kfe_joint">
-				<provideFeedback>true</provideFeedback>
-		</gazebo>
-		<xacro:if value="${load_force_sensors}">
-				<gazebo>
-						<plugin name="${prefix}_kfe_sensor" filename="libgazebo_ros_ft_sensor.so">
-								<ros>
-									<namespace>${robot_name}</namespace>
-								</ros>
-								<update_rate>100.0</update_rate>
-								<joint_name>${prefix}_kfe_joint</joint_name>
-						</plugin>
-				</gazebo>
-		</xacro:if>
-		<gazebo reference="${prefix}_foot_joint">
-			<disableFixedJointLumping>true</disableFixedJointLumping>
-		</gazebo>
-		<gazebo reference="${prefix}_upperleg">
-			<kp>1000000.0</kp>
-			<kd>100.0</kd>
-			<mu1>1.5</mu1>
-			<mu2>1.5</mu2>
-			<fdir1>1 0 0</fdir1>
-			<maxVel>1.0</maxVel>
-			<maxContacts>1</maxContacts>
-			<minDepth>0.00</minDepth>
-		</gazebo>
-		<gazebo reference="${prefix}_lowerleg">
-			<kp>1000000.0</kp>
-			<kd>100.0</kd>
-			<mu1>1.0</mu1>
-			<mu2>1.0</mu2>
-			<maxVel>1.0</maxVel>
-			<maxContacts>1</maxContacts>
-			<sensor name="${prefix}_shin_contact_sensor" type="contact">
-					<always_on>true</always_on>
-					<update_rate>250.0</update_rate>
-					<contact>
-						<collision>${prefix}_lowerleg_collision</collision>
-					</contact>
-					<plugin name="${prefix}_shin_bumper" filename="libgazebo_ros_bumper.so">
-						<frame_name>${prefix}_lowerleg</frame_name>
-						   <ros>
-							<namespace>${robot_name}</namespace>
-							<remapping>bumper_states:=${prefix}_shin_bumper</remapping>
-						  </ros>
-					</plugin>
-			</sensor>
-		</gazebo>
-                <gazebo reference="${prefix}_foot">
-                        <kp>1000000.0</kp>
-                        <kd>100.0</kd>
-                        <mu1>1.0</mu1>
-                        <mu2>1.0</mu2>
-                        <maxVel>1.0</maxVel>
-                        <maxContacts>1</maxContacts>
-                        <sensor name="${prefix}_foot_contact_sensor" type="contact">
-				<always_on>true</always_on>
-				<update_rate>250.0</update_rate>
-				<contact>
-						<collision>${prefix}_foot_collision</collision>
-				</contact>
-				<plugin name="${prefix}_foot_bumper" filename="libgazebo_ros_bumper.so">
-						<frame_name>${prefix}_foot</frame_name>
-						  <ros>
-							<namespace>${robot_name}</namespace>
-							<remapping>bumper_states:=${prefix}_foot_bumper</remapping>
-						  </ros>
-				</plugin>
-			</sensor>
-		</gazebo>
-	</xacro:macro>
+  <xacro:macro name="leg_gazebo" params="prefix robot_name load_force_sensors">
+    <gazebo reference="${prefix}_haa_joint">
+      <provideFeedback>true</provideFeedback>
+    </gazebo>
+    <gazebo reference="${prefix}_hfe_joint">
+      <provideFeedback>true</provideFeedback>
+    </gazebo>
+    <gazebo reference="${prefix}_kfe_joint">
+      <provideFeedback>true</provideFeedback>
+    </gazebo>
+    <gazebo reference="${prefix}_foot_joint">
+      <disableFixedJointLumping>true</disableFixedJointLumping>
+    </gazebo>
+    <gazebo reference="${prefix}_upperleg">
+      <kp>1000000.0</kp>
+      <kd>100.0</kd>
+      <mu1>1.5</mu1>
+      <mu2>1.5</mu2>
+      <fdir1>1 0 0</fdir1>
+      <maxVel>1.0</maxVel>
+      <maxContacts>1</maxContacts>
+      <minDepth>0.00</minDepth>
+    </gazebo>
+    <gazebo reference="${prefix}_lowerleg">
+      <kp>1000000.0</kp>
+      <kd>100.0</kd>
+      <mu1>1.0</mu1>
+      <mu2>1.0</mu2>
+      <maxVel>1.0</maxVel>
+      <maxContacts>1</maxContacts>
+      <sensor name="${prefix}_shin_contact_sensor" type="contact">
+        <always_on>true</always_on>
+        <update_rate>250.0</update_rate>
+        <topic>${robot_name}/${prefix}_shin_bumper</topic>
+        <contact>
+          <collision>${prefix}_lowerleg_collision</collision>
+        </contact>
+      </sensor>
+    </gazebo>
+    <gazebo reference="${prefix}_foot">
+      <kp>1000000.0</kp>
+      <kd>100.0</kd>
+      <mu1>1.0</mu1>
+      <mu2>1.0</mu2>
+      <maxVel>1.0</maxVel>
+      <maxContacts>1</maxContacts>
+      <sensor name="${prefix}_foot_contact_sensor" type="contact">
+        <always_on>true</always_on>
+        <update_rate>250.0</update_rate>
+        <topic>${robot_name}/${prefix}_foot_bumper</topic>
+        <contact>
+          <collision>${prefix}_foot_collision</collision>
+        </contact>
+      </sensor>
+    </gazebo>
+  </xacro:macro>
 </robot>
