Commit message: Use Ignition

File: wolf_description_utils/urdfs/leg.hardware.xacro (robot description, xacro)
@@ -1,5 +1,5 @@
 <?xml version="1.0"?>
 <robot xmlns:xacro="http://ros.org/wiki/xacro">
-        <xacro:macro name="leg_hardware" params="prefix">
+        <xacro:macro name="leg_hardware" params="prefix imu_name:='' imu_frame:=''">
         <!-- ROS1 -->
     	<!-- Hip assembly -->
@@ -39,5 +39,5 @@
                 <ros2_control name="${prefix}_leg_system" type="system">
                     <hardware>
-                      <plugin>gazebo_ros2_control/GazeboSystem</plugin>
+                      <plugin>ign_ros2_control/IgnitionSystem</plugin>
                     </hardware>
                     <!-- Hip assembly -->
@@ -71,4 +71,19 @@
                       <state_interface name="effort"/>
                     </joint>
+                    <xacro:if value="${imu_name != ''}">
+                      <sensor name="${imu_name}">
+                        <param name="frame_id">${imu_frame}</param>
+                        <state_interface name="orientation.x"/>
+                        <state_interface name="orientation.y"/>
+                        <state_interface name="orientation.z"/>
+                        <state_interface name="orientation.w"/>
+                        <state_interface name="angular_velocity.x"/>
+                        <state_interface name="angular_velocity.y"/>
+                        <state_interface name="angular_velocity.z"/>
+                        <state_interface name="linear_acceleration.x"/>
+                        <state_interface name="linear_acceleration.y"/>
+                        <state_interface name="linear_acceleration.z"/>
+                      </sensor>
+                    </xacro:if>
             </ros2_control>
 	</xacro:macro>

File: wolf_description_utils/urdfs/wheels.hardware.xacro (robot description, xacro)
@@ -4,6 +4,19 @@
   <ros2_control name="wheels_system" type="system">
     <hardware>
-      <plugin>gazebo_ros2_control/GazeboSystem</plugin>
+      <plugin>ign_ros2_control/IgnitionSystem</plugin>
     </hardware>
+    <sensor name="$(arg robot_name)_imu">
+      <param name="frame_id">trunk_imu</param>
+      <state_interface name="orientation.x"/>
+      <state_interface name="orientation.y"/>
+      <state_interface name="orientation.z"/>
+      <state_interface name="orientation.w"/>
+      <state_interface name="angular_velocity.x"/>
+      <state_interface name="angular_velocity.y"/>
+      <state_interface name="angular_velocity.z"/>
+      <state_interface name="linear_acceleration.x"/>
+      <state_interface name="linear_acceleration.y"/>
+      <state_interface name="linear_acceleration.z"/>
+    </sensor>
     <joint name="front_left_wheel_joint">
       <command_interface name="velocity">

Commit message: Spot working with imu

File: go1_description/robots/go1.urdf.xacro (robot description, xacro)
@@ -115,5 +115,5 @@
     <!-- IMU sensor -->
     <xacro:imu_sensor
-        sensor_name="$(arg robot_name)_imu"
+        sensor_name="imu"
         frame_name="trunk_imu"
         imu_topic="trunk_imu/data"
@@ -129,12 +129,14 @@
         accel_bias_stddev="0">
     </xacro:imu_sensor>
+    <!-- ROS2 control -->
+    <xacro:quadruped_ros2_control imu_name="imu" imu_frame="trunk_imu"/>
     <!-- Extensions -->
-    <xacro:leg_hardware prefix="rf" imu_name="$(arg robot_name)_imu" imu_frame="trunk_imu"/>
+    <xacro:leg_hardware prefix="rf" with_ros2_control="false"/>
     <xacro:leg_gazebo prefix="rf" robot_name="$(arg robot_name)" load_force_sensors="$(arg load_force_sensors)"/>
-    <xacro:leg_hardware prefix="lf" imu_name="" imu_frame=""/>
+    <xacro:leg_hardware prefix="lf" with_ros2_control="false"/>
     <xacro:leg_gazebo prefix="lf" robot_name="$(arg robot_name)" load_force_sensors="$(arg load_force_sensors)"/>
-    <xacro:leg_hardware prefix="rh" imu_name="" imu_frame=""/>
+    <xacro:leg_hardware prefix="rh" with_ros2_control="false"/>
     <xacro:leg_gazebo prefix="rh" robot_name="$(arg robot_name)" load_force_sensors="$(arg load_force_sensors)"/>
-    <xacro:leg_hardware prefix="lh" imu_name="" imu_frame=""/>
+    <xacro:leg_hardware prefix="lh" with_ros2_control="false"/>
     <xacro:leg_gazebo prefix="lh" robot_name="$(arg robot_name)" load_force_sensors="$(arg load_force_sensors)"/>
 </robot>

File: husky_description/robots/husky.urdf.xacro (robot description, xacro)
@@ -22,5 +22,5 @@
     <!-- IMU sensor -->
     <xacro:imu_sensor
-        sensor_name="$(arg robot_name)_imu"
+        sensor_name="imu"
         frame_name="trunk_imu"
         imu_topic="trunk_imu/data"

File: sensors_description/urdfs/sensors/imu.gazebo.xacro (robot description, xacro)
@@ -4,8 +4,8 @@
         rate_bias_mean rate_bias_stddev accel_mean accel_stddev accel_bias_mean accel_bias_stddev">
       <xacro:if value="${namespace == ''}">
-                <xacro:property name="imu_topic_ns" value="${imu_topic}"/>
+                <xacro:property name="imu_topic_ns" value="${'/' + imu_topic}"/>
       </xacro:if>
       <xacro:if value="${namespace != ''}">
-                <xacro:property name="imu_topic_ns" value="${namespace+'/'+imu_topic}"/>
+                <xacro:property name="imu_topic_ns" value="${'/' + namespace + '/' + imu_topic}"/>
       </xacro:if>
         <gazebo reference="${frame_name}">

File: spot_description/robots/spot.urdf.xacro (robot description, xacro)
@@ -630,5 +630,5 @@
     <!-- IMU sensor -->
     <xacro:imu_sensor
-        sensor_name="$(arg robot_name)_imu"
+        sensor_name="imu"
         frame_name="trunk_imu"
         imu_topic="trunk_imu/data"
@@ -644,12 +644,14 @@
         accel_bias_stddev="0">
     </xacro:imu_sensor>
+    <!-- ROS2 control -->
+    <xacro:quadruped_ros2_control imu_name="imu" imu_frame="trunk_imu"/>
     <!-- Extensions -->
-    <xacro:leg_hardware prefix="rf" imu_name="$(arg robot_name)_imu" imu_frame="trunk_imu"/>
+    <xacro:leg_hardware prefix="rf" with_ros2_control="false"/>
     <xacro:leg_gazebo prefix="rf" robot_name="$(arg robot_name)" load_force_sensors="$(arg load_force_sensors)"/>
-    <xacro:leg_hardware prefix="lf" imu_name="" imu_frame=""/>
+    <xacro:leg_hardware prefix="lf" with_ros2_control="false"/>
     <xacro:leg_gazebo prefix="lf" robot_name="$(arg robot_name)" load_force_sensors="$(arg load_force_sensors)"/>
-    <xacro:leg_hardware prefix="rh" imu_name="" imu_frame=""/>
+    <xacro:leg_hardware prefix="rh" with_ros2_control="false"/>
     <xacro:leg_gazebo prefix="rh" robot_name="$(arg robot_name)" load_force_sensors="$(arg load_force_sensors)"/>
-    <xacro:leg_hardware prefix="lh" imu_name="" imu_frame=""/>
+    <xacro:leg_hardware prefix="lh" with_ros2_control="false"/>
     <xacro:leg_gazebo prefix="lh" robot_name="$(arg robot_name)" load_force_sensors="$(arg load_force_sensors)"/>
     <xacro:if value="$(eval arm_name != '')">

File: wolf_description_utils/urdfs/gazebo.urdf.xacro (robot description, xacro)
@@ -6,15 +6,22 @@
 <xacro:arg name="base_name"   default="base_link"/>
 <xacro:property name="model_name" value="$(arg robot_model)"/>
-	<gazebo>
-        <plugin name="ign_ros2_control::IgnitionROS2ControlPlugin" filename="libign_ros2_control-system.so">
-                <robot_param_node>robot_state_publisher</robot_param_node>
-                <ros>
-                        <namespace>/$(arg robot_name)</namespace>
-                        <!--<remapping>tf:=$(arg robot_name)/tf</remapping>-->
-                        <remapping>wolf_controller/odom:=odometry/robot</remapping>
-                        <remapping>diffdrive_controller/odom:=odometry/robot</remapping>
-                </ros>
+		<gazebo>
+		        <plugin name="gz_ros2_control::GazeboSimROS2ControlPlugin" filename="gz_ros2_control-system">
+		                <!-- Keep ros2_control URDF source consistent with the model actually spawned by go0 -->
+		                <robot_param>description</robot_param>
+		                <robot_param_node>gazebo_robot_description</robot_param_node>
+		                <ros>
+	                        <xacro:if value="$(eval robot_name != '')">
+	                                <namespace>/$(arg robot_name)</namespace>
+	                        </xacro:if>
+	                        <!--<remapping>tf:=$(arg robot_name)/tf</remapping>-->
+	                        <remapping>wolf_controller/odom:=odometry/robot</remapping>
+	                        <remapping>diffdrive_controller/odom:=odometry/robot</remapping>
+	                </ros>
                 <parameters>$(find ${model_name}_description)/params/${model_name}_params_$(arg robot_name).ros2.yaml</parameters>
         </plugin>
+        <!-- Gazebo Sim IMU system is required so IMU sensors expose topics/components
+             that gz_ros2_control can subscribe to and populate ros2_control IMU interfaces. -->
+        <plugin filename="ignition-gazebo-imu-system" name="gz::sim::systems::Imu"/>
 	</gazebo>
 </robot>

File: wolf_description_utils/urdfs/imu.hardware.xacro (robot description, xacro)
@@ -5,5 +5,5 @@
                 <ros2_control name="sim_hardware_system" type="system">
                     <hardware>
-                      <plugin>ign_ros2_control/IgnitionSystem</plugin>
+                      <plugin>gz_ros2_control/GazeboSimSystem</plugin>
                     </hardware>
                     <sensor name="${imu_name}">

File: wolf_description_utils/urdfs/leg.hardware.xacro (robot description, xacro)
@@ -1,5 +1,75 @@
 <?xml version="1.0"?>
 <robot xmlns:xacro="http://ros.org/wiki/xacro">
-        <xacro:macro name="leg_hardware" params="prefix imu_name:='' imu_frame:=''">
+        <xacro:macro name="leg_ros2_control_joints" params="prefix">
+                    <!-- Hip assembly -->
+                    <joint name="${prefix}_haa_joint">
+                      <command_interface name="effort">
+                        <param name="min">-500.0</param>
+                        <param name="max">500.0</param>
+                      </command_interface>
+                      <state_interface name="position">
+                        <param name="initial_value">0.0</param>
+                      </state_interface>
+                      <state_interface name="velocity">
+                        <param name="initial_value">0.0</param>
+                      </state_interface>
+                      <state_interface name="effort"/>
+                    </joint>
+                    <!-- Upper leg -->
+                    <joint name="${prefix}_hfe_joint">
+                      <command_interface name="effort">
+                        <param name="min">-500.0</param>
+                        <param name="max">500.0</param>
+                      </command_interface>
+                      <state_interface name="position">
+                        <param name="initial_value">0.0</param>
+                      </state_interface>
+                      <state_interface name="velocity">
+                        <param name="initial_value">0.0</param>
+                      </state_interface>
+                      <state_interface name="effort"/>
+                    </joint>
+                    <!-- Lower leg -->
+                    <joint name="${prefix}_kfe_joint">
+                      <command_interface name="effort">
+                        <param name="min">-500.0</param>
+                        <param name="max">500.0</param>
+                      </command_interface>
+                      <state_interface name="position">
+                        <param name="initial_value">0.0</param>
+                      </state_interface>
+                      <state_interface name="velocity">
+                        <param name="initial_value">0.0</param>
+                      </state_interface>
+                      <state_interface name="effort"/>
+                    </joint>
+        </xacro:macro>
+        <xacro:macro name="quadruped_ros2_control" params="imu_name:='' imu_frame:=''">
+                <ros2_control name="quadruped_system" type="system">
+                    <hardware>
+                      <plugin>gz_ros2_control/GazeboSimSystem</plugin>
+                    </hardware>
+                    <xacro:leg_ros2_control_joints prefix="rf"/>
+                    <xacro:leg_ros2_control_joints prefix="lf"/>
+                    <xacro:leg_ros2_control_joints prefix="rh"/>
+                    <xacro:leg_ros2_control_joints prefix="lh"/>
+                    <xacro:if value="${imu_name != ''}">
+                      <sensor name="${imu_name}" type="imu">
+                        <param name="frame_id">${imu_frame}</param>
+                        <state_interface name="orientation.x"/>
+                        <state_interface name="orientation.y"/>
+                        <state_interface name="orientation.z"/>
+                        <state_interface name="orientation.w"/>
+                        <state_interface name="angular_velocity.x"/>
+                        <state_interface name="angular_velocity.y"/>
+                        <state_interface name="angular_velocity.z"/>
+                        <state_interface name="linear_acceleration.x"/>
+                        <state_interface name="linear_acceleration.y"/>
+                        <state_interface name="linear_acceleration.z"/>
+                      </sensor>
+                    </xacro:if>
+                </ros2_control>
+        </xacro:macro>
+        <xacro:macro name="leg_hardware" params="prefix imu_name:='' imu_frame:='' with_ros2_control:='true'">
         <!-- ROS1 -->
     	<!-- Hip assembly -->
@@ -37,54 +107,27 @@
 		</transmission>
                 <!-- ROS2 -->
-                <ros2_control name="${prefix}_leg_system" type="system">
-                    <hardware>
-                      <plugin>ign_ros2_control/IgnitionSystem</plugin>
-                    </hardware>
-                    <!-- Hip assembly -->
-                    <joint name="${prefix}_haa_joint">
-                      <command_interface name="effort">
-                        <param name="min">-500.0</param>
-                        <param name="max">500.0</param>
-                      </command_interface>
-                      <state_interface name="position"/>
-                      <state_interface name="velocity"/>
-                      <state_interface name="effort"/>
-                    </joint>
-                    <!-- Upper leg -->
-                    <joint name="${prefix}_hfe_joint">
-                      <command_interface name="effort">
-                        <param name="min">-500.0</param>
-                        <param name="max">500.0</param>
-                      </command_interface>
-                      <state_interface name="position"/>
-                      <state_interface name="velocity"/>
-                      <state_interface name="effort"/>
-                    </joint>
-                    <!-- Lower leg -->
-                    <joint name="${prefix}_kfe_joint">
-                      <command_interface name="effort">
-                        <param name="min">-500.0</param>
-                        <param name="max">500.0</param>
-                      </command_interface>
-                      <state_interface name="position"/>
-                      <state_interface name="velocity"/>
-                      <state_interface name="effort"/>
-                    </joint>
-                    <xacro:if value="${imu_name != ''}">
-                      <sensor name="${imu_name}">
-                        <param name="frame_id">${imu_frame}</param>
-                        <state_interface name="orientation.x"/>
-                        <state_interface name="orientation.y"/>
-                        <state_interface name="orientation.z"/>
-                        <state_interface name="orientation.w"/>
-                        <state_interface name="angular_velocity.x"/>
-                        <state_interface name="angular_velocity.y"/>
-                        <state_interface name="angular_velocity.z"/>
-                        <state_interface name="linear_acceleration.x"/>
-                        <state_interface name="linear_acceleration.y"/>
-                        <state_interface name="linear_acceleration.z"/>
-                      </sensor>
-                    </xacro:if>
-            </ros2_control>
+                <xacro:if value="${str(with_ros2_control).lower() not in ['false', '0', 'no']}">
+                  <ros2_control name="${prefix}_leg_system" type="system">
+                      <hardware>
+                        <plugin>gz_ros2_control/GazeboSimSystem</plugin>
+                      </hardware>
+                      <xacro:leg_ros2_control_joints prefix="${prefix}"/>
+                      <xacro:if value="${imu_name != ''}">
+                        <sensor name="${imu_name}" type="imu">
+                          <param name="frame_id">${imu_frame}</param>
+                          <state_interface name="orientation.x"/>
+                          <state_interface name="orientation.y"/>
+                          <state_interface name="orientation.z"/>
+                          <state_interface name="orientation.w"/>
+                          <state_interface name="angular_velocity.x"/>
+                          <state_interface name="angular_velocity.y"/>
+                          <state_interface name="angular_velocity.z"/>
+                          <state_interface name="linear_acceleration.x"/>
+                          <state_interface name="linear_acceleration.y"/>
+                          <state_interface name="linear_acceleration.z"/>
+                        </sensor>
+                      </xacro:if>
+                  </ros2_control>
+                </xacro:if>
 	</xacro:macro>
 </robot>

File: wolf_description_utils/urdfs/wheels.hardware.xacro (robot description, xacro)
@@ -4,7 +4,7 @@
   <ros2_control name="wheels_system" type="system">
     <hardware>
-      <plugin>ign_ros2_control/IgnitionSystem</plugin>
+      <plugin>gz_ros2_control/GazeboSimSystem</plugin>
     </hardware>
-    <sensor name="$(arg robot_name)_imu">
+    <sensor name="imu">
       <param name="frame_id">trunk_imu</param>
       <state_interface name="orientation.x"/>
