Commit message: file -> package for meshes

File: go1_description/robots/go1.urdf.xacro (robot description, xacro)
@@ -37,5 +37,5 @@
             <origin rpy="0 0 0" xyz="0 0 0"/>
             <geometry>
-                <mesh filename="file://$(find go1_description)/meshes/trunk.dae" scale="1 1 1"/>
+                <mesh filename="package://go1_description/meshes/trunk.dae" scale="1 1 1"/>
             </geometry>
             <material name="orange"/>
@@ -50,5 +50,5 @@
             <origin rpy="0 0 0" xyz="0 0 0"/>
             <geometry>
-                <mesh filename="file://$(find go1_description)/meshes/trunk.dae" scale="1 1 1"/>
+                <mesh filename="package://go1_description/meshes/trunk.dae" scale="1 1 1"/>
             </geometry>
         </collision> -->

File: go1_description/urdfs/depthCamera.xacro (robot description, xacro)
@@ -17,5 +17,5 @@
             <origin xyz="0 0 0" rpy="0 0 0"/>
             <geometry>
-                <mesh filename="file://$(find go1_description)/meshes/depthCamera.dae" scale="1 1 1"/>
+                <mesh filename="package://go1_description/meshes/depthCamera.dae" scale="1 1 1"/>
             </geometry>
             </visual>

File: go1_description/urdfs/leg.xacro (robot description, xacro)
@@ -30,5 +30,5 @@
                 </xacro:if>
                 <geometry>
-                    <mesh filename="file://$(find go1_description)/meshes/hip.dae" scale="1 1 1"/>
+                    <mesh filename="package://go1_description/meshes/hip.dae" scale="1 1 1"/>
                 </geometry>
                 <!-- <material name="orange"/> -->
@@ -76,8 +76,8 @@
                 <geometry>
                     <xacro:if value="${mirror_dae == True}">
-                        <mesh filename="file://$(find go1_description)/meshes/thigh.dae" scale="1 1 1"/>
+                        <mesh filename="package://go1_description/meshes/thigh.dae" scale="1 1 1"/>
                     </xacro:if>
                     <xacro:if value="${mirror_dae == False}">
-                        <mesh filename="file://$(find go1_description)/meshes/thigh_mirror.dae" scale="1 1 1"/>
+                        <mesh filename="package://go1_description/meshes/thigh_mirror.dae" scale="1 1 1"/>
                     </xacro:if>
                 </geometry>
@@ -111,5 +111,5 @@
                 <origin rpy="0 0 0" xyz="0 0 0"/>
                 <geometry>
-                    <mesh filename="file://$(find go1_description)/meshes/calf.dae" scale="1 1 1"/>
+                    <mesh filename="package://go1_description/meshes/calf.dae" scale="1 1 1"/>
                 </geometry>
                 <!-- <material name="orange"/> -->

File: go1_description/urdfs/ultraSound.xacro (robot description, xacro)
@@ -17,5 +17,5 @@
             <origin xyz="0 0 0" rpy="0 0 0"/>
             <geometry>
-                <mesh filename="file://$(find go1_description)/meshes/ultraSound.dae" scale="1 1 1"/>
+                <mesh filename="package://go1_description/meshes/ultraSound.dae" scale="1 1 1"/>
             </geometry>
             <material name="black"/>

File: husky_description/urdfs/accessories/sensor_arch.urdf.xacro (robot description, xacro)
@@ -7,5 +7,5 @@
              <visual>
                  <geometry>
-                     <mesh filename="file://$(find husky_description)/meshes/accessories/${size}_mm_sensor_arch.dae" />
+                     <mesh filename="package://husky_description/meshes/accessories/${size}_mm_sensor_arch.dae" />
                  </geometry>
              </visual>
@@ -13,5 +13,5 @@
                  <origin xyz="0 0 0" rpy="0 0 0"/>
                  <geometry>
-                     <mesh filename="file://$(find husky_description)/meshes/accessories/${size}_mm_sensor_arch.dae" />
+                     <mesh filename="package://husky_description/meshes/accessories/${size}_mm_sensor_arch.dae" />
                  </geometry>
              </collision>

File: husky_description/urdfs/decorations.urdf.xacro (robot description, xacro)
@@ -18,5 +18,5 @@
         <origin xyz="0 0 0" rpy="0 0 0" />
         <geometry>
-          <mesh filename="file://$(find husky_description)/meshes/top_chassis.dae" />
+          <mesh filename="package://husky_description/meshes/top_chassis.dae" />
         </geometry>
       </visual>
@@ -32,5 +32,5 @@
         <visual>
           <geometry>
-            <mesh filename="file://$(find husky_description)/meshes/user_rail.dae" />
+            <mesh filename="package://husky_description/meshes/user_rail.dae" />
           </geometry>
         </visual>
@@ -47,5 +47,5 @@
       <visual>
         <geometry>
-          <mesh filename="file://$(find husky_description)/meshes/bumper.dae" />
+          <mesh filename="package://husky_description/meshes/bumper.dae" />
         </geometry>
       </visual>
@@ -61,5 +61,5 @@
           <visual>
               <geometry>
-                  <mesh filename="file://$(find husky_description)/meshes/bumper_extension.dae" />
+                  <mesh filename="package://husky_description/meshes/bumper_extension.dae" />
               </geometry>
           </visual>
@@ -75,5 +75,5 @@
       <visual>
         <geometry>
-          <mesh filename="file://$(find husky_description)/meshes/bumper.dae" />
+          <mesh filename="package://husky_description/meshes/bumper.dae" />
         </geometry>
       </visual>
@@ -89,5 +89,5 @@
           <visual>
               <geometry>
-                  <mesh filename="file://$(find husky_description)/meshes/bumper_extension.dae" />
+                  <mesh filename="package://husky_description/meshes/bumper_extension.dae" />
               </geometry>
           </visual>
@@ -106,5 +106,5 @@
             <origin xyz="0 0 0" rpy="0 0 0" />
             <geometry>
-              <mesh filename="file://$(find husky_description)/meshes/large_top_plate.dae" />
+              <mesh filename="package://husky_description/meshes/large_top_plate.dae" />
             </geometry>
           </visual>
@@ -112,5 +112,5 @@
             <origin xyz="0 0 0" rpy="0 0 0"/>
             <geometry>
-              <mesh filename="file://$(find husky_description)/meshes/large_top_plate_collision.stl" />
+              <mesh filename="package://husky_description/meshes/large_top_plate_collision.stl" />
             </geometry>
           </collision>
@@ -140,5 +140,5 @@
             <origin xyz="0 0 0" rpy="0 0 0" />
             <geometry>
-              <mesh filename="file://$(find husky_description)/meshes/top_plate.dae" />
+              <mesh filename="package://husky_description/meshes/top_plate.dae" />
             </geometry>
           </visual>
@@ -146,5 +146,5 @@
             <origin xyz="0 0 0" rpy="0 0 0"/>
             <geometry>
-              <mesh filename="file://$(find husky_description)/meshes/top_plate.stl" />
+              <mesh filename="package://husky_description/meshes/top_plate.stl" />
             </geometry>
           </collision>

File: husky_description/urdfs/husky_macro.urdf.xacro (robot description, xacro)
@@ -39,5 +39,5 @@
         <origin xyz="0 0 0" rpy="0 0 0" />
         <geometry>
-          <mesh filename="file://$(find husky_description)/meshes/base_link.dae" />
+          <mesh filename="package://husky_description/meshes/base_link.dae" />
         </geometry>
       </visual>
@@ -102,5 +102,5 @@
         <origin xyz="0 0 0" rpy="0 0 ${-M_PI/2}" />
         <geometry>
-          <mesh filename="file://$(find husky_description)/meshes/accessories/lms1xx_mount.dae" />
+          <mesh filename="package://husky_description/meshes/accessories/lms1xx_mount.dae" />
         </geometry>
       </visual>
@@ -121,5 +121,5 @@
       <visual>
         <geometry>
-          <mesh filename="file://$(find husky_description)/meshes/accessories/300_mm_sensor_arch.dae" />
+          <mesh filename="package://husky_description/meshes/accessories/300_mm_sensor_arch.dae" />
         </geometry>
       </visual>
@@ -127,5 +127,5 @@
         <origin xyz="0 0 0" rpy="0 0 0" />
         <geometry>
-          <mesh filename="file://$(find husky_description)/meshes/accessories/300_mm_sensor_arch.dae" />
+          <mesh filename="package://husky_description/meshes/accessories/300_mm_sensor_arch.dae" />
         </geometry>
       </collision>
@@ -139,5 +139,5 @@
       <visual>
         <geometry>
-          <mesh filename="file://$(find husky_description)/meshes/accessories/depth_camera.dae"/>
+          <mesh filename="package://husky_description/meshes/accessories/depth_camera.dae"/>
         </geometry>
       </visual>
@@ -156,10 +156,10 @@
       <visual>
         <geometry>
-          <mesh filename="file://$(find husky_description)/meshes/accessories/lidar.dae"/>
+          <mesh filename="package://husky_description/meshes/accessories/lidar.dae"/>
         </geometry>
       </visual>
       <collision>
         <geometry>
-          <mesh filename="file://$(find husky_description)/meshes/accessories/lidar_collision.stl"/>
+          <mesh filename="package://husky_description/meshes/accessories/lidar_collision.stl"/>
         </geometry>
       </collision>

File: sensors_description/urdfs/sensors/bumblebee.urdf.xacro (robot description, xacro)
@@ -19,5 +19,5 @@
 				<origin xyz="0 0 0.018" rpy="${PI/2} 0 ${PI/2}"/>
 				<geometry>
-					<mesh filename="file://$(find sensors_description)/meshes/sensors/bumblebee.dae"/>
+					<mesh filename="package://sensors_description/meshes/sensors/bumblebee.dae"/>
 				</geometry>
 			</visual>
@@ -25,5 +25,5 @@
 				<origin xyz="0 0 0.018" rpy="${PI/2} 0 ${PI/2}"/>
 				<geometry>
-					<mesh filename="file://$(find sensors_description)/meshes/sensors/bumblebee.dae"/>
+					<mesh filename="package://sensors_description/meshes/sensors/bumblebee.dae"/>
 				</geometry>
 			</collision>

File: sensors_description/urdfs/sensors/hokuyo_laser.urdf.xacro (robot description, xacro)
@@ -25,5 +25,5 @@
 				<origin xyz="0 0 0" rpy="0 0 0" />
 				<geometry>
-					<mesh filename="file://$(find sensors_description)/meshes/sensors/hokuyo.dae" scale="0.0254 0.0254 0.0254" />
+					<mesh filename="package://sensors_description/meshes/sensors/hokuyo.dae" scale="0.0254 0.0254 0.0254" />
 				</geometry>
 			</visual>

File: sensors_description/urdfs/sensors/kinect.urdf.xacro (robot description, xacro)
@@ -46,5 +46,5 @@
 				<origin xyz="0.0 0.0 0.0" rpy="0.0 0.0 0"/>
 				<geometry>
-					<mesh filename="file://$(find sensors_description)/meshes/sensors/kinect.dae" scale="1 1 1" />
+					<mesh filename="package://sensors_description/meshes/sensors/kinect.dae" scale="1 1 1" />
 				</geometry>
 				<material name="gray">
@@ -55,5 +55,5 @@
 				<origin xyz="0.0 0.0 0.0" rpy="0.0 0.0 0.0"/>
 				<geometry>
-					<mesh filename="file://$(find sensors_description)/meshes/sensors/kinect.dae" scale="1 1 1" />
+					<mesh filename="package://sensors_description/meshes/sensors/kinect.dae" scale="1 1 1" />
 				</geometry>
 			</collision>

File: sensors_description/urdfs/sensors/kvh_1775_imu.urdf.xacro (robot description, xacro)
@@ -115,5 +115,5 @@
 				<origin xyz="0.0 0.0 0.0" rpy="0 0 0"/>
 				<geometry>
-					<mesh filename="file://$(find sensors_description)/meshes/sensors/kvh_1775.dae" scale="1 1 1" />
+					<mesh filename="package://sensors_description/meshes/sensors/kvh_1775.dae" scale="1 1 1" />
 				</geometry>
 				<material name="aluminium">

File: sensors_description/urdfs/sensors/realsense_d435.urdf.xacro (robot description, xacro)
@@ -49,5 +49,5 @@
           <!-- <box size="${d435_cam_width} ${d435_cam_height} ${d435_cam_depth}"/> -->
 <!--          <mesh filename="package://realsense2_description/meshes/d435.dae" />-->
-          <mesh filename="file://$(find sensors_description)/meshes/sensors/realsense_d435.stl" />
+          <mesh filename="package://sensors_description/meshes/sensors/realsense_d435.stl" />
           <!--<mesh filename="package://realsense2_description/meshes/d435/d435.dae" />-->
         </geometry>

File: sensors_description/urdfs/sensors/realsense_d455.urdf.xacro (robot description, xacro)
@@ -53,5 +53,5 @@
       <origin xyz="${d455_zero_depth_to_glass + d455_glass_to_front} ${-d455_cam_depth_py} 0" rpy="${M_PI/2} 0 ${M_PI/2}"/>
         <geometry>
-          <mesh filename="file://$(find sensors_description)/meshes/sensors/realsense_d455.stl" scale="0.001 0.001 0.001" />
+          <mesh filename="package://sensors_description/meshes/sensors/realsense_d455.stl" scale="0.001 0.001 0.001" />
         </geometry>
         <material name="${name}_aluminum"/>

File: sensors_description/urdfs/sensors/realsense_t265.urdf.xacro (robot description, xacro)
@@ -90,5 +90,5 @@
             <origin rpy="1.57 0 1.57" xyz="0 0 0"/>
             <geometry>
-                <mesh filename="file://$(find sensors_description)/meshes/sensors/realsense_t265.stl" scale="0.001 0.001 0.001"/>
+                <mesh filename="package://sensors_description/meshes/sensors/realsense_t265.stl" scale="0.001 0.001 0.001"/>
             </geometry>
         </visual>

File: sensors_description/urdfs/sensors/velodyne.urdf.xacro (robot description, xacro)
@@ -27,5 +27,5 @@
 				<origin xyz="0 0 0" rpy="0 0 0"/>
 				<geometry>
-					<mesh filename="file://$(find sensors_description)/meshes/sensors/velodyne_hdl32e.dae" scale="1 1 1" />
+					<mesh filename="package://sensors_description/meshes/sensors/velodyne_hdl32e.dae" scale="1 1 1" />
 				</geometry>
 				<material name="gray">
@@ -36,5 +36,5 @@
 				<origin xyz="0 0 0" rpy="0 0 0"/>
 				<geometry>
-					<mesh filename="file://$(find sensors_description)/meshes/sensors/velodyne_hdl32e.dae" scale="1 1 1" />
+					<mesh filename="package://sensors_description/meshes/sensors/velodyne_hdl32e.dae" scale="1 1 1" />
 				</geometry>
 			</collision>

File: sensors_description/urdfs/sensors/vislab_3dve.urdf.xacro (robot description, xacro)
@@ -18,5 +18,5 @@
 				<origin xyz="0.018 0 0" rpy="${PI/2} 0 ${-PI/2}"/>
 				<geometry>
-					<mesh filename="file://$(find sensors_description)/meshes/sensors/vislab_3dve.stl"/>
+					<mesh filename="package://sensors_description/meshes/sensors/vislab_3dve.stl"/>
 				</geometry>
 			</visual>
@@ -24,5 +24,5 @@
 				<origin xyz="0.018 0 0" rpy="${PI/2} 0 ${-PI/2}"/>
 				<geometry>
-					<mesh filename="file://$(find sensors_description)/meshes/sensors/vislab_3dve.stl"/>
+					<mesh filename="package://sensors_description/meshes/sensors/vislab_3dve.stl"/>
 				</geometry>
 			</collision>

File: sensors_description/urdfs/sensors/zed_mini.urdf.xacro (robot description, xacro)
@@ -68,5 +68,5 @@
         <origin xyz="${screw_offset_x} 0 0" rpy="0 0 0"/>
         <geometry>
-          <mesh filename="file://$(find sensors_description)/meshes/sensors/zed_mini.stl" />
+          <mesh filename="package://sensors_description/meshes/sensors/zed_mini.stl" />
         </geometry>
         <!-- <material name="${model}_mat" /> -->
@@ -74,5 +74,5 @@
       <collision>
         <geometry>
-          <mesh filename="file://$(find sensors_description)/meshes/sensors/zed_mini.stl" />
+          <mesh filename="package://sensors_description/meshes/sensors/zed_mini.stl" />
         </geometry>
       </collision>
