Commit message: file -> package for meshes

File: spot_description/robots/spot.urdf.xacro (robot description, xacro)
@@ -100,10 +100,10 @@
         <visual>
             <geometry>
-                <mesh filename="file://$(find spot_description)/meshes/body.dae" />
-            </geometry>
-        </visual>
-        <!--<collision>
-            <geometry>
-                <mesh filename="file://$(find spot_description)/meshes/body_collision.stl" />
+                <mesh filename="package://spot_description/meshes/body.dae" />
+            </geometry>
+        </visual>
+        <!--<collision>
+            <geometry>
+                <mesh filename="package://spot_description/meshes/body_collision.stl" />
             </geometry>
         </collision>-->
@@ -138,10 +138,10 @@
         <visual>
             <geometry>
-                <mesh filename="file://$(find spot_description)/meshes/front_left_hip.dae" />
-            </geometry>
-        </visual>
-        <!--<collision>
-            <geometry>
-                <mesh filename="file://$(find spot_description)/meshes/front_left_hip_collision.stl" />
+                <mesh filename="package://spot_description/meshes/front_left_hip.dae" />
+            </geometry>
+        </visual>
+        <!--<collision>
+            <geometry>
+                <mesh filename="package://spot_description/meshes/front_left_hip_collision.stl" />
             </geometry>
         </collision>-->
@@ -165,10 +165,10 @@
         <visual>
             <geometry>
-                <mesh filename="file://$(find spot_description)/meshes/front_left_upper_leg.dae" />
-            </geometry>
-        </visual>
-        <!--<collision>
-            <geometry>
-                <mesh filename="file://$(find spot_description)/meshes/front_left_upper_leg_collision.stl" />
+                <mesh filename="package://spot_description/meshes/front_left_upper_leg.dae" />
+            </geometry>
+        </visual>
+        <!--<collision>
+            <geometry>
+                <mesh filename="package://spot_description/meshes/front_left_upper_leg_collision.stl" />
             </geometry>
         </collision>-->
@@ -198,10 +198,10 @@
         <visual>
             <geometry>
-                <mesh filename="file://$(find spot_description)/meshes/front_left_lower_leg.dae" />
-            </geometry>
-        </visual>
-        <!--<collision>
-            <geometry>
-                <mesh filename="file://$(find spot_description)/meshes/front_left_lower_leg_collision.stl" />
+                <mesh filename="package://spot_description/meshes/front_left_lower_leg.dae" />
+            </geometry>
+        </visual>
+        <!--<collision>
+            <geometry>
+                <mesh filename="package://spot_description/meshes/front_left_lower_leg_collision.stl" />
             </geometry>
         </collision>-->
@@ -260,10 +260,10 @@
         <visual>
             <geometry>
-                <mesh filename="file://$(find spot_description)/meshes/front_right_hip.dae" />
-            </geometry>
-        </visual>
-        <!--<collision>
-            <geometry>
-                <mesh filename="file://$(find spot_description)/meshes/front_right_hip_collision.stl" />
+                <mesh filename="package://spot_description/meshes/front_right_hip.dae" />
+            </geometry>
+        </visual>
+        <!--<collision>
+            <geometry>
+                <mesh filename="package://spot_description/meshes/front_right_hip_collision.stl" />
             </geometry>
         </collision>-->
@@ -287,10 +287,10 @@
         <visual>
             <geometry>
-                <mesh filename="file://$(find spot_description)/meshes/front_right_upper_leg.dae" />
-            </geometry>
-        </visual>
-        <!--<collision>
-            <geometry>
-                <mesh filename="file://$(find spot_description)/meshes/front_right_upper_leg_collision.stl" />
+                <mesh filename="package://spot_description/meshes/front_right_upper_leg.dae" />
+            </geometry>
+        </visual>
+        <!--<collision>
+            <geometry>
+                <mesh filename="package://spot_description/meshes/front_right_upper_leg_collision.stl" />
             </geometry>
         </collision>-->
@@ -320,10 +320,10 @@
         <visual>
             <geometry>
-                <mesh filename="file://$(find spot_description)/meshes/front_right_lower_leg.dae" />
-            </geometry>
-        </visual>
-        <!--<collision>
-            <geometry>
-                <mesh filename="file://$(find spot_description)/meshes/front_right_lower_leg_collision.stl" />
+                <mesh filename="package://spot_description/meshes/front_right_lower_leg.dae" />
+            </geometry>
+        </visual>
+        <!--<collision>
+            <geometry>
+                <mesh filename="package://spot_description/meshes/front_right_lower_leg_collision.stl" />
             </geometry>
         </collision>-->
@@ -382,10 +382,10 @@
         <visual>
             <geometry>
-                <mesh filename="file://$(find spot_description)/meshes/rear_left_hip.dae" />
-            </geometry>
-        </visual>
-        <!--<collision>
-            <geometry>
-                <mesh filename="file://$(find spot_description)/meshes/rear_left_hip_collision.stl" />
+                <mesh filename="package://spot_description/meshes/rear_left_hip.dae" />
+            </geometry>
+        </visual>
+        <!--<collision>
+            <geometry>
+                <mesh filename="package://spot_description/meshes/rear_left_hip_collision.stl" />
             </geometry>
         </collision>-->
@@ -409,10 +409,10 @@
         <visual>
             <geometry>
-                <mesh filename="file://$(find spot_description)/meshes/rear_left_upper_leg.dae" />
-            </geometry>
-        </visual>
-        <!--<collision>
-            <geometry>
-                <mesh filename="file://$(find spot_description)/meshes/rear_left_upper_leg_collision.stl" />
+                <mesh filename="package://spot_description/meshes/rear_left_upper_leg.dae" />
+            </geometry>
+        </visual>
+        <!--<collision>
+            <geometry>
+                <mesh filename="package://spot_description/meshes/rear_left_upper_leg_collision.stl" />
             </geometry>
         </collision>-->
@@ -442,10 +442,10 @@
         <visual>
             <geometry>
-                <mesh filename="file://$(find spot_description)/meshes/rear_left_lower_leg.dae" />
-            </geometry>
-        </visual>
-        <!--<collision>
-            <geometry>
-                <mesh filename="file://$(find spot_description)/meshes/rear_left_lower_leg_collision.stl" />
+                <mesh filename="package://spot_description/meshes/rear_left_lower_leg.dae" />
+            </geometry>
+        </visual>
+        <!--<collision>
+            <geometry>
+                <mesh filename="package://spot_description/meshes/rear_left_lower_leg_collision.stl" />
             </geometry>
         </collision>-->
@@ -504,10 +504,10 @@
         <visual>
             <geometry>
-                <mesh filename="file://$(find spot_description)/meshes/rear_right_hip.dae" />
-            </geometry>
-        </visual>
-        <!--<collision>
-            <geometry>
-                <mesh filename="file://$(find spot_description)/meshes/rear_right_hip_collision.stl" />
+                <mesh filename="package://spot_description/meshes/rear_right_hip.dae" />
+            </geometry>
+        </visual>
+        <!--<collision>
+            <geometry>
+                <mesh filename="package://spot_description/meshes/rear_right_hip_collision.stl" />
             </geometry>
         </collision>-->
@@ -531,10 +531,10 @@
         <visual>
             <geometry>
-                <mesh filename="file://$(find spot_description)/meshes/rear_right_upper_leg.dae" />
-            </geometry>
-        </visual>
-        <!--<collision>
-            <geometry>
-                <mesh filename="file://$(find spot_description)/meshes/rear_right_upper_leg_collision.stl" />
+                <mesh filename="package://spot_description/meshes/rear_right_upper_leg.dae" />
+            </geometry>
+        </visual>
+        <!--<collision>
+            <geometry>
+                <mesh filename="package://spot_description/meshes/rear_right_upper_leg_collision.stl" />
             </geometry>
         </collision>-->
@@ -564,10 +564,10 @@
         <visual>
             <geometry>
-                <mesh filename="file://$(find spot_description)/meshes/rear_right_lower_leg.dae" />
-            </geometry>
-        </visual>
-        <!--<collision>
-            <geometry>
-                <mesh filename="file://$(find spot_description)/meshes/rear_right_lower_leg_collision.stl" />
+                <mesh filename="package://spot_description/meshes/rear_right_lower_leg.dae" />
+            </geometry>
+        </visual>
+        <!--<collision>
+            <geometry>
+                <mesh filename="package://spot_description/meshes/rear_right_lower_leg_collision.stl" />
             </geometry>
         </collision>-->

File: spot_description/urdfs/accessories.urdf.xacro (robot description, xacro)
@@ -19,15 +19,15 @@
       <visual>
         <geometry>
-          <mesh filename="file://$(find spot_description)/meshes/pack_top.dae"/>
+          <mesh filename="package://spot_description/meshes/pack_top.dae"/>
         </geometry>
       </visual>
       <visual>
         <geometry>
-          <mesh filename="file://$(find spot_description)/meshes/pack_body.dae"/>
+          <mesh filename="package://spot_description/meshes/pack_body.dae"/>
         </geometry>
       </visual>
       <collision>
         <geometry>
-          <mesh filename="file://$(find spot_description)/meshes/pack_body.dae"/>
+          <mesh filename="package://spot_description/meshes/pack_body.dae"/>
         </geometry>
       </collision>
@@ -44,10 +44,10 @@
       <visual>
         <geometry>
-          <mesh filename="file://$(find spot_description)/meshes/lidar_mount.dae"/>
+          <mesh filename="package://spot_description/meshes/lidar_mount.dae"/>
         </geometry>
       </visual>
       <collision>
         <geometry>
-          <mesh filename="file://$(find spot_description)/meshes/lidar_mount_collision.stl"/>
+          <mesh filename="package://spot_description/meshes/lidar_mount_collision.stl"/>
         </geometry>
       </collision>
@@ -63,10 +63,10 @@
         <visual>
           <geometry>
-            <mesh filename="file://$(find spot_description)/meshes/velo.dae"/>
+            <mesh filename="package://spot_description/meshes/velo.dae"/>
           </geometry>
         </visual>
         <collision>
           <geometry>
-            <mesh filename="file://$(find spot_description)/meshes/velo_collision.stl"/>
+            <mesh filename="package://spot_description/meshes/velo_collision.stl"/>
           </geometry>
         </collision>

Commit message: Make it work with jazzy

File: go1_description/robots/go1.urdf.xacro (robot description, xacro)
@@ -10,5 +10,5 @@
     <xacro:arg name="robot_name"         default=""/>
     <xacro:arg name="base_name"          default="base_link"/>
-    <xacro:arg name="simulator"          default="ignition"/>
+    <xacro:arg name="simulator"          default="gz"/>
     <!-- load generic materials -->
     <xacro:include filename="$(find wolf_description_utils)/urdfs/materials.xacro"/>

File: go1_description/urdfs/accessories.urdf.xacro (robot description, xacro)
@@ -1,5 +1,5 @@
 <?xml version="1.0"?>
 <robot xmlns:xacro="http://www.ros.org/wiki/xacro">
-  <xacro:arg name="simulator" default="ignition"/>
+  <xacro:arg name="simulator" default="gz"/>
   <xacro:include filename="$(find sensors_description)/urdfs/common.xacro"/>
   <xacro:include filename="$(find sensors_description)/urdfs/sensors/depth_camera.gazebo.xacro"/>

File: husky_description/robots/husky.urdf.xacro (robot description, xacro)
@@ -9,5 +9,5 @@
   <xacro:arg name="robot_name"         default=""/>
   <xacro:arg name="base_name"          default="base_link"/>
-  <xacro:arg name="simulator"          default="ignition"/>
+  <xacro:arg name="simulator"          default="gz"/>
   <!-- generic simulator_gazebo plugins for starting mechanism control, ros time -->
   <xacro:include filename="$(find wolf_description_utils)/urdfs/gazebo.urdf.xacro"/>

File: husky_description/urdfs/accessories.urdf.xacro (robot description, xacro)
@@ -1,5 +1,5 @@
 <?xml version="1.0"?>
 <robot xmlns:xacro="http://www.ros.org/wiki/xacro">
-  <xacro:arg name="simulator" default="ignition"/>
+  <xacro:arg name="simulator" default="gz"/>
   <xacro:include filename="$(find sensors_description)/urdfs/common.xacro"/>
   <xacro:include filename="$(find sensors_description)/urdfs/sensors/depth_camera.gazebo.xacro"/>

File: spot_description/robots/spot.urdf.xacro (robot description, xacro)
@@ -10,5 +10,5 @@
     <xacro:arg name="robot_name"         default=""/>
     <xacro:arg name="base_name"          default="base_link"/>
-    <xacro:arg name="simulator"          default="ignition"/>
+    <xacro:arg name="simulator"          default="gz"/>
     <!-- load generic materials -->
     <xacro:include filename="$(find wolf_description_utils)/urdfs/materials.xacro"/>

File: spot_description/urdfs/accessories.urdf.xacro (robot description, xacro)
@@ -1,5 +1,5 @@
 <?xml version="1.0"?>
 <robot xmlns:xacro="http://www.ros.org/wiki/xacro">
-  <xacro:arg name="simulator" default="ignition"/>
+  <xacro:arg name="simulator" default="gz"/>
   <xacro:include filename="$(find sensors_description)/urdfs/common.xacro"/>
   <xacro:include filename="$(find sensors_description)/urdfs/sensors/depth_camera.gazebo.xacro"/>

File: wolf_description_utils/urdfs/gazebo.urdf.xacro (robot description, xacro)
@@ -6,6 +6,14 @@
 <xacro:arg name="base_name"   default="base_link"/>
 <xacro:arg name="sensors"     default="false"/>
+<xacro:arg name="simulator"   default="gz"/>
 <xacro:arg name="load_global_gazebo_systems" default="true"/>
+<xacro:arg name="controller_params_file" default="$(find $(arg robot_model)_description)/params/$(arg robot_model)_params.ros2.yaml"/>
 <xacro:property name="model_name" value="$(arg robot_model)"/>
+<xacro:property name="imu_plugin_filename" value="gz-sim-imu-system"/>
+<xacro:property name="imu_plugin_name" value="gz::sim::systems::Imu"/>
+<xacro:property name="sensors_plugin_filename" value="gz-sim-sensors-system"/>
+<xacro:property name="sensors_plugin_name" value="gz::sim::systems::Sensors"/>
+<xacro:property name="navsat_plugin_filename" value="gz-sim-navsat-system"/>
+<xacro:property name="navsat_plugin_name" value="gz::sim::systems::NavSat"/>
 		<gazebo>
 		        <plugin name="gz_ros2_control::GazeboSimROS2ControlPlugin" filename="gz_ros2_control-system">
@@ -21,15 +29,15 @@
 	                        <remapping>diffdrive_controller/odom:=odometry/robot</remapping>
 	                </ros>
-                <parameters>$(find ${model_name}_description)/params/${model_name}_params_$(arg robot_name).ros2.yaml</parameters>
+                <parameters>$(arg controller_params_file)</parameters>
         </plugin>
         <xacro:if value="$(arg load_global_gazebo_systems)">
                 <!-- Gazebo Sim sensor systems are global to the running world.
                      Loading them once avoids multi-robot duplicate visual/rendering crashes. -->
-                <plugin filename="ignition-gazebo-imu-system" name="gz::sim::systems::Imu"/>
+                <plugin filename="${imu_plugin_filename}" name="${imu_plugin_name}"/>
                 <xacro:if value="$(arg sensors)">
-                        <plugin filename="ignition-gazebo-sensors-system" name="gz::sim::systems::Sensors">
+                        <plugin filename="${sensors_plugin_filename}" name="${sensors_plugin_name}">
                                 <render_engine>ogre2</render_engine>
                         </plugin>
-                        <plugin filename="ignition-gazebo-navsat-system" name="ignition::gazebo::systems::NavSat"/>
+                        <plugin filename="${navsat_plugin_filename}" name="${navsat_plugin_name}"/>
                 </xacro:if>
         </xacro:if>
