Commit message: Update go1 navigation params and description

File: go1_description/urdfs/accessories.urdf.xacro (robot description, xacro)
@@ -2,8 +2,8 @@
 <robot xmlns:xacro="http://www.ros.org/wiki/xacro">
   <xacro:include filename="$(find sensors_description)/urdfs/common.xacro"/>
-  <!--<xacro:include filename="$(find sensors_description)/urdfs/sensors/velodyne.gazebo.xacro"/>-->
+  <xacro:include filename="$(find go1_description)/urdfs/ultraSound.xacro"/>
+  <xacro:include filename="$(find go1_description)/urdfs/depthCamera.xacro"/>
   <xacro:include filename="$(find velodyne_description)/urdf/VLP-16.urdf.xacro"/>
-  <xacro:include filename="$(find sensors_description)/urdfs/sensors/realsense_d435.urdf.xacro" />
-  <xacro:include filename="$(find sensors_description)/urdfs/sensors/realsense_t265.xacro" />
+  <xacro:include filename="$(find sensors_description)/urdfs/sensors/realsense_t265.xacro"/>
   <xacro:depthCamera camID="1" name="face">
       <origin rpy="${PI} 0 0" xyz="0.2785 0.0125 0.0167"/>
@@ -44,3 +44,22 @@
       <origin rpy="0 0 0" xyz="0.2747 0.0 -0.0088"/>
   </xacro:ultraSound>
+  <xacro:realsense_T265 sensor_name="t265" parent_link="trunk" rate="30.0">
+    <origin xyz="0.3 0 0.05" rpy="0 0.24 0" />
+  </xacro:realsense_T265>
+  <joint name="lidar_cage_to_lidar" type="fixed">
+      <parent link="trunk"/>
+      <child link="lidar"/>
+      <origin rpy="0.0 0.0 0.0" xyz="0.0 0.0 0.05"/>
+  </joint>
+  <link name="lidar">
+      <inertial>
+          <origin rpy="0.0 0.0 0.0" xyz="-0.012 0.001 -0.008"/>
+          <mass value="0.695"/>
+          <inertia ixx="0.000846765" ixy="6.9565e-05" ixz="0.00027111" iyy="0.001367583" iyz="5.8984e-05" izz="0.001363673"/>
+      </inertial>
+  </link>
+  <xacro:VLP-16 parent="lidar" name="velodyne" topic="/velodyne_points"
+                organize_cloud="true" hz="10" gpu="true">
+    <origin xyz="0 0 0" rpy="0 0 0" />
+  </xacro:VLP-16>
 </robot>

File: go1_description/urdfs/depthCamera.xacro (robot description, xacro)
@@ -17,5 +17,5 @@
             <origin xyz="0 0 0" rpy="0 0 0"/>
             <geometry>
-                <mesh filename="file://$$(find go1_description)/meshes/depthCamera.dae" scale="1 1 1"/>
+                <mesh filename="package://go1_description/meshes/depthCamera.dae" scale="1 1 1"/>
             </geometry>
             </visual>
@@ -59,5 +59,5 @@
                     <depthImageInfoTopicName>/camera_${name}/depth/camera_info</depthImageInfoTopicName>
                     <!-- <pointCloudTopicName>/camera_${name}/depth/points</pointCloudTopicName> -->
-                    <pointCloudTopicName>/cam${camID}/point_cloud_${name}</pointCloudTopicName>
+                    <pointCloudTopicName>/camera${camID}/point_cloud_${name}</pointCloudTopicName>
                     <frameName>camera_optical_${name}</frameName>
                     <pointCloudCutoff>0.1</pointCloudCutoff>

Commit message: Some modifications to have compatibility with go1

File: go1_description/urdfs/accessories.urdf.xacro (robot description, xacro)
@@ -49,8 +49,8 @@
   <joint name="lidar_cage_to_lidar" type="fixed">
       <parent link="trunk"/>
-      <child link="lidar"/>
+      <child link="rslidar"/>
       <origin rpy="0.0 0.0 0.0" xyz="0.0 0.0 0.05"/>
   </joint>
-  <link name="lidar">
+  <link name="rslidar">
       <inertial>
           <origin rpy="0.0 0.0 0.0" xyz="-0.012 0.001 -0.008"/>
@@ -59,5 +59,5 @@
       </inertial>
   </link>
-  <xacro:VLP-16 parent="lidar" name="velodyne" topic="/velodyne_points"
+  <xacro:VLP-16 parent="rslidar" name="rslidar-16" topic="/rslidar_points"
                 organize_cloud="true" hz="10" gpu="true">
     <origin xyz="0 0 0" rpy="0 0 0" />

Commit message: added realsense

File: go1_description/urdfs/accessories.urdf.xacro (robot description, xacro)
@@ -8,5 +8,9 @@
   <xacro:include filename="$(find sensors_description)/urdfs/sensors/imu.gazebo.xacro"/>
   <xacro:include filename="$(find sensors_description)/urdfs/sensors/gps.gazebo.xacro"/>
+  <xacro:include filename="$(find sensors_description)/urdfs/sensors/realsense_d435.urdf.xacro" />
 <!-- Comment out to save computational power -->
+  <xacro:realsense_d435 name="d435" topics_ns="/camera" parent="trunk">
+	<origin xyz="0.25 0 0.08" rpy="0 0.3 0" />
+  </xacro:realsense_d435>
   <xacro:depthCamera camID="1" name="face">
       <origin rpy="${PI} 0 0" xyz="0.2785 0.0125 0.0167"/>
@@ -47,7 +51,7 @@
       <origin rpy="0 0 0" xyz="0.2747 0.0 -0.0088"/>
   </xacro:ultraSound>
-  <xacro:realsense_T265 name="t265" topics_ns="/$(arg robot_name)" parent="trunk" rate="30.0">
+  <!--xacro:realsense_T265 name="t265" topics_ns="/$(arg robot_name)" parent="trunk" rate="30.0">
     <origin xyz="0.3 0 0.05" rpy="0 0.24 0" />
-  </xacro:realsense_T265>
+  </xacro:realsense_T265-->
   <xacro:VLP-16 parent="rslidar" name="rslidar-16" topic="/$(arg robot_name)/lidar_points"
                 organize_cloud="true" hz="10" gpu="true">

Commit message: updated realsense position

File: go1_description/urdfs/accessories.urdf.xacro (robot description, xacro)
@@ -11,5 +11,5 @@
 <!-- Comment out to save computational power -->
   <xacro:realsense_d435 name="d435" topics_ns="/camera" parent="trunk">
-	<origin xyz="0.25 0 0.08" rpy="0 0.3 0" />
+	<origin xyz="0.04 0 0.15" rpy="0 0.3 0" />
   </xacro:realsense_d435>
   <xacro:depthCamera camID="1" name="face">

Commit message: Add t265

File: go1_description/urdfs/accessories.urdf.xacro (robot description, xacro)
@@ -9,7 +9,7 @@
   <xacro:include filename="$(find sensors_description)/urdfs/sensors/gps.gazebo.xacro"/>
   <xacro:include filename="$(find sensors_description)/urdfs/sensors/realsense_d435.urdf.xacro" />
-<!-- Comment out to save computational power -->
-  <xacro:realsense_d435 name="d435" topics_ns="/camera" parent="trunk">
-	<origin xyz="0.04 0 0.15" rpy="0 0.3 0" />
+  <!-- Comment out to save computational power -->
+  <xacro:realsense_d435 name="d435" topics_ns="/$(arg robot_name)/d435" parent="trunk">
+      <origin xyz="0.04 0 0.15" rpy="0 0.3 0" />
   </xacro:realsense_d435>
   <xacro:depthCamera camID="1" name="face">
@@ -51,7 +51,7 @@
       <origin rpy="0 0 0" xyz="0.2747 0.0 -0.0088"/>
   </xacro:ultraSound>
-  <!--xacro:realsense_T265 name="t265" topics_ns="/$(arg robot_name)" parent="trunk" rate="30.0">
+  <xacro:realsense_T265 name="t265" topics_ns="/$(arg robot_name)" parent="trunk" rate="30.0">
     <origin xyz="0.3 0 0.05" rpy="0 0.24 0" />
-  </xacro:realsense_T265-->
+  </xacro:realsense_T265>
   <xacro:VLP-16 parent="rslidar" name="rslidar-16" topic="/$(arg robot_name)/lidar_points"
                 organize_cloud="true" hz="10" gpu="true">

Commit message: alligned camera and lidar with eagle

File: go1_description/urdfs/accessories.urdf.xacro (robot description, xacro)
@@ -11,5 +11,5 @@
   <!-- Comment out to save computational power -->
   <xacro:realsense_d435 name="d435" topics_ns="/$(arg robot_name)/d435" parent="trunk">
-      <origin xyz="0.04 0 0.15" rpy="0 0.3 0" />
+      <origin xyz="0.14 0 0.15" rpy="0 0.3 0" />
   </xacro:realsense_d435>
   <xacro:depthCamera camID="1" name="face">
@@ -56,5 +56,5 @@
   <xacro:VLP-16 parent="rslidar" name="rslidar-16" topic="/$(arg robot_name)/lidar_points"
                 organize_cloud="true" hz="10" gpu="true">
-    <origin xyz="0 0 0" rpy="0 0 0" />
+    <origin xyz="0.1 0 0" rpy="0 0 0" />
   </xacro:VLP-16>
   <!-- IMU sensor -->

Commit message: Update go1
still not working!

File: go1_description/urdfs/accessories.urdf.xacro (robot description, xacro)
@@ -2,68 +2,44 @@
 <robot xmlns:xacro="http://www.ros.org/wiki/xacro">
   <xacro:include filename="$(find sensors_description)/urdfs/common.xacro"/>
-  <xacro:include filename="$(find go1_description)/urdfs/ultraSound.xacro"/>
-  <xacro:include filename="$(find go1_description)/urdfs/depthCamera.xacro"/>
-  <xacro:include filename="$(find velodyne_description)/urdf/VLP-16.urdf.xacro"/>
-  <xacro:include filename="$(find sensors_description)/urdfs/sensors/realsense_t265.urdf.xacro"/>
+  <xacro:include filename="$(find sensors_description)/urdfs/sensors/depth_camera.gazebo.xacro"/>
   <xacro:include filename="$(find sensors_description)/urdfs/sensors/gps.gazebo.xacro"/>
-  <xacro:include filename="$(find sensors_description)/urdfs/sensors/realsense_d435.urdf.xacro" />
-  <xacro:realsense_d435 name="camera" topics_ns="/$(arg robot_name)/camera" parent="base_link">
-      <origin xyz="0.14 0 0.15" rpy="0 0.3 0" />
-  </xacro:realsense_d435>
- <!-- Comment out to save computational power -->
- <!--
-  <xacro:depthCamera camID="1" name="face">
-      <origin rpy="${PI} 0 0" xyz="0.2785 0.0125 0.0167"/>
-  </xacro:depthCamera>
-  <xacro:depthCamera camID="2" name="chin">
-      <origin rpy="${PI} ${PI/2} 0" xyz="0.2522 0.0125 -0.0436"/>
-  </xacro:depthCamera>
-  <xacro:depthCamera camID="3" name="left">
-      <origin rpy="${PI} 0.2618 ${PI/2}" xyz="-0.066 0.082 -0.0176"/>
-  </xacro:depthCamera>
-  <xacro:depthCamera camID="4" name="right">
-      <origin rpy="${PI} 0.2618 ${-PI/2}" xyz="-0.041 -0.082 -0.0176"/>
-  </xacro:depthCamera>
-  <xacro:depthCamera camID="5" name="rearDown">
-      <origin rpy="${PI} ${PI/2} 0" xyz="-0.0825 0.0125 -0.04365"/>
-  </xacro:depthCamera>
-  <joint name="camera_laserscan_joint_left" type="fixed">
-      <origin rpy="0 0.2618 0" xyz="0 0 0"/>
-      <parent link="camera_left"/>
-      <child link="camera_laserscan_link_left"/>
-  </joint>
-  <link name="camera_laserscan_link_left">
-  </link>
-  <joint name="camera_laserscan_joint_right" type="fixed">
-      <origin rpy="0 0.2618 0" xyz="0 0 0"/>
-      <parent link="camera_right"/>
-      <child link="camera_laserscan_link_right"/>
-  </joint>
-  <link name="camera_laserscan_link_right">
-  </link>
-  <xacro:ultraSound name="left">
-      <origin rpy="0 0.2618 ${PI/2}" xyz="-0.0535  0.0826 0.00868"/>
-  </xacro:ultraSound>
-  <xacro:ultraSound name="right">
-      <origin rpy="0 0.2618 ${-PI/2}" xyz="-0.0535 -0.0826 0.00868"/>
-  </xacro:ultraSound>
-  <xacro:ultraSound name="face">
-      <origin rpy="0 0 0" xyz="0.2747 0.0 -0.0088"/>
-  </xacro:ultraSound>
-   -->
-  <xacro:realsense_T265 name="t265" topics_ns="/$(arg robot_name)" parent="base_link" rate="30.0">
-    <origin xyz="0.3 0 0.05" rpy="0 0.24 0" />
-  </xacro:realsense_T265>
-  <xacro:VLP-16 parent="lidar_mount" name="rslidar" topic="/$(arg robot_name)/lidar_points"
-                organize_cloud="true" hz="10" gpu="true">
-    <origin xyz="0.1 0 0" rpy="0 0 0" />
-  </xacro:VLP-16>
+  <xacro:include filename="$(find sensors_description)/urdfs/sensors/lidar.gazebo.xacro"/>
+   <xacro:depth_camera
+     name="camera"
+     namespace="$(arg robot_name)"
+     update_rate="30"
+     image_width="640"
+     image_height="480"
+     fov="1.047"
+     near="0.1"
+     far="10.0"
+     parent_link="base_link"
+     image_topic="$(arg robot_name)/camera/rgb/image_raw"
+     depth_topic="$(arg robot_name)/camera/depth/image_raw"
+     pointcloud_topic="$(arg robot_name)/camera/points"
+     camera_info_topic="$(arg robot_name)/camera/camera_info"
+     origin_xyz="0.14 0 0.15"
+     origin_rpy="0 0.3 0"/>
+  <xacro:velodyne_laser_gazebo_sensor
+    sensor_name="lidar"
+    topic_name="lidar_points"
+    update_rate="10.0"
+    frame_id="lidar_mount"
+    namespace="$(arg robot_name)"
+    min_range="0.9"
+    max_range="130.0"
+    number_of_beams="32"
+    horizontal_samples="220"
+    horizontal_fov="6.28319"
+    vertical_fov="0.2618"
+    noise_stddev="0.01"/>
+    <!--<origin xyz="0.1 0 0" rpy="0 0 0" />-->
   <!-- GPS sensor -->
-  <xacro:gps_sensor
-      gps_topic="fix"
-      vel_topic="velocity_fix"
-      namespace="$(arg robot_name)"
-      frame_name="base_link"
-      update_rate="10.0">
-  </xacro:gps_sensor>
+  <xacro:gazebo_gps_sensor
+    sensor_name="gps_sensor"
+    namespace="$(arg robot_name)"
+    gps_topic="gps/fix"
+    velocity_topic="gps/velocity_fix"
+    update_rate="10.0"
+    frame_id="base_link" />
 </robot>
