Commit message: Use kinect depth

File: go1_description/urdfs/accessories.urdf.xacro (robot description, xacro)
@@ -7,10 +7,7 @@
   <xacro:include filename="$(find sensors_description)/urdfs/sensors/realsense_t265.urdf.xacro"/>
   <xacro:include filename="$(find sensors_description)/urdfs/sensors/gps.gazebo.xacro"/>
-  <xacro:include filename="$(find sensors_description)/urdfs/sensors/realsense_d435.urdf.xacro" />
-  <xacro:realsense_d435 name="camera" topics_ns="/$(arg robot_name)/camera" parent="base_link">
-      <origin xyz="0.14 0 0.15" rpy="0 0.3 0" />
-  </xacro:realsense_d435>
- <!-- Comment out to save computational power -->
- <!--
+  <xacro:include filename="$(find sensors_description)/urdfs/sensors/kinect.gazebo.xacro"/>
+  <!-- Optional Go1 depth cameras / ultrasounds (currently commented) -->
+  <!--
   <xacro:depthCamera camID="1" name="face">
       <origin rpy="${PI} 0 0" xyz="0.2785 0.0125 0.0167"/>
@@ -51,12 +48,45 @@
       <origin rpy="0 0 0" xyz="0.2747 0.0 -0.0088"/>
   </xacro:ultraSound>
-   -->
+  -->
+  <!-- T265 tracking camera -->
   <xacro:realsense_T265 name="t265" topics_ns="/$(arg robot_name)" parent="base_link" rate="30.0">
     <origin xyz="0.3 0 0.05" rpy="0 0.24 0" />
   </xacro:realsense_T265>
+  <!-- Velodyne lidar on lidar_mount (from main URDF) -->
   <xacro:VLP-16 parent="lidar_mount" name="rslidar" topic="/$(arg robot_name)/lidar_points"
                 organize_cloud="true" hz="10" gpu="true">
     <origin xyz="0.1 0 0" rpy="0 0 0" />
   </xacro:VLP-16>
+  <!-- Kinect-style RGBD camera with explicit optical frame -->
+  <!-- Base camera link attached to base_link -->
+  <link name="kinect_camera_link"/>
+  <joint name="kinect_camera_mount_joint" type="fixed">
+    <parent link="base_link"/>
+    <!-- Pose of Kinect relative to robot body (tune as you like) -->
+    <origin xyz="0.14 0 0.15" rpy="0 0.3 0"/>
+    <child link="kinect_camera_link"/>
+  </joint>
+  <!-- Optical frame: REP-103 camera convention (z forward, x right, y down) -->
+  <link name="kinect_camera_optical_frame"/>
+  <joint name="kinect_camera_optical_joint" type="fixed">
+    <parent link="kinect_camera_link"/>
+    <!-- rotation from x-forward, z-up to z-forward, x-right, y-down -->
+    <origin xyz="0 0 0" rpy="-1.5707963 0 -1.5707963"/>
+    <child link="kinect_camera_optical_frame"/>
+  </joint>
+  <!-- Kinect RGB(+depth) sensor using our fixed macro -->
+  <xacro:kinect_rgb_sensor
+    link_name="kinect_camera_link"
+    frame_name="kinect_camera_optical_frame"
+    camera_name="camera">
+  </xacro:kinect_rgb_sensor>
+  <!-- Optional IR variant, aligned identically -->
+  <!--
+  <xacro:kinect_ir_sensor
+    link_name="kinect_camera_link"
+    frame_name="kinect_camera_optical_frame"
+    camera_name="/$(arg robot_name)/kinect">
+  </xacro:kinect_ir_sensor>
+  -->
   <!-- GPS sensor -->
   <xacro:gps_sensor

File: husky_description/robots/husky.urdf.xacro (robot description, xacro)
@@ -16,28 +16,59 @@
   <xacro:include filename="$(find velodyne_description)/urdf/VLP-16.urdf.xacro"/>
   <xacro:include filename="$(find sensors_description)/urdfs/sensors/gps.gazebo.xacro"/>
+  <xacro:include filename="$(find sensors_description)/urdfs/sensors/kinect.gazebo.xacro"/>
   <xacro:include filename="$(find husky_description)/urdfs/husky_macro.urdf.xacro" />
   <xacro:husky floating_base_link="$(arg floating_base_link)" />
-    <!-- IMU sensor -->
-    <xacro:imu_sensor
-        frame_name="trunk_imu"
-        imu_topic="trunk_imu/data"
-        namespace="$(arg robot_name)"
-        update_rate="${1.0 / $(arg period)}"
-        rate_mean="0"
-        rate_stddev="0.01"
-        rate_bias_mean="0"
-        rate_bias_stddev="0"
-        accel_mean="0"
-        accel_stddev="0.001"
-        accel_bias_mean="0"
-        accel_bias_stddev="0">
-    </xacro:imu_sensor>
-    <xacro:imu_hardware imu_name="trunk_imu" imu_frame="trunk_imu"/>
+  <!-- IMU sensor -->
+  <xacro:imu_sensor
+      frame_name="trunk_imu"
+      imu_topic="trunk_imu/data"
+      namespace="$(arg robot_name)"
+      update_rate="${1.0 / $(arg period)}"
+      rate_mean="0"
+      rate_stddev="0.01"
+      rate_bias_mean="0"
+      rate_bias_stddev="0"
+      accel_mean="0"
+      accel_stddev="0.001"
+      accel_bias_mean="0"
+      accel_bias_stddev="0">
+  </xacro:imu_sensor>
+  <xacro:imu_hardware imu_name="trunk_imu" imu_frame="trunk_imu"/>
   <!-- Standard accessories. -->
   <xacro:if value="$(arg sensors)">
+    <!-- LIDAR sensor -->
     <xacro:VLP-16 parent="lidar_arch_mount_link" name="lidar" topic="/$(arg robot_name)/lidar_points"
                   organize_cloud="true" hz="10" gpu="true">
       <origin xyz="0 0 0" rpy="0 0 0" />
     </xacro:VLP-16>
+    <!-- RGBD camera mount + optical frame for Kinect plugin -->
+    <link name="camera_link"/>
+    <joint name="camera_mount_joint" type="fixed">
+      <!-- Pose of the simulated RGBD camera relative to the Husky mount -->
+      <origin xyz="0 0 0" rpy="0 0 0"/>
+      <parent link="realsense_mountpoint_link"/>
+      <child link="camera_link"/>
+    </joint>
+    <!-- Optical frame (camera convention: z forward, x right, y down) -->
+    <link name="camera_optical_frame"/>
+    <joint name="camera_optical_joint" type="fixed">
+      <!-- rotation from x-forward, z-up to z-forward, x-right, y-down -->
+      <origin xyz="0 0 0" rpy="-1.5707963 0 -1.5707963"/>
+      <parent link="camera_link"/>
+      <child link="camera_optical_frame"/>
+    </joint>
+    <!-- Kinect RGB(+depth) sensor using the optical frame -->
+    <xacro:kinect_rgb_sensor
+      link_name="camera_link"
+      frame_name="camera_optical_frame"
+      camera_name="camera">
+    </xacro:kinect_rgb_sensor>
+    <!-- (optional) IR variant, if you want it:
+    <xacro:kinect_ir_sensor
+      link_name="camera_link"
+      frame_name="camera_optical_frame"
+      camera_name="camera">
+    </xacro:kinect_ir_sensor>
+    -->
     <!-- GPS sensor -->
     <xacro:gps_sensor
@@ -48,4 +79,4 @@
         update_rate="10.0">
     </xacro:gps_sensor>
-    </xacro:if>
+  </xacro:if>
 </robot>

File: husky_description/urdfs/husky_macro.urdf.xacro (robot description, xacro)
@@ -1,4 +1,4 @@
 <?xml version="1.0"?>
-<robot xmlns:xacro="http://ros.org/wiki/xacro">
+<robot xmlns:xacro="http://www.ros.org/wiki/xacro">
   <xacro:property name="husky_front_bumper_extend" value="$(optenv HUSKY_FRONT_BUMPER_EXTEND 0)" />
   <xacro:property name="husky_rear_bumper_extend" value="$(optenv HUSKY_REAR_BUMPER_EXTEND 0)" />

File: sensors_description/urdfs/sensors/kinect.gazebo.xacro (robot description, xacro)
@@ -1,90 +1,99 @@
 <?xml version="1.0"?>
 <root xmlns:xacro="http://ros.org/wiki/xacro">
-	<xacro:macro name="kinect_ir_sensor" params="link_name frame_name camera_name">
-		<gazebo reference="${link_name}">
-			<sensor type="depth" name="${link_name}_ir_sensor">
-				<always_on>true</always_on>
-				<update_rate>1.0</update_rate>
-				<camera>
-					<horizontal_fov>${57.0*PI/180.0}</horizontal_fov>
-						<image>
-							<format>L8</format>
-							<width>640</width>
-							<height>480</height>
-						</image>
-					<clip>
-						<near>1.2</near>
-						<far>3.5</far>
-					</clip>
-				</camera>
-				<plugin name="${link_name}_controller" filename="libgazebo_ros_openni_kinect.so">
-					<baseline>0.2</baseline>
-					<alwaysOn>true</alwaysOn>
-					<updateRate>1.0</updateRate>
-					<cameraName>${camera_name}_ir</cameraName>
-					<imageTopicName>/${camera_name}/depth/image_raw</imageTopicName>
-					<cameraInfoTopicName>/${camera_name}/depth/camera_info</cameraInfoTopicName>
-					<depthImageTopicName>/${camera_name}/depth/image_raw</depthImageTopicName>
-					<depthImageCameraInfoTopicName>/${camera_name}/depth/camera_info</depthImageCameraInfoTopicName>
-					<pointCloudTopicName>/${camera_name}/depth/points</pointCloudTopicName>
-					<frameName>${frame_name}</frameName>
-					<pointCloudCutoff>0.5</pointCloudCutoff>
-					<distortionK1>0.00000001</distortionK1>
-					<distortionK2>0.00000001</distortionK2>
-					<distortionK3>0.00000001</distortionK3>
-					<distortionT1>0.00000001</distortionT1>
-					<distortionT2>0.00000001</distortionT2>
-					<CxPrime>0</CxPrime>
-					<Cx>0</Cx>
-					<Cy>0</Cy>
-					<focalLength>0</focalLength>
-					<hackBaseline>0</hackBaseline>
-				</plugin>
-			</sensor>
-			<material value="Gazebo/Red"/>
-		</gazebo>
-	</xacro:macro>
-	<xacro:macro name="kinect_rgb_sensor" params="link_name frame_name camera_name">
-		<gazebo reference="${link_name}">
-			<sensor type="depth" name="${link_name}_rgb_sensor">
-				<always_on>true</always_on>
-				<update_rate>1.0</update_rate>
-				<camera>
-					<horizontal_fov>${57.0*PI/180.0}</horizontal_fov>
-					<image>
-						<format>R8G8B8</format>
-						<width>640</width>
-						<height>480</height>
-					</image>
-					<clip>
-						<near>1.2</near>
-						<far>3.5</far>
-					</clip>
-				</camera>
-				<plugin name="${link_name}_controller" filename="libgazebo_ros_openni_kinect.so">
-					<alwaysOn>true</alwaysOn>
-					<updateRate>1.0</updateRate>
-					<cameraName>${camera_name}_rgb</cameraName>
-					<imageTopicName>/${camera_name}/rgb/image_raw</imageTopicName>
-					<cameraInfoTopicName>/${camera_name}/rgb/camera_info</cameraInfoTopicName>
-					<depthImageTopicName>/${camera_name}/depth/image_raw</depthImageTopicName>
-					<depthImageCameraInfoTopicName>/${camera_name}/depth/camera_info</depthImageCameraInfoTopicName>
-					<pointCloudTopicName>/${camera_name}/depth_registered/points</pointCloudTopicName>
-					<frameName>${frame_name}</frameName>
-					<pointCloudCutoff>0.5</pointCloudCutoff>
-					<distortionK1>0.00000001</distortionK1>
-					<distortionK2>0.00000001</distortionK2>
-					<distortionK3>0.00000001</distortionK3>
-					<distortionT1>0.00000001</distortionT1>
-					<distortionT2>0.00000001</distortionT2>
-					<CxPrime>0</CxPrime>
-					<Cx>0</Cx>
-					<Cy>0</Cy>
-					<focalLength>0</focalLength>
-					<hackBaseline>0</hackBaseline>
-				</plugin>
-			</sensor>
-			<material value="Gazebo/Red"/>
-		</gazebo>
-	</xacro:macro>
+  <xacro:property name="PI" value="3.1415926535897931" />
+  <!-- IR depth sensor -->
+  <xacro:macro name="kinect_ir_sensor" params="link_name frame_name camera_name">
+    <gazebo reference="${link_name}">
+      <sensor type="depth" name="${link_name}_ir_sensor">
+        <always_on>true</always_on>
+        <update_rate>1.0</update_rate>
+        <camera>
+          <horizontal_fov>${57.0*PI/180.0}</horizontal_fov>
+          <image>
+            <format>L8</format>
+            <width>640</width>
+            <height>480</height>
+          </image>
+          <clip>
+            <near>1.2</near>
+            <far>3.5</far>
+          </clip>
+        </camera>
+        <plugin name="${link_name}_ir_controller" filename="libgazebo_ros_openni_kinect.so">
+          <baseline>0.2</baseline>
+          <alwaysOn>true</alwaysOn>
+          <updateRate>1.0</updateRate>
+          <!-- Namespace for this IR camera -->
+          <cameraName>${camera_name}_ir</cameraName>
+          <!-- Same pattern as RGB: relative topics inside cameraName ns -->
+          <imageTopicName>image_raw</imageTopicName>
+          <cameraInfoTopicName>camera_info</cameraInfoTopicName>
+          <depthImageTopicName>depth/image_raw</depthImageTopicName>
+          <depthImageCameraInfoTopicName>depth/camera_info</depthImageCameraInfoTopicName>
+          <pointCloudTopicName>depth/points</pointCloudTopicName>
+          <!-- Frame already passed as optical frame from outside -->
+          <frameName>${frame_name}</frameName>
+          <pointCloudCutoff>0.5</pointCloudCutoff>
+          <distortionK1>0.00000001</distortionK1>
+          <distortionK2>0.00000001</distortionK2>
+          <distortionK3>0.00000001</distortionK3>
+          <distortionT1>0.00000001</distortionT1>
+          <distortionT2>0.00000001</distortionT2>
+          <CxPrime>0</CxPrime>
+          <Cx>0</Cx>
+          <Cy>0</Cy>
+          <focalLength>0</focalLength>
+          <hackBaseline>0</hackBaseline>
+        </plugin>
+      </sensor>
+      <material value="Gazebo/Red"/>
+    </gazebo>
+  </xacro:macro>
+  <!-- RGB(+depth) sensor -->
+  <xacro:macro name="kinect_rgb_sensor" params="link_name frame_name camera_name">
+    <gazebo reference="${link_name}">
+      <sensor type="depth" name="${link_name}_rgb_sensor">
+        <always_on>true</always_on>
+        <update_rate>1.0</update_rate>
+        <camera>
+          <horizontal_fov>${57.0*PI/180.0}</horizontal_fov>
+          <image>
+            <format>R8G8B8</format>
+            <width>640</width>
+            <height>480</height>
+          </image>
+          <clip>
+            <near>1.2</near>
+            <far>3.5</far>
+          </clip>
+        </camera>
+        <plugin name="${link_name}_rgb_controller" filename="libgazebo_ros_openni_kinect.so">
+          <alwaysOn>true</alwaysOn>
+          <updateRate>1.0</updateRate>
+          <!-- Base RGB camera namespace -->
+          <cameraName>${camera_name}</cameraName>
+          <!-- Relative topics; will resolve to ${cameraName}/... -->
+          <imageTopicName>image_raw</imageTopicName>
+          <cameraInfoTopicName>camera_info</cameraInfoTopicName>
+          <depthImageTopicName>depth/image_raw</depthImageTopicName>
+          <depthImageCameraInfoTopicName>depth/camera_info</depthImageCameraInfoTopicName>
+          <pointCloudTopicName>depth/points</pointCloudTopicName>
+          <!-- Optical frame passed from outside -->
+          <frameName>${frame_name}</frameName>
+          <pointCloudCutoff>0.5</pointCloudCutoff>
+          <distortionK1>0.00000001</distortionK1>
+          <distortionK2>0.00000001</distortionK2>
+          <distortionK3>0.00000001</distortionK3>
+          <distortionT1>0.00000001</distortionT1>
+          <distortionT2>0.00000001</distortionT2>
+          <CxPrime>0</CxPrime>
+          <Cx>0</Cx>
+          <Cy>0</Cy>
+          <focalLength>0</focalLength>
+          <hackBaseline>0</hackBaseline>
+        </plugin>
+      </sensor>
+      <material value="Gazebo/Red"/>
+    </gazebo>
+  </xacro:macro>
 </root>

File: spot_description/urdfs/accessories.urdf.xacro (robot description, xacro)
@@ -1,9 +1,13 @@
 <?xml version="1.0"?>
-<robot xmlns:xacro="http://www.ros.org/wiki/xacro">
+<robot xmlns:xacro="http://www.ros.org/wiki/xacro" name="spot_sensors">
+  <!-- Common + sensors includes -->
   <xacro:include filename="$(find sensors_description)/urdfs/common.xacro"/>
   <xacro:include filename="$(find velodyne_description)/urdf/VLP-16.urdf.xacro"/>
-  <xacro:include filename="$(find sensors_description)/urdfs/sensors/realsense_d435.urdf.xacro" />
+  <xacro:include filename="$(find sensors_description)/urdfs/sensors/kinect.gazebo.xacro"/>
   <xacro:include filename="$(find sensors_description)/urdfs/sensors/realsense_t265.urdf.xacro" />
   <xacro:include filename="$(find sensors_description)/urdfs/sensors/gps.gazebo.xacro"/>
+  <!-- PI (only needed if not already defined in included xacros) -->
+  <xacro:property name="PI" value="3.1415926535897931"/>
+  <!-- Pack mount on Spot -->
   <xacro:if value="$(optenv SPOT_PACK 1)">
     <joint name="pack_mount_joint" type="fixed">
@@ -30,4 +34,5 @@
     </link>
   </xacro:if>
+  <!-- Lidar mount on pack -->
   <xacro:if value="$(optenv SPOT_LIDAR_MOUNT 1)">
     <joint name="lidar_mount_joint" type="fixed">
@@ -48,4 +53,5 @@
       </collision>
     </link>
+    <!-- Velodyne + front sensors -->
     <xacro:if value="$(optenv SPOT_VELODYNE 1)">
       <joint name="velodyne_mount_joint" type="fixed">
@@ -66,12 +72,47 @@
         </collision>
       </link>
-      <xacro:VLP-16 parent="velodyne_mount" name="velodyne" topic="/$(arg robot_name)/lidar_points"
+      <!-- Velodyne VLP-16 -->
+      <xacro:VLP-16 parent="velodyne_mount" name="velodyne"
+                    topic="/$(arg robot_name)/lidar_points"
                     organize_cloud="true" hz="10" gpu="true">
         <origin xyz="0 0 0" rpy="0 0 0" />
       </xacro:VLP-16>
-      <xacro:realsense_d435 name="camera" topics_ns="/$(arg robot_name)/camera" parent="front_rail">
-        <origin xyz="0.13 0 0" rpy="0 0 0" />
-      </xacro:realsense_d435>
-      <xacro:realsense_T265 name="t265" topics_ns="/$(arg robot_name)" parent="front_rail" rate="30.0">
+      <!-- FRONT RAIL is assumed to be defined in the base Spot model -->
+      <!-- Camera base link on front_rail -->
+      <link name="camera_link"/>
+      <joint name="camera_mount_joint" type="fixed">
+        <parent link="front_rail"/>
+        <child link="camera_link"/>
+        <!-- Physical pose of the RGBD camera wrt front_rail -->
+        <!-- tune xyz/rpy if needed to match your model -->
+        <origin xyz="0.13 0 0.0" rpy="0 0 0"/>
+      </joint>
+      <!-- Optical frame (REP-103: z forward, x right, y down) -->
+      <link name="camera_optical_frame"/>
+      <joint name="camera_optical_joint" type="fixed">
+        <parent link="camera_link"/>
+        <child link="camera_optical_frame"/>
+        <!-- rotation from x-forward,z-up to z-forward,x-right,y-down -->
+        <origin xyz="0 0 0" rpy="${-PI/2} 0 ${-PI/2}"/>
+      </joint>
+      <!-- Kinect RGB (depth) sensor using the optical frame for the point cloud -->
+      <xacro:kinect_rgb_sensor
+        link_name="camera_link"
+        frame_name="camera_optical_frame"
+        camera_name="camera">
+      </xacro:kinect_rgb_sensor>
+      <!-- Optional: IR depth sensor variant, if you want it too -->
+      <!--
+      <xacro:kinect_ir_sensor
+        link_name="camera_link"
+        frame_name="camera_optical_frame"
+        camera_name="camera_ir">
+      </xacro:kinect_ir_sensor>
+      -->
+      <!-- T265 tracking camera -->
+      <xacro:realsense_T265 name="t265"
+                            topics_ns="/$(arg robot_name)"
+                            parent="front_rail"
+                            rate="30.0">
         <origin xyz="0.13 0 0.04" rpy="0 0 0" />
       </xacro:realsense_T265>
