Commit message: Husky!

File: husky_description/robots/husky.urdf.xacro (robot description, xacro)
@@ -14,6 +14,9 @@
   <xacro:include filename="$(find sensors_description)/urdfs/sensors/imu.gazebo.xacro"/>
   <xacro:include filename="$(find wolf_description_utils)/urdfs/wheels.hardware.xacro"/>
+  <xacro:include filename="$(find sensors_description)/urdfs/sensors/depth_camera.gazebo.xacro"/>
+  <xacro:include filename="$(find sensors_description)/urdfs/sensors/gps.gazebo.xacro"/>
+  <xacro:include filename="$(find sensors_description)/urdfs/sensors/lidar.gazebo.xacro"/>
   <xacro:include filename="$(find husky_description)/urdfs/husky_macro.urdf.xacro" />
-  <xacro:husky prefix="" floating_base_link="$(arg floating_base_link)" />
+  <xacro:husky floating_base_link="$(arg floating_base_link)" />
     <!-- IMU sensor -->
     <xacro:imu_sensor
@@ -32,3 +35,42 @@
     </xacro:imu_sensor>
     <xacro:imu_hardware imu_name="trunk_imu" imu_frame="trunk_imu"/>
+    <!-- Standard accessories. -->
+    <xacro:if value="$(arg sensors)">
+        <xacro:depth_camera
+          name="camera"
+          namespace="$(arg robot_name)"
+          update_rate="30"
+          image_width="640"
+          image_height="480"
+          fov="1.047"
+          near="0.1"
+          far="10.0"
+          parent_link="realsense_mountpoint_link"
+          image_topic="$(arg robot_name)/camera/rgb/image_raw"
+          depth_topic="$(arg robot_name)/camera/depth/image_raw"
+          pointcloud_topic="$(arg robot_name)/camera/points"
+          camera_info_topic="$(arg robot_name)/camera/camera_info"
+          origin_xyz="0.13 0 0"
+          origin_rpy="0 0 0"/>
+        <xacro:velodyne_laser_gazebo_sensor
+          sensor_name="lidar"
+          topic_name="lidar_points"
+          update_rate="10.0"
+          frame_id="lidar_arch_mount_link"
+          namespace="$(arg robot_name)"
+          min_range="0.9"
+          max_range="130.0"
+          number_of_beams="32"
+          horizontal_samples="220"
+          horizontal_fov="6.28319"
+          vertical_fov="0.2618"
+          noise_stddev="0.01" />
+      <xacro:gazebo_gps_sensor
+          sensor_name="gps_sensor"
+          namespace="$(arg robot_name)"
+          gps_topic="gps/fix"
+          velocity_topic="gps/velocity_fix"
+          update_rate="10.0"
+          frame_id="base_link" />
+    </xacro:if>
 </robot>

File: husky_description/urdfs/decorations.urdf.xacro (robot description, xacro)
@@ -11,4 +11,6 @@
     <xacro:property name="husky_front_bumper_extend" value="$(optenv HUSKY_FRONT_BUMPER_EXTEND 0)" />
     <xacro:property name="husky_rear_bumper_extend" value="$(optenv HUSKY_REAR_BUMPER_EXTEND 0)" />
+    <xacro:property name="husky_top_plate" value="$(optenv HUSKY_TOP_PLATE_ENABLED 1)" />
+    <xacro:property name="husky_large_top_plate" value="$(optenv HUSKY_LARGE_TOP_PLATE 1)" />
     <!-- Spawn Husky chassis -->
     <link name="top_chassis_link">
@@ -97,7 +99,7 @@
       </joint>
     </xacro:if>
-    <xacro:if value="$(optenv HUSKY_TOP_PLATE_ENABLED true)">
+    <xacro:if value="${husky_top_plate}">
       <!-- Spawn the top plate -->
-      <xacro:if value="$(optenv HUSKY_LARGE_TOP_PLATE false)">
+      <xacro:unless value="${husky_large_top_plate}">
         <link name="top_plate_link">
           <visual>
@@ -132,6 +134,6 @@
           <origin xyz="-0.4125 0 0.00672" rpy="0 0 0"/>
         </joint>
-      </xacro:if>
-      <xacro:unless value="$(optenv HUSKY_LARGE_TOP_PLATE false)">
+      </xacro:unless>
+      <xacro:if value="${husky_large_top_plate}">
         <link name="top_plate_link">
           <visual>
@@ -166,5 +168,5 @@
           <origin xyz="-0.36633 0 0.00639" rpy="0 0 0"/>
         </joint>
-      </xacro:unless>
+      </xacro:if>
       <link name="top_plate_front_link"/>
       <link name="top_plate_rear_link"/>

File: husky_description/urdfs/husky_macro.urdf.xacro (robot description, xacro)
@@ -1,45 +1,33 @@
 <?xml version="1.0"?>
 <robot xmlns:xacro="http://ros.org/wiki/xacro">
-  <xacro:arg name="laser_enabled" default="$(optenv CPR_LASER_ENABLED 0)" />
-  <xacro:arg name="laser_xyz" default="$(optenv CPR_LASER_XYZ 0.2206 0.0 0.00635)" />
-  <xacro:arg name="laser_rpy" default="$(optenv CPR_LASER_RPY 0.0 0.0 0.0)" />
-  <xacro:arg name="realsense_enabled" default="$(optenv CPR_REALSENSE 0)" />
-  <xacro:arg name="realsense_xyz" default="$(optenv CPR_REALSENSE_XYZ 0 0 0)" />
-  <xacro:arg name="realsense_rpy" default="$(optenv CPR_REALSENSE_RPY 0 0 0)" />
-  <xacro:arg name="realsense_mount" default="$(optenv CPR_REALSENSE_MOUNT_FRAME sensor_arch_mount_link)" />
   <xacro:property name="husky_front_bumper_extend" value="$(optenv HUSKY_FRONT_BUMPER_EXTEND 0)" />
   <xacro:property name="husky_rear_bumper_extend" value="$(optenv HUSKY_REAR_BUMPER_EXTEND 0)" />
   <xacro:arg name="robot_namespace" default="/" />
-  <xacro:arg name="urdf_extras" default="$(optenv CPR_URDF_EXTRAS empty.urdf)" />
   <!-- Included URDF/XACRO Files -->
   <xacro:include filename="$(find husky_description)/urdfs/decorations.urdf.xacro" />
   <xacro:include filename="$(find husky_description)/urdfs/wheel.urdf.xacro" />
-  <!--<xacro:include filename="$(find husky_description)/urdfs/accessories/intel_realsense.urdf.xacro"/>-->
-  <!--<xacro:include filename="$(find husky_description)/urdf/accessories/sick_lms1xx_mount.urdf.xacro"/>-->
-  <!--<xacro:include filename="$(find husky_description)/urdfs/accessories/sensor_arch.urdf.xacro"/>-->
   <xacro:property name="M_PI" value="3.14159"/>
-  <xacro:macro name="husky" params="prefix floating_base_link">
-    <!-- Base Size -->
-    <xacro:property name="base_x_size" value="0.98740000" />
-    <xacro:property name="base_y_size" value="0.57090000" />
-    <xacro:property name="base_z_size" value="0.24750000" />
-    <!-- Wheel Mounting Positions -->
+  <xacro:macro name="husky" params="floating_base_link">
+    <!-- Base Dimensions -->
+    <xacro:property name="base_x_size" value="0.9874" />
+    <xacro:property name="base_y_size" value="0.5709" />
+    <xacro:property name="base_z_size" value="0.2475" />
+    <!-- Wheel Configuration -->
     <xacro:property name="wheelbase" value="0.5120" />
     <xacro:property name="track" value="0.5708" />
     <xacro:property name="wheel_vertical_offset" value="0.03282" />
-    <!-- Wheel Properties -->
     <xacro:property name="wheel_length" value="0.1143" />
     <xacro:property name="wheel_radius" value="0.1651" />
-    <!-- Floating-base Joint -->
+    <!-- Floating base (optional) -->
     <xacro:if value="$(arg floating_base_link)">
-        <link name="world"/>
-        <joint name="${prefix}floating_base_joint" type="floating">
-          <origin rpy="0 0 0" xyz="0 0 0"/>
-          <parent link="world"/>
-          <child link="${prefix}base_link"/>
-        </joint>
+      <link name="world"/>
+      <joint name="floating_base_joint" type="floating">
+        <origin rpy="0 0 0" xyz="0 0 0"/>
+        <parent link="world"/>
+        <child link="base_link"/>
+      </joint>
     </xacro:if>
-    <!-- Base link is the center of the robot's bottom plate -->
-    <link name="${prefix}base_link">
+    <!-- Base Link -->
+    <link name="base_link">
       <visual>
         <origin xyz="0 0 0" rpy="0 0 0" />
@@ -49,7 +37,7 @@
       </visual>
       <collision>
-        <origin xyz="${( husky_front_bumper_extend - husky_rear_bumper_extend ) / 2.0} 0 ${base_z_size/4}" rpy="0 0 0" />
+        <origin xyz="${(husky_front_bumper_extend - husky_rear_bumper_extend) / 2.0} 0 ${base_z_size/4}" rpy="0 0 0" />
         <geometry>
-          <box size="${ base_x_size + husky_front_bumper_extend + husky_rear_bumper_extend } ${base_y_size} ${base_z_size/2}"/>
+          <box size="${base_x_size + husky_front_bumper_extend + husky_rear_bumper_extend} ${base_y_size} ${base_z_size/2}" />
         </geometry>
       </collision>
@@ -57,17 +45,16 @@
         <origin xyz="0 0 ${base_z_size*3/4-0.01}" rpy="0 0 0" />
         <geometry>
-          <box size="${base_x_size*4/5} ${base_y_size} ${base_z_size/2-0.02}"/>
+          <box size="${base_x_size*4/5} ${base_y_size} ${base_z_size/2-0.02}" />
         </geometry>
       </collision>
     </link>
-    <!-- Base footprint is on the ground under the robot -->
-    <link name="${prefix}base_footprint"/>
-    <joint name="${prefix}base_footprint_joint" type="fixed">
+    <link name="base_footprint" />
+    <joint name="base_footprint_joint" type="fixed">
       <origin xyz="0 0 ${wheel_vertical_offset - wheel_radius}" rpy="0 0 0" />
-      <parent link="${prefix}base_link" />
-      <child link="${prefix}base_footprint" />
+      <parent link="base_link" />
+      <child link="base_footprint" />
     </joint>
-    <!-- Inertial link stores the robot's inertial information -->
-    <link name="${prefix}inertial_link">
+    <!-- Inertial -->
+    <link name="inertial_link">
       <inertial>
         <mass value="46.034" />
@@ -76,69 +63,106 @@
       </inertial>
     </link>
-    <joint name="${prefix}inertial_joint" type="fixed">
+    <joint name="inertial_joint" type="fixed">
       <origin xyz="0 0 0" rpy="0 0 0" />
-      <parent link="${prefix}base_link" />
-      <child link="${prefix}inertial_link" />
+      <parent link="base_link" />
+      <child link="inertial_link" />
     </joint>
-    <!-- IMU Link-->
-    <!-- Can be modified with environment variables in /etc/ros/setup.bash -->
-    <link name="${prefix}trunk_imu"/>
-    <joint name="${prefix}imu_joint" type="fixed">
+    <!-- IMU -->
+    <link name="trunk_imu" />
+    <joint name="imu_joint" type="fixed">
       <origin xyz="$(optenv CPR_IMU_XYZ 0 0 0)" rpy="$(optenv CPR_IMU_RPY 0 0 0)" />
-      <parent link="${prefix}base_link" />
-      <child link="${prefix}trunk_imu" />
+      <parent link="base_link" />
+      <child link="trunk_imu" />
     </joint>
-    <!-- GPS Link-->
-    <!-- Can be modified with environment variables in /etc/ros/setup.bash -->
-    <link name="${prefix}gps_link"/>
-    <joint name="${prefix}gps_joint" type="fixed">
+    <!-- GPS -->
+    <link name="gps_link" />
+    <joint name="gps_joint" type="fixed">
       <origin xyz="$(optenv CPR_GPS_XYZ 0 0 0)" rpy="$(optenv CPR_GPS_RPY 0 0 0)" />
-      <parent link="${prefix}base_link" />
-      <child link="${prefix}gps_link" />
+      <parent link="base_link" />
+      <child link="gps_link" />
     </joint>
-    <!-- Husky wheel macros -->
-    <xacro:husky_wheel wheel_prefix="${prefix}front_left">
+    <!-- Wheels -->
+    <xacro:husky_wheel wheel_prefix="front_left">
       <origin xyz="${wheelbase/2} ${track/2} ${wheel_vertical_offset}" rpy="0 0 0" />
     </xacro:husky_wheel>
-    <xacro:husky_wheel wheel_prefix="${prefix}front_right">
+    <xacro:husky_wheel wheel_prefix="front_right">
       <origin xyz="${wheelbase/2} ${-track/2} ${wheel_vertical_offset}" rpy="0 0 0" />
     </xacro:husky_wheel>
-    <xacro:husky_wheel wheel_prefix="${prefix}rear_left">
+    <xacro:husky_wheel wheel_prefix="rear_left">
       <origin xyz="${-wheelbase/2} ${track/2} ${wheel_vertical_offset}" rpy="0 0 0" />
     </xacro:husky_wheel>
-    <xacro:husky_wheel wheel_prefix="${prefix}rear_right">
+    <xacro:husky_wheel wheel_prefix="rear_right">
       <origin xyz="${-wheelbase/2} ${-track/2} ${wheel_vertical_offset}" rpy="0 0 0" />
     </xacro:husky_wheel>
+    <!-- Decorations -->
     <xacro:husky_decorate />
-    <!-- <xacro:if value="$(arg laser_enabled)">
-      <xacro:sick_lms1xx_mount prefix="base"/>
-      <xacro:sick_lms1xx frame="base_laser" topic="scan" robot_namespace="$(arg robot_namespace)"/>
-      <joint name="laser_mount_joint" type="fixed">
-        <origin xyz="$(arg laser_xyz)" rpy="$(arg laser_rpy)" />
-        <parent link="top_plate_link" />
-        <child link="base_laser_mount" />
-      </joint>
-    </xacro:if> -->
-    <!--
-      top sensor arch; include this if we have realsense enabled
-      keep this as a property to make it easier to add multiple conditions, should we need
-      the top bar for any additional sensors in the future
-    -->
-    <!-- <xacro:property name="topbar_needed_realsense" value="$(arg realsense_enabled)" />
-    <xacro:if value="${topbar_needed_realsense}">
-      <xacro:sensor_arch prefix="" parent="top_plate_link">
-        <origin xyz="-0.35 0 0.51" rpy="0 0 -3.14"/>
-      </xacro:sensor_arch>
-    </xacro:if> -->
-    <!-- add the intel realsense to the topbar if needed -->
-    <xacro:if value="$(arg realsense_enabled)">
-      <link name="realsense_mountpoint"/>
-      <joint name="realsense_mountpoint_joint" type="fixed">
-        <origin xyz="$(arg realsense_xyz)" rpy="$(arg realsense_rpy)" />
-        <parent link="$(arg realsense_mount)"/>
-        <child link="realsense_mountpoint" />
-      </joint>
-      <xacro:intel_realsense_mount prefix="camera" topic="realsense" parent_link="realsense_mountpoint"/>
-    </xacro:if>
+    <!-- Laser Mount -->
+    <link name="base_laser_mount">
+      <visual>
+        <origin xyz="0 0 0" rpy="0 0 ${-M_PI/2}" />
+        <geometry>
+          <mesh filename="file://$(find husky_description)/meshes/accessories/lms1xx_mount.dae" />
+        </geometry>
+      </visual>
+      <collision>
+        <origin xyz="0 0 .0585" rpy="0 0 0" />
+        <geometry>
+          <box size=".1 .108 .117" />
+        </geometry>
+      </collision>
+    </link>
+    <joint name="laser_mount_joint" type="fixed">
+      <origin xyz="0.2206 0.0 0.00635" rpy="0.0 0.0 0.0" />
+      <parent link="top_plate_link" />
+      <child link="base_laser_mount" />
+    </joint>
+    <!-- Sensor Arch -->
+    <link name="sensor_arch_mount_link">
+      <visual>
+        <geometry>
+          <mesh filename="file://$(find husky_description)/meshes/accessories/300_mm_sensor_arch.dae" />
+        </geometry>
+      </visual>
+      <collision>
+        <origin xyz="0 0 0" rpy="0 0 0" />
+        <geometry>
+          <mesh filename="file://$(find husky_description)/meshes/accessories/300_mm_sensor_arch.dae" />
+        </geometry>
+      </collision>
+    </link>
+    <joint name="realsense_mountpoint" type="fixed">
+      <origin xyz="0.05 0.0 0.1" rpy="0.0 0.0 0.0" />
+      <parent link="base_laser_mount" />
+      <child link="realsense_mountpoint_link" />
+    </joint>
+    <link name="realsense_mountpoint_link">
+      <visual>
+        <geometry>
+          <mesh filename="file://$(find husky_description)/meshes/accessories/depth_camera.dae"/>
+        </geometry>
+      </visual>
+    </link>
+    <joint name="sensor_arch_mount" type="fixed">
+      <origin xyz="-0.35 0 0.3" rpy="0 0 -3.14" /> <!-- with 510mm use 0.51 on z-->
+      <parent link="top_plate_link" />
+      <child link="sensor_arch_mount_link" />
+    </joint>
+    <joint name="lidar_arch_mount" type="fixed">
+      <origin xyz="0 0 0" rpy="0 0 0" />
+      <parent link="sensor_arch_mount_link" />
+      <child link="lidar_arch_mount_link" />
+    </joint>
+    <link name="lidar_arch_mount_link">
+      <visual>
+        <geometry>
+          <mesh filename="file://$(find husky_description)/meshes/accessories/lidar.dae"/>
+        </geometry>
+      </visual>
+      <collision>
+        <geometry>
+          <mesh filename="file://$(find husky_description)/meshes/accessories/lidar_collision.stl"/>
+        </geometry>
+      </collision>
+    </link>
   </xacro:macro>
 </robot>
