Commit message: Fix wildcards and ros2 gazebo sensor plugins

File: husky_description/robots/husky.urdf.xacro (robot description, xacro)
@@ -21,4 +21,5 @@
     <!-- IMU sensor -->
     <xacro:imu_sensor
+        sensor_name="$(arg robot_name)_imu"
         frame_name="trunk_imu"
         imu_topic="trunk_imu/data"
@@ -34,8 +35,8 @@
         accel_bias_stddev="0">
     </xacro:imu_sensor>
-    <xacro:imu_hardware imu_name="trunk_imu" imu_frame="trunk_imu"/>
+    <xacro:imu_hardware imu_name="$(arg robot_name)_imu" imu_frame="trunk_imu"/>
     <!-- Standard accessories. -->
     <xacro:if value="$(arg sensors)">
-        <xacro:depth_camera
+      <xacro:depth_camera
           name="camera"
           namespace="$(arg robot_name)"
@@ -47,25 +48,21 @@
           far="10.0"
           parent_link="realsense_mountpoint_link"
-          image_topic="$(arg robot_name)/camera/rgb/image_raw"
-          depth_topic="$(arg robot_name)/camera/depth/image_raw"
-          pointcloud_topic="$(arg robot_name)/camera/points"
-          camera_info_topic="$(arg robot_name)/camera/camera_info"
           origin_xyz="0.13 0 0"
           origin_rpy="0 0 0"/>
-        <xacro:velodyne_laser_gazebo_sensor
-          sensor_name="lidar"
-          topic_name="lidar_points"
-          update_rate="10.0"
-          frame_id="lidar_arch_mount_link"
-          namespace="$(arg robot_name)"
-          min_range="0.9"
-          max_range="130.0"
-          number_of_beams="32"
-          horizontal_samples="220"
-          horizontal_fov="6.28319"
-          vertical_fov="0.2618"
-          noise_stddev="0.01" />
+      <xacro:velodyne_laser_gazebo_sensor
+        sensor_name="$(arg robot_name)_lidar"
+        topic_name="lidar_points"
+        update_rate="10.0"
+        frame_id="lidar_arch_mount_link"
+        namespace="$(arg robot_name)"
+        min_range="0.9"
+        max_range="130.0"
+        number_of_beams="32"
+        horizontal_samples="220"
+        horizontal_fov="6.28319"
+        vertical_fov="0.2618"
+        noise_stddev="0.01" />
       <xacro:gazebo_gps_sensor
-          sensor_name="gps_sensor"
+          sensor_name="$(arg robot_name)_gps"
           namespace="$(arg robot_name)"
           gps_topic="gps/fix"

File: husky_description/urdfs/husky_macro.urdf.xacro (robot description, xacro)
@@ -1,7 +1,6 @@
 <?xml version="1.0"?>
-<robot xmlns:xacro="http://ros.org/wiki/xacro">
+<robot name="husky" xmlns:xacro="http://ros.org/wiki/xacro">
   <xacro:property name="husky_front_bumper_extend" value="$(optenv HUSKY_FRONT_BUMPER_EXTEND 0)" />
   <xacro:property name="husky_rear_bumper_extend" value="$(optenv HUSKY_REAR_BUMPER_EXTEND 0)" />
-  <xacro:arg name="robot_namespace" default="/" />
   <!-- Included URDF/XACRO Files -->
   <xacro:include filename="$(find husky_description)/urdfs/decorations.urdf.xacro" />

File: sensors_description/urdfs/sensors/depth_camera.gazebo.xacro (robot description, xacro)
@@ -2,6 +2,5 @@
 <robot xmlns:xacro="http://ros.org/wiki/xacro">
   <xacro:macro name="depth_camera" params="
-    name namespace update_rate image_width image_height fov near far parent_link
-    image_topic camera_info_topic depth_topic pointcloud_topic origin_xyz origin_rpy
+    name namespace update_rate image_width image_height fov near far parent_link origin_xyz origin_rpy
   ">
     <!-- Camera Link -->
@@ -39,5 +38,5 @@
         <always_on>true</always_on>
         <pose>${origin_xyz} ${origin_rpy}</pose>
-        <camera name="${name}_depth_camera">
+        <camera name="${name}">
           <horizontal_fov>${fov}</horizontal_fov>
           <image>
@@ -52,11 +51,19 @@
         </camera>
         <!-- Plugin for Depth Camera -->
-        <plugin name="gazebo_ros_depth_camera_plugin" filename="libgazebo_ros_camera.so">
+        <plugin name="${namespace}_${name}_plugin" filename="libgazebo_ros_camera.so">
+          <robotNamespace>/${namespace}</robotNamespace>
           <ros>
-            <namespace>${namespace}</namespace>
-            <remapping>~/image_raw:=${image_topic}</remapping>
-            <remapping>~/camera_info:=${camera_info_topic}</remapping>
-            <remapping>~/depth/image_raw:=${depth_topic}</remapping>
-            <remapping>~/points:=${pointcloud_topic}</remapping>
+            <namespace>/${namespace}</namespace>
+            <remapping>${name}/image_raw:=/${namespace}/${name}/image_raw</remapping>
+            <remapping>${name}/image_raw/compressed:=/${namespace}/${name}/image_raw/compressed</remapping>
+            <remapping>${name}/image_raw/compressedDepth:=/${namespace}/${name}/image_raw/compressedDepth</remapping>
+            <remapping>${name}/image_raw/theora:=/${namespace}/${name}/image_raw/theora</remapping>
+            <remapping>${name}/depth/image_raw:=/${namespace}/${name}/depth/image_raw</remapping>
+            <remapping>${name}/depth/camera_info:=/${namespace}/${name}/depth/camera_info</remapping>
+            <remapping>${name}/depth/image_raw/compressed:=/${namespace}/${name}/depth/image_raw/compressed</remapping>
+            <remapping>${name}/depth/image_raw/compressedDepth:=/${namespace}/${name}/depth/image_raw/compressedDepth</remapping>
+            <remapping>${name}/depth/image_raw/theora:=/${namespace}/${name}/depth/image_raw/theora</remapping>
+            <remapping>${name}/camera_info:=/${namespace}/${name}/camera_info</remapping>
+            <remapping>${name}/points:=/${namespace}/${name}/points</remapping>
           </ros>
           <camera_name>${name}</camera_name>

File: sensors_description/urdfs/sensors/gps.gazebo.xacro (robot description, xacro)
@@ -20,5 +20,5 @@
       </xacro:if>
     <gazebo reference="${frame_id}">
-      <sensor type="gps" name="${sensor_name}">
+      <sensor name="${sensor_name}" type="gps" >
         <always_on>1</always_on>
         <update_rate>${update_rate}</update_rate>
@@ -26,10 +26,11 @@
           <!-- Optionally, include additional sensor-specific parameters here -->
         </gps>
-        <plugin name="gps_plugin" filename="libgazebo_ros_gps_sensor.so">
+        <plugin name="${sensor_name}_plugin" filename="libgazebo_ros_gps_sensor.so">
+          <robotNamespace>/${namespace}</robotNamespace>
           <ros>
             <namespace>/${namespace}</namespace>
             <!-- Additional ROS plugin configuration can be added here -->
-            <remapping>gps_plugin/out:=${gps_topic}</remapping>
-            <remapping>gps_plugin/vel:=${velocity_topic}</remapping>
+            <remapping>${sensor_name}_plugin/out:=/${namespace}/${gps_topic}</remapping>
+            <remapping>${sensor_name}_plugin/vel:=/${namespace}/${velocity_topic}</remapping>
           </ros>
           <frame_name>${frame_name_ns}</frame_name>

File: sensors_description/urdfs/sensors/imu.gazebo.xacro (robot description, xacro)
@@ -1,23 +1,24 @@
 <?xml version="1.0"?>
 <robot xmlns:xacro="http://ros.org/wiki/xacro">
-    <xacro:macro name="imu_sensor" params="frame_name imu_topic namespace update_rate rate_mean rate_stddev
+    <xacro:macro name="imu_sensor" params="sensor_name frame_name imu_topic namespace update_rate rate_mean rate_stddev
         rate_bias_mean rate_bias_stddev accel_mean accel_stddev accel_bias_mean accel_bias_stddev">
       <xacro:if value="${namespace == ''}">
-                    <xacro:property name="frame_name_ns" value="${frame_name}"/>
+                <xacro:property name="frame_name_ns" value="${frame_name}"/>
       </xacro:if>
       <xacro:if value="${namespace != ''}">
-                    <xacro:property name="frame_name_ns" value="${namespace+'/'+frame_name}"/>
+                <xacro:property name="frame_name_ns" value="${namespace+'/'+frame_name}"/>
       </xacro:if>
-        <gazebo reference="trunk_imu">
+        <gazebo reference="${frame_name}">
             <gravity>true</gravity>
-            <sensor name="trunk_imu" type="imu">
+            <sensor name="${sensor_name}" type="imu">
                 <always_on>true</always_on>
                 <update_rate>${update_rate}</update_rate>
                 <visualize>true</visualize>
                 <topic>${imu_topic}</topic>
-                <plugin name="imu_sensor_plugin" filename="libgazebo_ros_imu_sensor.so">
+                <plugin name="${sensor_name}_plugin" filename="libgazebo_ros_imu_sensor.so">
+                    <robotNamespace>/${namespace}</robotNamespace>
                     <ros>
-                        <namespace>${namespace}</namespace>
-                        <remapping>imu_sensor_plugin/out:=${imu_topic}</remapping>
+                        <namespace>/${namespace}</namespace>
+                        <remapping>${sensor_name}_plugin/out:=/${namespace}/${imu_topic}</remapping>
                     </ros>
                     <update_rate>${update_rate}</update_rate>

File: sensors_description/urdfs/sensors/lidar.gazebo.xacro (robot description, xacro)
@@ -1,55 +1,58 @@
 <?xml version="1.0"?>
 <robot xmlns:xacro="http://ros.org/wiki/xacro">
-<xacro:macro name="velodyne_laser_gazebo_sensor" params="sensor_name topic_name update_rate frame_id namespace min_range max_range number_of_beams horizontal_samples horizontal_fov vertical_fov noise_stddev">
-      <xacro:if value="${namespace == ''}">
-                    <xacro:property name="frame_name_ns" value="${frame_id}"/>
-      </xacro:if>
-      <xacro:if value="${namespace != ''}">
-                    <xacro:property name="frame_name_ns" value="${namespace+'/'+frame_id}"/>
-      </xacro:if>
-  <gazebo reference="${frame_id}">
-        <sensor type="ray" name="${sensor_name}">
-          <pose>0 0 0 0 0 0</pose>
-          <visualize>false</visualize>
-          <update_rate>${update_rate}</update_rate>
-          <ray>
-                <scan>
-                    <horizontal>
-                        <samples>${horizontal_samples}</samples>
-                        <resolution>1</resolution>
-                        <min_angle>${-0.5 * horizontal_fov}</min_angle>
-                        <max_angle>${0.5 * horizontal_fov}</max_angle>
-                    </horizontal>
-                    <vertical>
-                        <samples>${number_of_beams}</samples>
-                        <resolution>1</resolution>
-                        <min_angle>${-0.5 * vertical_fov}</min_angle>
-                        <max_angle>${0.5 * vertical_fov}</max_angle>
-                    </vertical>
-                </scan>
-                <range>
-                    <min>${min_range}</min>
-                    <max>${max_range}</max>
-                    <resolution>0.001</resolution>
-                </range>
-                <noise>
-                    <type>gaussian</type>
-                    <mean>0.0</mean>
-                    <stddev>0.0</stddev>
-                </noise>
-          </ray>
-          <plugin name="gazebo_ros_laser_controller" filename="libgazebo_ros_velodyne_laser.so">
-            <ros>
-              <namespace>/${namespace}</namespace>
-              <remapping>gazebo_ros_laser_controller/out:=${topic_name}</remapping>
-            </ros>
-            <frame_name>${frame_name_ns}</frame_name>
-            <organize_cloud>true</organize_cloud>
-            <min_range>${min_range}</min_range>
-            <max_range>${max_range}</max_range>
-            <gaussian_noise>${noise_stddev}</gaussian_noise>
-          </plugin>
-        </sensor>
+  <xacro:macro name="velodyne_laser_gazebo_sensor" params="sensor_name topic_name update_rate frame_id namespace min_range max_range number_of_beams horizontal_samples horizontal_fov vertical_fov noise_stddev">
+    <!-- Construct full frame name -->
+    <xacro:if value="${namespace == ''}">
+      <xacro:property name="frame_name_ns" value="${frame_id}"/>
+    </xacro:if>
+    <xacro:if value="${namespace != ''}">
+      <xacro:property name="frame_name_ns" value="${namespace + '/' + frame_id}"/>
+    </xacro:if>
+    <!-- Sensor definition -->
+    <gazebo reference="${frame_id}">
+      <sensor type="ray" name="${sensor_name}">
+        <pose>0 0 0 0 0 0</pose>
+        <visualize>false</visualize>
+        <update_rate>${update_rate}</update_rate>
+        <ray>
+          <scan>
+            <horizontal>
+              <samples>${horizontal_samples}</samples>
+              <resolution>1</resolution>
+              <min_angle>${-0.5 * horizontal_fov}</min_angle>
+              <max_angle>${0.5 * horizontal_fov}</max_angle>
+            </horizontal>
+            <vertical>
+              <samples>${number_of_beams}</samples>
+              <resolution>1</resolution>
+              <min_angle>${-0.5 * vertical_fov}</min_angle>
+              <max_angle>${0.5 * vertical_fov}</max_angle>
+            </vertical>
+          </scan>
+          <range>
+            <min>${min_range}</min>
+            <max>${max_range}</max>
+            <resolution>0.001</resolution>
+          </range>
+          <noise>
+            <type>gaussian</type>
+            <mean>0.0</mean>
+            <stddev>0.0</stddev>
+          </noise>
+        </ray>
+        <plugin name="${sensor_name}_plugin" filename="libgazebo_ros_velodyne_laser.so">
+          <robotNamespace>/${namespace}</robotNamespace>
+          <ros>
+            <namespace>/${namespace}</namespace>
+            <remapping>${sensor_name}_plugin/out:=/${namespace}/${topic_name}</remapping>
+          </ros>
+          <frame_name>${frame_name_ns}</frame_name>
+          <organize_cloud>true</organize_cloud>
+          <min_range>${min_range}</min_range>
+          <max_range>${max_range}</max_range>
+          <gaussian_noise>${noise_stddev}</gaussian_noise>
+        </plugin>
+      </sensor>
     </gazebo>
-</xacro:macro>
+  </xacro:macro>
 </robot>

File: spot_description/robots/spot.urdf.xacro (robot description, xacro)
@@ -629,4 +629,5 @@
     <!-- IMU sensor -->
     <xacro:imu_sensor
+        sensor_name="$(arg robot_name)_imu"
         frame_name="trunk_imu"
         imu_topic="trunk_imu/data"
@@ -651,5 +652,5 @@
     <xacro:leg_hardware prefix="lh"/>
     <xacro:leg_gazebo prefix="lh" robot_name="$(arg robot_name)" load_force_sensors="$(arg load_force_sensors)"/>
-    <xacro:imu_hardware imu_name="trunk_imu" imu_frame="trunk_imu"/>
+    <xacro:imu_hardware imu_name="$(arg robot_name)_imu" imu_frame="trunk_imu"/>
     <xacro:if value="$(eval arm_name != '')">
         <xacro:include filename="$(find spot_description)/urdfs/arm/$(arg arm_name)_adapter.urdf.xacro" />

File: spot_description/urdfs/accessories.urdf.xacro (robot description, xacro)
@@ -71,12 +71,8 @@
      far="10.0"
      parent_link="front_rail"
-     image_topic="$(arg robot_name)/camera/rgb/image_raw"
-     depth_topic="$(arg robot_name)/camera/depth/image_raw"
-     pointcloud_topic="$(arg robot_name)/camera/points"
-     camera_info_topic="$(arg robot_name)/camera/camera_info"
      origin_xyz="0.13 0 0"
      origin_rpy="0 0 0"/>
   <xacro:velodyne_laser_gazebo_sensor
-    sensor_name="lidar"
+    sensor_name="$(arg robot_name)_lidar"
     topic_name="lidar_points"
     update_rate="10.0"
@@ -91,5 +87,5 @@
     noise_stddev="0.01" />
 <xacro:gazebo_gps_sensor
-    sensor_name="gps_sensor"
+    sensor_name="$(arg robot_name)_gps"
     namespace="$(arg robot_name)"
     gps_topic="gps/fix"

File: wolf_description_utils/urdfs/gazebo.urdf.xacro (robot description, xacro)
@@ -8,4 +8,5 @@
 	<gazebo>
         <plugin name="controller_manager" filename="libgazebo_ros2_control.so">
+                <robot_param_node>/$(arg robot_name)/robot_state_publisher</robot_param_node>
                 <ros>
                         <namespace>/$(arg robot_name)</namespace>
@@ -14,5 +15,5 @@
                         <remapping>diffdrive_controller/odom:=odometry/robot</remapping>
                 </ros>
-                <parameters>$(find ${model_name}_description)/params/${model_name}_params.ros2.yaml</parameters>
+                <parameters>$(find ${model_name}_description)/params/${model_name}_params_$(arg robot_name).ros2.yaml</parameters>
         </plugin>
     	<plugin name="ground_truth" filename="libgazebo_ros_p3d.so">

Commit message: Make husky control works in ROS1 and add controller launch files

File: husky_description/robots/husky.urdf.xacro (robot description, xacro)
@@ -14,7 +14,6 @@
   <xacro:include filename="$(find sensors_description)/urdfs/sensors/imu.gazebo.xacro"/>
   <xacro:include filename="$(find wolf_description_utils)/urdfs/wheels.hardware.xacro"/>
-  <xacro:include filename="$(find sensors_description)/urdfs/sensors/depth_camera.gazebo.xacro"/>
+  <xacro:include filename="$(find velodyne_description)/urdf/VLP-16.urdf.xacro"/>
   <xacro:include filename="$(find sensors_description)/urdfs/sensors/gps.gazebo.xacro"/>
-  <xacro:include filename="$(find sensors_description)/urdfs/sensors/lidar.gazebo.xacro"/>
   <xacro:include filename="$(find husky_description)/urdfs/husky_macro.urdf.xacro" />
   <xacro:husky floating_base_link="$(arg floating_base_link)" />
@@ -35,42 +34,18 @@
     </xacro:imu_sensor>
     <xacro:imu_hardware imu_name="trunk_imu" imu_frame="trunk_imu"/>
-    <!-- Standard accessories. -->
-    <xacro:if value="$(arg sensors)">
-        <xacro:depth_camera
-          name="camera"
-          namespace="$(arg robot_name)"
-          update_rate="30"
-          image_width="640"
-          image_height="480"
-          fov="1.047"
-          near="0.1"
-          far="10.0"
-          parent_link="realsense_mountpoint_link"
-          image_topic="$(arg robot_name)/camera/rgb/image_raw"
-          depth_topic="$(arg robot_name)/camera/depth/image_raw"
-          pointcloud_topic="$(arg robot_name)/camera/points"
-          camera_info_topic="$(arg robot_name)/camera/camera_info"
-          origin_xyz="0.13 0 0"
-          origin_rpy="0 0 0"/>
-        <xacro:velodyne_laser_gazebo_sensor
-          sensor_name="lidar"
-          topic_name="lidar_points"
-          update_rate="10.0"
-          frame_id="lidar_arch_mount_link"
-          namespace="$(arg robot_name)"
-          min_range="0.9"
-          max_range="130.0"
-          number_of_beams="32"
-          horizontal_samples="220"
-          horizontal_fov="6.28319"
-          vertical_fov="0.2618"
-          noise_stddev="0.01" />
-      <xacro:gazebo_gps_sensor
-          sensor_name="gps_sensor"
-          namespace="$(arg robot_name)"
-          gps_topic="gps/fix"
-          velocity_topic="gps/velocity_fix"
-          update_rate="10.0"
-          frame_id="base_link" />
+  <!-- Standard accessories. -->
+  <xacro:if value="$(arg sensors)">
+    <xacro:VLP-16 parent="lidar_arch_mount_link" name="lidar" topic="/$(arg robot_name)/lidar_points"
+                  organize_cloud="true" hz="10" gpu="true">
+      <origin xyz="0 0 0" rpy="0 0 0" />
+    </xacro:VLP-16>
+    <!-- GPS sensor -->
+    <xacro:gps_sensor
+        gps_topic="fix"
+        vel_topic="velocity_fix"
+        namespace="$(arg robot_name)"
+        frame_name="base_link"
+        update_rate="10.0">
+    </xacro:gps_sensor>
     </xacro:if>
 </robot>
