Commit message: Load ignition sensors

File: husky_description/robots/husky.urdf.xacro (robot description, xacro)
@@ -17,7 +17,13 @@
   <xacro:include filename="$(find husky_description)/urdfs/husky_macro.urdf.xacro" />
   <xacro:husky floating_base_link="$(arg floating_base_link)" />
+  <xacro:if value="$(eval robot_name != '')">
+    <xacro:property name="husky_imu_sensor_name" value="$(arg robot_name)_imu"/>
+  </xacro:if>
+  <xacro:if value="$(eval robot_name == '')">
+    <xacro:property name="husky_imu_sensor_name" value="imu"/>
+  </xacro:if>
     <!-- IMU sensor -->
     <xacro:imu_sensor
-        sensor_name="imu"
+        sensor_name="${husky_imu_sensor_name}"
         frame_name="trunk_imu"
         imu_topic="trunk_imu/data"

File: sensors_description/urdfs/sensors/depth_camera.gazebo.xacro (robot description, xacro)
@@ -40,7 +40,9 @@
       <xacro:property name="camera_frame_id" value="${namespace + '/' + name + '_link'}"/>
     </xacro:if>
-    <!-- Gazebo Sim depth camera sensor -->
+    <!-- Gazebo Sim RGB-D camera sensor.
+         It publishes ${camera_topic_ns}/image, ${camera_topic_ns}/camera_info,
+         ${camera_topic_ns}/depth_image, and ${camera_topic_ns}/points. -->
     <gazebo reference="${name}_link">
-      <sensor type="depth_camera" name="${name}">
+      <sensor type="rgbd_camera" name="${name}">
         <update_rate>${update_rate}</update_rate>
         <always_on>true</always_on>

File: wolf_description_utils/urdfs/gazebo.urdf.xacro (robot description, xacro)
@@ -6,4 +6,5 @@
 <xacro:arg name="base_name"   default="base_link"/>
 <xacro:arg name="sensors"     default="false"/>
+<xacro:arg name="load_global_gazebo_systems" default="true"/>
 <xacro:property name="model_name" value="$(arg robot_model)"/>
 		<gazebo>
@@ -22,14 +23,14 @@
                 <parameters>$(find ${model_name}_description)/params/${model_name}_params_$(arg robot_name).ros2.yaml</parameters>
         </plugin>
-        <!-- Gazebo Sim IMU system is required so IMU sensors expose topics/components
-             that gz_ros2_control can subscribe to and populate ros2_control IMU interfaces. -->
-        <plugin filename="ignition-gazebo-imu-system" name="gz::sim::systems::Imu"/>
-        <xacro:if value="$(arg sensors)">
-                <!-- Gazebo Sim Sensors system drives rendering-based sensors (camera, lidar). -->
-                <plugin filename="ignition-gazebo-sensors-system" name="gz::sim::systems::Sensors">
-                        <render_engine>ogre2</render_engine>
-                </plugin>
-                <!-- Gazebo Sim NavSat system enables GPS sensor data publication. -->
-                <plugin filename="ignition-gazebo-navsat-system" name="ignition::gazebo::systems::NavSat"/>
+        <xacro:if value="$(arg load_global_gazebo_systems)">
+                <!-- Gazebo Sim sensor systems are global to the running world.
+                     Loading them once avoids multi-robot duplicate visual/rendering crashes. -->
+                <plugin filename="ignition-gazebo-imu-system" name="gz::sim::systems::Imu"/>
+                <xacro:if value="$(arg sensors)">
+                        <plugin filename="ignition-gazebo-sensors-system" name="gz::sim::systems::Sensors">
+                                <render_engine>ogre2</render_engine>
+                        </plugin>
+                        <plugin filename="ignition-gazebo-navsat-system" name="ignition::gazebo::systems::NavSat"/>
+                </xacro:if>
         </xacro:if>
 	</gazebo>

File: wolf_description_utils/urdfs/wheels.hardware.xacro (robot description, xacro)
@@ -1,4 +1,10 @@
 <?xml version="1.0"?>
 <robot xmlns:xacro="http://ros.org/wiki/xacro">
+  <xacro:if value="$(eval robot_name != '')">
+    <xacro:property name="wheel_imu_sensor_name" value="$(arg robot_name)_imu"/>
+  </xacro:if>
+  <xacro:if value="$(eval robot_name == '')">
+    <xacro:property name="wheel_imu_sensor_name" value="imu"/>
+  </xacro:if>
   <!-- ros2_control system definition -->
   <ros2_control name="wheels_system" type="system">
@@ -6,5 +12,5 @@
       <plugin>gz_ros2_control/GazeboSimSystem</plugin>
     </hardware>
-    <sensor name="imu">
+    <sensor name="${wheel_imu_sensor_name}">
       <param name="frame_id">trunk_imu</param>
       <state_interface name="orientation.x"/>
